Commit message: add joint_state_publisher & fixed sonar

File: pandora_sensors_description/urdf/sonar_sensor.urdf.xacro (robot description, xacro)
@@ -2,63 +2,63 @@
 <robot xmlns:xacro="http://ros.org/wiki/xacro">
 <xacro:macro name="sonar_caster" params="name parent *origin">
-	<joint name="${name}_sonar_joint" type="fixed">
-      <xacro:insert_block name="origin" />
-      <parent link="${parent}"/>
-      <child link="${name}_sonar_link"/>
-    </joint>
-    <link name="${name}_sonar_link">
-      <inertial>
-        <origin xyz="0 0 0.186" rpy="0 0 0"/>
-        <mass value="0.001"/>
-		<inertia ixx="1.0" ixy="0.0" ixz="0.0"
-				 iyy="1.0" iyz="0.0" izz="1.0"/>
-      </inertial>
-      <collision name="collision">
-        <geometry>
-            <box size="0.01 0.01 0.01"/>
-        </geometry>
-      </collision>
-      <visual name="visual">
-        <geometry>
-          <mesh filename="package://pandora_sensors_description/meshes/sonar_sensor/max_sonar_ez4.dae"/>
-        </geometry>
-      </visual>
-    </link>
-    <gazebo reference="${name}_sonar_link">
-		<sensor name="${name}_sonar" type="ray">
-        <pose>0.01 0 0.0175 0 -0 0</pose>
-        <ray>
-          <scan>
-            <horizontal>
-              <samples>10</samples>
-              <resolution>1</resolution>
-              <min_angle>-0.01</min_angle>
-              <max_angle>0.01</max_angle>
-            </horizontal>
-            <vertical>
-              <samples>10</samples>
-              <resolution>1</resolution>
-              <min_angle>-0.1</min_angle>
-              <max_angle>0.1</max_angle>
-            </vertical>
-          </scan>
-          <range>
-            <min>0.1</min>
-            <max>2.5</max>
-            <resolution>0.01</resolution>
-          </range>
-        </ray>
-        <always_on>1</always_on>
-        <update_rate>10</update_rate>
-        <visualize>true</visualize>
-        <plugin name="sonar2ros" filename="libpandora_sonar_plugin.so">
-			<topicName>/sensors/sonar</topicName>
-			<updateRate>10</updateRate>
-			<gaussianNoise>0.0</gaussianNoise>
-			<frameName>rear_sonar</frameName>
-			<robotNamespace></robotNamespace>
-		</plugin>
-      </sensor>
-    </gazebo>
+  <joint name="${name}_sonar_joint" type="fixed">
+    <xacro:insert_block name="origin" />
+    <parent link="${parent}"/>
+    <child link="${name}_sonar_link"/>
+  </joint>
+  <link name="${name}_sonar_link">
+    <inertial>
+      <origin xyz="0 0 0.186" rpy="0 0 0"/>
+      <mass value="0.001"/>
+      <inertia ixx="1.0" ixy="0.0" ixz="0.0"
+       iyy="1.0" iyz="0.0" izz="1.0"/>
+    </inertial>
+    <collision name="collision">
+      <geometry>
+          <box size="0.01 0.01 0.01"/>
+      </geometry>
+    </collision>
+    <visual name="visual">
+      <geometry>
+        <mesh filename="package://pandora_sensors_description/meshes/sonar_sensor/max_sonar_ez4.dae"/>
+      </geometry>
+    </visual>
+  </link>
+  <gazebo reference="${name}_sonar_link">
+    <sensor name="${name}_sonar" type="ray">
+      <pose>0.01 0 0.0175 0 -0 0</pose>
+      <ray>
+        <scan>
+          <horizontal>
+            <samples>10</samples>
+            <resolution>1</resolution>
+            <min_angle>-0.01</min_angle>
+            <max_angle>0.01</max_angle>
+          </horizontal>
+          <vertical>
+            <samples>10</samples>
+            <resolution>1</resolution>
+            <min_angle>-0.1</min_angle>
+            <max_angle>0.1</max_angle>
+          </vertical>
+        </scan>
+        <range>
+          <min>0.1</min>
+          <max>2.5</max>
+          <resolution>0.01</resolution>
+        </range>
+      </ray>
+      <always_on>1</always_on>
+      <update_rate>10</update_rate>
+      <visualize>true</visualize>
+      <plugin name="sonar2ros" filename="libpandora_sonar_plugin.so">
+        <topicName>/sensors/sonar</topicName>
+        <updateRate>10</updateRate>
+        <gaussianNoise>0.0</gaussianNoise>
+        <frameName>rear_sonar_link</frameName>
+        <robotNamespace></robotNamespace>
+      </plugin>
+    </sensor>
+  </gazebo>
 </xacro:macro>
 </robot>
