Commit message: Refactor gears description and separate robot files.

File: pandora_sensors_description/urdf/co2_sensor.urdf.xacro (robot description, xacro)
@@ -1,26 +1,34 @@
 <?xml version="1.0" ?>
-<robot xmlns:xacro="http://ros.org/wiki/xacro">
-<xacro:macro name="co2_caster" params="parent *origin">
-      <link name="co2_link">
-		  <inertial>
-			<mass value="0.1"/>
-			<origin xyz="0 0 0"/>
-			<inertia ixx="1" ixy="0" ixz="0" iyy="1" iyz="0" izz="1" />
-		  </inertial>
-        <visual name="visual">
-		  <origin xyz="0 0 0" rpy="0 0 0"/>
-          <geometry>
-			<mesh filename="package://pandora_sensors_description/meshes/co2_sensor/co2_small.dae"/>
-          </geometry>
-        </visual>
-        <collision name="collision">
-		  <origin xyz="0 0 0" rpy="0 0 0"/>
-          <geometry>
-            <box size="0.01 0.01 0.01"/>
-          </geometry>
-        </collision>
+<robot xmlns:xacro="http://ros.org/wiki/xacro" >
+  <xacro:macro name="co2_caster"
+               params="parent *origin" >
+    <link name="co2_link" >
+      <inertial>
+        <mass value="0.1" />
+        <origin xyz="0 0 0" />
+        <inertia ixx="1"
+                 ixy="0"
+                 ixz="0"
+                 iyy="1"
+                 iyz="0"
+                 izz="1" />
+      </inertial>
+      <visual name="visual" >
+        <origin xyz="0 0 0"
+                rpy="0 0 0" />
+        <geometry>
+          <mesh filename="package://pandora_sensors_description/meshes/co2_sensor/co2_small.dae" />
+        </geometry>
+      </visual>
+      <collision name="collision" >
+        <origin xyz="0 0 0"
+                rpy="0 0 0" />
+        <geometry>
+          <box size="0.01 0.01 0.01" />
+        </geometry>
+      </collision>
     </link>
-    <gazebo reference="co2_link">
-		<sensor name="co2" type="camera">
+    <gazebo reference="co2_link" >
+      <sensor name="co2" type="camera" >
         <camera>
           <horizontal_fov>1.5</horizontal_fov>
@@ -37,15 +45,17 @@
         <update_rate>5</update_rate>
         <visualize>false</visualize>
-        <plugin name="co2ros" filename="libpandora_co2_plugin.so">
-			<frameName>co2</frameName>
-			<topicName>sensors/co2</topicName>
-		</plugin>
+        <plugin name="co2ros"
+                filename="libpandora_co2_plugin.so" >
+          <frameName>co2</frameName>
+          <topicName>sensors/co2</topicName>
+        </plugin>
       </sensor>
-   </gazebo>
-   	<joint name="co2_joint" type="fixed">
-	  <xacro:insert_block name="origin" />
-      <parent link="${parent}"/>
-	  <child link="co2_link"/>
-	</joint>
-</xacro:macro>
+    </gazebo>
+    <joint name="co2_joint"
+           type="fixed" >
+      <parent link="${parent}" />
+      <child link="co2_link" />
+      <xacro:insert_block name="origin" />
+    </joint>
+  </xacro:macro>
 </robot>

File: pandora_sensors_description/urdf/hokuyo_utm_30lx.urdf.xacro (robot description, xacro)
@@ -1,99 +1,117 @@
 <?xml version="1.0" ?>
-<robot xmlns:xacro="http://ros.org/wiki/xacro">
-<xacro:macro name="hokuyo_caster" params="parent *origin">
-  <link name="laser_link">
-    <inertial>
-      <mass value="0.1"/>
-      <origin xyz="0 0 0"/>
-      <inertia ixx="0.0002632" ixy="0" ixz="0"
-       iyy="0.0002632" iyz="0" izz="0.000162" />
-    </inertial>
-  <!--
-    <inertial>
-      <mass value="0.1"/>
-      <origin xyz="0 0 0"/>
-      <inertia ixx="1" ixy="0" ixz="0" iyy="1" iyz="0" izz="1" />
-    </inertial>
-  -->
-    <visual name="visual">
-      <geometry>
-        <mesh filename="package://pandora_sensors_description/meshes/hokuyo_utm_30lx/hokuyo_utm_30lx.dae"/>
-      </geometry>
-    </visual>
-    <collision name="collision-base">
-      <origin xyz="0 0 -0.0145" rpy="0 0 0"/>
-      <geometry>
-    <box size="0.05 0.05 0.041"/>
-      </geometry>
-    </collision>
-    <collision name="collision-top">
-      <origin xyz="0 0 0.0205" rpy="0 0 0"/>
-      <geometry>
-        <cylinder radius="0.021" length="0.029"/>
-      </geometry>
-    </collision>
-  </link>
-  <gazebo reference="laser_link">
-    <sensor name="laser" type="ray">
-      <pose>0.01 0 0.0175 0 -0 0</pose>
-      <ray>
-        <scan>
-          <horizontal>
-            <samples>640</samples>
-            <resolution>1</resolution>
-            <min_angle>-2.26889</min_angle>
-            <max_angle>2.268899</max_angle>
-          </horizontal>
-        </scan>
-        <range>
-          <min>0.08</min>
-          <max>10</max>
-          <resolution>0.01</resolution>
-        </range>
-      </ray>
-      <plugin name="laser" filename="libRayPlugin.so" />
-      <plugin name="laser2Ros" filename="libgazebo_ros_laser.so">
-        <topicName>/slam/scan</topicName>
-        <frameName>/laser_link</frameName>
-      </plugin>
-      <always_on>1</always_on>
-      <update_rate>30</update_rate>
-      <visualize>true</visualize>
-    </sensor>
-  </gazebo>
-  <link name="hokuyo_base_link">
-    <inertial>
-      <mass value="0.001"/>
-      <origin xyz="0 0 0"/>
-      <inertia ixx="0.00000001" ixy="0" ixz="0"
-           iyy="0.00000001" iyz="0" izz="0.00000001"/>
-    </inertial>
-    <visual>
-      <origin xyz="0 0 0" rpy="0 0 0"/>
-      <geometry>
-        <box size="0 0 0"/>
-      </geometry>
-    </visual>
-    <collision>
-      <origin xyz="0 0 0" rpy="0 0 0"/>
-      <geometry>
-        <box size="0 0 0"/>
-      </geometry>
-    </collision>
-  </link>
-  <joint name="laser_roll_joint" type="revolute">
-    <xacro:insert_block name="origin" />
-    <parent link="${parent}"/>
-    <child link="hokuyo_base_link"/>
-    <axis xyz="1 0 0"/>
-    <limit effort="300" velocity="100.0" lower="-1.57" upper="1.57"/>
-  </joint>
-  <joint name="laser_pitch_joint" type="revolute">
-    <origin xyz="0 0 0" rpy="0 0 0"/>
-    <parent link="hokuyo_base_link"/>
-    <child link="laser_link"/>
-    <axis xyz="0 1 0"/>
-    <limit effort="300" velocity="100.0" lower="-1.57" upper="1.57"/>
-  </joint>
-</xacro:macro>
+<robot xmlns:xacro="http://ros.org/wiki/xacro" >
+  <xacro:macro name="hokuyo_caster"
+               params="parent *origin" >
+    <link name="laser_link" >
+      <inertial>
+        <mass value="0.01" />
+        <origin xyz="0 0 0" />
+        <inertia ixx="0.0002632"
+                 ixy="0"
+                 ixz="0"
+                 iyy="0.0002632"
+                 iyz="0"
+                 izz="0.000162" />
+      </inertial>
+      <visual name="visual" >
+        <geometry>
+          <mesh filename="package://pandora_sensors_description/meshes/hokuyo_utm_30lx/hokuyo_utm_30lx.dae" />
+        </geometry>
+      </visual>
+      <collision name="collision-base" >
+        <origin xyz="0 0 -0.0145"
+                rpy="0 0 0" />
+        <geometry>
+      <box size="0.05 0.05 0.041" />
+        </geometry>
+      </collision>
+      <collision name="collision-top" >
+        <origin xyz="0 0 0.0205"
+                rpy="0 0 0" />
+        <geometry>
+          <cylinder radius="0.021"
+                    length="0.029" />
+        </geometry>
+      </collision>
+    </link>
+    <gazebo reference="laser_link" >
+      <sensor name="laser"
+              type="ray" >
+        <pose>0.01 0 0.0175 0 -0 0</pose>
+        <ray>
+          <scan>
+            <horizontal>
+              <samples>640</samples>
+              <resolution>1</resolution>
+              <min_angle>-2.26889</min_angle>
+              <max_angle>2.268899</max_angle>
+            </horizontal>
+          </scan>
+          <range>
+            <min>0.08</min>
+            <max>10</max>
+            <resolution>0.01</resolution>
+          </range>
+        </ray>
+        <plugin name="laser"
+                filename="libRayPlugin.so" />
+        <plugin name="laser2Ros"
+                filename="libgazebo_ros_laser.so" >
+          <topicName>/slam/scan</topicName>
+          <frameName>/laser_link</frameName>
+        </plugin>
+        <always_on>1</always_on>
+        <update_rate>30</update_rate>
+        <visualize>true</visualize>
+      </sensor>
+    </gazebo>
+    <link name="hokuyo_base_link" >
+      <inertial>
+        <mass value="0.001" />
+        <origin xyz="0 0 0" />
+        <inertia ixx="0.00000001"
+                 ixy="0"
+                 ixz="0"
+                 iyy="0.00000001"
+                 iyz="0"
+                 izz="0.00000001" />
+      </inertial>
+      <visual>
+        <origin xyz="0 0 0"
+                rpy="0 0 0" />
+        <geometry>
+          <box size="0 0 0" />
+        </geometry>
+      </visual>
+      <collision>
+        <origin xyz="0 0 0"
+                rpy="0 0 0" />
+        <geometry>
+          <box size="0 0 0" />
+        </geometry>
+      </collision>
+    </link>
+    <joint name="laser_roll_joint"
+           type="revolute" >
+      <parent link="${parent}" />
+      <child link="hokuyo_base_link" />
+      <xacro:insert_block name="origin" />
+      <axis xyz="1 0 0" />
+      <limit lower="-1.57"
+             upper="1.57"
+             effort="300"
+             velocity="100.0" />
+    </joint>
+    <joint name="laser_pitch_joint"
+           type="revolute" >
+      <parent link="hokuyo_base_link" />
+      <child link="laser_link" />
+      <origin xyz="0 0 0" rpy="0 0 0" />
+      <axis xyz="0 1 0" />
+      <limit lower="-1.57"
+             upper="1.57"
+             effort="300"
+             velocity="100.0" />
+    </joint>
+  </xacro:macro>
 </robot>

File: pandora_sensors_description/urdf/kinect_camera.urdf.xacro (robot description, xacro)
@@ -1,110 +1,136 @@
 <?xml version="1.0" ?>
-<robot xmlns:xacro="http://ros.org/wiki/xacro">
-<xacro:macro name="kinect_caster" params="parent *origin">
-  <link name="kinect_link">
-    <inertial>
-      <origin xyz="0 0 0" rpy="0 0 0"/>
-      <mass value="0.1"/>
-      <inertia ixx="0.004075" ixy="0.0" ixz="0.0"
-                iyy="0.004075" iyz="0.0" izz="0.004075"/>
-    </inertial>
-    <collision name="collision">
-      <geometry>
-        <box size="0.073000 0.276000 0.072000"/>
-      </geometry>
-    </collision>
-    <visual name="visual">
-      <geometry>
-        <mesh filename="package://pandora_sensors_description/meshes/kinect_camera/kinect_camera_simple.dae"/>
-      </geometry>
-    </visual>
-  </link>
-  <link name="kinect_camera">
-    <inertial>
-      <origin xyz="0 0 0" rpy="0 0 0"/>
-      <mass value="0.001"/>
-      <inertia ixx="0.00004075" ixy="0.0" ixz="0.0"
-           iyy="0.00004075" iyz="0.0" izz="0.00004075"/>
-    </inertial>
-    <collision name="collision">
-      <geometry>
-        <box size="0.001 0.001 0.001"/>
-      </geometry>
-    </collision>
-    <visual name="visual">
-      <geometry>
-        <box size="0.001 0.001 0.001"/>
-      </geometry>
-    </visual>
-  </link>
-  <joint name="kinect_camera_joint" type="fixed">
-    <origin xyz="0 0 0" rpy="-1.57 0 -1.57"/>
-    <parent link="kinect_link"/>
-    <child link="kinect_camera"/>
-  </joint>
-  <gazebo reference="kinect_link">
-    <sensor name="kinect" type="depth">
-      <update_rate>20</update_rate>
-      <camera>
-        <horizontal_fov>1.047198</horizontal_fov>
-        <image>
-          <width>640</width>
-          <height>480</height>
-          <format>R8G8B8</format>
-        </image>
-        <clip>
-          <near>0.05</near>
-          <far>3</far>
-        </clip>
-      </camera>
-      <plugin name="depth2ros" filename="libgazebo_ros_openni_kinect.so">
-        <pointCloudTopicName>point_cloud</pointCloudTopicName>
-        <frameName>kinect_camera</frameName>
-        <cameraName>kinect</cameraName>
-        <imageTopicName>image</imageTopicName>
-        <depthImageTopicName>depth/image</depthImageTopicName>
-        <depthImageCameraInfoTopicName>depth/image/info</depthImageCameraInfoTopicName>
-        <pointCloudCutoff>0.4</pointCloudCutoff>
-      </plugin>
-    </sensor>
-  </gazebo>
-  <link name="kinect_base_link">
-    <inertial>
-      <mass value="0.001"/>
-      <origin xyz="0 0 0"/>
-      <inertia ixx="0.00000001" ixy="0" ixz="0"
-           iyy="0.00000001" iyz="0" izz="0.00000001"/>
-    </inertial>
-    <visual>
-      <origin xyz="0 0 0" rpy="0 0 0"/>
-      <geometry>
-        <box size="0 0 0"/>
-      </geometry>
-    </visual>
-    <collision>
-      <origin xyz="0 0 0" rpy="0 0 0"/>
-      <geometry>
-        <box size="0 0 0"/>
-      </geometry>
-    </collision>
-  </link>
-  <joint name="kinect_pitch_joint" type="fixed">
-    <xacro:insert_block name="origin" />
-      <parent link="${parent}"/>
-    <child link="kinect_base_link"/>
-    <axis xyz="0 1 0"/>
-  <!--
-    <limit effort="300" velocity="100.0" />
-  -->
-  </joint>
-  <joint name="kinect_yaw_joint" type="fixed">
-    <origin xyz="0 0 0" rpy="0 0 0"/>
-    <child link="kinect_link"/>
-    <parent link="kinect_base_link"/>
-    <axis xyz="0 0 1"/>
-  <!--
-    <limit effort="300" velocity="100.0" />
-  -->
-  </joint>
-</xacro:macro>
+<robot xmlns:xacro="http://ros.org/wiki/xacro" >
+  <xacro:macro name="kinect_caster"
+               params="parent *origin" >
+    <link name="kinect_link" >
+      <inertial>
+        <origin xyz="0 0 0"
+                rpy="0 0 0" />
+        <mass value="0.01" />
+        <inertia ixx="0.0004075"
+                 ixy="0.0"
+                 ixz="0.0"
+                 iyy="0.0004075"
+                 iyz="0.0"
+                 izz="0.0004075" />
+      </inertial>
+      <collision name="collision" >
+        <geometry>
+          <box size="0.073000 0.276000 0.072000" />
+        </geometry>
+      </collision>
+      <visual name="visual" >
+        <geometry>
+          <mesh filename="package://pandora_sensors_description/meshes/kinect_camera/kinect_camera_simple.dae" />
+        </geometry>
+      </visual>
+    </link>
+    <link name="kinect_camera" >
+      <inertial>
+        <origin xyz="0 0 0"
+                rpy="0 0 0" />
+        <mass value="0.001" />
+        <inertia ixx="0.00004075"
+                 ixy="0.0"
+                 ixz="0.0"
+                 iyy="0.00004075"
+                 iyz="0.0"
+                 izz="0.00004075" />
+      </inertial>
+      <collision name="collision" >
+        <geometry>
+          <box size="0.001 0.001 0.001" />
+        </geometry>
+      </collision>
+      <visual name="visual" >
+        <geometry>
+          <box size="0.001 0.001 0.001" />
+        </geometry>
+      </visual>
+    </link>
+    <joint name="kinect_camera_joint"
+           type="fixed" >
+      <parent link="kinect_link" />
+      <child link="kinect_camera" />
+      <origin xyz="0 0 0"
+              rpy="-1.57 0 -1.57" />
+    </joint>
+    <gazebo reference="kinect_link" >
+      <sensor name="kinect"
+              type="depth" >
+        <update_rate>20</update_rate>
+        <camera>
+          <horizontal_fov>1.047198</horizontal_fov>
+          <image>
+            <width>640</width>
+            <height>480</height>
+            <format>R8G8B8</format>
+          </image>
+          <clip>
+            <near>0.05</near>
+            <far>3</far>
+          </clip>
+        </camera>
+        <plugin name="depth2ros"
+                filename="libgazebo_ros_openni_kinect.so" >
+          <pointCloudTopicName>point_cloud</pointCloudTopicName>
+          <frameName>kinect_camera</frameName>
+          <cameraName>kinect</cameraName>
+          <imageTopicName>image</imageTopicName>
+          <depthImageTopicName>depth/image</depthImageTopicName>
+          <depthImageCameraInfoTopicName>depth/image/info</depthImageCameraInfoTopicName>
+          <pointCloudCutoff>0.4</pointCloudCutoff>
+        </plugin>
+      </sensor>
+    </gazebo>
+    <link name="kinect_base_link" >
+      <inertial>
+        <mass value="0.001" />
+        <origin xyz="0 0 0" />
+        <inertia ixx="0.00000001"
+                 ixy="0"
+                 ixz="0"
+                 iyy="0.00000001"
+                 iyz="0"
+                 izz="0.00000001" />
+      </inertial>
+      <visual>
+        <origin xyz="0 0 0"
+                rpy="0 0 0" />
+        <geometry>
+          <box size="0 0 0" />
+        </geometry>
+      </visual>
+      <collision>
+        <origin xyz="0 0 0"
+                rpy="0 0 0" />
+        <geometry>
+          <box size="0 0 0" />
+        </geometry>
+      </collision>
+    </link>
+    <joint name="kinect_pitch_joint"
+           type="revolute" >
+      <parent link="${parent}" />
+      <child link="kinect_base_link" />
+      <xacro:insert_block name="origin" />
+      <axis xyz="0 1 0" />
+      <limit lower="-1.57"
+             upper="1.57"
+             effort="300"
+             velocity="100.0" />
+    </joint>
+    <joint name="kinect_yaw_joint"
+           type="revolute" >
+      <parent link="kinect_base_link" />
+      <child link="kinect_link" />
+      <origin xyz="0 0 0"
+              rpy="0 0 0" />
+      <axis xyz="0 0 1" />
+      <limit lower="-1.57"
+             upper="1.57"
+             effort="300"
+             velocity="100.0" />
+    </joint>
+  </xacro:macro>
 </robot>

File: pandora_sensors_description/urdf/microphone_sensor.urdf.xacro (robot description, xacro)
@@ -1,26 +1,35 @@
 <?xml version="1.0" ?>
-<robot xmlns:xacro="http://ros.org/wiki/xacro">
-<xacro:macro name="microphone_caster" params="parent *origin">
-      <link name="microphone_link">
-        <inertial>
-			<mass value="0.1"/>
-			<origin xyz="0 0 0"/>
-			<inertia ixx="1" ixy="0" ixz="0" iyy="1" iyz="0" izz="1" />
-		 </inertial>
-        <visual name="visual">
-		  <origin xyz="0 0 0" rpy="0 0 0"/>
-          <geometry>
-			<mesh filename="package://pandora_sensors_description/meshes/microphone_sensor/microphone_small.dae"/>
-          </geometry>
-        </visual>
-        <collision name="collision">
-          <origin xyz="0 0 0" rpy="0 0 0"/>
-          <geometry>
-            <box size="0.01 0.01 0.01"/>
-          </geometry>
-        </collision>
+<robot xmlns:xacro="http://ros.org/wiki/xacro" >
+  <xacro:macro name="microphone_caster"
+               params="parent *origin" >
+    <link name="microphone_link" >
+      <inertial>
+        <mass value="0.1" />
+        <origin xyz="0 0 0" />
+        <inertia ixx="1"
+                 ixy="0"
+                 ixz="0"
+                 iyy="1"
+                 iyz="0"
+                 izz="1" />
+      </inertial>
+      <visual name="visual" >
+        <origin xyz="0 0 0"
+                rpy="0 0 0" />
+        <geometry>
+          <mesh filename="package://pandora_sensors_description/meshes/microphone_sensor/microphone_small.dae" />
+        </geometry>
+      </visual>
+      <collision name="collision" >
+        <origin xyz="0 0 0"
+                rpy="0 0 0" />
+        <geometry>
+          <box size="0.01 0.01 0.01" />
+        </geometry>
+      </collision>
     </link>
-    <gazebo reference="microphone_link">
-		<sensor name="microphone" type="camera">
+    <gazebo reference="microphone_link" >
+      <sensor name="microphone"
+              type="camera" >
         <camera>
           <horizontal_fov>1.5</horizontal_fov>
@@ -37,15 +46,16 @@
         <update_rate>10</update_rate>
         <visualize>false</visualize>
-        <plugin name="microphone2ros" filename="libpandora_microphone_plugin.so">
-			<frameName>sound</frameName>
-			<topicName>sensors/sound</topicName>
-		</plugin>
+        <plugin name="microphone2ros"
+                filename="libpandora_microphone_plugin.so" >
+          <frameName>sound</frameName>
+          <topicName>sensors/sound</topicName>
+        </plugin>
       </sensor>
-	</gazebo>
-	<joint name="microphone_joint" type="fixed">
-	  <xacro:insert_block name="origin" />
-      <parent link="${parent}"/>
-	  <child link="microphone_link"/>
-	</joint>
-</xacro:macro>
+    </gazebo>
+    <joint name="microphone_joint" type="fixed" >
+      <xacro:insert_block name="origin" />
+      <parent link="${parent}" />
+      <child link="microphone_link" />
+    </joint>
+  </xacro:macro>
 </robot>
