Commit message: Refactor gears description and separate robot files.

File: pandora_sensors_description/urdf/sonar_sensor.urdf.xacro (robot description, xacro)
@@ -1,64 +1,73 @@
 <?xml version="1.0" ?>
-<robot xmlns:xacro="http://ros.org/wiki/xacro">
-<xacro:macro name="sonar_caster" params="name parent *origin">
-  <joint name="${name}_sonar_joint" type="fixed">
-    <xacro:insert_block name="origin" />
-    <parent link="${parent}"/>
-    <child link="${name}_sonar_link"/>
-  </joint>
-  <link name="${name}_sonar_link">
-    <inertial>
-      <origin xyz="0 0 0.186" rpy="0 0 0"/>
-      <mass value="0.001"/>
-      <inertia ixx="1.0" ixy="0.0" ixz="0.0"
-       iyy="1.0" iyz="0.0" izz="1.0"/>
-    </inertial>
-    <collision name="collision">
-      <geometry>
-          <box size="0.01 0.01 0.01"/>
-      </geometry>
-    </collision>
-    <visual name="visual">
-      <geometry>
-        <mesh filename="package://pandora_sensors_description/meshes/sonar_sensor/max_sonar_ez4.dae"/>
-      </geometry>
-    </visual>
-  </link>
-  <gazebo reference="${name}_sonar_link">
-    <sensor name="${name}_sonar" type="ray">
-      <pose>0.01 0 0.0175 0 -0 0</pose>
-      <ray>
-        <scan>
-          <horizontal>
-            <samples>10</samples>
-            <resolution>1</resolution>
-            <min_angle>-0.01</min_angle>
-            <max_angle>0.01</max_angle>
-          </horizontal>
-          <vertical>
-            <samples>10</samples>
-            <resolution>1</resolution>
-            <min_angle>-0.1</min_angle>
-            <max_angle>0.1</max_angle>
-          </vertical>
-        </scan>
-        <range>
-          <min>0.1</min>
-          <max>2.5</max>
-          <resolution>0.01</resolution>
-        </range>
-      </ray>
-      <always_on>1</always_on>
-      <update_rate>10</update_rate>
-      <visualize>true</visualize>
-      <plugin name="sonar2ros" filename="libpandora_sonar_plugin.so">
-        <topicName>/sensors/sonar</topicName>
-        <updateRate>10</updateRate>
-        <gaussianNoise>0.0</gaussianNoise>
-        <frameName>rear_sonar_link</frameName>
-        <robotNamespace></robotNamespace>
-      </plugin>
-    </sensor>
-  </gazebo>
-</xacro:macro>
+<robot xmlns:xacro="http://ros.org/wiki/xacro" >
+  <xacro:macro name="sonar_caster"
+               params="name parent *origin" >
+    <joint name="${name}_sonar_joint"
+           type="fixed" >
+      <parent link="${parent}" />
+      <child link="${name}_sonar_link" />
+      <xacro:insert_block name="origin" />
+    </joint>
+    <link name="${name}_sonar_link" >
+      <inertial>
+        <origin xyz="0 0 0.186"
+                rpy="0 0 0" />
+        <mass value="0.001" />
+        <inertia ixx="1.0"
+                 ixy="0.0"
+                 ixz="0.0"
+                 iyy="1.0"
+                 iyz="0.0"
+                 izz="1.0" />
+      </inertial>
+      <visual name="visual" >
+        <geometry>
+          <mesh filename="package://pandora_sensors_description/meshes/sonar_sensor/max_sonar_ez4.dae" />
+        </geometry>
+      </visual>
+      <collision name="collision" >
+        <geometry>
+            <box size="0.01 0.01 0.01" />
+        </geometry>
+      </collision>
+    </link>
+    <gazebo reference="${name}_sonar_link" >
+      <sensor name="${name}_sonar"
+              type="ray" >
+        <pose>0.01 0 0.0175 0 -0 0</pose>
+        <ray>
+          <scan>
+            <horizontal>
+              <samples>10</samples>
+              <resolution>1</resolution>
+              <min_angle>-0.01</min_angle>
+              <max_angle>0.01</max_angle>
+            </horizontal>
+            <vertical>
+              <samples>10</samples>
+              <resolution>1</resolution>
+              <min_angle>-0.1</min_angle>
+              <max_angle>0.1</max_angle>
+            </vertical>
+          </scan>
+          <range>
+            <min>0.1</min>
+            <max>2.5</max>
+            <resolution>0.01</resolution>
+          </range>
+        </ray>
+        <always_on>1</always_on>
+        <update_rate>10</update_rate>
+        <visualize>true</visualize>
+        <plugin name="sonar2ros"
+                filename="libpandora_sonar_plugin.so" >
+          <topicName>/sensors/sonar</topicName>
+          <updateRate>10</updateRate>
+          <gaussianNoise>0.0</gaussianNoise>
+          <frameName>rear_sonar_link</frameName>
+          <robotNamespace></robotNamespace>
+        </plugin>
+      </sensor>
+    </gazebo>
+  </xacro:macro>
 </robot>

File: pandora_sensors_description/urdf/thermal_sensor.urdf.xacro (robot description, xacro)
@@ -1,25 +1,32 @@
 <?xml version="1.0" ?>
-<robot xmlns:xacro="http://ros.org/wiki/xacro">
-<xacro:macro name="thermal_caster" params="parent *origin">
-      <link name="thermal_link">
-        <inertial>
-			<origin xyz="0 0 0.186" rpy="0 0 0"/>
-			<mass value="0.1"/>
-			<inertia ixx="1.0" ixy="0.0" ixz="0.0"
-					 iyy="1.0" iyz="0.0" izz="1.0"/>
-		</inertial>
-        <visual name="visual">
-          <geometry>
-			 <mesh filename="package://pandora_sensors_description/meshes/thermal_sensor/thermal_small.dae"/>
-          </geometry>
-        </visual>
-        <collision name="collision">
-          <geometry>
-            <box size="0.01 0.01 0.01"/>
-          </geometry>
-        </collision>
+<robot xmlns:xacro="http://ros.org/wiki/xacro" >
+  <xacro:macro name="thermal_caster"
+               params="parent *origin" >
+    <link name="thermal_link" >
+      <inertial>
+        <origin xyz="0 0 0.186"
+                rpy="0 0 0" />
+        <mass value="0.1" />
+        <inertia ixx="1.0"
+                 ixy="0.0"
+                 ixz="0.0"
+                 iyy="1.0"
+                 iyz="0.0"
+                 izz="1.0" />
+      </inertial>
+      <visual name="visual" >
+        <geometry>
+          <mesh filename="package://pandora_sensors_description/meshes/thermal_sensor/thermal_small.dae" />
+        </geometry>
+      </visual>
+      <collision name="collision" >
+        <geometry>
+          <box size="0.01 0.01 0.01" />
+        </geometry>
+      </collision>
     </link>
-    <gazebo reference="thermal_link">
-		<sensor name="thermal" type="camera">
+    <gazebo reference="thermal_link" >
+      <sensor name="thermal"
+              type="camera" >
         <camera>
           <horizontal_fov>0.5</horizontal_fov>
@@ -36,15 +43,17 @@
         <update_rate>30</update_rate>
         <visualize>false</visualize>
-        <plugin name="thermal2ros" filename="libpandora_thermal_plugin.so">
-			<frameName>thermal_link</frameName>
-			<topicName>sensors/thermal</topicName>
-		</plugin>
+        <plugin name="thermal2ros"
+                filename="libpandora_thermal_plugin.so" >
+          <frameName>thermal_link</frameName>
+          <topicName>sensors/thermal</topicName>
+        </plugin>
       </sensor>
-	</gazebo>
-	<joint name="thermal_joint" type="fixed">
-	  <xacro:insert_block name="origin" />
-      <parent link="${parent}"/>
-	  <child link="thermal_link"/>
-	</joint>
-</xacro:macro>
+    </gazebo>
+    <joint name="thermal_joint"
+           type="fixed" >
+      <parent link="${parent}" />
+      <child link="thermal_link" />
+      <xacro:insert_block name="origin" />
+    </joint>
+  </xacro:macro>
 </robot>

Commit message: Adjust center of mass and mass of sensors.

File: pandora_sensors_description/urdf/co2_sensor.urdf.xacro (robot description, xacro)
@@ -5,6 +5,7 @@
     <link name="co2_link" >
       <inertial>
+        <origin xyz="0.008 0.0 0.0"
+                rpy="0 0 0" />
         <mass value="0.1" />
-        <origin xyz="0 0 0" />
         <inertia ixx="1"
                  ixy="0"
@@ -12,5 +13,5 @@
                  iyy="1"
                  iyz="0"
-                 izz="1" />
+                 izz="1" /><!-- FIXME -->
       </inertial>
       <visual name="visual" >

File: pandora_sensors_description/urdf/kinect_camera.urdf.xacro (robot description, xacro)
@@ -5,7 +5,7 @@
     <link name="kinect_link" >
       <inertial>
-        <origin xyz="0 0 0"
+        <origin xyz="-0.02891 -0.00024 0.00037"
                 rpy="0 0 0" />
-        <mass value="0.01" />
+        <mass value="0.1" />
         <inertia ixx="0.0004075"
                  ixy="0.0"
@@ -13,5 +13,5 @@
                  iyy="0.0004075"
                  iyz="0.0"
-                 izz="0.0004075" />
+                 izz="0.0004075" /><!-- FIXME -->
       </inertial>
       <collision name="collision" >

File: pandora_sensors_description/urdf/microphone_sensor.urdf.xacro (robot description, xacro)
@@ -5,6 +5,7 @@
     <link name="microphone_link" >
       <inertial>
+        <origin xyz="0.008 0.0 0.0"
+                rpy="0 0 0" />
         <mass value="0.1" />
-        <origin xyz="0 0 0" />
         <inertia ixx="1"
                  ixy="0"
@@ -12,5 +13,5 @@
                  iyy="1"
                  iyz="0"
-                 izz="1" />
+                 izz="1" /><!-- FIXME -->
       </inertial>
       <visual name="visual" >

File: pandora_sensors_description/urdf/sonar_sensor.urdf.xacro (robot description, xacro)
@@ -11,7 +11,7 @@
     <link name="${name}_sonar_link" >
       <inertial>
-        <origin xyz="0 0 0.186"
+        <origin xyz="0.008 0.0 0.0"
                 rpy="0 0 0" />
-        <mass value="0.001" />
+        <mass value="0.1" />
         <inertia ixx="1.0"
                  ixy="0.0"
@@ -19,5 +19,5 @@
                  iyy="1.0"
                  iyz="0.0"
-                 izz="1.0" />
+                 izz="1.0" /><!-- FIXME -->
       </inertial>
       <visual name="visual" >

File: pandora_sensors_description/urdf/thermal_sensor.urdf.xacro (robot description, xacro)
@@ -5,5 +5,5 @@
     <link name="${prefix_y}_thermal_link" >
       <inertial>
-        <origin xyz="0 0 0.186"
+        <origin xyz="0.008 0.0 0.0"
                 rpy="0 0 0" />
         <mass value="0.1" />
@@ -13,5 +13,5 @@
                  iyy="1.0"
                  iyz="0.0"
-                 izz="1.0" />
+                 izz="1.0" /><!-- FIXME -->
       </inertial>
       <visual name="visual" >
