Commit message: Add kinect base & asus xtion.

File: pandora_sensors_description/urdf/hokuyo_utm_30lx.urdf.xacro (robot description, xacro)
@@ -11,5 +11,5 @@
                        *origin" >
     <!-- ################################################################## -->
-    <link name="laser_base_link" >
+    <link name="laser_servo_link" >
       <inertial>
         <!-- ============================================================== -->
@@ -107,5 +107,5 @@
         <!-- ============================================================== -->
         <parent link="${parent}" />
-        <child link="laser_base_link" />
+        <child link="laser_servo_link" />
         <!-- ============================================================== -->
         <xacro:insert_block name="origin" />
@@ -118,5 +118,5 @@
         <!-- ============================================================== -->
         <parent link="${parent}" />
-        <child link="laser_base_link" />
+        <child link="laser_servo_link" />
         <!-- ============================================================== -->
         <xacro:insert_block name="origin" />
@@ -147,5 +147,5 @@
              type="fixed" >
         <!-- ============================================================== -->
-        <parent link="laser_base_link" />
+        <parent link="laser_servo_link" />
         <child link="laser_main_link" />
         <!-- ============================================================== -->
@@ -159,5 +159,5 @@
              type="revolute" >
         <!-- ============================================================== -->
-        <parent link="laser_base_link" />
+        <parent link="laser_servo_link" />
         <child link="laser_main_link" />
         <!-- ============================================================== -->

File: pandora_sensors_description/urdf/kinect_camera.urdf.xacro (robot description, xacro)
@@ -11,5 +11,5 @@
                        *origin" >
     <!-- ################################################################## -->
-    <link name="kinect_base_link" >
+    <link name="kinect_servo_link" >
       <inertial>
         <!-- ============================================================== -->
@@ -48,8 +48,45 @@
     </link>
     <!-- ################################################################## -->
+    <link name="kinect_base_link" >
+      <inertial>
+        <!-- ============================================================== -->
+        <origin xyz="0.03416 0.0 0.01146" />
+        <!-- ============================================================== -->
+        <mass value="0.0001" /><!--FIXME-->
+        <!-- ============================================================== -->
+        <inertia ixx="0.00000001"
+                 ixy="0"
+                 ixz="0"
+                 iyy="0.00000001"
+                 iyz="0"
+                 izz="0.00000001" /><!--FIXME-->
+        <!-- ============================================================== -->
+      </inertial>
+      <visual>
+        <!-- ============================================================== -->
+        <origin xyz="0 0 0"
+                rpy="0 0 0" />
+        <!-- ============================================================== -->
+        <geometry>
+          <mesh filename="package://pandora_sensors_description/meshes/kinect_camera/kinect_base.dae" />
+        </geometry>
+        <!-- ============================================================== -->
+      </visual>
+      <collision>
+        <!-- ============================================================== -->
+        <origin xyz="0.02131 0.0 0.01992"
+                rpy="0 0 0" />
+        <!-- ============================================================== -->
+        <geometry>
+          <box size="0.07 0.055 0.04" />
+        </geometry>
+        <!-- ============================================================== -->
+      </collision>
+    </link>
+    <!-- ################################################################## -->
     <link name="kinect_main_link" >
       <inertial>
         <!-- ============================================================== -->
-        <origin xyz="0.0023 -0.00024 0.01818" />
+        <origin xyz="0.00052 0.00048 0.02055" />
         <!-- ============================================================== -->
         <mass value="0.226796185" />
@@ -69,5 +106,5 @@
         <!-- ============================================================== -->
         <geometry>
-          <mesh filename="package://pandora_sensors_description/meshes/kinect_camera/kinect_camera_simple.dae" />
+          <mesh filename="package://pandora_sensors_description/meshes/kinect_camera/asus_xtion_pro.dae" />
         </geometry>
         <!-- ============================================================== -->
@@ -75,9 +112,9 @@
       <collision>
         <!-- ============================================================== -->
-        <origin xyz="0.0 0.0 0.018"
-                rpy="0 0 0" />
-        <!-- ============================================================== -->
-        <geometry>
-          <box size="0.079 0.295 0.055" />
+        <origin xyz="0.0 0.0 0.01342"
+                rpy="0 0 0" />
+        <!-- ============================================================== -->
+        <geometry>
+          <box size="0.037 0.18 0.042" />
         </geometry>
         <!-- ============================================================== -->
@@ -192,5 +229,5 @@
         <!-- ============================================================== -->
         <parent link="${parent}" />
-        <child link="kinect_base_link" />
+        <child link="kinect_servo_link" />
         <!-- ============================================================== -->
         <xacro:insert_block name="origin" />
@@ -203,5 +240,5 @@
         <!-- ============================================================== -->
         <parent link="${parent}" />
-        <child link="kinect_base_link" />
+        <child link="kinect_servo_link" />
         <!-- ============================================================== -->
         <xacro:insert_block name="origin" />
@@ -232,6 +269,6 @@
              type="fixed" >
         <!-- ============================================================== -->
-        <parent link="kinect_base_link" />
-        <child link="kinect_main_link" />
+        <parent link="kinect_servo_link" />
+        <child link="kinect_base_link" />
         <!-- ============================================================== -->
         <origin xyz="0.037 0.0 0.021"
@@ -244,6 +281,6 @@
              type="revolute" >
         <!-- ============================================================== -->
-        <parent link="kinect_base_link" />
-        <child link="kinect_main_link" />
+        <parent link="kinect_servo_link" />
+        <child link="kinect_base_link" />
         <!-- ============================================================== -->
         <origin xyz="0.037 0.0 0.021"
@@ -270,4 +307,15 @@
       </joint>
     </xacro:unless>
+    <!-- Base Joint ########################################################-->
+    <joint name="kinect_base_joint"
+           type="fixed" >
+      <!-- ================================================================ -->
+      <parent link="kinect_base_link" />
+      <child link="kinect_main_link" />
+      <!-- ================================================================ -->
+      <origin xyz="0.04274 0.0 0.03142"
+              rpy="0.0 0.0 0.0" />
+      <!-- ================================================================ -->
+    </joint>
     <!-- Camera Joint ##################################################### -->
     <joint name="kinect_joint"
@@ -277,5 +325,5 @@
       <child link="kinect_frame" />
       <!-- ================================================================ -->
-      <origin xyz="0.03016 0.0 0.01781"
+      <origin xyz="0.01784 0.0 0.02167"
               rpy="0.0 0.0 0.0" />
       <!-- ================================================================ -->
