Commit message: Refactor sensors_description package

File: pandora_sensors_description/urdf/camera.urdf.xacro (robot description, xacro)
@@ -3,15 +3,11 @@
   <xacro:include filename="$(find pandora_urdf_properties)/xacro/constants.xacro" />
   <xacro:include filename="$(find pandora_urdf_properties)/xacro/defaults.xacro" />
-<!-- ###################################################################### -->
   <xacro:macro name="camera_caster"
                params="parent prefix_y *origin" >
-    <!-- ################################################################## -->
-    <link name="${prefix_y}_camera_main_link" >
+    <!-- Links ############################################################ -->
+    <link name="${prefix_y}_camera_link" >
       <inertial>
-        <!-- ============================================================== -->
         <origin xyz="0.00972 0.0 0.04428" />
-        <!-- ============================================================== -->
         <mass value="0.005" />
-        <!-- ============================================================== -->
         <inertia ixx="2.1208E-7"
                  ixy="0"
@@ -20,95 +16,46 @@
                  iyz="0"
                  izz="2.1208E-7" />
-        <!-- ============================================================== -->
       </inertial>
       <visual>
-        <!-- ============================================================== -->
-        <origin xyz="0 0 0"
-                rpy="0 0 0" />
-        <!-- ============================================================== -->
         <geometry>
           <mesh filename="package://pandora_sensors_description/meshes/camera/logitech.dae" />
         </geometry>
-        <!-- ============================================================== -->
       </visual>
       <collision>
-        <!-- ============================================================== -->
         <origin xyz="0.00557 0.0 0.03624"
                 rpy="0 0 0" />
-        <!-- ============================================================== -->
         <geometry>
           <box size="0.049 0.095 0.073" />
         </geometry>
-        <!-- ============================================================== -->
       </collision>
     </link>
-    <!-- ################################################################## -->
+    <!-- Joints ########################################################### -->
+    <joint name="${prefix_y}_camera_parent_joint"
+           type="fixed" >
+      <parent link="${parent}" />
+      <child link="${prefix_y}_camera_link" />
+      <xacro:insert_block name="origin" />
+    </joint>
+    <!-- Frames ########################################################### -->
     <link name="${prefix_y}_camera_frame" >
-      <inertial>
-        <!-- ============================================================== -->
-        <origin xyz="0.0 0.0 0.0" />
-        <!-- ============================================================== -->
-        <mass value="0.005" />
-        <!-- ============================================================== -->
-        <inertia ixx="1.0E-6"
-                 ixy="0"
-                 ixz="0"
-                 iyy="1.0E-6"
-                 iyz="0"
-                 izz="1.0E-6" />
-        <!-- ============================================================== -->
-      </inertial>
+      <xacro:point_mass_inertial />
     </link>
-    <!-- ################################################################## -->
     <link name="${prefix_y}_camera_optical_frame" >
-      <inertial>
-        <!-- ============================================================== -->
-        <origin xyz="0.0 0.0 0.0" />
-        <!-- ============================================================== -->
-        <mass value="0.005" />
-        <!-- ============================================================== -->
-        <inertia ixx="1.0E-6"
-                 ixy="0"
-                 ixz="0"
-                 iyy="1.0E-6"
-                 iyz="0"
-                 izz="1.0E-6" />
-        <!-- ============================================================== -->
-      </inertial>
+      <xacro:point_mass_inertial />
     </link>
-    <!-- ################################################################## -->
-    <joint name="${prefix_y}_camera_main_joint"
-           type="fixed" >
-      <!-- ================================================================ -->
-      <parent link="${parent}" />
-      <child link="${prefix_y}_camera_main_link" />
-      <!-- ================================================================ -->
-      <xacro:insert_block name="origin" />
-      <!-- ================================================================ -->
-    </joint>
-    <!-- ################################################################## -->
     <joint name="${prefix_y}_camera_joint"
            type="fixed" >
-      <!-- ================================================================ -->
-      <parent link="${prefix_y}_camera_main_link" />
+      <parent link="${prefix_y}_camera_link" />
       <child link="${prefix_y}_camera_frame" />
-      <!-- ================================================================ -->
       <origin xyz="0.02499 0.0 0.05704"
               rpy="0.0 -0.2792 0.0" />
-      <!-- ================================================================ -->
     </joint>
-    <!-- ################################################################## -->
     <joint name="${prefix_y}_camera_optical_joint"
            type="fixed" >
-      <!-- ================================================================ -->
       <parent link="${prefix_y}_camera_frame" />
       <child link="${prefix_y}_camera_optical_frame" />
-      <!-- ================================================================ -->
       <origin xyz="0.0 0.0 0.0"
               rpy="-1.5708 0.0 -1.5708" />
-      <!-- ================================================================ -->
     </joint>
-    <!-- ################################################################## -->
   </xacro:macro>
-<!-- ###################################################################### -->
 </robot>

File: pandora_sensors_description/urdf/co2.urdf.xacro (robot description, xacro)
@@ -3,15 +3,11 @@
   <xacro:include filename="$(find pandora_urdf_properties)/xacro/constants.xacro" />
   <xacro:include filename="$(find pandora_urdf_properties)/xacro/defaults.xacro" />
-<!-- ###################################################################### -->
   <xacro:macro name="co2_caster"
                params="parent *origin" >
-    <!-- ################################################################## -->
+    <!-- Links ############################################################ -->
     <link name="co2_link" >
       <inertial>
-        <!-- ============================================================== -->
         <origin xyz="0.005 0.0 0.0" />
-        <!-- ============================================================== -->
         <mass value="0.005" />
-        <!-- ============================================================== -->
         <inertia ixx="2.1208E-7"
                  ixy="0"
@@ -20,67 +16,36 @@
                  iyz="0"
                  izz="2.1208E-7" />
-        <!-- ============================================================== -->
       </inertial>
       <visual>
-        <!-- ============================================================== -->
-        <origin xyz="0 0 0"
-                rpy="0 0 0" />
-        <!-- ============================================================== -->
         <geometry>
           <mesh filename="package://pandora_sensors_description/meshes/co2/dynament.dae" />
         </geometry>
-        <!-- ============================================================== -->
       </visual>
       <collision>
-        <!-- ============================================================== -->
         <origin xyz="0.0075 0.0 0.0"
                 rpy="0 0 0" />
-        <!-- ============================================================== -->
         <geometry>
           <box size="0.015 0.022 0.022" />
         </geometry>
-        <!-- ============================================================== -->
       </collision>
     </link>
-    <!-- ################################################################## -->
-    <link name="co2_frame" >
-      <inertial>
-        <!-- ============================================================== -->
-        <origin xyz="0.0 0.0 0.0" />
-        <!-- ============================================================== -->
-        <mass value="0.005" />
-        <!-- ============================================================== -->
-        <inertia ixx="1.0E-6"
-                 ixy="0"
-                 ixz="0"
-                 iyy="1.0E-6"
-                 iyz="0"
-                 izz="1.0E-6" />
-        <!-- ============================================================== -->
-      </inertial>
-    </link>
-    <!-- ################################################################## -->
-    <joint name="co2_main_joint"
+    <!-- Joints ########################################################### -->
+    <joint name="co2_parent_joint"
            type="fixed" >
-      <!-- ================================================================ -->
       <parent link="${parent}" />
       <child link="co2_link" />
-      <!-- ================================================================ -->
       <xacro:insert_block name="origin" />
-      <!-- ================================================================ -->
     </joint>
-    <!-- ################################################################## -->
+    <!-- Frames ########################################################### -->
+    <link name="co2_frame" >
+      <xacro:point_mass_inertial />
+    </link>
     <joint name="co2_joint"
            type="fixed" >
-      <!-- ================================================================ -->
       <parent link="co2_link" />
       <child link="co2_frame" />
-      <!-- ================================================================ -->
       <origin xyz="0.015 0.0 0.0"
               rpy="0.0 0.0 0.0" />
-      <!-- ================================================================ -->
     </joint>
-    <!-- ################################################################## -->
   </xacro:macro>
-<!-- ###################################################################### -->
 </robot>

File: pandora_sensors_description/urdf/flir.urdf.xacro (robot description, xacro)
@@ -3,15 +3,11 @@
   <xacro:include filename="$(find pandora_urdf_properties)/xacro/constants.xacro" />
   <xacro:include filename="$(find pandora_urdf_properties)/xacro/defaults.xacro" />
-<!-- ###################################################################### -->
   <xacro:macro name="flir_caster"
                params="parent *origin" >
-    <!-- ################################################################## -->
-    <link name="flir_main_link" >
+    <!-- Links ############################################################ -->
+    <link name="flir_link" >
       <inertial>
-        <!-- ============================================================== -->
         <origin xyz="0.00126 0.0 0.0" />
-        <!-- ============================================================== -->
         <mass value="0.005" />
-        <!-- ============================================================== -->
         <inertia ixx="2.1208E-7"
                  ixy="0"
@@ -20,95 +16,46 @@
                  iyz="0"
                  izz="2.1208E-7" />
-        <!-- ============================================================== -->
       </inertial>
       <visual>
-        <!-- ============================================================== -->
-        <origin xyz="0 0 0"
-                rpy="0 0 0" />
-        <!-- ============================================================== -->
         <geometry>
           <mesh filename="package://pandora_sensors_description/meshes/flir/flir.dae" />
         </geometry>
-        <!-- ============================================================== -->
       </visual>
       <collision>
-        <!-- ============================================================== -->
         <origin xyz="0.00225 0.0 0.0"
                 rpy="0 0 0" />
-        <!-- ============================================================== -->
         <geometry>
           <box size="0.004 0.020 0.037" />
         </geometry>
-        <!-- ============================================================== -->
       </collision>
     </link>
-    <!-- ################################################################## -->
+    <!-- Joints ########################################################### -->
+    <joint name="flir_parent_joint"
+           type="fixed" >
+      <parent link="${parent}" />
+      <child link="flir_link" />
+      <xacro:insert_block name="origin" />
+    </joint>
+    <!-- Frames ########################################################### -->
     <link name="flir_frame" >
-      <inertial>
-        <!-- ============================================================== -->
-        <origin xyz="0.0 0.0 0.0" />
-        <!-- ============================================================== -->
-        <mass value="0.005" />
-        <!-- ============================================================== -->
-        <inertia ixx="1.0E-6"
-                 ixy="0"
-                 ixz="0"
-                 iyy="1.0E-6"
-                 iyz="0"
-                 izz="1.0E-6" />
-        <!-- ============================================================== -->
-      </inertial>
+      <xacro:point_mass_inertial />
     </link>
-    <!-- ################################################################## -->
     <link name="flir_optical_frame" >
-      <inertial>
-        <!-- ============================================================== -->
-        <origin xyz="0.0 0.0 0.0" />
-        <!-- ============================================================== -->
-        <mass value="0.005" />
-        <!-- ============================================================== -->
-        <inertia ixx="1.0E-6"
-                 ixy="0"
-                 ixz="0"
-                 iyy="1.0E-6"
-                 iyz="0"
-                 izz="1.0E-6" />
-        <!-- ============================================================== -->
-      </inertial>
+      <xacro:point_mass_inertial />
     </link>
-    <!-- ################################################################## -->
-    <joint name="flir_main_joint"
-           type="fixed" >
-      <!-- ================================================================ -->
-      <parent link="${parent}" />
-      <child link="flir_main_link" />
-      <!-- ================================================================ -->
-      <xacro:insert_block name="origin" />
-      <!-- ================================================================ -->
-    </joint>
-    <!-- ################################################################## -->
     <joint name="flir_joint"
            type="fixed" >
-      <!-- ================================================================ -->
-      <parent link="flir_main_link" />
+      <parent link="flir_link" />
       <child link="flir_frame" />
-      <!-- ================================================================ -->
       <origin xyz="0.0045 0.0 0.00125"
               rpy="0.0 0.0 0.0" />
-      <!-- ================================================================ -->
     </joint>
-    <!-- ################################################################## -->
     <joint name="flir_optical_joint"
            type="fixed" >
-      <!-- ================================================================ -->
       <parent link="flir_frame" />
       <child link="flir_optical_frame" />
-      <!-- ================================================================ -->
       <origin xyz="0.0 0.0 0.0"
               rpy="-1.5708 0.0 -1.5708" />
-      <!-- ================================================================ -->
     </joint>
-    <!-- ################################################################## -->
   </xacro:macro>
-<!-- ###################################################################### -->
 </robot>

File: pandora_sensors_description/urdf/microphone.urdf.xacro (robot description, xacro)
@@ -3,15 +3,11 @@
   <xacro:include filename="$(find pandora_urdf_properties)/xacro/constants.xacro" />
   <xacro:include filename="$(find pandora_urdf_properties)/xacro/defaults.xacro" />
-<!-- ###################################################################### -->
   <xacro:macro name="microphone_caster"
                params="parent *origin" >
-    <!-- ################################################################## -->
+    <!-- Links ############################################################ -->
     <link name="microphone_link" >
       <inertial>
-        <!-- ============================================================== -->
         <origin xyz="0.01177 0.0 0.0" />
-        <!-- ============================================================== -->
         <mass value="0.005" />
-        <!-- ============================================================== -->
         <inertia ixx="2.1208E-7"
                  ixy="0"
@@ -20,67 +16,36 @@
                  iyz="0"
                  izz="2.1208E-7" />
-        <!-- ============================================================== -->
       </inertial>
       <visual>
-        <!-- ============================================================== -->
-        <origin xyz="0 0 0"
-                rpy="0 0 0" />
-        <!-- ============================================================== -->
         <geometry>
           <mesh filename="package://pandora_sensors_description/meshes/microphone/kinect_array.dae" />
         </geometry>
-        <!-- ============================================================== -->
       </visual>
       <collision>
-        <!-- ============================================================== -->
         <origin xyz="0.0 0.0 0.01"
                 rpy="0 0 0" />
-        <!-- ============================================================== -->
         <geometry>
           <box size="0.053 0.055 0.020" />
         </geometry>
-        <!-- ============================================================== -->
       </collision>
     </link>
-    <!-- ################################################################## -->
-    <link name="microphone_frame" >
-      <inertial>
-        <!-- ============================================================== -->
-        <origin xyz="0.0 0.0 0.0" />
-        <!-- ============================================================== -->
-        <mass value="0.005" />
-        <!-- ============================================================== -->
-        <inertia ixx="1.0E-6"
-                 ixy="0"
-                 ixz="0"
-                 iyy="1.0E-6"
-                 iyz="0"
-                 izz="1.0E-6" />
-        <!-- ============================================================== -->
-      </inertial>
-    </link>
-    <!-- ################################################################## -->
-    <joint name="microphone_main_joint"
+    <!-- Joints ########################################################### -->
+    <joint name="microphone_parent_joint"
            type="fixed" >
-      <!-- ================================================================ -->
       <parent link="${parent}" />
       <child link="microphone_link" />
-      <!-- ================================================================ -->
       <xacro:insert_block name="origin" />
-      <!-- ================================================================ -->
     </joint>
-    <!-- ################################################################## -->
+    <!-- Frames ########################################################### -->
+    <link name="microphone_frame" >
+      <xacro:point_mass_inertial />
+    </link>
     <joint name="microphone_joint"
            type="fixed" >
-      <!-- ================================================================ -->
       <parent link="microphone_link" />
       <child link="microphone_frame" />
-      <!-- ================================================================ -->
       <origin xyz="0.0 0.0 0.0125"
               rpy="0.0 0.0 0.0" />
-      <!-- ================================================================ -->
     </joint>
-    <!-- ################################################################## -->
   </xacro:macro>
-<!-- ###################################################################### -->
 </robot>
