Commit message: Refactor sensors_description package

File: pandora_sensors_description/urdf/sonar.urdf.xacro (robot description, xacro)
@@ -3,15 +3,11 @@
   <xacro:include filename="$(find pandora_urdf_properties)/xacro/constants.xacro" />
   <xacro:include filename="$(find pandora_urdf_properties)/xacro/defaults.xacro" />
-<!-- ###################################################################### -->
   <xacro:macro name="sonar_caster"
                params="parent name *origin" >
-    <!-- ################################################################## -->
+    <!-- Links ############################################################ -->
     <link name="${name}_sonar_link" >
       <inertial>
-        <!-- ============================================================== -->
         <origin xyz="0.005 0.0 0.0" />
-        <!-- ============================================================== -->
         <mass value="0.010" />
-        <!-- ============================================================== -->
         <inertia ixx="4.2416E-7"
                  ixy="0.0"
@@ -20,67 +16,36 @@
                  iyz="0.0"
                  izz="1.6341E-6" />
-        <!-- ============================================================== -->
       </inertial>
       <visual>
-        <!-- ============================================================== -->
-        <origin xyz="0 0 0"
-                rpy="0 0 0" />
-        <!-- ============================================================== -->
         <geometry>
           <mesh filename="package://pandora_sensors_description/meshes/sonar/sonar_new.dae" />
         </geometry>
-        <!-- ============================================================== -->
       </visual>
       <collision>
-        <!-- ============================================================== -->
         <origin xyz="0.0075 0.0 0.0"
                 rpy="0 0 0" />
-        <!-- ============================================================== -->
         <geometry>
           <box size="0.015 0.044 0.022" />
         </geometry>
-        <!-- ============================================================== -->
       </collision>
     </link>
-    <!-- ################################################################## -->
-    <link name="${name}_sonar_frame" >
-      <inertial>
-        <!-- ============================================================== -->
-        <origin xyz="0.0 0.0 0.0" />
-        <!-- ============================================================== -->
-        <mass value="0.005" />
-        <!-- ============================================================== -->
-        <inertia ixx="1.0E-6"
-                 ixy="0"
-                 ixz="0"
-                 iyy="1.0E-6"
-                 iyz="0"
-                 izz="1.0E-6" />
-        <!-- ============================================================== -->
-      </inertial>
-    </link>
-    <!-- ################################################################## -->
-    <joint name="${name}_sonar_main_joint"
+    <!-- Joints ########################################################### -->
+    <joint name="${name}_sonar_parent_joint"
            type="fixed" >
-      <!-- ================================================================ -->
       <parent link="${parent}" />
       <child link="${name}_sonar_link" />
-      <!-- ================================================================ -->
       <xacro:insert_block name="origin" />
-      <!-- ================================================================ -->
     </joint>
-    <!-- ################################################################## -->
+    <!-- Frames ########################################################### -->
+    <link name="${name}_sonar_frame" >
+      <xacro:point_mass_inertial />
+    </link>
     <joint name="${name}_sonar_joint"
            type="fixed" >
-      <!-- ================================================================ -->
       <parent link="${name}_sonar_link" />
       <child link="${name}_sonar_frame" />
-      <!-- ================================================================ -->
       <origin xyz="0.015 0.0 0.0"
               rpy="0.0 0.0 0.0" />
-      <!-- ================================================================ -->
     </joint>
-    <!-- ################################################################## -->
   </xacro:macro>
-<!-- ###################################################################### -->
 </robot>

File: pandora_sensors_description/urdf/thermal.urdf.xacro (robot description, xacro)
@@ -3,15 +3,11 @@
   <xacro:include filename="$(find pandora_urdf_properties)/xacro/constants.xacro" />
   <xacro:include filename="$(find pandora_urdf_properties)/xacro/defaults.xacro" />
-<!-- ###################################################################### -->
   <xacro:macro name="thermal_caster"
                params="parent prefix_y *origin" >
-    <!-- ################################################################## -->
-    <link name="${prefix_y}_thermal_main_link" >
+    <!-- Links ############################################################ -->
+    <link name="${prefix_y}_thermal_link" >
       <inertial>
-        <!-- ============================================================== -->
         <origin xyz="0.00126 0.0 0.0" />
-        <!-- ============================================================== -->
         <mass value="0.005" />
-        <!-- ============================================================== -->
         <inertia ixx="2.1208E-7"
                  ixy="0"
@@ -20,95 +16,46 @@
                  iyz="0"
                  izz="2.1208E-7" />
-        <!-- ============================================================== -->
       </inertial>
       <visual>
-        <!-- ============================================================== -->
-        <origin xyz="0 0 0"
-                rpy="0 0 0" />
-        <!-- ============================================================== -->
         <geometry>
           <mesh filename="package://pandora_sensors_description/meshes/thermal/grid_eye.dae" />
         </geometry>
-        <!-- ============================================================== -->
       </visual>
       <collision>
-        <!-- ============================================================== -->
         <origin xyz="0.00225 0.0 0.0"
                 rpy="0 0 0" />
-        <!-- ============================================================== -->
         <geometry>
           <box size="0.004 0.020 0.037" />
         </geometry>
-        <!-- ============================================================== -->
       </collision>
     </link>
-    <!-- ################################################################## -->
+    <!-- Joints ########################################################### -->
+    <joint name="${prefix_y}_thermal_parent_joint"
+           type="fixed" >
+      <parent link="${parent}" />
+      <child link="${prefix_y}_thermal_link" />
+      <xacro:insert_block name="origin" />
+    </joint>
+    <!-- Frames ########################################################### -->
     <link name="${prefix_y}_thermal_frame" >
-      <inertial>
-        <!-- ============================================================== -->
-        <origin xyz="0.0 0.0 0.0" />
-        <!-- ============================================================== -->
-        <mass value="0.005" />
-        <!-- ============================================================== -->
-        <inertia ixx="1.0E-6"
-                 ixy="0"
-                 ixz="0"
-                 iyy="1.0E-6"
-                 iyz="0"
-                 izz="1.0E-6" />
-        <!-- ============================================================== -->
-      </inertial>
+      <xacro:point_mass_inertial />
     </link>
-    <!-- ################################################################## -->
     <link name="${prefix_y}_thermal_optical_frame" >
-      <inertial>
-        <!-- ============================================================== -->
-        <origin xyz="0.0 0.0 0.0" />
-        <!-- ============================================================== -->
-        <mass value="0.005" />
-        <!-- ============================================================== -->
-        <inertia ixx="1.0E-6"
-                 ixy="0"
-                 ixz="0"
-                 iyy="1.0E-6"
-                 iyz="0"
-                 izz="1.0E-6" />
-        <!-- ============================================================== -->
-      </inertial>
+      <xacro:point_mass_inertial />
     </link>
-    <!-- ################################################################## -->
-    <joint name="${prefix_y}_thermal_main_joint"
-           type="fixed" >
-      <!-- ================================================================ -->
-      <parent link="${parent}" />
-      <child link="${prefix_y}_thermal_main_link" />
-      <!-- ================================================================ -->
-      <xacro:insert_block name="origin" />
-      <!-- ================================================================ -->
-    </joint>
-    <!-- ################################################################## -->
     <joint name="${prefix_y}_thermal_joint"
            type="fixed" >
-      <!-- ================================================================ -->
-      <parent link="${prefix_y}_thermal_main_link" />
+      <parent link="${prefix_y}_thermal_link" />
       <child link="${prefix_y}_thermal_frame" />
-      <!-- ================================================================ -->
       <origin xyz="0.0045 0.0 0.00125"
               rpy="0.0 0.0 0.0" />
-      <!-- ================================================================ -->
     </joint>
-    <!-- ################################################################## -->
     <joint name="${prefix_y}_thermal_optical_joint"
            type="fixed" >
-      <!-- ================================================================ -->
       <parent link="${prefix_y}_thermal_frame" />
       <child link="${prefix_y}_thermal_optical_frame" />
-      <!-- ================================================================ -->
       <origin xyz="0.0 0.0 0.0"
               rpy="-1.5708 0.0 -1.5708" />
-      <!-- ================================================================ -->
     </joint>
-    <!-- ################################################################## -->
   </xacro:macro>
-<!-- ###################################################################### -->
 </robot>
