Commit message: Fix logitech stick pose

File: pandora_sensors_description/urdf/logitec_stick.urdf.xacro (robot description, xacro)
@@ -69,8 +69,8 @@
            type="fixed" >
       <!-- ================================================================ -->
-      <parent link="kinect_link" />
+      <parent link="base_link" />
       <child link="logitec_stick_base_link" />
       <!-- ================================================================ -->
-      <origin xyz="0.0 0.0 0.013"
+      <origin xyz="0.022 0.015 0.484"
               rpy="0.0 0.0 0.0" />
       <!-- ================================================================ -->
@@ -83,5 +83,5 @@
       <child link="logitec_stick_camera_frame" />
       <!-- ================================================================ -->
-      <origin xyz="0.027 0.0 0.266"
+      <origin xyz="0.0 0.0 0.0"
               rpy="0.0 0.0 0.0" />
       <!-- ================================================================ -->

Commit message: Removes visual box from logitec_stick urdf

File: pandora_sensors_description/urdf/logitec_stick.urdf.xacro (robot description, xacro)
@@ -20,14 +20,4 @@
         <!-- ============================================================== -->
       </inertial>>
-      <visual>
-        <!-- ============================================================== -->
-        <!-- <origin xyz="0 0 1" /> -->
-        <!-- ============================================================== -->
-        <geometry>
-          <origin xyz="0 0 1" />
-          <box size="0.5 0.5 0.3" />
-        </geometry>
-        <!-- ============================================================== -->
-      </visual>
     </link>
     <!-- ################################################################## -->
