Commit message: Changed inertia in sensors' and pioneer3at's urdfs and file names from smp to gears_smp

File: pandora_robots_description/urdf/gears_smp.urdf.xacro (robot description, xacro)
@@ -5,5 +5,5 @@
        xmlns:xacro="http://ros.org/wiki/xacro"
        name="smp">
-  <xacro:include filename="$(find pandora_robots_description)/urdf/smp_skeleton.urdf.xacro" />
+  <xacro:include filename="$(find pandora_robots_description)/urdf/gears_smp_skeleton.urdf.xacro" />
   <link
     name="base_link">
@@ -52,4 +52,9 @@
     <origin xyz="0 -0.0915 0" rpy="0 0 0" />
   </xacro:skeleton_caster>
+  <!--Insert kinect-->
+  <xacro:include filename="$(find pandora_sensors_description)/urdf/kinect_camera.urdf.xacro" />
+  <xacro:kinect_caster parent="base_link">
+    <origin xyz="0.2 0 0.33" rpy="0 0 0"/>
+  </xacro:kinect_caster>
   <!-- Add ros_control plugin-->
   <gazebo>

File: pandora_robots_description/urdf/gears_smp_skeleton.urdf.xacro (robot description, xacro)
@@ -1,5 +1,5 @@
 <?xml version="1.0" ?>
 <robot xmlns:xacro="http://ros.org/wiki/xacro">
-  <xacro:include filename="$(find pandora_robots_description)/urdf/smp_wheel.urdf.xacro" />
+  <xacro:include filename="$(find pandora_robots_description)/urdf/gears_smp_wheel.urdf.xacro" />
   <xacro:macro name="skeleton_caster" params="suffix reflect parent *origin">
     <link

File: pandora_robots_description/urdf/pioneer3at.urdf.xacro (robot description, xacro)
@@ -8,8 +8,7 @@
   <link name="base_link">
     <inertial>
-      <mass value="10.0"/>
-      <origin xyz="0 0 0"/>
-      <inertia ixx="0.3338" ixy="0.0" ixz="0.0"
-         iyy="0.4783" iyz="0.0"
+      <mass value="14.0"/>
+      <inertia ixx="0.3338" ixy="0" ixz="0"
+         iyy="0.4783" iyz="0"
          izz="0.3338"/>
     </inertial>
@@ -38,7 +37,7 @@
       <mass value="0.1"/>
       <origin xyz="0 0 0" rpy="0 0 0"/>
-      <inertia ixx="1.0" ixy="0.0" ixz="0.0"
-         iyy="1.0" iyz="0.0"
-        izz="1.0"/>
+      <inertia ixx="0.001" ixy="0.0" ixz="0.0"
+         iyy="0.001" iyz="0.0"
+        izz="0.001"/>
     </inertial>
     <visual name="base_visual">
@@ -72,6 +71,6 @@
         <mass value="0.1"/>
         <origin xyz="0 0 0"/>
-        <inertia ixx="1.0" ixy="0.0" ixz="0.0"
-           iyy="1.0" iyz="0.0" izz="1.0"/>
+        <inertia ixx="0.001" ixy="0.0" ixz="0.0"
+           iyy="0.001" iyz="0.0" izz="0.001"/>
         </inertial>
     <visual name="base_visual">
@@ -103,6 +102,6 @@
         <mass value="0.1"/>
         <origin xyz="0 0 0"/>
-        <inertia ixx="1.0" ixy="0.0" ixz="0.0"
-           iyy="1.0" iyz="0.0" izz="1.0"/>
+        <inertia ixx="0.001" ixy="0.0" ixz="0.0"
+           iyy="0.001" iyz="0.0" izz="0.001"/>
         </inertial>
     <visual name="base_visual">
@@ -171,6 +170,6 @@
         <mass value="0.1"/>
         <origin xyz="0 0 0"/>
-        <inertia ixx="1.0" ixy="0.0" ixz="0.0"
-           iyy="1.0" iyz="0.0" izz="1.0"/>
+        <inertia ixx="0.001" ixy="0.0" ixz="0.0"
+           iyy="0.001" iyz="0.0" izz="0.001"/>
         </inertial>
     <visual name="base_visual">
@@ -202,6 +201,6 @@
         <mass value="0.1"/>
         <origin xyz="0 0 0"/>
-        <inertia ixx="1.0" ixy="0.0" ixz="0.0"
-           iyy="1.0" iyz="0.0" izz="1.0"/>
+        <inertia ixx="0.001" ixy="0.0" ixz="0.0"
+           iyy="0.001" iyz="0.0" izz="0.001"/>
         </inertial>
     <visual name="base_visual">
@@ -343,5 +342,5 @@
   <xacro:include filename="$(find pandora_sensors_description)/urdf/kinect_camera.urdf.xacro" />
   <xacro:kinect_caster parent="base_link">
-    <origin xyz="0.2 0 0.33" rpy="0 0 0"/>
+    <origin xyz="0.2 0 0.33" rpy="0 0.53 0"/>
   </xacro:kinect_caster>
   <!--Insert sonars-->

File: pandora_sensors_description/urdf/co2_sensor.urdf.xacro (robot description, xacro)
@@ -3,17 +3,17 @@
 <xacro:macro name="co2_caster" params="parent *origin">
       <link name="co2_link">
-		  <inertial>
-			<mass value="0.1"/>
-			<origin xyz="0 0 0"/>
-			<inertia ixx="1" ixy="0" ixz="0" iyy="1" iyz="0" izz="1" />
-		  </inertial>
+      <inertial>
+      <mass value="0.1"/>
+      <origin xyz="0 0 0"/>
+      <inertia ixx="0.0001" ixy="0" ixz="0" iyy="0.0001" iyz="0" izz="0.0001" />
+      </inertial>
         <visual name="visual">
-		  <origin xyz="0 0 0" rpy="0 0 0"/>
+      <origin xyz="0 0 0" rpy="0 0 0"/>
           <geometry>
-			<mesh filename="package://pandora_sensors_description/meshes/co2_sensor/co2_small.dae"/>
+      <mesh filename="package://pandora_sensors_description/meshes/co2_sensor/co2_small.dae"/>
           </geometry>
         </visual>
         <collision name="collision">
-		  <origin xyz="0 0 0" rpy="0 0 0"/>
+      <origin xyz="0 0 0" rpy="0 0 0"/>
           <geometry>
             <box size="0.01 0.01 0.01"/>
@@ -22,30 +22,30 @@
     </link>
     <gazebo reference="co2_link">
-		<sensor name="co2" type="camera">
-        <camera>
-          <horizontal_fov>1.5</horizontal_fov>
-          <image>
-            <width>640</width>
-            <height>480</height>
-          </image>
-          <clip>
-            <near>0.1</near>
-            <far>0.8</far>
-          </clip>
-        </camera>
-        <always_on>1</always_on>
-        <update_rate>5</update_rate>
-        <visualize>false</visualize>
-        <plugin name="co2ros" filename="libpandora_co2_plugin.so">
-			<frameName>co2</frameName>
-			<topicName>sensors/co2</topicName>
-		</plugin>
-      </sensor>
-   </gazebo>
-   	<joint name="co2_joint" type="fixed">
-	  <xacro:insert_block name="origin" />
-      <parent link="${parent}"/>
-	  <child link="co2_link"/>
-	</joint>
+    <sensor name="co2" type="camera">
+      <camera>
+        <horizontal_fov>1.5</horizontal_fov>
+        <image>
+          <width>640</width>
+          <height>480</height>
+        </image>
+        <clip>
+          <near>0.1</near>
+          <far>0.8</far>
+        </clip>
+      </camera>
+      <always_on>1</always_on>
+      <update_rate>5</update_rate>
+      <visualize>false</visualize>
+      <plugin name="co2ros" filename="libpandora_co2_plugin.so">
+        <frameName>co2</frameName>
+        <topicName>sensors/co2</topicName>
+      </plugin>
+    </sensor>
+  </gazebo>
+  <joint name="co2_joint" type="fixed">
+    <xacro:insert_block name="origin" />
+    <parent link="${parent}"/>
+    <child link="co2_link"/>
+  </joint>
 </xacro:macro>
 </robot>

File: pandora_sensors_description/urdf/microphone_sensor.urdf.xacro (robot description, xacro)
@@ -2,50 +2,50 @@
 <robot xmlns:xacro="http://ros.org/wiki/xacro">
 <xacro:macro name="microphone_caster" params="parent *origin">
-      <link name="microphone_link">
-        <inertial>
-			<mass value="0.1"/>
-			<origin xyz="0 0 0"/>
-			<inertia ixx="1" ixy="0" ixz="0" iyy="1" iyz="0" izz="1" />
-		 </inertial>
-        <visual name="visual">
-		  <origin xyz="0 0 0" rpy="0 0 0"/>
-          <geometry>
-			<mesh filename="package://pandora_sensors_description/meshes/microphone_sensor/microphone_small.dae"/>
-          </geometry>
-        </visual>
-        <collision name="collision">
-          <origin xyz="0 0 0" rpy="0 0 0"/>
-          <geometry>
-            <box size="0.01 0.01 0.01"/>
-          </geometry>
-        </collision>
-    </link>
-    <gazebo reference="microphone_link">
-		<sensor name="microphone" type="camera">
-        <camera>
-          <horizontal_fov>1.5</horizontal_fov>
-          <image>
-            <width>640</width>
-            <height>480</height>
-          </image>
-          <clip>
-            <near>0.1</near>
-            <far>2</far>
-          </clip>
-        </camera>
-        <always_on>1</always_on>
-        <update_rate>10</update_rate>
-        <visualize>false</visualize>
-        <plugin name="microphone2ros" filename="libpandora_microphone_plugin.so">
-			<frameName>sound</frameName>
-			<topicName>sensors/sound</topicName>
-		</plugin>
-      </sensor>
-	</gazebo>
-	<joint name="microphone_joint" type="fixed">
-	  <xacro:insert_block name="origin" />
+  <link name="microphone_link">
+    <inertial>
+      <mass value="0.1"/>
+      <origin xyz="0 0 0"/>
+      <inertia ixx="0.0001" ixy="0" ixz="0" iyy="0.0001" iyz="0" izz="0.0001" />
+    </inertial>
+    <visual name="visual">
+      <origin xyz="0 0 0" rpy="0 0 0"/>
+      <geometry>
+        <mesh filename="package://pandora_sensors_description/meshes/microphone_sensor/microphone_small.dae"/>
+      </geometry>
+    </visual>
+    <collision name="collision">
+      <origin xyz="0 0 0" rpy="0 0 0"/>
+      <geometry>
+        <box size="0.01 0.01 0.01"/>
+      </geometry>
+    </collision>
+  </link>
+  <gazebo reference="microphone_link">
+    <sensor name="microphone" type="camera">
+      <camera>
+        <horizontal_fov>1.5</horizontal_fov>
+        <image>
+          <width>640</width>
+          <height>480</height>
+        </image>
+        <clip>
+          <near>0.1</near>
+          <far>2</far>
+        </clip>
+      </camera>
+      <always_on>1</always_on>
+      <update_rate>10</update_rate>
+      <visualize>false</visualize>
+      <plugin name="microphone2ros" filename="libpandora_microphone_plugin.so">
+        <frameName>sound</frameName>
+        <topicName>sensors/sound</topicName>
+      </plugin>
+    </sensor>
+  </gazebo>
+  <joint name="microphone_joint" type="fixed">
+    <xacro:insert_block name="origin" />
       <parent link="${parent}"/>
-	  <child link="microphone_link"/>
-	</joint>
+    <child link="microphone_link"/>
+  </joint>
 </xacro:macro>
 </robot>

File: pandora_sensors_description/urdf/sonar_sensor.urdf.xacro (robot description, xacro)
@@ -11,6 +11,6 @@
       <origin xyz="0 0 0.186" rpy="0 0 0"/>
       <mass value="0.001"/>
-      <inertia ixx="1.0" ixy="0.0" ixz="0.0"
-       iyy="1.0" iyz="0.0" izz="1.0"/>
+      <inertia ixx="0.0001" ixy="0.0" ixz="0.0"
+       iyy="0.0001" iyz="0.0" izz="0.0001"/>
     </inertial>
     <collision name="collision">

File: pandora_sensors_description/urdf/thermal_sensor.urdf.xacro (robot description, xacro)
@@ -2,24 +2,24 @@
 <robot xmlns:xacro="http://ros.org/wiki/xacro">
 <xacro:macro name="thermal_caster" params="parent *origin">
-      <link name="thermal_link">
-        <inertial>
-			<origin xyz="0 0 0.186" rpy="0 0 0"/>
-			<mass value="0.1"/>
-			<inertia ixx="1.0" ixy="0.0" ixz="0.0"
-					 iyy="1.0" iyz="0.0" izz="1.0"/>
-		</inertial>
-        <visual name="visual">
-          <geometry>
-			 <mesh filename="package://pandora_sensors_description/meshes/thermal_sensor/thermal_small.dae"/>
-          </geometry>
-        </visual>
-        <collision name="collision">
-          <geometry>
-            <box size="0.01 0.01 0.01"/>
-          </geometry>
-        </collision>
+    <link name="thermal_link">
+      <inertial>
+        <origin xyz="0 0 0.186" rpy="0 0 0"/>
+        <mass value="0.1"/>
+        <inertia ixx="0.0001" ixy="0.0" ixz="0.0"
+             iyy="0.0001" iyz="0.0" izz="0.0001"/>
+      </inertial>
+      <visual name="visual">
+        <geometry>
+         <mesh filename="package://pandora_sensors_description/meshes/thermal_sensor/thermal_small.dae"/>
+        </geometry>
+      </visual>
+      <collision name="collision">
+        <geometry>
+          <box size="0.01 0.01 0.01"/>
+        </geometry>
+      </collision>
     </link>
     <gazebo reference="thermal_link">
-		<sensor name="thermal" type="camera">
+    <sensor name="thermal" type="camera">
         <camera>
           <horizontal_fov>0.5</horizontal_fov>
@@ -37,14 +37,14 @@
         <visualize>false</visualize>
         <plugin name="thermal2ros" filename="libpandora_thermal_plugin.so">
-			<frameName>thermal_link</frameName>
-			<topicName>sensors/thermal</topicName>
-		</plugin>
+        <frameName>thermal_link</frameName>
+        <topicName>sensors/thermal</topicName>
+      </plugin>
       </sensor>
-	</gazebo>
-	<joint name="thermal_joint" type="fixed">
-	  <xacro:insert_block name="origin" />
+  </gazebo>
+  <joint name="thermal_joint" type="fixed">
+    <xacro:insert_block name="origin" />
       <parent link="${parent}"/>
-	  <child link="thermal_link"/>
-	</joint>
+    <child link="thermal_link"/>
+  </joint>
 </xacro:macro>
 </robot>
