Commit message: simulation with standalone models

File: pandora_robots_description/urdf/pioneer3at.urdf.xacro (robot description, xacro)
@@ -4,373 +4,373 @@
        xmlns:interface="http://playerstage.sourceforge.net/gazebo/xmlschema/#interface"
        xmlns:xacro="http://ros.org/wiki/xacro"
-	   name="pioneer3at">
+       name="pioneer3at">
 <!-- base_link -->
-	<link name="base_footprint"/>
-	<joint name="base_footprint_joint" type="fixed">
-		<origin xyz="0 0 0.177" rpy="0 0 0"/>
-		<parent link="base_footprint"/>
-		<child link="base_link"/>
-	</joint>
-	<link name="base_link">
-		<inertial>
-			<mass value="10.0"/>
-			<origin xyz="0 0 0"/>
-			<inertia ixx="0.3338" ixy="0.0" ixz="0.0"
-				 iyy="0.4783" iyz="0.0"
-				 izz="0.3338"/>
-		</inertial>
-		<visual name="base_visual">
-			<origin xyz="0 0 0" rpy="0 0 0"/>
-			<geometry name="pioneer_geom">
-				<mesh filename="package://pandora_robots_description/meshes/pioneer3at/p3at_meshes/chassis.stl"/>
-			</geometry>
-			<material name="ChassisRed">
-				<color rgba="0.851 0.0 0.0 1.0"/>
-			</material>
-		</visual>
-		<collision>
-			<origin xyz="0 0 0" rpy="0 0 0"/>
-				<geometry>
-					<mesh filename="package://pandora_robots_description/meshes/pioneer3at/p3at_meshes/chassis.stl"/>
-				</geometry>
-		</collision>
-	</link>
-	<gazebo reference="base_link">
-		<material value="Gazebo/Red"/>
-	</gazebo>
+  <link name="base_footprint"/>
+  <joint name="base_footprint_joint" type="fixed">
+    <origin xyz="0 0 0.177" rpy="0 0 0"/>
+    <parent link="base_footprint"/>
+    <child link="base_link"/>
+  </joint>
+  <link name="base_link">
+    <inertial>
+      <mass value="10.0"/>
+      <origin xyz="0 0 0"/>
+      <inertia ixx="0.3338" ixy="0.0" ixz="0.0"
+         iyy="0.4783" iyz="0.0"
+         izz="0.3338"/>
+    </inertial>
+    <visual name="base_visual">
+      <origin xyz="0 0 0" rpy="0 0 0"/>
+      <geometry name="pioneer_geom">
+        <mesh filename="package://pandora_robots_description/meshes/pioneer3at/p3at_meshes/chassis.stl"/>
+      </geometry>
+      <material name="ChassisRed">
+        <color rgba="0.851 0.0 0.0 1.0"/>
+      </material>
+    </visual>
+    <collision>
+      <origin xyz="0 0 0" rpy="0 0 0"/>
+        <geometry>
+          <mesh filename="package://pandora_robots_description/meshes/pioneer3at/p3at_meshes/chassis.stl"/>
+        </geometry>
+    </collision>
+  </link>
+  <gazebo reference="base_link">
+    <material value="Gazebo/Red"/>
+  </gazebo>
 <!-- Top -->
-	<link name="top_plate">
-		<inertial>
-			<mass value="0.1"/>
-			<origin xyz="0 0 0" rpy="0 0 0"/>
-			<inertia ixx="1.0" ixy="0.0" ixz="0.0"
-				 iyy="1.0" iyz="0.0"
- 				izz="1.0"/>
-		</inertial>
-		<visual name="base_visual">
-			<origin xyz="0 0 0" rpy="0 0 0"/>
-			<geometry name="pioneer_geom">
-				<mesh filename="package://pandora_robots_description/meshes/pioneer3at/p3at_meshes/top.stl"/>
-			</geometry>
-			<material name="TopBlack">
-					<color rgba="0.038 0.038 0.038 1.0"/>
-			</material>
-		</visual>
-		<collision>
-			<origin xyz="0 0 0" rpy="0 0 0"/>
-			<geometry>
-				<box size="0 0 0"/>
-			</geometry>
-		</collision>
-	</link>
-	<gazebo reference="top_plate">
-		<material value="Gazebo/Black"/>
-	</gazebo>
-	<joint name="base_top_joint" type="fixed">
-		<origin xyz="-0.025 0 0.096"/>
-		<parent link="base_link"/>
-		<child link="top_plate"/>
-	</joint>
-<!-- Front Axles + Wheels + Hubcaps -->
-<xacro:macro name="p3at_front" params="suffix reflect">
-	<link name="p3at_front_${suffix}_axle">
-		<inertial>
-			<mass value="0.1"/>
-			<origin xyz="0 0 0"/>
-			<inertia ixx="1.0" ixy="0.0" ixz="0.0"
-				 iyy="1.0" iyz="0.0" izz="1.0"/>
-  	 	</inertial>
-	<visual name="base_visual">
-		<origin xyz="0 0 0" rpy="0 0 0"/>
-		<geometry name="pioneer_geom">
-			<mesh filename="package://pandora_robots_description/meshes/pioneer3at/p3at_meshes/axle.stl"/>
-		</geometry>
-		<material name="AxleGrey">
-			<color rgba="0.5 0.5 0.5 1"/>
-		</material>
-	</visual>
-	<collision>
-		<origin xyz="0 0 0" rpy="0 0 0"/>
-		<geometry>
-			<box size="0 0 0"/>
-		</geometry>
-	</collision>
-	</link>
-	<gazebo reference="p3at_front_${suffix}_axle">
-		<material value="Gazebo/Grey"/>
-	</gazebo>
-	<joint name="base_front_${suffix}_axle_joint" type="fixed">
-		<origin xyz="0.135 ${reflect*0.156} -0.066" rpy="0 0 0"/>
-		<parent link="base_link"/>
-		<child link="p3at_front_${suffix}_axle"/>
-	</joint>
-	<link name="p3at_front_${suffix}_hub">
-		<inertial>
-			<mass value="0.1"/>
-			<origin xyz="0 0 0"/>
-			<inertia ixx="1.0" ixy="0.0" ixz="0.0"
-				 iyy="1.0" iyz="0.0" izz="1.0"/>
-  	 	</inertial>
-	<visual name="base_visual">
-		<origin xyz="0 0 0" rpy="0 0 0"/>
-		<geometry name="pioneer_geom">
-			<mesh filename="package://pandora_robots_description/meshes/pioneer3at/p3at_meshes/${suffix}_hubcap.stl"/>
-		</geometry>
-		<material name="HubcapYellow">
-			<color rgba="1.0 0.811 0.151 1.0"/>
-		</material>
-	</visual>
-	<collision>
-		<origin xyz="0 0 0" rpy="0 0 0"/>
-		<geometry>
-			<box size="0 0 0"/>
-		</geometry>
-	</collision>
-	</link>
-	<gazebo reference="p3at_front_${suffix}_hub">
-		<material value="Gazebo/Yellow"/>
-	</gazebo>
-	<joint name="base_front_${suffix}_hub_joint" type="fixed">
-		<origin xyz="0 ${reflect*0.041} 0" rpy="0 0 0"/>
-		<parent link="p3at_front_${suffix}_axle"/>
-		<child link="p3at_front_${suffix}_hub"/>
-	</joint>
-	<link name="p3at_front_${suffix}_wheel">
-		<inertial>
-			<mass value="0.5"/>
-			<origin xyz="0 0 0"/>
-			<inertia ixx="0.012411765597" ixy="0" ixz="0"
-         iyy="0.015218160428" iyz="0" izz="0.011763977943"/>
-      </inertial>
-	<visual name="base_visual">
-		<origin xyz="0 0 0" rpy="0 0 0"/>
-		<geometry name="pioneer_geom">
-			<mesh filename="package://pandora_robots_description/meshes/pioneer3at/p3at_meshes/wheel.stl"/>
-		</geometry>
-		<material name="WheelBlack">
-			<color rgba="0.117 0.117 0.117 1"/>
-		</material>
-	</visual>
-	<collision>
-		<origin xyz="0 0 0" rpy="${-3.1415927/2} 0 0"/>
-		<geometry>
-	    <!--mesh filename="package://pandora_robots_description/meshes/pioneer3at/p3at_meshes/wheel.stl"/-->
-	    <cylinder radius="0.111" length="0.075"/>
-		</geometry>
-	</collision>
-	</link>
-	<gazebo reference="p3at_front_${suffix}_wheel">
-		<material value="Gazebo/Black"/>
-	</gazebo>
-	<joint name="p3at_front_${suffix}_wheel_joint" type="continuous">
-  	<axis xyz="0 1 0"/>
-    <anchor xyz="0 0 0"/>
-    <limit effort="100" velocity="100" />
-    <joint_properties damping="0.7"/>
-		<origin xyz="0 0 0" rpy="0 0 0"/>
-		<parent link="p3at_front_${suffix}_hub"/>
-		<child link="p3at_front_${suffix}_wheel"/>
-	</joint>
-<!-- Back Axles + Wheels + Hubcaps -->
-	<link name="p3at_back_${suffix}_axle">
-		<inertial>
-			<mass value="0.1"/>
-			<origin xyz="0 0 0"/>
-			<inertia ixx="1.0" ixy="0.0" ixz="0.0"
-				 iyy="1.0" iyz="0.0" izz="1.0"/>
-  	 	</inertial>
-	<visual name="base_visual">
-		<origin xyz="0 0 0" rpy="0 0 0"/>
-		<geometry name="pioneer_geom">
-			<mesh filename="package://pandora_robots_description/meshes/pioneer3at/p3at_meshes/axle.stl"/>
-		</geometry>
-		<material name="AxleGrey">
-			<color rgba="0.5 0.5 0.5 1"/>
-		</material>
-	</visual>
-	<collision>
-		<origin xyz="0 0 0" rpy="0 0 0"/>
-		<geometry>
-			<mesh filename="package://pandora_robots_description/meshes/pioneer3at/p3at_meshes/axle.stl"/>
-		</geometry>
-	</collision>
-	</link>
-	<gazebo reference="p3at_back_${suffix}_axle">
-		<material value="Gazebo/Grey"/>
-	</gazebo>
-	<joint name="bp3at_back_${suffix}_axle_joint" type="fixed">
-		<origin xyz="-0.134 ${reflect*0.156} -0.066" rpy="0 0 0"/>
-		<parent link="base_link"/>
-		<child link="p3at_back_${suffix}_axle"/>
-	</joint>
-	<link name="p3at_back_${suffix}_hub">
-		<inertial>
-			<mass value="0.1"/>
-			<origin xyz="0 0 0"/>
-			<inertia ixx="1.0" ixy="0.0" ixz="0.0"
-				 iyy="1.0" iyz="0.0" izz="1.0"/>
-  	 	</inertial>
-	<visual name="base_visual">
-		<origin xyz="0 0 0" rpy="0 0 0"/>
-		<geometry name="pioneer_geom">
-			<mesh filename="package://pandora_robots_description/meshes/pioneer3at/p3at_meshes/${suffix}_hubcap.stl"/>
-		</geometry>
-		<material name="HubcapYellow"/>
-	</visual>
-	<collision>
-		<origin xyz="0 0 0" rpy="0 0 0"/>
-		<geometry>
-			<mesh filename="package://pandora_robots_description/meshes/pioneer3at/p3at_meshes/${suffix}_hubcap.stl"/>
-		</geometry>
-	</collision>
-	</link>
-	<gazebo reference="p3at_back_${suffix}_hub">
-		<material value="Gazebo/Yellow"/>
-	</gazebo>
-	<joint name="p3at_back_${suffix}_hub_joint" type="fixed">
-		<origin xyz="-0 ${reflect*0.041} 0" rpy="0 0 0"/>
-		<parent link="p3at_back_${suffix}_axle"/>
-		<child link="p3at_back_${suffix}_hub"/>
-	</joint>
-	<link name="p3at_back_${suffix}_wheel">
-		<inertial>
-			<mass value="0.5"/>
-			<origin xyz="0 0 0"/>
-			<inertia ixx="0.012411765597" ixy="0" ixz="0"
-         iyy="0.015218160428" iyz="0" izz="0.011763977943"/>
-      </inertial>
-	<visual name="base_visual">
-		<origin xyz="0 0 0" rpy="0 0 0"/>
-		<geometry name="pioneer_geom">
-			<mesh filename="package://pandora_robots_description/meshes/pioneer3at/p3at_meshes/wheel.stl"/>
-		</geometry>
-		<material name="WheelBlack"/>
-	</visual>
-	<collision>
-		<origin xyz="0 0 0" rpy="${-3.1415927/2} 0 0"/>
-		<geometry>
-			<!--<mesh filename="package://pandora_robots_description/meshes/pioneer3at/p3at_meshes/wheel.stl"/>-->
-			<cylinder radius="0.111" length="0.075"/>
-		</geometry>
-	</collision>
-	</link>
-	<gazebo reference="p3at_back_${suffix}_wheel">
-		<material value="Gazebo/Black"/>
-	</gazebo>
-	<joint name="p3at_back_${suffix}_wheel_joint" type="continuous">
-	  <axis xyz="0 1 0"/>
-    <anchor xyz="0 0 0"/>
-    <limit effort="100" velocity="100" />
-    <joint_properties damping="0.7"/>
-		<origin xyz="0 0 0" rpy="0 0 0"/>
-		<parent link="p3at_back_${suffix}_hub"/>
-		<child link="p3at_back_${suffix}_wheel"/>
-	</joint>
-  <gazebo reference="p3at_back_${suffix}_wheel">
-    <kp>1000000.0</kp> <!-- kp and kd for rubber -->
-    <kd>100.0</kd>
-    <mu1>10.0</mu1>
-    <mu2>1.0</mu2>
-    <fdir1>0 1 0</fdir1> <!-- is this correct? -->
-    <maxVel>1.0</maxVel>
-    <minDepth>0.00</minDepth>
+  <link name="top_plate">
+    <inertial>
+      <mass value="0.1"/>
+      <origin xyz="0 0 0" rpy="0 0 0"/>
+      <inertia ixx="1.0" ixy="0.0" ixz="0.0"
+         iyy="1.0" iyz="0.0"
+        izz="1.0"/>
+    </inertial>
+    <visual name="base_visual">
+      <origin xyz="0 0 0" rpy="0 0 0"/>
+      <geometry name="pioneer_geom">
+        <mesh filename="package://pandora_robots_description/meshes/pioneer3at/p3at_meshes/top.stl"/>
+      </geometry>
+      <material name="TopBlack">
+          <color rgba="0.038 0.038 0.038 1.0"/>
+      </material>
+    </visual>
+    <collision>
+      <origin xyz="0 0 0" rpy="0 0 0"/>
+      <geometry>
+        <box size="0 0 0"/>
+      </geometry>
+    </collision>
+  </link>
+  <gazebo reference="top_plate">
+    <material value="Gazebo/Black"/>
   </gazebo>
-  <gazebo reference="p3at_front_${suffix}_wheel">
-    <kp>1000000.0</kp> <!--<limit effort="30" velocity="10.0" /> kp and kd for rubber -->
-    <kd>100.0</kd>
-    <mu1>10.0</mu1>
-    <mu2>1.0</mu2>
-    <fdir1>0 1 0</fdir1> <!-- is this correct? -->
-    <maxVel>1.0</maxVel>
-    <minDepth>0.00</minDepth>
+  <joint name="base_top_joint" type="fixed">
+    <origin xyz="-0.025 0 0.096"/>
+    <parent link="base_link"/>
+    <child link="top_plate"/>
+  </joint>
+  <!-- Front Axles + Wheels + Hubcaps -->
+  <xacro:macro name="p3at_front" params="suffix reflect">
+    <link name="p3at_front_${suffix}_axle">
+      <inertial>
+        <mass value="0.1"/>
+        <origin xyz="0 0 0"/>
+        <inertia ixx="1.0" ixy="0.0" ixz="0.0"
+           iyy="1.0" iyz="0.0" izz="1.0"/>
+        </inertial>
+    <visual name="base_visual">
+      <origin xyz="0 0 0" rpy="0 0 0"/>
+      <geometry name="pioneer_geom">
+        <mesh filename="package://pandora_robots_description/meshes/pioneer3at/p3at_meshes/axle.stl"/>
+      </geometry>
+      <material name="AxleGrey">
+        <color rgba="0.5 0.5 0.5 1"/>
+      </material>
+    </visual>
+    <collision>
+      <origin xyz="0 0 0" rpy="0 0 0"/>
+      <geometry>
+        <box size="0 0 0"/>
+      </geometry>
+    </collision>
+    </link>
+    <gazebo reference="p3at_front_${suffix}_axle">
+      <material value="Gazebo/Grey"/>
+    </gazebo>
+    <joint name="base_front_${suffix}_axle_joint" type="fixed">
+      <origin xyz="0.135 ${reflect*0.156} -0.066" rpy="0 0 0"/>
+      <parent link="base_link"/>
+      <child link="p3at_front_${suffix}_axle"/>
+    </joint>
+    <link name="p3at_front_${suffix}_hub">
+      <inertial>
+        <mass value="0.1"/>
+        <origin xyz="0 0 0"/>
+        <inertia ixx="1.0" ixy="0.0" ixz="0.0"
+           iyy="1.0" iyz="0.0" izz="1.0"/>
+        </inertial>
+    <visual name="base_visual">
+      <origin xyz="0 0 0" rpy="0 0 0"/>
+      <geometry name="pioneer_geom">
+        <mesh filename="package://pandora_robots_description/meshes/pioneer3at/p3at_meshes/${suffix}_hubcap.stl"/>
+      </geometry>
+      <material name="HubcapYellow">
+        <color rgba="1.0 0.811 0.151 1.0"/>
+      </material>
+    </visual>
+    <collision>
+      <origin xyz="0 0 0" rpy="0 0 0"/>
+      <geometry>
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
File: pandora_sensors_description/urdf/hokuyo_utm_30lx.urdf.xacro (robot description, xacro)
@@ -2,120 +2,98 @@
 <robot xmlns:xacro="http://ros.org/wiki/xacro">
 <xacro:macro name="hokuyo_caster" params="parent *origin">
-    <link name="laser_link">
-      <inertial>
-        <mass value="0.1"/>
-        <origin xyz="0 0 0"/>
-        <inertia ixx="0.0002632" ixy="0" ixz="0"
-				 iyy="0.0002632" iyz="0" izz="0.000162" />
-      </inertial>
-<!--
-      <inertial>
-        <mass value="0.1"/>
-        <origin xyz="0 0 0"/>
-        <inertia ixx="1" ixy="0" ixz="0" iyy="1" iyz="0" izz="1" />
-      </inertial>
--->
-      <visual name="visual">
-        <geometry>
-          <mesh filename="package://pandora_sensors_description/meshes/hokuyo_utm_30lx/hokuyo_utm_30lx.dae"/>
-        </geometry>
-      </visual>
-      <collision name="collision-base">
-        <origin xyz="0 0 -0.0145" rpy="0 0 0"/>
-        <geometry>
-			<box size="0.05 0.05 0.041"/>
-        </geometry>
-      </collision>
-      <collision name="collision-top">
-        <origin xyz="0 0 0.0205" rpy="0 0 0"/>
-        <geometry>
-          <cylinder radius="0.021" length="0.029"/>
-        </geometry>
-      </collision>
-    </link>
-    <gazebo reference="laser_link">
-		<sensor name="laser" type="ray">
-        <pose>0.01 0 0.0175 0 -0 0</pose>
-        <ray>
-          <scan>
-            <horizontal>
-              <samples>640</samples>
-              <resolution>1</resolution>
-              <min_angle>-2.26889</min_angle>
-              <max_angle>2.268899</max_angle>
-            </horizontal>
-          </scan>
-          <range>
-            <min>0.08</min>
-            <max>10</max>
-            <resolution>0.01</resolution>
-          </range>
-        </ray>
-        <plugin name="laser" filename="libRayPlugin.so" />
-        <plugin name="laser2Ros" filename="libgazebo_ros_laser.so">
-			<topicName>/slam/scan</topicName>
-			<frameName>/laser</frameName>
-		</plugin>
-        <always_on>1</always_on>
-        <update_rate>30</update_rate>
-        <visualize>true</visualize>
-        </sensor>
-    </gazebo>
-	<link name="hokuyo_base_link">
-		<inertial>
-			<mass value="0.001"/>
-			<origin xyz="0 0 0"/>
-			<inertia ixx="0.00000001" ixy="0" ixz="0"
-					 iyy="0.00000001" iyz="0" izz="0.00000001"/>
-		</inertial>
-		<visual>
-			<origin xyz="0 0 0" rpy="0 0 0"/>
-			<geometry>
-				<box size="0 0 0"/>
-			</geometry>
-		</visual>
-		<collision>
-			<origin xyz="0 0 0" rpy="0 0 0"/>
-			<geometry>
-				<box size="0 0 0"/>
-			</geometry>
-		</collision>
-	</link>
-	<joint name="laser_roll_joint" type="fixed">
-		<xacro:insert_block name="origin" />
-		<parent link="${parent}"/>
-		<child link="hokuyo_base_link"/>
-		<axis xyz="1 0 0"/>
-<!--
-		<limit effort="300" velocity="100.0" />
--->
-	</joint>
-	<joint name="laser_pitch_joint" type="fixed">
-		<origin xyz="0 0 0" rpy="0 0 0"/>
-		<parent link="hokuyo_base_link"/>
-		<child link="laser_link"/>
-		<axis xyz="0 1 0"/>
-<!--
-		<limit effort="300" velocity="100.0" />
--->
-	</joint>
-<!--
-	<transmission name="laser_roll_transmission">
-		<type>transmission_interface/SimpleTransmission</type>
-		<joint name="laser_roll_joint"/>
-		<actuator name="laser_roll_motor">
-		  <hardwareInterface>EffortJointInterface</hardwareInterface>
-		  <mechanicalReduction>1</mechanicalReduction>
-		</actuator>
-	</transmission>
-	<transmission name="laser_pitch_transmission">
-		<type>transmission_interface/SimpleTransmission</type>
-		<joint name="laser_pitch_joint"/>
-		<actuator name="laser_pitch_motor">
-		  <hardwareInterface>EffortJointInterface</hardwareInterface>
-		  <mechanicalReduction>1</mechanicalReduction>
-		</actuator>
-	</transmission>
--->
+  <link name="laser_link">
+    <inertial>
+      <mass value="0.1"/>
+      <origin xyz="0 0 0"/>
+      <inertia ixx="0.0002632" ixy="0" ixz="0"
+       iyy="0.0002632" iyz="0" izz="0.000162" />
+    </inertial>
+  <!--
+    <inertial>
+      <mass value="0.1"/>
+      <origin xyz="0 0 0"/>
+      <inertia ixx="1" ixy="0" ixz="0" iyy="1" iyz="0" izz="1" />
+    </inertial>
+  -->
+    <visual name="visual">
+      <geometry>
+        <mesh filename="package://pandora_sensors_description/meshes/hokuyo_utm_30lx/hokuyo_utm_30lx.dae"/>
+      </geometry>
+    </visual>
+    <collision name="collision-base">
+      <origin xyz="0 0 -0.0145" rpy="0 0 0"/>
+      <geometry>
+    <box size="0.05 0.05 0.041"/>
+      </geometry>
+    </collision>
+    <collision name="collision-top">
+      <origin xyz="0 0 0.0205" rpy="0 0 0"/>
+      <geometry>
+        <cylinder radius="0.021" length="0.029"/>
+      </geometry>
+    </collision>
+  </link>
+  <gazebo reference="laser_link">
+    <sensor name="laser" type="ray">
+      <pose>0.01 0 0.0175 0 -0 0</pose>
+      <ray>
+        <scan>
+          <horizontal>
+            <samples>640</samples>
+            <resolution>1</resolution>
+            <min_angle>-2.26889</min_angle>
+            <max_angle>2.268899</max_angle>
+          </horizontal>
+        </scan>
+        <range>
+          <min>0.08</min>
+          <max>10</max>
+          <resolution>0.01</resolution>
+        </range>
+      </ray>
+      <plugin name="laser" filename="libRayPlugin.so" />
+      <plugin name="laser2Ros" filename="libgazebo_ros_laser.so">
+        <topicName>/slam/scan</topicName>
+        <frameName>/laser</frameName>
+      </plugin>
+      <always_on>1</always_on>
+      <update_rate>30</update_rate>
+      <visualize>true</visualize>
+    </sensor>
+  </gazebo>
+  <link name="hokuyo_base_link">
+    <inertial>
+      <mass value="0.001"/>
+      <origin xyz="0 0 0"/>
+      <inertia ixx="0.00000001" ixy="0" ixz="0"
+           iyy="0.00000001" iyz="0" izz="0.00000001"/>
+    </inertial>
+    <visual>
+      <origin xyz="0 0 0" rpy="0 0 0"/>
+      <geometry>
+        <box size="0 0 0"/>
+      </geometry>
+    </visual>
+    <collision>
+      <origin xyz="0 0 0" rpy="0 0 0"/>
+      <geometry>
+        <box size="0 0 0"/>
+      </geometry>
+    </collision>
+  </link>
+  <joint name="laser_roll_joint" type="revolute">
+    <xacro:insert_block name="origin" />
+    <parent link="${parent}"/>
+    <child link="hokuyo_base_link"/>
+    <axis xyz="1 0 0"/>
+    <limit effort="300" velocity="100.0" lower="-1.57" upper="1.57"/>
+  </joint>
+  <joint name="laser_pitch_joint" type="revolute">
+    <origin xyz="0 0 0" rpy="0 0 0"/>
+    <parent link="hokuyo_base_link"/>
+    <child link="laser_link"/>
+    <axis xyz="0 1 0"/>
+    <limit effort="300" velocity="100.0" lower="-1.57" upper="1.57"/>
+  </joint>
 </xacro:macro>
 </robot>
