Commit message: simulation with standalone models

File: pandora_sensors_description/urdf/kinect_camera.urdf.xacro (robot description, xacro)
@@ -2,127 +2,109 @@
 <robot xmlns:xacro="http://ros.org/wiki/xacro">
 <xacro:macro name="kinect_caster" params="parent *origin">
-    <link name="kinect_link">
-      <inertial>
-		<origin xyz="0 0 0" rpy="0 0 0"/>
-        <mass value="0.1"/>
-		<inertia ixx="0.004075" ixy="0.0" ixz="0.0"
-				 iyy="0.004075" iyz="0.0" izz="0.004075"/>
-      </inertial>
-      <collision name="collision">
-        <geometry>
-          <box size="0.073000 0.276000 0.072000"/>
-        </geometry>
-      </collision>
-      <visual name="visual">
-        <geometry>
-          <mesh filename="package://pandora_sensors_description/meshes/kinect_camera/kinect_camera_simple.dae"/>
-        </geometry>
-      </visual>
-    </link>
-    <link name="kinect_camera">
-      <inertial>
-		<origin xyz="0 0 0" rpy="0 0 0"/>
-        <mass value="0.001"/>
-		<inertia ixx="0.00004075" ixy="0.0" ixz="0.0"
-				 iyy="0.00004075" iyz="0.0" izz="0.00004075"/>
-      </inertial>
-      <collision name="collision">
-        <geometry>
-          <box size="0.001 0.001 0.001"/>
-        </geometry>
-      </collision>
-      <visual name="visual">
-        <geometry>
-          <box size="0.001 0.001 0.001"/>
-        </geometry>
-      </visual>
-    </link>
-    <joint name="kinect_camera_joint" type="fixed">
-	  <origin xyz="0 0 0" rpy="-1.57 0 -1.57"/>
-	  <parent link="kinect_link"/>
-	  <child link="kinect_camera"/>
-	</joint>
-	<gazebo reference="kinect_link">
-      <sensor name="kinect" type="depth">
-        <update_rate>20</update_rate>
-        <camera>
-          <horizontal_fov>1.047198</horizontal_fov>
-          <image>
-            <width>640</width>
-            <height>480</height>
-            <format>R8G8B8</format>
-          </image>
-          <clip>
-            <near>0.05</near>
-            <far>3</far>
-          </clip>
-        </camera>
-        <plugin name="depth2ros" filename="libgazebo_ros_openni_kinect.so">
-			<pointCloudTopicName>point_cloud</pointCloudTopicName>
-			<frameName>kinect_camera</frameName>
-			<cameraName>kinect</cameraName>
-			<imageTopicName>image</imageTopicName>
-			<depthImageTopicName>depth/image</depthImageTopicName>
-			<depthImageCameraInfoTopicName>depth/image/info</depthImageCameraInfoTopicName>
-			<pointCloudCutoff>0.4</pointCloudCutoff>
-		</plugin>
-      </sensor>
-	</gazebo>
-	<link name="kinect_base_link">
-		<inertial>
-			<mass value="0.001"/>
-			<origin xyz="0 0 0"/>
-			<inertia ixx="0.00000001" ixy="0" ixz="0"
-					 iyy="0.00000001" iyz="0" izz="0.00000001"/>
-		</inertial>
-		<visual>
-			<origin xyz="0 0 0" rpy="0 0 0"/>
-			<geometry>
-				<box size="0 0 0"/>
-			</geometry>
-		</visual>
-		<collision>
-			<origin xyz="0 0 0" rpy="0 0 0"/>
-			<geometry>
-				<box size="0 0 0"/>
-			</geometry>
-		</collision>
-	</link>
-	<joint name="kinect_pitch_joint" type="fixed">
-	  <xacro:insert_block name="origin" />
+  <link name="kinect_link">
+    <inertial>
+      <origin xyz="0 0 0" rpy="0 0 0"/>
+      <mass value="0.1"/>
+      <inertia ixx="0.004075" ixy="0.0" ixz="0.0"
+                iyy="0.004075" iyz="0.0" izz="0.004075"/>
+    </inertial>
+    <collision name="collision">
+      <geometry>
+        <box size="0.073000 0.276000 0.072000"/>
+      </geometry>
+    </collision>
+    <visual name="visual">
+      <geometry>
+        <mesh filename="package://pandora_sensors_description/meshes/kinect_camera/kinect_camera_simple.dae"/>
+      </geometry>
+    </visual>
+  </link>
+  <link name="kinect_camera">
+    <inertial>
+      <origin xyz="0 0 0" rpy="0 0 0"/>
+      <mass value="0.001"/>
+      <inertia ixx="0.00004075" ixy="0.0" ixz="0.0"
+           iyy="0.00004075" iyz="0.0" izz="0.00004075"/>
+    </inertial>
+    <collision name="collision">
+      <geometry>
+        <box size="0.001 0.001 0.001"/>
+      </geometry>
+    </collision>
+    <visual name="visual">
+      <geometry>
+        <box size="0.001 0.001 0.001"/>
+      </geometry>
+    </visual>
+  </link>
+  <joint name="kinect_camera_joint" type="fixed">
+    <origin xyz="0 0 0" rpy="-1.57 0 -1.57"/>
+    <parent link="kinect_link"/>
+    <child link="kinect_camera"/>
+  </joint>
+  <gazebo reference="kinect_link">
+    <sensor name="kinect" type="depth">
+      <update_rate>20</update_rate>
+      <camera>
+        <horizontal_fov>1.047198</horizontal_fov>
+        <image>
+          <width>640</width>
+          <height>480</height>
+          <format>R8G8B8</format>
+        </image>
+        <clip>
+          <near>0.05</near>
+          <far>3</far>
+        </clip>
+      </camera>
+      <plugin name="depth2ros" filename="libgazebo_ros_openni_kinect.so">
+        <pointCloudTopicName>point_cloud</pointCloudTopicName>
+        <frameName>kinect_camera</frameName>
+        <cameraName>kinect</cameraName>
+        <imageTopicName>image</imageTopicName>
+        <depthImageTopicName>depth/image</depthImageTopicName>
+        <depthImageCameraInfoTopicName>depth/image/info</depthImageCameraInfoTopicName>
+        <pointCloudCutoff>0.4</pointCloudCutoff>
+      </plugin>
+    </sensor>
+  </gazebo>
+  <link name="kinect_base_link">
+    <inertial>
+      <mass value="0.001"/>
+      <origin xyz="0 0 0"/>
+      <inertia ixx="0.00000001" ixy="0" ixz="0"
+           iyy="0.00000001" iyz="0" izz="0.00000001"/>
+    </inertial>
+    <visual>
+      <origin xyz="0 0 0" rpy="0 0 0"/>
+      <geometry>
+        <box size="0 0 0"/>
+      </geometry>
+    </visual>
+    <collision>
+      <origin xyz="0 0 0" rpy="0 0 0"/>
+      <geometry>
+        <box size="0 0 0"/>
+      </geometry>
+    </collision>
+  </link>
+  <joint name="kinect_pitch_joint" type="fixed">
+    <xacro:insert_block name="origin" />
       <parent link="${parent}"/>
-	  <child link="kinect_base_link"/>
-	  <axis xyz="0 1 0"/>
-<!--
-	  <limit effort="300" velocity="100.0" />
--->
-	</joint>
-	<joint name="kinect_yaw_joint" type="fixed">
-	  <origin xyz="0 0 0" rpy="0 0 0"/>
-	  <child link="kinect_link"/>
-	  <parent link="kinect_base_link"/>
-	  <axis xyz="0 0 1"/>
-<!--
-	  <limit effort="300" velocity="100.0" />
--->
-	</joint>
-<!--
-	<transmission name="kinect_pitch_transmission">
-		<type>transmission_interface/SimpleTransmission</type>
-		<joint name="kinect_pitch_joint"/>
-		<actuator name="kinect_pitch_motor">
-		  <hardwareInterface>EffortJointInterface</hardwareInterface>
-		  <mechanicalReduction>1</mechanicalReduction>
-		</actuator>
-	</transmission>
-	<transmission name="kinect_yaw_transmission">
-		<type>transmission_interface/SimpleTransmission</type>
-		<joint name="kinect_yaw_joint"/>
-		<actuator name="kinect_yaw_motor">
-		  <hardwareInterface>EffortJointInterface</hardwareInterface>
-		  <mechanicalReduction>1</mechanicalReduction>
-		</actuator>
-	</transmission>
--->
+    <child link="kinect_base_link"/>
+    <axis xyz="0 1 0"/>
+  <!--
+    <limit effort="300" velocity="100.0" />
+  -->
+  </joint>
+  <joint name="kinect_yaw_joint" type="fixed">
+    <origin xyz="0 0 0" rpy="0 0 0"/>
+    <child link="kinect_link"/>
+    <parent link="kinect_base_link"/>
+    <axis xyz="0 0 1"/>
+  <!--
+    <limit effort="300" velocity="100.0" />
+  -->
+  </joint>
 </xacro:macro>
 </robot>

Commit message: remove base_footprint link

File: pandora_robots_description/urdf/pioneer3at.urdf.xacro (robot description, xacro)
@@ -6,10 +6,4 @@
        name="pioneer3at">
 <!-- base_link -->
-  <link name="base_footprint"/>
-  <joint name="base_footprint_joint" type="fixed">
-    <origin xyz="0 0 0.177" rpy="0 0 0"/>
-    <parent link="base_footprint"/>
-    <child link="base_link"/>
-  </joint>
   <link name="base_link">
     <inertial>
@@ -317,5 +311,5 @@
       <wheelSeparation>0.4</wheelSeparation>
       <wheelDiameter>0.220</wheelDiameter>
-      <robotBaseFrame>base_footprint</robotBaseFrame>
+      <robotBaseFrame>base_link</robotBaseFrame>
       <topicName>cmd_vel</topicName>
       <broadcastTF>0</broadcastTF>

Commit message: Add model with separately exported meshes. All sensors and plugins are disabled.

File: pandora_robots_description/urdf/pioneer3at.urdf.xacro (robot description, xacro)
@@ -6,16 +6,9 @@
        name="pioneer3at">
 <!-- base_link -->
-  <link name="base_footprint"/>
-  <joint name="base_footprint_joint" type="fixed">
-    <origin xyz="0 0 0.177" rpy="0 0 0"/>
-    <parent link="base_footprint"/>
-    <child link="base_link"/>
-  </joint>
   <link name="base_link">
     <inertial>
-      <mass value="10.0"/>
-      <origin xyz="0 0 0"/>
-      <inertia ixx="0.3338" ixy="0.0" ixz="0.0"
-         iyy="0.4783" iyz="0.0"
+      <mass value="14.0"/>
+      <inertia ixx="0.3338" ixy="0" ixz="0"
+         iyy="0.4783" iyz="0"
          izz="0.3338"/>
     </inertial>
@@ -44,7 +37,7 @@
       <mass value="0.1"/>
       <origin xyz="0 0 0" rpy="0 0 0"/>
-      <inertia ixx="1.0" ixy="0.0" ixz="0.0"
-         iyy="1.0" iyz="0.0"
-        izz="1.0"/>
+      <inertia ixx="0.001" ixy="0.0" ixz="0.0"
+         iyy="0.001" iyz="0.0"
+        izz="0.001"/>
     </inertial>
     <visual name="base_visual">
@@ -78,6 +71,6 @@
         <mass value="0.1"/>
         <origin xyz="0 0 0"/>
-        <inertia ixx="1.0" ixy="0.0" ixz="0.0"
-           iyy="1.0" iyz="0.0" izz="1.0"/>
+        <inertia ixx="0.001" ixy="0.0" ixz="0.0"
+           iyy="0.001" iyz="0.0" izz="0.001"/>
         </inertial>
     <visual name="base_visual">
@@ -109,6 +102,6 @@
         <mass value="0.1"/>
         <origin xyz="0 0 0"/>
-        <inertia ixx="1.0" ixy="0.0" ixz="0.0"
-           iyy="1.0" iyz="0.0" izz="1.0"/>
+        <inertia ixx="0.001" ixy="0.0" ixz="0.0"
+           iyy="0.001" iyz="0.0" izz="0.001"/>
         </inertial>
     <visual name="base_visual">
@@ -177,6 +170,6 @@
         <mass value="0.1"/>
         <origin xyz="0 0 0"/>
-        <inertia ixx="1.0" ixy="0.0" ixz="0.0"
-           iyy="1.0" iyz="0.0" izz="1.0"/>
+        <inertia ixx="0.001" ixy="0.0" ixz="0.0"
+           iyy="0.001" iyz="0.0" izz="0.001"/>
         </inertial>
     <visual name="base_visual">
@@ -208,6 +201,6 @@
         <mass value="0.1"/>
         <origin xyz="0 0 0"/>
-        <inertia ixx="1.0" ixy="0.0" ixz="0.0"
-           iyy="1.0" iyz="0.0" izz="1.0"/>
+        <inertia ixx="0.001" ixy="0.0" ixz="0.0"
+           iyy="0.001" iyz="0.0" izz="0.001"/>
         </inertial>
     <visual name="base_visual">
@@ -317,5 +310,5 @@
       <wheelSeparation>0.4</wheelSeparation>
       <wheelDiameter>0.220</wheelDiameter>
-      <robotBaseFrame>base_footprint</robotBaseFrame>
+      <robotBaseFrame>base_link</robotBaseFrame>
       <topicName>cmd_vel</topicName>
       <broadcastTF>0</broadcastTF>
@@ -349,5 +342,5 @@
   <xacro:include filename="$(find pandora_sensors_description)/urdf/kinect_camera.urdf.xacro" />
   <xacro:kinect_caster parent="base_link">
-    <origin xyz="0.2 0 0.33" rpy="0 0 0"/>
+    <origin xyz="0.2 0 0.33" rpy="0 0.53 0"/>
   </xacro:kinect_caster>
   <!--Insert sonars-->
