Commit message: Change friction coefficients and enable the differential plugin.

File: pandora_robots_description/urdf/base.urdf.xacro (robot description, xacro)
@@ -59,12 +59,4 @@
     </plugin>
   </gazebo>
-  Add differential plugin
-  <gazebo>
-    <plugin name="RosDifferantialSkeletonPlugin" filename="libpandora_differential_skeleton_plugin.so">
-      <robotNamespace></robotNamespace>
-      <leftSkeletonJoint>left_side_joint</leftSkeletonJoint>
-      <rightSkeletonJoint>right_side_joint</rightSkeletonJoint>
-    </plugin>
-  </gazebo>
   Add ros_control plugin
   <gazebo>
@@ -75,4 +67,12 @@
   </gazebo>
   -->
+  <!-- Add differential plugin -->
+  <gazebo>
+    <plugin name="RosDifferantialSkeletonPlugin" filename="libpandora_differential_skeleton_plugin.so">
+      <robotNamespace></robotNamespace>
+      <leftSkeletonJoint>left_side_joint</leftSkeletonJoint>
+      <rightSkeletonJoint>right_side_joint</rightSkeletonJoint>
+    </plugin>
+  </gazebo>
   <!-- Add skid steer drive plugin-->
   <gazebo>
@@ -89,5 +89,4 @@
       <topicName>cmd_vel</topicName>
       <broadcastTF>0</broadcastTF>
-	    <!-- TODO: Fix torque -->
       <torque>5.0</torque>
       <commandTopic>cmd_vel</commandTopic>

File: pandora_robots_description/urdf/side.urdf.xacro (robot description, xacro)
@@ -28,13 +28,11 @@
       </collision>
     </link>
-    <joint name="${prefix_y}_side_joint" type="fixed" >
+    <joint name="${prefix_y}_side_joint" type="revolute" >
       <xacro:insert_block name="origin" />
       <parent link="${parent}" />
       <child link="${prefix_y}_side_link" />
-	  <!--
       <axis xyz="0 1 0" />
       <limit effort="100" velocity="100"
              lower="-0.785" upper="0.785" />
-	  -->
     </joint>
     <xacro:wheel_caster prefix_y="${prefix_y}" prefix_x="front"

File: pandora_robots_description/urdf/wheel.urdf.xacro (robot description, xacro)
@@ -38,14 +38,11 @@
     </joint>
     <gazebo reference="${prefix_y}_${prefix_x}_wheel_link" >
-      <!-- TODO: Fix coefficients -->
-	    <!-- <material>Gazebo/Black</material> -->
-      <!-- <maxVel>1.0</maxVel> -->
-      <mu1>0.75</mu1>
-      <mu2>0.75</mu2>
-      <fdir1>1 0 0</fdir1>
+      <mu1>0.3</mu1>
+      <mu2>0.3</mu2>
+      <!-- <fdir1>1 0 0</fdir1> -->
       <kp>10000000.0</kp>
       <kd>1.0</kd>
       <!-- Increase min depth -->
-      <minDepth>0.001</minDepth>
+      <minDepth>0.005</minDepth>
       <maxContacts>1</maxContacts>
     </gazebo>

Commit message: Add the new differential plugin in the model and simplify the wheel meshes.
TODO: Tune PID parameters and fix physics.

File: pandora_robots_description/urdf/base.urdf.xacro (robot description, xacro)
@@ -21,5 +21,5 @@
       <origin xyz="0 0 0" rpy="0 0 0" />
       <geometry>
-		    <!-- TODO: Simplify mesh -->
+		     <!-- TODO: Simplify mesh -->
         <mesh filename="package://pandora_robots_description/meshes/gears/base_link.stl" />
       </geometry>
@@ -32,6 +32,5 @@
     <origin xyz="0 -0.110 0" rpy="0 0 0" />
   </xacro:side_caster>
-  <!-- Disable sensors and plugins -->
-  <!--
+  <!-- Disable sensors and plugins
   Insert kinect
   <xacro:include filename="$(find pandora_sensors_description)/urdf/kinect_camera.urdf.xacro" />
@@ -69,8 +68,21 @@
   <!-- Add differential plugin -->
   <gazebo>
-    <plugin name="RosDifferantialSkeletonPlugin" filename="libpandora_differential_skeleton_plugin.so">
+    <plugin name="RosDifferantialPlugin" filename="libpandora_differential_plugin.so">
       <robotNamespace></robotNamespace>
-      <leftSkeletonJoint>left_side_joint</leftSkeletonJoint>
-      <rightSkeletonJoint>right_side_joint</rightSkeletonJoint>
+	    <baseLink>base_link</baseLink>
+      <leftFrontWheelLink>left_front_wheel_link</leftFrontWheelLink>
+      <leftRearWheelLink>left_rear_wheel_link</leftRearWheelLink>
+      <rightFrontWheelLink>right_front_wheel_link</rightFrontWheelLink>
+      <rightRearWheelLink>right_rear_wheel_link</rightRearWheelLink>
+      <leftSideJoint>left_side_joint</leftSideJoint>
+      <rightSideJoint>right_side_joint</rightSideJoint>
+      <maxAngle>0.785</maxAngle>
+      <sideJointDamping>0.0</sideJointDamping>
+      <maxDownforce>0.0</maxDownforce>
+      <forceAdjustment>1.0</forceAdjustment>
+      <!-- TODO: Tune PID -->
+      <P>100.0</P>
+      <I>1</I>
+      <D>10.0</D>
     </plugin>
   </gazebo>

File: pandora_robots_description/urdf/side.urdf.xacro (robot description, xacro)
@@ -9,5 +9,5 @@
         <mass value="0.93539" />
         <inertia ixx="0.001211" ixy="-4.0495E-05" ixz="${reflect_y*(1.0211E-06)}"
-	               iyy="0.026668" iyz="${reflect_y*(-0.00024586)}" izz="0.026454" />
+	             iyy="0.026668" iyz="${reflect_y*(-0.00024586)}" izz="0.026454" />
       </inertial>
       <visual>
@@ -33,7 +33,14 @@
       <child link="${prefix_y}_side_link" />
       <axis xyz="0 1 0" />
+	    <!-- TODO: Set damping -->
+      <dynamics damping="0" />
       <limit effort="100" velocity="100"
              lower="-0.785" upper="0.785" />
     </joint>
+    <!--
+    <gazebo reference="${prefix_y}_side_joint" >
+      <implicitSpringDamper>true</implicitSpringDamper>
+    </gazebo>
+    -->
     <xacro:wheel_caster prefix_y="${prefix_y}" prefix_x="front"
 	                      reflect_y="${reflect_y}" reflect_x="1" />

File: pandora_robots_description/urdf/wheel.urdf.xacro (robot description, xacro)
@@ -3,4 +3,5 @@
   <xacro:macro name="wheel_caster" params="prefix_y prefix_x reflect_y reflect_x" >
     <link name="${prefix_y}_${prefix_x}_wheel_link" >
+      <!--
       <inertial>
         <origin xyz="${reflect_y*(-2.2235E-05)} ${reflect_y*(-0.00052624)} 2.4287E-05"
@@ -8,5 +9,5 @@
         <mass value="1.2128" />
         <inertia ixx="0.0032586" ixy="5.862E-08" ixz="${reflect_y*(4.2142E-07)}"
-	               iyy="0.0054812" iyz="${reflect_y*(-6.4028E-08)}" izz="0.0032574" />
+	             iyy="0.0054812" iyz="${reflect_y*(-6.4028E-08)}" izz="0.0032574" />
       </inertial>
       <visual>
@@ -14,4 +15,5 @@
         <geometry>
           <mesh filename="package://pandora_robots_description/meshes/gears/wheel_link.stl" />
+          <mesh filename="package://pandora_robots_description/meshes/gears/simplified_wheel_link.stl" />
         </geometry>
         <material name="" >
@@ -22,6 +24,28 @@
         <origin xyz="0 0 0" rpy="0 0 ${(1-reflect_y)*1.57}" />
         <geometry>
-		      <!-- TODO: Simplify mesh -->
           <mesh filename="package://pandora_robots_description/meshes/gears/wheel_link.stl" />
+          <mesh filename="package://pandora_robots_description/meshes/gears/simplified_wheel_link.stl" />
+        </geometry>
+      </collision>
+      -->
+      <inertial>
+        <origin xyz="0 0 0" rpy="0 0 0" />
+        <mass value="1.2128" />
+        <inertia ixx="0.002982821" ixy="0" ixz="0"
+	               iyy="0.002982821" iyz="0" izz="0.004791967" />
+      </inertial>
+      <visual>
+        <origin xyz="0 0 0" rpy="1.57 0 0" />
+        <geometry>
+          <cylinder length="0.0762" radius="0.088895"/>
+        </geometry>
+        <material name="" >
+          <color rgba="0.753 0.753 0.753 1" />
+        </material>
+      </visual>
+      <collision>
+        <origin xyz="0 0 0" rpy="1.57 0 0" />
+        <geometry>
+          <cylinder length="0.0762" radius="0.088895"/>
         </geometry>
       </collision>
@@ -29,19 +53,19 @@
     <joint name="${prefix_y}_${prefix_x}_wheel_joint" type="continuous" >
       <origin xyz="${reflect_x*0.198785} ${reflect_y*0.110545} -0.052795"
-	            rpy="0 0 0" />
+	          rpy="0 0 0" />
       <parent link="${prefix_y}_side_link" />
       <child link="${prefix_y}_${prefix_x}_wheel_link" />
       <axis xyz="0 1 0" />
-	    <limit effort="100" velocity="100" />
-      <joint_properties damping="0.0" friction="0.0" />
-      <anchor xyz="0 0 0" />
+	  <limit effort="100" velocity="100" />
+      <!-- <anchor xyz="0 0 0" /> -->
     </joint>
+	<!-- TODO: Fix physics -->
     <gazebo reference="${prefix_y}_${prefix_x}_wheel_link" >
-      <mu1>0.3</mu1>
-      <mu2>0.3</mu2>
+      <mu1>0.8</mu1>
+      <mu2>0.8</mu2>
       <!-- <fdir1>1 0 0</fdir1> -->
       <kp>10000000.0</kp>
       <kd>1.0</kd>
-      <!-- Increase min depth -->
+      <!-- TODO: Adjust min depth -->
       <minDepth>0.005</minDepth>
       <maxContacts>1</maxContacts>

Commit message: Fix identation.

File: pandora_robots_description/urdf/base.urdf.xacro (robot description, xacro)
@@ -21,5 +21,5 @@
       <origin xyz="0 0 0" rpy="0 0 0" />
       <geometry>
-		     <!-- TODO: Simplify mesh -->
+         <!-- TODO: Simplify mesh -->
         <mesh filename="package://pandora_robots_description/meshes/gears/base_link.stl" />
       </geometry>
@@ -70,5 +70,5 @@
     <plugin name="RosDifferantialPlugin" filename="libpandora_differential_plugin.so">
       <robotNamespace></robotNamespace>
-	    <baseLink>base_link</baseLink>
+      <baseLink>base_link</baseLink>
       <leftFrontWheelLink>left_front_wheel_link</leftFrontWheelLink>
       <leftRearWheelLink>left_rear_wheel_link</leftRearWheelLink>

File: pandora_robots_description/urdf/side.urdf.xacro (robot description, xacro)
@@ -5,9 +5,9 @@
     <link name="${prefix_y}_side_link" >
       <inertial>
-	    <origin xyz="${reflect_y*(-9.2074E-08)} ${reflect_y*(0.010782)} -0.028501"
-	            rpy="0 0 0" />
+      <origin xyz="${reflect_y*(-9.2074E-08)} ${reflect_y*(0.010782)} -0.028501"
+              rpy="0 0 0" />
         <mass value="0.93539" />
         <inertia ixx="0.001211" ixy="-4.0495E-05" ixz="${reflect_y*(1.0211E-06)}"
-	             iyy="0.026668" iyz="${reflect_y*(-0.00024586)}" izz="0.026454" />
+               iyy="0.026668" iyz="${reflect_y*(-0.00024586)}" izz="0.026454" />
       </inertial>
       <visual>
@@ -23,5 +23,5 @@
         <origin xyz="0 0 0" rpy="0 0 ${(1-reflect_y)*1.57}" />
         <geometry>
-		      <!-- TODO: Simplify mesh -->
+          <!-- TODO: Simplify mesh -->
           <mesh filename="package://pandora_robots_description/meshes/gears/side_link.stl" />
         </geometry>
@@ -33,5 +33,5 @@
       <child link="${prefix_y}_side_link" />
       <axis xyz="0 1 0" />
-	    <!-- TODO: Set damping -->
+      <!-- TODO: Set damping -->
       <dynamics damping="0" />
       <limit effort="100" velocity="100"
@@ -44,7 +44,7 @@
     -->
     <xacro:wheel_caster prefix_y="${prefix_y}" prefix_x="front"
-	                      reflect_y="${reflect_y}" reflect_x="1" />
+                        reflect_y="${reflect_y}" reflect_x="1" />
     <xacro:wheel_caster prefix_y="${prefix_y}" prefix_x="rear"
-	                      reflect_y="${reflect_y}" reflect_x="-1" />
+                        reflect_y="${reflect_y}" reflect_x="-1" />
   </xacro:macro>
 </robot>

File: pandora_robots_description/urdf/wheel.urdf.xacro (robot description, xacro)
@@ -9,5 +9,5 @@
         <mass value="1.2128" />
         <inertia ixx="0.0032586" ixy="5.862E-08" ixz="${reflect_y*(4.2142E-07)}"
-	             iyy="0.0054812" iyz="${reflect_y*(-6.4028E-08)}" izz="0.0032574" />
+               iyy="0.0054812" iyz="${reflect_y*(-6.4028E-08)}" izz="0.0032574" />
       </inertial>
       <visual>
@@ -33,5 +33,5 @@
         <mass value="1.2128" />
         <inertia ixx="0.002982821" ixy="0" ixz="0"
-	               iyy="0.002982821" iyz="0" izz="0.004791967" />
+                 iyy="0.002982821" iyz="0" izz="0.004791967" />
       </inertial>
       <visual>
@@ -53,12 +53,12 @@
     <joint name="${prefix_y}_${prefix_x}_wheel_joint" type="continuous" >
       <origin xyz="${reflect_x*0.198785} ${reflect_y*0.110545} -0.052795"
-	          rpy="0 0 0" />
+            rpy="0 0 0" />
       <parent link="${prefix_y}_side_link" />
       <child link="${prefix_y}_${prefix_x}_wheel_link" />
       <axis xyz="0 1 0" />
-	  <limit effort="100" velocity="100" />
+    <limit effort="100" velocity="100" />
       <!-- <anchor xyz="0 0 0" /> -->
     </joint>
-	<!-- TODO: Fix physics -->
+  <!-- TODO: Fix physics -->
     <gazebo reference="${prefix_y}_${prefix_x}_wheel_link" >
       <mu1>0.8</mu1>
@@ -71,15 +71,15 @@
       <maxContacts>1</maxContacts>
     </gazebo>
-	<!--
+  <!--
     <transmission name="${prefix_y}_${prefix_x}_wheel_trans" >
-	  <type>transmission_interface/SimpleTransmission</type>
+    <type>transmission_interface/SimpleTransmission</type>
       <joint name="${prefix_y}_${prefix_x}_wheel_joint" />
       <actuator name="${prefix_y}_${prefix_x}_motor_link">
-	    <hardwareInterface>VelocityJointInterface</hardwareInterface>
+      <hardwareInterface>VelocityJointInterface</hardwareInterface>
         <mechanicalReduction>1.0</mechanicalReduction>
         <!- <motorTorqueConstant>1</motorTorqueConstant> ->
-	  </actuator>
+    </actuator>
     </transmission>
-	-->
+  -->
   </xacro:macro>
 </robot>

Commit message: Add new super simplified wheel mesh for better adhesion.

File: pandora_robots_description/urdf/base.urdf.xacro (robot description, xacro)
@@ -13,4 +13,5 @@
       <geometry>
         <mesh filename="package://pandora_robots_description/meshes/gears/base_link.stl" />
+        <!-- <mesh filename="package://pandora_robots_description/meshes/gears/simplified_base_link.stl" /> -->
       </geometry>
       <material name="" >
@@ -21,6 +22,6 @@
       <origin xyz="0 0 0" rpy="0 0 0" />
       <geometry>
-         <!-- TODO: Simplify mesh -->
         <mesh filename="package://pandora_robots_description/meshes/gears/base_link.stl" />
+        <!-- <mesh filename="package://pandora_robots_description/meshes/gears/simplified_base_link.stl" /> -->
       </geometry>
     </collision>
@@ -78,11 +79,13 @@
       <rightSideJoint>right_side_joint</rightSideJoint>
       <maxAngle>0.785</maxAngle>
+      <correctionForceModifier>200.0</correctionForceModifier>
+      <!-- TODO: Tune PID -->
+      <P>120.0</P>
+      <I>0.005</I>
+      <D>8.0</D>
       <sideJointDamping>0.0</sideJointDamping>
       <maxDownforce>0.0</maxDownforce>
-      <forceAdjustment>1.0</forceAdjustment>
-      <!-- TODO: Tune PID -->
-      <P>100.0</P>
-      <I>1</I>
-      <D>10.0</D>
+      <maxDifferentialForceZ>0.0</maxDifferentialForceZ>
+      <maxDifferentialForceY>0.0</maxDifferentialForceY>
     </plugin>
   </gazebo>

File: pandora_robots_description/urdf/side.urdf.xacro (robot description, xacro)
@@ -15,4 +15,5 @@
         <geometry>
           <mesh filename="package://pandora_robots_description/meshes/gears/side_link.stl" />
+          <!-- <mesh filename="package://pandora_robots_description/meshes/gears/simplified_side_link.stl" /> -->
         </geometry>
         <material name="" >
@@ -23,6 +24,6 @@
         <origin xyz="0 0 0" rpy="0 0 ${(1-reflect_y)*1.57}" />
         <geometry>
-          <!-- TODO: Simplify mesh -->
           <mesh filename="package://pandora_robots_description/meshes/gears/side_link.stl" />
+          <!-- <mesh filename="package://pandora_robots_description/meshes/gears/simplified_side_link.stl" /> -->
         </geometry>
       </collision>
@@ -34,5 +35,5 @@
       <axis xyz="0 1 0" />
       <!-- TODO: Set damping -->
-      <dynamics damping="0" />
+      <dynamics damping="0.1" />
       <limit effort="100" velocity="100"
              lower="-0.785" upper="0.785" />

File: pandora_robots_description/urdf/wheel.urdf.xacro (robot description, xacro)
@@ -3,5 +3,4 @@
   <xacro:macro name="wheel_caster" params="prefix_y prefix_x reflect_y reflect_x" >
     <link name="${prefix_y}_${prefix_x}_wheel_link" >
-      <!--
       <inertial>
         <origin xyz="${reflect_y*(-2.2235E-05)} ${reflect_y*(-0.00052624)} 2.4287E-05"
@@ -14,6 +13,7 @@
         <origin xyz="0 0 0" rpy="0 0 ${(1-reflect_y)*1.57}" />
         <geometry>
-          <mesh filename="package://pandora_robots_description/meshes/gears/wheel_link.stl" />
-          <mesh filename="package://pandora_robots_description/meshes/gears/simplified_wheel_link.stl" />
+          <!-- <mesh filename="package://pandora_robots_description/meshes/gears/wheel_link.stl" /> -->
+          <!-- <mesh filename="package://pandora_robots_description/meshes/gears/simplified_wheel_link.stl" /> -->
+          <mesh filename="package://pandora_robots_description/meshes/gears/super_simplified_wheel_link.stl" />
         </geometry>
         <material name="" >
@@ -24,9 +24,10 @@
         <origin xyz="0 0 0" rpy="0 0 ${(1-reflect_y)*1.57}" />
         <geometry>
-          <mesh filename="package://pandora_robots_description/meshes/gears/wheel_link.stl" />
-          <mesh filename="package://pandora_robots_description/meshes/gears/simplified_wheel_link.stl" />
+          <!-- <mesh filename="package://pandora_robots_description/meshes/gears/wheel_link.stl" /> -->
+          <!-- <mesh filename="package://pandora_robots_description/meshes/gears/simplified_wheel_link.stl" /> -->
+          <mesh filename="package://pandora_robots_description/meshes/gears/super_simplified_wheel_link.stl" />
         </geometry>
       </collision>
-      -->
+      <!--
       <inertial>
         <origin xyz="0 0 0" rpy="0 0 0" />
@@ -50,4 +51,5 @@
         </geometry>
       </collision>
+      -->
     </link>
     <joint name="${prefix_y}_${prefix_x}_wheel_joint" type="continuous" >
@@ -58,18 +60,17 @@
       <axis xyz="0 1 0" />
     <limit effort="100" velocity="100" />
-      <!-- <anchor xyz="0 0 0" /> -->
+    <!-- <anchor xyz="0 0 0" /> -->
     </joint>
-  <!-- TODO: Fix physics -->
+    <!-- TODO: Fix physics -->
     <gazebo reference="${prefix_y}_${prefix_x}_wheel_link" >
-      <mu1>0.8</mu1>
-      <mu2>0.8</mu2>
+      <mu1>0.75</mu1>
+      <mu2>0.75</mu2>
       <!-- <fdir1>1 0 0</fdir1> -->
       <kp>10000000.0</kp>
       <kd>1.0</kd>
-      <!-- TODO: Adjust min depth -->
-      <minDepth>0.005</minDepth>
+      <minDepth>0.001</minDepth>
       <maxContacts>1</maxContacts>
     </gazebo>
-  <!--
+    <!--
     <transmission name="${prefix_y}_${prefix_x}_wheel_trans" >
     <type>transmission_interface/SimpleTransmission</type>
@@ -81,5 +82,5 @@
     </actuator>
     </transmission>
-  -->
+    -->
   </xacro:macro>
 </robot>

Commit message: Add laser and kinect.

File: pandora_robots_description/urdf/base.urdf.xacro (robot description, xacro)
@@ -13,5 +13,4 @@
       <geometry>
         <mesh filename="package://pandora_robots_description/meshes/gears/base_link.stl" />
-        <!-- <mesh filename="package://pandora_robots_description/meshes/gears/simplified_base_link.stl" /> -->
       </geometry>
       <material name="" >
@@ -23,4 +22,5 @@
       <geometry>
         <mesh filename="package://pandora_robots_description/meshes/gears/base_link.stl" />
+        <!-- TODO -->
         <!-- <mesh filename="package://pandora_robots_description/meshes/gears/simplified_base_link.stl" /> -->
       </geometry>
@@ -33,15 +33,15 @@
     <origin xyz="0 -0.110 0" rpy="0 0 0" />
   </xacro:side_caster>
-  <!-- Disable sensors and plugins
-  Insert kinect
+  <!-- Insert kinect -->
   <xacro:include filename="$(find pandora_sensors_description)/urdf/kinect_camera.urdf.xacro" />
   <xacro:kinect_caster parent="base_link">
-    <origin xyz="0.2 0 0.33" rpy="0 0 0"/>
+    <origin xyz="0.156 0 0.526" rpy="0 0 0"/>
   </xacro:kinect_caster>
-  Insert hokuyo laser
+  <!-- Insert hokuyo laser -->
   <xacro:include filename="$(find pandora_sensors_description)/urdf/hokuyo_utm_30lx.urdf.xacro" />
   <xacro:hokuyo_caster parent="base_link">
-    <origin xyz="0.25 0 0.15" rpy="0 0 0"/>
+    <origin xyz="0.2 0 0.15" rpy="0 0 0"/>
   </xacro:hokuyo_caster>
+  <!--
   Add imu plugin
   <gazebo>

File: pandora_robots_description/urdf/side.urdf.xacro (robot description, xacro)
@@ -15,5 +15,4 @@
         <geometry>
           <mesh filename="package://pandora_robots_description/meshes/gears/side_link.stl" />
-          <!-- <mesh filename="package://pandora_robots_description/meshes/gears/simplified_side_link.stl" /> -->
         </geometry>
         <material name="" >
@@ -25,4 +24,5 @@
         <geometry>
           <mesh filename="package://pandora_robots_description/meshes/gears/side_link.stl" />
+          <!-- TODO -->
           <!-- <mesh filename="package://pandora_robots_description/meshes/gears/simplified_side_link.stl" /> -->
         </geometry>
@@ -34,5 +34,5 @@
       <child link="${prefix_y}_side_link" />
       <axis xyz="0 1 0" />
-      <!-- TODO: Set damping -->
+      <!-- TODO: Adjust damping -->
       <dynamics damping="0.1" />
       <limit effort="100" velocity="100"

File: pandora_robots_description/urdf/wheel.urdf.xacro (robot description, xacro)
@@ -13,7 +13,6 @@
         <origin xyz="0 0 0" rpy="0 0 ${(1-reflect_y)*1.57}" />
         <geometry>
-          <!-- <mesh filename="package://pandora_robots_description/meshes/gears/wheel_link.stl" /> -->
+          <mesh filename="package://pandora_robots_description/meshes/gears/wheel_link.stl" />
           <!-- <mesh filename="package://pandora_robots_description/meshes/gears/simplified_wheel_link.stl" /> -->
-          <mesh filename="package://pandora_robots_description/meshes/gears/super_simplified_wheel_link.stl" />
         </geometry>
         <material name="" >
@@ -24,32 +23,7 @@
         <origin xyz="0 0 0" rpy="0 0 ${(1-reflect_y)*1.57}" />
         <geometry>
-          <!-- <mesh filename="package://pandora_robots_description/meshes/gears/wheel_link.stl" /> -->
-          <!-- <mesh filename="package://pandora_robots_description/meshes/gears/simplified_wheel_link.stl" /> -->
-          <mesh filename="package://pandora_robots_description/meshes/gears/super_simplified_wheel_link.stl" />
+          <mesh filename="package://pandora_robots_description/meshes/gears/simplified_wheel_link.stl" />
         </geometry>
       </collision>
-      <!--
-      <inertial>
-        <origin xyz="0 0 0" rpy="0 0 0" />
-        <mass value="1.2128" />
-        <inertia ixx="0.002982821" ixy="0" ixz="0"
-                 iyy="0.002982821" iyz="0" izz="0.004791967" />
-      </inertial>
-      <visual>
-        <origin xyz="0 0 0" rpy="1.57 0 0" />
-        <geometry>
-          <cylinder length="0.0762" radius="0.088895"/>
-        </geometry>
-        <material name="" >
-          <color rgba="0.753 0.753 0.753 1" />
-        </material>
-      </visual>
-      <collision>
-        <origin xyz="0 0 0" rpy="1.57 0 0" />
-        <geometry>
-          <cylinder length="0.0762" radius="0.088895"/>
-        </geometry>
-      </collision>
-      -->
     </link>
     <joint name="${prefix_y}_${prefix_x}_wheel_joint" type="continuous" >
@@ -60,5 +34,4 @@
       <axis xyz="0 1 0" />
     <limit effort="100" velocity="100" />
-    <!-- <anchor xyz="0 0 0" /> -->
     </joint>
     <!-- TODO: Fix physics -->
