Commit message: Add simplified meshes for base and side links.

File: pandora_robots_description/urdf/base.urdf.xacro (robot description, xacro)
@@ -21,7 +21,5 @@
       <origin xyz="0 0 0" rpy="0 0 0" />
       <geometry>
-        <mesh filename="package://pandora_robots_description/meshes/gears/base_link.stl" />
-        <!-- TODO -->
-        <!-- <mesh filename="package://pandora_robots_description/meshes/gears/simplified_base_link.stl" /> -->
+        <mesh filename="package://pandora_robots_description/meshes/gears/simplified_base_link.stl" />
       </geometry>
     </collision>

File: pandora_robots_description/urdf/side.urdf.xacro (robot description, xacro)
@@ -23,7 +23,5 @@
         <origin xyz="0 0 0" rpy="0 0 ${(1-reflect_y)*1.57}" />
         <geometry>
-          <mesh filename="package://pandora_robots_description/meshes/gears/side_link.stl" />
-          <!-- TODO -->
-          <!-- <mesh filename="package://pandora_robots_description/meshes/gears/simplified_side_link.stl" /> -->
+          <mesh filename="package://pandora_robots_description/meshes/gears/simplified_side_link.stl" />
         </geometry>
       </collision>

File: pandora_robots_description/urdf/wheel.urdf.xacro (robot description, xacro)
@@ -14,5 +14,4 @@
         <geometry>
           <mesh filename="package://pandora_robots_description/meshes/gears/wheel_link.stl" />
-          <!-- <mesh filename="package://pandora_robots_description/meshes/gears/simplified_wheel_link.stl" /> -->
         </geometry>
         <material name="" >

Commit message: Tune differential PID and disable sensors.

File: pandora_robots_description/urdf/base.urdf.xacro (robot description, xacro)
@@ -31,14 +31,16 @@
     <origin xyz="0 -0.110 0" rpy="0 0 0" />
   </xacro:side_caster>
-  <!-- Insert kinect -->
+  <!--
+  Insert kinect
   <xacro:include filename="$(find pandora_sensors_description)/urdf/kinect_camera.urdf.xacro" />
   <xacro:kinect_caster parent="base_link">
     <origin xyz="0.156 0 0.526" rpy="0 0 0"/>
   </xacro:kinect_caster>
-  <!-- Insert hokuyo laser -->
+  Insert hokuyo laser
   <xacro:include filename="$(find pandora_sensors_description)/urdf/hokuyo_utm_30lx.urdf.xacro" />
   <xacro:hokuyo_caster parent="base_link">
     <origin xyz="0.2 0 0.15" rpy="0 0 0"/>
   </xacro:hokuyo_caster>
+  -->
   <!--
   Add imu plugin
@@ -77,9 +79,9 @@
       <rightSideJoint>right_side_joint</rightSideJoint>
       <maxAngle>0.785</maxAngle>
-      <correctionForceModifier>200.0</correctionForceModifier>
+      <correctionForceModifier>100.0</correctionForceModifier>
       <!-- TODO: Tune PID -->
-      <P>120.0</P>
-      <I>0.005</I>
-      <D>8.0</D>
+      <P>250.0</P>
+      <I>0.001</I>
+      <D>1000.0</D>
       <sideJointDamping>0.0</sideJointDamping>
       <maxDownforce>0.0</maxDownforce>

File: pandora_robots_description/urdf/side.urdf.xacro (robot description, xacro)
@@ -33,5 +33,5 @@
       <axis xyz="0 1 0" />
       <!-- TODO: Adjust damping -->
-      <dynamics damping="0.1" />
+      <dynamics damping="0.0" />
       <limit effort="100" velocity="100"
              lower="-0.785" upper="0.785" />
