Commit message: Add ros control plugin and wheel transmission for pioneer3at.

File: pandora_robots_description/urdf/pioneer3at/pioneer3at.urdf.xacro (robot description, xacro)
@@ -1,9 +1,6 @@
 <?xml version="1.0"?>
-<robot xmlns:sensor="http://playerstage.sourceforge.net/gazebo/xmlschema/#sensor"
-       xmlns:controller="http://playerstage.sourceforge.net/gazebo/xmlschema/#controller"
-       xmlns:interface="http://playerstage.sourceforge.net/gazebo/xmlschema/#interface"
-       xmlns:xacro="http://ros.org/wiki/xacro"
-       name="pioneer3at">
-<!-- base_link -->
+<robot name="pioneer3at"
+       xacro="http://ros.org/wiki/xacro" >
+  <!-- Base Link -->
   <link name="base_link">
     <inertial>
@@ -32,5 +29,5 @@
     <material value="Gazebo/Red"/>
   </gazebo>
-<!-- Top -->
+  <!-- Top -->
   <link name="top_plate">
     <inertial>
@@ -104,20 +101,20 @@
         <inertia ixx="0.001" ixy="0.0" ixz="0.0"
            iyy="0.001" iyz="0.0" izz="0.001"/>
-        </inertial>
-    <visual name="base_visual">
-      <origin xyz="0 0 0" rpy="0 0 0"/>
-      <geometry name="pioneer_geom">
-        <mesh filename="package://pandora_robots_description/meshes/pioneer3at/p3at_meshes/${suffix}_hubcap.stl"/>
-      </geometry>
-      <material name="HubcapYellow">
-        <color rgba="1.0 0.811 0.151 1.0"/>
-      </material>
-    </visual>
-    <collision>
-      <origin xyz="0 0 0" rpy="0 0 0"/>
-      <geometry>
-        <box size="0 0 0"/>
-      </geometry>
-    </collision>
+      </inertial>
+      <visual name="base_visual">
+        <origin xyz="0 0 0" rpy="0 0 0"/>
+        <geometry name="pioneer_geom">
+          <mesh filename="package://pandora_robots_description/meshes/pioneer3at/p3at_meshes/${suffix}_hubcap.stl"/>
+        </geometry>
+        <material name="HubcapYellow">
+          <color rgba="1.0 0.811 0.151 1.0"/>
+        </material>
+      </visual>
+      <collision>
+        <origin xyz="0 0 0" rpy="0 0 0"/>
+        <geometry>
+          <box size="0 0 0"/>
+        </geometry>
+      </collision>
     </link>
     <gazebo reference="p3at_front_${suffix}_hub">
@@ -135,21 +132,21 @@
         <inertia ixx="0.012411765597" ixy="0" ixz="0"
            iyy="0.015218160428" iyz="0" izz="0.011763977943"/>
-        </inertial>
-    <visual name="base_visual">
-      <origin xyz="0 0 0" rpy="0 0 0"/>
-      <geometry name="pioneer_geom">
-        <mesh filename="package://pandora_robots_description/meshes/pioneer3at/p3at_meshes/wheel.stl"/>
-      </geometry>
-      <material name="WheelBlack">
-        <color rgba="0.117 0.117 0.117 1"/>
-      </material>
-    </visual>
-    <collision>
-      <origin xyz="0 0 0" rpy="${-3.1415927/2} 0 0"/>
-      <geometry>
-        <!--mesh filename="package://pandora_robots_description/meshes/pioneer3at/p3at_meshes/wheel.stl"/-->
-        <cylinder radius="0.111" length="0.075"/>
-      </geometry>
-    </collision>
+      </inertial>
+      <visual name="base_visual">
+        <origin xyz="0 0 0" rpy="0 0 0"/>
+        <geometry name="pioneer_geom">
+          <mesh filename="package://pandora_robots_description/meshes/pioneer3at/p3at_meshes/wheel.stl"/>
+        </geometry>
+        <material name="WheelBlack">
+          <color rgba="0.117 0.117 0.117 1"/>
+        </material>
+      </visual>
+      <collision>
+        <origin xyz="0 0 0" rpy="${-3.1415927/2} 0 0"/>
+        <geometry>
+          <!--mesh filename="package://pandora_robots_description/meshes/pioneer3at/p3at_meshes/wheel.stl"/-->
+          <cylinder radius="0.111" length="0.075"/>
+        </geometry>
+      </collision>
     </link>
     <gazebo reference="p3at_front_${suffix}_wheel">
@@ -165,5 +162,5 @@
       <child link="p3at_front_${suffix}_wheel"/>
     </joint>
-  <!-- Back Axles + Wheels + Hubcaps -->
+    <!-- Back Axles + Wheels + Hubcaps -->
     <link name="p3at_back_${suffix}_axle">
       <inertial>
@@ -172,20 +169,20 @@
         <inertia ixx="0.001" ixy="0.0" ixz="0.0"
            iyy="0.001" iyz="0.0" izz="0.001"/>
-        </inertial>
-    <visual name="base_visual">
-      <origin xyz="0 0 0" rpy="0 0 0"/>
-      <geometry name="pioneer_geom">
-        <mesh filename="package://pandora_robots_description/meshes/pioneer3at/p3at_meshes/axle.stl"/>
-      </geometry>
-      <material name="AxleGrey">
-        <color rgba="0.5 0.5 0.5 1"/>
-      </material>
-    </visual>
-    <collision>
-      <origin xyz="0 0 0" rpy="0 0 0"/>
-      <geometry>
-        <mesh filename="package://pandora_robots_description/meshes/pioneer3at/p3at_meshes/axle.stl"/>
-      </geometry>
-    </collision>
+      </inertial>
+      <visual name="base_visual">
+        <origin xyz="0 0 0" rpy="0 0 0"/>
+        <geometry name="pioneer_geom">
+          <mesh filename="package://pandora_robots_description/meshes/pioneer3at/p3at_meshes/axle.stl"/>
+        </geometry>
+        <material name="AxleGrey">
+          <color rgba="0.5 0.5 0.5 1"/>
+        </material>
+      </visual>
+      <collision>
+        <origin xyz="0 0 0" rpy="0 0 0"/>
+        <geometry>
+          <mesh filename="package://pandora_robots_description/meshes/pioneer3at/p3at_meshes/axle.stl"/>
+        </geometry>
+      </collision>
     </link>
     <gazebo reference="p3at_back_${suffix}_axle">
@@ -203,18 +200,18 @@
         <inertia ixx="0.001" ixy="0.0" ixz="0.0"
            iyy="0.001" iyz="0.0" izz="0.001"/>
-        </inertial>
-    <visual name="base_visual">
-      <origin xyz="0 0 0" rpy="0 0 0"/>
-      <geometry name="pioneer_geom">
-        <mesh filename="package://pandora_robots_description/meshes/pioneer3at/p3at_meshes/${suffix}_hubcap.stl"/>
-      </geometry>
-      <material name="HubcapYellow"/>
-    </visual>
-    <collision>
-      <origin xyz="0 0 0" rpy="0 0 0"/>
-      <geometry>
-        <mesh filename="package://pandora_robots_description/meshes/pioneer3at/p3at_meshes/${suffix}_hubcap.stl"/>
-      </geometry>
-    </collision>
+      </inertial>
+      <visual name="base_visual">
+        <origin xyz="0 0 0" rpy="0 0 0"/>
+        <geometry name="pioneer_geom">
+          <mesh filename="package://pandora_robots_description/meshes/pioneer3at/p3at_meshes/${suffix}_hubcap.stl"/>
+        </geometry>
+        <material name="HubcapYellow"/>
+      </visual>
+      <collision>
+        <origin xyz="0 0 0" rpy="0 0 0"/>
+        <geometry>
+          <mesh filename="package://pandora_robots_description/meshes/pioneer3at/p3at_meshes/${suffix}_hubcap.stl"/>
+        </geometry>
+      </collision>
     </link>
     <gazebo reference="p3at_back_${suffix}_hub">
@@ -232,19 +229,19 @@
         <inertia ixx="0.012411765597" ixy="0" ixz="0"
            iyy="0.015218160428" iyz="0" izz="0.011763977943"/>
-        </inertial>
-    <visual name="base_visual">
-      <origin xyz="0 0 0" rpy="0 0 0"/>
-      <geometry name="pioneer_geom">
-        <mesh filename="package://pandora_robots_description/meshes/pioneer3at/p3at_meshes/wheel.stl"/>
-      </geometry>
-      <material name="WheelBlack"/>
-    </visual>
-    <collision>
-      <origin xyz="0 0 0" rpy="${-3.1415927/2} 0 0"/>
-      <geometry>
-        <!--<mesh filename="package://pandora_robots_description/meshes/pioneer3at/p3at_meshes/wheel.stl"/>-->
-        <cylinder radius="0.111" length="0.075"/>
-      </geometry>
-    </collision>
+      </inertial>
+      <visual name="base_visual">
+        <origin xyz="0 0 0" rpy="0 0 0"/>
+        <geometry name="pioneer_geom">
+          <mesh filename="package://pandora_robots_description/meshes/pioneer3at/p3at_meshes/wheel.stl"/>
+        </geometry>
+        <material name="WheelBlack"/>
+      </visual>
+      <collision>
+        <origin xyz="0 0 0" rpy="${-3.1415927/2} 0 0"/>
+        <geometry>
+          <!--<mesh filename="package://pandora_robots_description/meshes/pioneer3at/p3at_meshes/wheel.stl"/>-->
+          <cylinder radius="0.111" length="0.075"/>
+        </geometry>
+      </collision>
     </link>
     <gazebo reference="p3at_back_${suffix}_wheel">
@@ -278,5 +275,6 @@
       <minDepth>0.00</minDepth>
     </gazebo>
-      <transmission name="p3at_front_${suffix}_wheel_transmission">
+    <!-- Wheel Transmission -->
+    <transmission name="p3at_front_${suffix}_wheel_transmission">
       <type>transmission_interface/SimpleTransmission</type>
       <joint name="p3at_front_${suffix}_wheel_joint"/>
@@ -295,8 +293,16 @@
     </transmission>
   </xacro:macro>
+  <!-- Add wheels -->
   <xacro:p3at_front suffix="left" reflect="1"/>
   <xacro:p3at_front suffix="right" reflect="-1"/>
   <xacro:p3at_back suffix="left" reflect="1"/>
   <xacro:p3at_back suffix="right" reflect="-1"/>
+  <!-- Plugins ============================================================ -->
+  <!-- Add ros control plugin-->
+  <gazebo>
+    <plugin name="gazebo_ros_control" filename="libgazebo_ros_control.so">
+      <robotNamespace></robotNamespace>
+    </plugin>
+  </gazebo>
   <!-- Add skid steer drive plugin-->
   <gazebo>
@@ -319,4 +325,28 @@
     </plugin>
   </gazebo>
+  <!-- Add 3D pose plugin -->
+  <gazebo>
+    <plugin name="Pandora3dPosePlugin" filename="libpandora_p3d_plugin.so">
+      <robotNamespace></robotNamespace>
+      <bodyName>base_link</bodyName>
+      <frameName>map</frameName>
+      <topicName>perfect_pose</topicName>
+      <broadcastTF>0</broadcastTF>
+    </plugin>
+  </gazebo>
+  <!-- Add imu plugin-->
+  <gazebo>
+    <plugin filename="libgazebo_ros_imu.so" name="imu_en_ros">
+      <bodyName>base_link</bodyName>
+      <robotNamespace></robotNamespace>
+      <topicName>/sensors/imu</topicName>
+    </plugin>
+  </gazebo>
+  <!-- Sensors ============================================================ -->
+  <!--Insert kinect-->
+  <xacro:include filename="$(find pandora_sensors_description)/urdf/kinect_camera.urdf.xacro" />
+  <xacro:kinect_caster parent="base_link">
+    <origin xyz="0.2 0 0.33" rpy="0 0 0"/>
+  </xacro:kinect_caster>
   <!--Insert hokuyo laser-->
   <xacro:include filename="$(find pandora_sensors_description)/urdf/hokuyo_utm_30lx.urdf.xacro" />
@@ -324,24 +354,4 @@
     <origin xyz="0.25 0 0.15" rpy="0 0 0"/>
   </xacro:hokuyo_caster>
-  <!-- Add imu plugin-->
-  <gazebo>
-    <plugin name="RosImuPlugin" filename="libpandora_imu_stabilizer_plugin.so">
-      <topicName>/sensors/imu</topicName>
-      <bodyName>base_link</bodyName>
-      <updateRate>50.0</updateRate>
-      <robotNamespace></robotNamespace>
-      <serviceName>default_imu</serviceName>
-      <gaussianNoise>0.0</gaussianNoise>
-      <xyzOffset>0 0 0</xyzOffset>
-      <rpyOffset>0 0 0</rpyOffset>
-      <rollCorrectionJoint>laser_roll_joint</rollCorrectionJoint>
-      <pitchCorrectionJoint>laser_pitch_joint</pitchCorrectionJoint>
-    </plugin>
-  </gazebo>
-  <!--Insert kinect-->
-  <xacro:include filename="$(find pandora_sensors_description)/urdf/kinect_camera.urdf.xacro" />
-  <xacro:kinect_caster parent="base_link">
-    <origin xyz="0.2 0 0.33" rpy="0 0.53 0"/>
-  </xacro:kinect_caster>
   <!--Insert sonars-->
   <xacro:include filename="$(find pandora_sensors_description)/urdf/sonar_sensor.urdf.xacro" />
