Commit message: Add color to visual meshes.

File: pandora_robots_description/urdf/gears/config/gears_physics.gazebo.xacro (robot description, xacro)
@@ -11,5 +11,5 @@
   <xacro:macro name="base_link_sdf_physics" >
     <gazebo reference="${base_link_name}_link" >
-      <material>Gazebo/Grey</material>
+      <!-- <material>Gazebo/Grey</material> -->
       <!-- <gravity>false</gravity> -->
       <!-- <dampingFactor>0.0</dampingFactor> -->
@@ -30,5 +30,5 @@
                params="prefix_y" >
     <gazebo reference="${prefix_y}_${side_link_name}_link" >
-      <material>Gazebo/FlatBlack</material>
+      <!-- <material>Gazebo/FlatBlack</material> -->
       <!-- <gravity>false</gravity> -->
       <!-- <dampingFactor>0.0</dampingFactor> -->
@@ -49,5 +49,5 @@
                params="prefix_y prefix_x" >
     <gazebo reference="${prefix_y}_${prefix_x}_${wheel_link_name}_link" >
-      <material>Gazebo/FlatBlack</material>
+      <!-- <material>Gazebo/FlatBlack</material> -->
       <!-- <gravity>true</gravity> -->
       <!-- <dampingFactor>0</dampingFactor> -->

File: pandora_robots_description/urdf/gears/config/properties/meshes.xacro (robot description, xacro)
@@ -5,5 +5,5 @@
   <xacro:macro name="base_link_visual_mesh" >
     <geometry>
-      <mesh filename="package://pandora_robots_description/meshes/gears/visual/base_link.stl" />
+      <mesh filename="package://pandora_robots_description/meshes/gears/visual/base_link.dae" />
       <!-- <mesh filename="package://pandora_robots_description/meshes/gears/collision/base_link.stl" /> -->
     </geometry>
@@ -12,5 +12,5 @@
   <xacro:macro name="side_link_visual_mesh" >
     <geometry>
-      <mesh filename="package://pandora_robots_description/meshes/gears/visual/side_link.stl" />
+      <mesh filename="package://pandora_robots_description/meshes/gears/visual/side_link.dae" />
       <!-- <mesh filename="package://pandora_robots_description/meshes/gears/collision/side_link.stl" /> -->
     </geometry>
@@ -19,5 +19,5 @@
   <xacro:macro name="wheel_link_visual_mesh" >
     <geometry>
-      <mesh filename="package://pandora_robots_description/meshes/gears/visual/wheel_link.stl" />
+      <mesh filename="package://pandora_robots_description/meshes/gears/visual/wheel_link.dae" />
       <!-- <mesh filename="package://pandora_robots_description/meshes/gears/collision/wheel_link.stl" /> -->
     </geometry>
@@ -29,5 +29,5 @@
     <geometry>
       <mesh filename="package://pandora_robots_description/meshes/gears/collision/base_link.stl" />
-      <!-- <mesh filename="package://pandora_robots_description/meshes/gears/visual/base_link.stl" /> -->
+      <!-- <mesh filename="package://pandora_robots_description/meshes/gears/visual/base_link.dae" /> -->
     </geometry>
   </xacro:macro>
@@ -36,5 +36,5 @@
     <geometry>
       <mesh filename="package://pandora_robots_description/meshes/gears/collision/side_link.stl" />
-      <!-- <mesh filename="package://pandora_robots_description/meshes/gears/visual/side_link.stl" /> -->
+      <!-- <mesh filename="package://pandora_robots_description/meshes/gears/visual/side_link.dae" /> -->
     </geometry>
   </xacro:macro>
@@ -43,5 +43,5 @@
     <geometry>
       <mesh filename="package://pandora_robots_description/meshes/gears/collision/wheel_link.stl" />
-      <!-- <mesh filename="package://pandora_robots_description/meshes/gears/visual/wheel_link.stl" /> -->
+      <!-- <mesh filename="package://pandora_robots_description/meshes/gears/visual/wheel_link.dae" /> -->
     </geometry>
   </xacro:macro>

Commit message: Add new visual and collision meshes for base and linear links.

File: pandora_robots_description/urdf/gears/config/gears_physics.gazebo.xacro (robot description, xacro)
@@ -134,5 +134,5 @@
     <dynamics damping="0.0" />
          <!-- friction="0.0" /> -->
-    <limit lower="-${linear_elevator_joint_max_limit}"
+    <limit lower="0"
            upper="${linear_elevator_joint_max_limit}"
            effort="100.0"
@@ -150,5 +150,5 @@
     <dynamics damping="${side_joint_damping}" />
          <!-- friction="0.0" /> -->
-    <limit lower="0"
+    <limit lower="-${side_joint_max_limit}"
            upper="${side_joint_max_limit}"
            effort="100.0"
