Commit message: Add 'xacro if' to enable sensor transimission.

File: pandora_robots_description/urdf/gears/config/gears_configurations.xacro (robot description, xacro)
@@ -6,39 +6,39 @@
   <!-- Links ============================================================== -->
   <xacro:property name="enable_links" value="true" />
-  <xacro:property name="enable_base_link" value="true" />
-  <xacro:property name="enable_side_links" value="true" />
-  <xacro:property name="enable_wheel_links" value="true" />
+    <xacro:property name="enable_base_link" value="true" />
+    <xacro:property name="enable_side_links" value="true" />
+    <xacro:property name="enable_wheel_links" value="true" />
   <!-- Joints ============================================================= -->
   <xacro:property name="enable_joints" value="true" />
-  <xacro:property name="enable_side_joints" value="true" />
-  <xacro:property name="enable_wheel_joints" value="true" />
+    <xacro:property name="enable_side_joints" value="true" />
+    <xacro:property name="enable_wheel_joints" value="true" />
   <!-- Sensors ============================================================ -->
   <xacro:property name="enable_sensors" value="false" />
-  <xacro:property name="enable_kinect_sensor" value="true" />
-  <xacro:property name="enable_hokuyo_laser_sensor" value="true" />
-  <xacro:property name="enable_sonar_sensor" value="false" />
-  <xacro:property name="enable_thermal_sensor" value="false" />
-  <xacro:property name="enable_co2_sensor" value="false" />
-  <xacro:property name="enable_microphone_sensor" value="false" />
+    <xacro:property name="enable_kinect_sensor" value="true" />
+    <xacro:property name="enable_hokuyo_laser_sensor" value="true" />
+    <xacro:property name="enable_sonar_sensor" value="false" />
+    <xacro:property name="enable_thermal_sensor" value="false" />
+    <xacro:property name="enable_co2_sensor" value="false" />
+    <xacro:property name="enable_microphone_sensor" value="false" />
   <!-- Transmission ======================================================= -->
-  <xacro:property name="enable_transmission" value="false" />
-  <xacro:property name="enable_wheel_transmission" value="true" />
-  <xacro:property name="enable_sensor_transmission" value="true" />
-  <xacro:property name="enable_laser_sensor_transmission" value="true" />
-  <xacro:property name="enable_kinect_sensor_transmission" value="true" />
+  <xacro:property name="enable_transmission" value="true" />
+    <xacro:property name="enable_sensor_transmission" value="false" />
+      <xacro:property name="enable_laser_sensor_transmission" value="true" />
+      <xacro:property name="enable_kinect_sensor_transmission" value="true" />
+    <xacro:property name="enable_wheel_transmission" value="true" />
   <!-- Plugins ============================================================ -->
   <xacro:property name="enable_plugins" value="true" />
-  <xacro:property name="enable_pandora_differential_plugin" value="true" />
-  <xacro:property name="enable_pandora_p3d_plugin" value="false" />
-  <xacro:property name="enable_ros_imu_plugin" value="false" />
-  <xacro:property name="enable_ros_control_plugin" value="false" />
-  <xacro:property name="enable_ros_skid_steer_drive_plugin" value="true" />
+    <xacro:property name="enable_pandora_differential_plugin" value="true" />
+    <xacro:property name="enable_pandora_p3d_plugin" value="false" />
+    <xacro:property name="enable_ros_imu_plugin" value="false" />
+    <xacro:property name="enable_ros_control_plugin" value="true" />
+    <xacro:property name="enable_ros_skid_steer_drive_plugin" value="true" />
   <!-- SDF Physics ======================================================== -->
   <xacro:property name="enable_sdf_physics" value="true" />
-  <xacro:property name="enable_base_link_sdf_physics" value="true" />
-  <xacro:property name="enable_side_link_sdf_physics" value="true" />
-  <xacro:property name="enable_wheel_link_sdf_physics" value="true" />
-  <xacro:property name="enable_side_joint_sdf_physics" value="false" />
-  <xacro:property name="enable_wheel_joint_sdf_physics" value="false" />
+    <xacro:property name="enable_base_link_sdf_physics" value="true" />
+    <xacro:property name="enable_side_link_sdf_physics" value="true" />
+    <xacro:property name="enable_wheel_link_sdf_physics" value="true" />
+    <xacro:property name="enable_side_joint_sdf_physics" value="false" />
+    <xacro:property name="enable_wheel_joint_sdf_physics" value="false" />
   <!-- Meshes ============================================================= -->
   <!-- TODO -->

File: pandora_robots_description/urdf/gears/gears.urdf.xacro (robot description, xacro)
@@ -123,12 +123,14 @@
     </xacro:if>
     <!-- ================================================================== -->
-    <xacro:if value="${enable_kinect_sensor_transmission}" >
-      <xacro:sensor_transmission sensor="kinect" rotation="pitch" />
-      <xacro:sensor_transmission sensor="kinect" rotation="yaw" />
-    </xacro:if>
-    <!-- ================================================================== -->
-    <xacro:if value="${enable_laser_sensor_transmission}" >
-      <xacro:sensor_transmission sensor="laser" rotation="roll" />
-      <xacro:sensor_transmission sensor="laser" rotation="pitch" />
+    <xacro:if value="${enable_sensor_transmission}" >
+      <xacro:if value="${enable_kinect_sensor_transmission}" >
+        <xacro:sensor_transmission sensor="kinect" rotation="pitch" />
+        <xacro:sensor_transmission sensor="kinect" rotation="yaw" />
+      </xacro:if>
+      <!-- ================================================================ -->
+      <xacro:if value="${enable_laser_sensor_transmission}" >
+        <xacro:sensor_transmission sensor="laser" rotation="roll" />
+        <xacro:sensor_transmission sensor="laser" rotation="pitch" />
+      </xacro:if>
     </xacro:if>
     <!-- ================================================================== -->
