Commit message: Fix transmission hardware interface in gears and refactor pioneer3at.

File: pandora_robots_description/urdf/gears/config/gears_configurations.xacro (robot description, xacro)
@@ -63,9 +63,12 @@
   <xacro:property name="side_joint_damping" value="0.0" />
   <!-- ==================================================================== -->
-  <xacro:property name="max_linear_velocity" value="2.0" />
-  <xacro:property name="max_angular_velocity" value="2.0" />
+  <xacro:property name="max_robot_linear_velocity" value="2.0" />
+  <xacro:property name="max_robot_angular_velocity" value="2.0" />
+  <xacro:property name="max_kinect_angular_velocity" value="2.5" />
+  <xacro:property name="max_laser_angular_velocity" value="2.5" />
   <!-- ==================================================================== -->
-  <xacro:property name="max_linear_acceleration" value="1.0" />
-  <xacro:property name="max_angular_acceleration" value="1.0" />
+  <xacro:property name="max_robot_linear_acceleration" value="1.0" />
+  <xacro:property name="max_kinect_angular_acceleration" value="0.0" />
+  <xacro:property name="max_laser_angular_acceleration" value="0.0" />
   <!-- ==================================================================== -->
   <!-- TODO -->

File: pandora_robots_description/urdf/gears/config/gears_physics.gazebo.xacro (robot description, xacro)
@@ -7,5 +7,5 @@
     </gazebo>
   </xacro:macro>
-<!-- Links ################################################################ -->
+<!-- Links (SDF) ########################################################## -->
   <!-- ==================================================================== -->
   <xacro:macro name="base_link_sdf_physics" >

File: pandora_robots_description/urdf/gears/gazebo/plugins.gazebo.xacro (robot description, xacro)
@@ -1,5 +1,5 @@
 <?xml version="1.0"?>
 <robot xmlns:xacro="http://ros.org/wiki/xacro" >
-<!-- Differential Plugin ################################################## -->
+<!-- Differential ######################################################### -->
   <xacro:macro name="pandora_differential_plugin" >
     <!-- ================================================================== -->
@@ -28,5 +28,5 @@
     <!-- ================================================================== -->
   </xacro:macro>
-<!-- 3D Pose Plugin ####################################################### -->
+<!-- 3D Pose ############################################################## -->
   <xacro:macro name="pandora_p3d_plugin" >
     <!-- ================================================================== -->
@@ -43,5 +43,5 @@
     <!-- ================================================================== -->
   </xacro:macro>
-<!-- Imu Plugin ########################################################### -->
+<!-- Imu ################################################################## -->
   <xacro:macro name="ros_imu_plugin" >
     <!-- ================================================================== -->
@@ -49,12 +49,19 @@
       <plugin name="imu_en_ros"
               filename="libgazebo_ros_imu.so" >
+        <updateRate>50.0</updateRate>
+        <topicName>/sensors/imu</topicName>
+        <serviceName>default_imu</serviceName>
         <robotNamespace>${robot_namespace}</robotNamespace>
         <bodyName>${base_link_name}_link</bodyName>
-        <topicName>/sensors/imu</topicName>
+        <!-- <rollCorrectionJoint>laser_roll_joint</rollCorrectionJoint> -->
+        <!-- <pitchCorrectionJoint>laser_pitch_joint</pitchCorrectionJoint> -->
+        <gaussianNoise>0.0</gaussianNoise>
+        <xyzOffset>0 0 0</xyzOffset>
+        <rpyOffset>0 0 0</rpyOffset>
       </plugin>
     </gazebo>
     <!-- ================================================================== -->
   </xacro:macro>
-<!-- Ros Control Plugin ################################################### -->
+<!-- Ros Control ########################################################## -->
   <xacro:macro name="ros_control_plugin" >
     <!-- ================================================================== -->
@@ -68,5 +75,5 @@
     <!-- ================================================================== -->
   </xacro:macro>
-<!-- Skid Steer Drive Plugin ############################################## -->
+<!-- Skid Steer Drive ##################################################### -->
   <xacro:macro name="ros_skid_steer_drive_plugin" >
     <!-- ================================================================== -->

File: pandora_robots_description/urdf/gears/gazebo/transmission.xacro (robot description, xacro)
@@ -1,13 +1,13 @@
 <?xml version="1.0"?>
 <robot xmlns:xacro="http://ros.org/wiki/xacro" >
-<!-- Wheel Macro ########################################################## -->
+<!-- Wheel ################################################################ -->
   <xacro:macro name="wheel_transmission"
                params="prefix_y prefix_x" >
     <!-- ================================================================== -->
     <transmission name="${prefix_y}_${prefix_x}_${wheel_link_name}_transmission" >
+      <type>transmission_interface/SimpleTransmission</type>
       <joint name="${prefix_y}_${prefix_x}_${wheel_joint_name}_joint" />
-      <type>transmission_interface/SimpleTransmission</type>
       <actuator name="${prefix_y}_${prefix_x}_motor" >
-        <hardwareInterface>VelocityJointInterface</hardwareInterface>
+        <hardwareInterface>EffortJointInterface</hardwareInterface>
         <mechanicalReduction>1.0</mechanicalReduction>
       </actuator>
@@ -15,11 +15,11 @@
     <!-- ================================================================== -->
   </xacro:macro>
-<!-- Sensor Macro ######################################################### -->
+<!-- Sensor ############################################################### -->
   <xacro:macro name="sensor_transmission"
                params="sensor rotation" >
     <!-- ================================================================== -->
     <transmission name="${sensor}_${rotation}_transmission" >
+      <type>transmission_interface/SimpleTransmission</type>
       <joint name="${sensor}_${rotation}_joint" />
-      <type>transmission_interface/SimpleTransmission</type>
       <actuator name="${sensor}_${rotation}_motor" >
         <hardwareInterface>EffortJointInterface</hardwareInterface>

File: pandora_robots_description/urdf/gears/model/joints.urdf.xacro (robot description, xacro)
@@ -1,5 +1,5 @@
 <?xml version="1.0" ?>
 <robot xmlns:xacro="http://ros.org/wiki/xacro" >
-<!-- Side Macro ########################################################### -->
+<!-- Side ################################################################# -->
   <xacro:macro name="side_joint"
                params="prefix_y reflect_y" >
@@ -14,5 +14,5 @@
     <!-- ================================================================== -->
   </xacro:macro>
-<!-- Wheel Macro ########################################################## -->
+<!-- Wheel ################################################################ -->
   <xacro:macro name="wheel_joint"
                params="prefix_y prefix_x reflect_y reflect_x" >

File: pandora_robots_description/urdf/gears/model/links.urdf.xacro (robot description, xacro)
@@ -1,5 +1,5 @@
 <?xml version="1.0" ?>
 <robot xmlns:xacro="http://ros.org/wiki/xacro" >
-<!-- Base Macro ################################################################# -->
+<!-- Base ################################################################# -->
   <xacro:macro name="base_link" >
     <!-- ================================================================== -->
@@ -22,5 +22,5 @@
     <!-- ================================================================== -->
   </xacro:macro>
-<!-- Side Macro ########################################################### -->
+<!-- Side ################################################################# -->
   <xacro:macro name="side_link"
                params="prefix_y reflect_y" >
@@ -44,5 +44,5 @@
     <!-- ================================================================== -->
   </xacro:macro>
-<!-- Wheel Macro ########################################################## -->
+<!-- Wheel ################################################################ -->
   <xacro:macro name="wheel_link"
                params="prefix_y prefix_x reflect_y reflect_x" >

File: pandora_robots_description/urdf/pioneer3at/pioneer3at.urdf.xacro (robot description, xacro)
@@ -1,311 +1,383 @@
 <?xml version="1.0"?>
 <robot name="pioneer3at"
-       xacro="http://ros.org/wiki/xacro" >
-  <!-- Base Link -->
-  <link name="base_link">
+       xmlns:xacro="http://ros.org/wiki/xacro" >
+<!-- Links and Joints ##################################################### -->
+  <!-- Base =============================================================== -->
+  <link name="base_link" >
     <inertial>
-      <mass value="14.0"/>
-      <inertia ixx="0.3338" ixy="0" ixz="0"
-         iyy="0.4783" iyz="0"
-         izz="0.3338"/>
+      <mass value="14.0" />
+      <origin xyz="0 0 0"
+              rpy="0 0 0" />
+      <inertia ixx="0.3338"
+               ixy="0"
+               ixz="0"
+               iyy="0.4783"
+               iyz="0"
+               izz="0.3338" />
     </inertial>
-    <visual name="base_visual">
-      <origin xyz="0 0 0" rpy="0 0 0"/>
-      <geometry name="pioneer_geom">
-        <mesh filename="package://pandora_robots_description/meshes/pioneer3at/p3at_meshes/chassis.stl"/>
+    <visual>
+      <origin xyz="0 0 0"
+              rpy="0 0 0" />
+      <geometry>
+        <mesh filename="package://pandora_robots_description/meshes/pioneer3at/p3at_meshes/chassis.stl" />
       </geometry>
-      <material name="ChassisRed">
-        <color rgba="0.851 0.0 0.0 1.0"/>
+      <material name="ChassisRed" >
+        <color rgba="0.851 0.0 0.0 1.0" />
       </material>
     </visual>
     <collision>
-      <origin xyz="0 0 0" rpy="0 0 0"/>
-        <geometry>
-          <mesh filename="package://pandora_robots_description/meshes/pioneer3at/p3at_meshes/chassis.stl"/>
-        </geometry>
+      <origin xyz="0 0 0"
+              rpy="0 0 0" />
+      <geometry>
+        <mesh filename="package://pandora_robots_description/meshes/pioneer3at/p3at_meshes/chassis.stl" />
+      </geometry>
     </collision>
   </link>
-  <gazebo reference="base_link">
-    <material value="Gazebo/Red"/>
-  </gazebo>
-  <!-- Top -->
-  <link name="top_plate">
+  <gazebo reference="base_link" >
+    <material value="Gazebo/Red" />
+  </gazebo>
+  <!-- Top ================================================================ -->
+  <link name="top_plate" >
     <inertial>
-      <mass value="0.1"/>
-      <origin xyz="0 0 0" rpy="0 0 0"/>
-      <inertia ixx="0.001" ixy="0.0" ixz="0.0"
-         iyy="0.001" iyz="0.0"
-        izz="0.001"/>
+      <mass value="0.1" />
+      <origin xyz="0 0 0"
+              rpy="0 0 0" />
+      <inertia ixx="0.001"
+               ixy="0.0"
+               ixz="0.0"
+               iyy="0.001"
+               iyz="0.0"
+               izz="0.001" />
     </inertial>
-    <visual name="base_visual">
-      <origin xyz="0 0 0" rpy="0 0 0"/>
-      <geometry name="pioneer_geom">
-        <mesh filename="package://pandora_robots_description/meshes/pioneer3at/p3at_meshes/top.stl"/>
+    <visual>
+      <origin xyz="0 0 0"
+              rpy="0 0 0" />
+      <geometry>
+        <mesh filename="package://pandora_robots_description/meshes/pioneer3at/p3at_meshes/top.stl" />
       </geometry>
-      <material name="TopBlack">
-          <color rgba="0.038 0.038 0.038 1.0"/>
+      <material name="TopBlack" >
+          <color rgba="0.038 0.038 0.038 1.0" />
       </material>
     </visual>
     <collision>
-      <origin xyz="0 0 0" rpy="0 0 0"/>
+      <origin xyz="0 0 0"
+              rpy="0 0 0" />
       <geometry>
-        <box size="0 0 0"/>
+        <box size="0 0 0" />
       </geometry>
     </collision>
   </link>
-  <gazebo reference="top_plate">
-    <material value="Gazebo/Black"/>
-  </gazebo>
-  <joint name="base_top_joint" type="fixed">
-    <origin xyz="-0.025 0 0.096"/>
-    <parent link="base_link"/>
-    <child link="top_plate"/>
+  <gazebo reference="top_plate" >
+    <material value="Gazebo/Black" />
+  </gazebo>
+  <joint name="base_top_joint"
+         type="fixed" >
+    <parent link="base_link" />
+    <child link="top_plate" />
+    <origin xyz="-0.025 0 0.096" />
   </joint>
-  <!-- Front Axles + Wheels + Hubcaps -->
-  <xacro:macro name="p3at_front" params="suffix reflect">
-    <link name="p3at_front_${suffix}_axle">
-      <inertial>
-        <mass value="0.1"/>
-        <origin xyz="0 0 0"/>
-        <inertia ixx="0.001" ixy="0.0" ixz="0.0"
-           iyy="0.001" iyz="0.0" izz="0.001"/>
-        </inertial>
-    <visual name="base_visual">
-      <origin xyz="0 0 0" rpy="0 0 0"/>
-      <geometry name="pioneer_geom">
-        <mesh filename="package://pandora_robots_description/meshes/pioneer3at/p3at_meshes/axle.stl"/>
-      </geometry>
-      <material name="AxleGrey">
-        <color rgba="0.5 0.5 0.5 1"/>
-      </material>
-    </visual>
-    <collision>
-      <origin xyz="0 0 0" rpy="0 0 0"/>
-      <geometry>
-        <box size="0 0 0"/>
-      </geometry>
-    </collision>
-    </link>
-    <gazebo reference="p3at_front_${suffix}_axle">
-      <material value="Gazebo/Grey"/>
-    </gazebo>
-    <joint name="base_front_${suffix}_axle_joint" type="fixed">
-      <origin xyz="0.135 ${reflect*0.156} -0.066" rpy="0 0 0"/>
-      <parent link="base_link"/>
-      <child link="p3at_front_${suffix}_axle"/>
-    </joint>
-    <link name="p3at_front_${suffix}_hub">
-      <inertial>
-        <mass value="0.1"/>
-        <origin xyz="0 0 0"/>
-        <inertia ixx="0.001" ixy="0.0" ixz="0.0"
-           iyy="0.001" iyz="0.0" izz="0.001"/>
-      </inertial>
-      <visual name="base_visual">
-        <origin xyz="0 0 0" rpy="0 0 0"/>
-        <geometry name="pioneer_geom">
-          <mesh filename="package://pandora_robots_description/meshes/pioneer3at/p3at_meshes/${suffix}_hubcap.stl"/>
-        </geometry>
-        <material name="HubcapYellow">
-          <color rgba="1.0 0.811 0.151 1.0"/>
+  <!-- Front Axles + Wheels + Hubcaps ===================================== -->
+  <xacro:macro name="p3at_front"
+               params="suffix reflect" >
+    <link name="p3at_front_${suffix}_axle" >
+      <inertial>
+        <mass value="0.1" />
+        <origin xyz="0 0 0"
+                rpy="0 0 0" />
+        <inertia ixx="0.001"
+                 ixy="0.0"
+                 ixz="0.0"
+                 iyy="0.001"
+                 iyz="0.0"
+                 izz="0.001" />
+      </inertial>
+      <visual>
+        <origin xyz="0 0 0"
+                rpy="0 0 0" />
+        <geometry>
+          <mesh filename="package://pandora_robots_description/meshes/pioneer3at/p3at_meshes/axle.stl" />
+        </geometry>
+        <material name="AxleGrey" >
+          <color rgba="0.5 0.5 0.5 1" />
         </material>
       </visual>
       <collision>
-        <origin xyz="0 0 0" rpy="0 0 0"/>
-        <geometry>
-          <box size="0 0 0"/>
-        </geometry>
-      </collision>
-    </link>
-    <gazebo reference="p3at_front_${suffix}_hub">
-      <material value="Gazebo/Yellow"/>
-    </gazebo>
-    <joint name="base_front_${suffix}_hub_joint" type="fixed">
-      <origin xyz="0 ${reflect*0.041} 0" rpy="0 0 0"/>
-      <parent link="p3at_front_${suffix}_axle"/>
-      <child link="p3at_front_${suffix}_hub"/>
-    </joint>
-    <link name="p3at_front_${suffix}_wheel">
-      <inertial>
-        <mass value="0.5"/>
-        <origin xyz="0 0 0"/>
-        <inertia ixx="0.012411765597" ixy="0" ixz="0"
-           iyy="0.015218160428" iyz="0" izz="0.011763977943"/>
-      </inertial>
-      <visual name="base_visual">
-        <origin xyz="0 0 0" rpy="0 0 0"/>
-        <geometry name="pioneer_geom">
-          <mesh filename="package://pandora_robots_description/meshes/pioneer3at/p3at_meshes/wheel.stl"/>
-        </geometry>
-        <material name="WheelBlack">
-          <color rgba="0.117 0.117 0.117 1"/>
+        <origin xyz="0 0 0"
+                rpy="0 0 0" />
+        <geometry>
+          <box size="0 0 0" />
+        </geometry>
+      </collision>
+    </link>
+    <gazebo reference="p3at_front_${suffix}_axle" >
+      <material value="Gazebo/Grey" />
+    </gazebo>
+    <joint name="base_front_${suffix}_axle_joint"
+           type="fixed" >
+      <parent link="base_link" />
+      <child link="p3at_front_${suffix}_axle" />
+      <origin xyz="0.135 ${reflect*0.156} -0.066"
+              rpy="0 0 0" />
+    </joint>
+    <link name="p3at_front_${suffix}_hub" >
+      <inertial>
+        <mass value="0.1" />
+        <origin xyz="0 0 0"
+                rpy="0 0 0" />
+        <inertia ixx="0.001"
+                 ixy="0.0"
+                 ixz="0.0"
+                 iyy="0.001"
+                 iyz="0.0"
+                 izz="0.001" />
+      </inertial>
+      <visual>
+        <origin xyz="0 0 0"
+                rpy="0 0 0" />
+        <geometry>
+          <mesh filename="package://pandora_robots_description/meshes/pioneer3at/p3at_meshes/${suffix}_hubcap.stl" />
+        </geometry>
+        <material name="HubcapYellow" >
+          <color rgba="1.0 0.811 0.151 1.0" />
         </material>
       </visual>
       <collision>
-        <origin xyz="0 0 0" rpy="${-3.1415927/2} 0 0"/>
+        <origin xyz="0 0 0"
+                rpy="0 0 0" />
+        <geometry>
+          <box size="0 0 0" />
+        </geometry>
+      </collision>
+    </link>
+    <gazebo reference="p3at_front_${suffix}_hub" >
+      <material value="Gazebo/Yellow" />
+    </gazebo>
+    <joint name="base_front_${suffix}_hub_joint"
+           type="fixed" >
+      <parent link="p3at_front_${suffix}_axle" />
+      <child link="p3at_front_${suffix}_hub" />
+      <origin xyz="0 ${reflect*0.041} 0"
+              rpy="0 0 0" />
+    </joint>
+    <link name="p3at_front_${suffix}_wheel" >
+      <inertial>
+        <mass value="0.5" />
+        <origin xyz="0 0 0"
+                rpy="0 0 0" />
+        <inertia ixx="0.012411765597"
+                 ixy="0"
+                 ixz="0"
+                 iyy="0.015218160428"
+                 iyz="0"
+                 izz="0.011763977943" />
+      </inertial>
+      <visual>
+        <origin xyz="0 0 0"
+                rpy="0 0 0" />
+        <geometry>
+          <mesh filename="package://pandora_robots_description/meshes/pioneer3at/p3at_meshes/wheel.stl" />
+        </geometry>
+        <material name="WheelBlack" >
+          <color rgba="0.117 0.117 0.117 1" />
+        </material>
+      </visual>
+      <collision>
+        <origin xyz="0 0 0"
+                rpy="${-3.1415927/2} 0 0" />
         <geometry>
           <!--mesh filename="package://pandora_robots_description/meshes/pioneer3at/p3at_meshes/wheel.stl"/-->
-          <cylinder radius="0.111" length="0.075"/>
-        </geometry>
-      </collision>
-    </link>
-    <gazebo reference="p3at_front_${suffix}_wheel">
-      <material value="Gazebo/Black"/>
-    </gazebo>
-    <joint name="p3at_front_${suffix}_wheel_joint" type="continuous">
-      <axis xyz="0 1 0"/>
-      <anchor xyz="0 0 0"/>
-      <limit effort="100" velocity="100" />
-      <joint_properties damping="0.7"/>
-      <origin xyz="0 0 0" rpy="0 0 0"/>
-      <parent link="p3at_front_${suffix}_hub"/>
-      <child link="p3at_front_${suffix}_wheel"/>
-    </joint>
-    <!-- Back Axles + Wheels + Hubcaps -->
-    <link name="p3at_back_${suffix}_axle">
-      <inertial>
-        <mass value="0.1"/>
-        <origin xyz="0 0 0"/>
-        <inertia ixx="0.001" ixy="0.0" ixz="0.0"
-           iyy="0.001" iyz="0.0" izz="0.001"/>
-      </inertial>
-      <visual name="base_visual">
-        <origin xyz="0 0 0" rpy="0 0 0"/>
-        <geometry name="pioneer_geom">
-          <mesh filename="package://pandora_robots_description/meshes/pioneer3at/p3at_meshes/axle.stl"/>
-        </geometry>
-        <material name="AxleGrey">
-          <color rgba="0.5 0.5 0.5 1"/>
+          <cylinder radius="0.111"
+                    length="0.075" />
+        </geometry>
+      </collision>
+    </link>
+    <gazebo reference="p3at_front_${suffix}_wheel" >
+      <material value="Gazebo/Black" />
+    </gazebo>
+    <joint name="p3at_front_${suffix}_wheel_joint"
+           type="continuous" >
+      <parent link="p3at_front_${suffix}_hub" />
+      <child link="p3at_front_${suffix}_wheel" />
+      <origin xyz="0 0 0"
+              rpy="0 0 0" />
+      <axis xyz="0 1 0" />
+      <limit effort="100"
+             velocity="100" />
+      <joint_properties damping="0.7" />
+    </joint>
+    <!-- Back Axles + Wheels + Hubcaps ==================================== -->
+    <link name="p3at_back_${suffix}_axle" >
+      <inertial>
+        <mass value="0.1" />
+        <origin xyz="0 0 0"
+                rpy="0 0 0" />
+        <inertia ixx="0.001"
+                 ixy="0.0"
+                 ixz="0.0"
+                 iyy="0.001"
+                 iyz="0.0"
+                 izz="0.001" />
+      </inertial>
+      <visual>
+        <origin xyz="0 0 0"
+                rpy="0 0 0" />
+        <geometry>
+          <mesh filename="package://pandora_robots_description/meshes/pioneer3at/p3at_meshes/axle.stl" />
+        </geometry>
+        <material name="AxleGrey" >
+          <color rgba="0.5 0.5 0.5 1" />
         </material>
       </visual>
       <collision>
-        <origin xyz="0 0 0" rpy="0 0 0"/>
-        <geometry>
-          <mesh filename="package://pandora_robots_description/meshes/pioneer3at/p3at_meshes/axle.stl"/>
-        </geometry>
-      </collision>
-    </link>
-    <gazebo reference="p3at_back_${suffix}_axle">
-      <material value="Gazebo/Grey"/>
-    </gazebo>
-    <joint name="bp3at_back_${suffix}_axle_joint" type="fixed">
-      <origin xyz="-0.134 ${reflect*0.156} -0.066" rpy="0 0 0"/>
-      <parent link="base_link"/>
-      <child link="p3at_back_${suffix}_axle"/>
-    </joint>
-    <link name="p3at_back_${suffix}_hub">
-      <inertial>
-        <mass value="0.1"/>
-        <origin xyz="0 0 0"/>
-        <inertia ixx="0.001" ixy="0.0" ixz="0.0"
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