Commit message: Include gazebo controller launcher in robot launchers and add arg to enable ros_control.

File: pandora_robots_description/urdf/gears/config/gears_configurations.xacro (robot description, xacro)
@@ -1,5 +1,5 @@
 <?xml version="1.0"?>
 <robot xmlns:xacro="http://ros.org/wiki/xacro" >
-<!-- Elements Status ###################################################### -->
+<!-- Element Status ####################################################### -->
   <!-- Robot ============================================================== -->
   <xacro:property name="static_robot" value="false" />
@@ -22,9 +22,8 @@
     <xacro:property name="enable_microphone_sensor" value="false" />
   <!-- Transmission ======================================================= -->
-  <xacro:property name="enable_transmission" value="true" />
-    <xacro:property name="enable_sensor_transmission" value="false" />
-      <xacro:property name="enable_laser_sensor_transmission" value="true" />
-      <xacro:property name="enable_kinect_sensor_transmission" value="true" />
-    <xacro:property name="enable_wheel_transmission" value="true" />
+  <xacro:property name="enable_sensor_transmission" value="true" />
+    <xacro:property name="enable_laser_sensor_transmission" value="true" />
+    <xacro:property name="enable_kinect_sensor_transmission" value="true" />
+  <xacro:property name="enable_wheel_transmission" value="true" />
   <!-- Plugins ============================================================ -->
   <xacro:property name="enable_plugins" value="true" />

File: pandora_robots_description/urdf/gears/gears.urdf.xacro (robot description, xacro)
@@ -114,22 +114,32 @@
   </xacro:if>
 <!-- Load Transmissions ################################################### -->
-  <xacro:if value="${enable_transmission}" >
+  <xacro:if value="$(arg control)" >
     <!-- ================================================================== -->
-    <xacro:if value="${enable_wheel_transmission}" >
-      <xacro:wheel_transmission prefix_y="left" prefix_x="front" />
-      <xacro:wheel_transmission prefix_y="left" prefix_x="rear" />
-      <xacro:wheel_transmission prefix_y="right" prefix_x="front" />
-      <xacro:wheel_transmission prefix_y="right" prefix_x="rear" />
+    <xacro:if value="${enable_wheel_links}" >
+      <xacro:if value="${enable_wheel_transmission}" >
+        <xacro:wheel_transmission prefix_y="left" prefix_x="front" />
+        <xacro:wheel_transmission prefix_y="left" prefix_x="rear" />
+        <xacro:wheel_transmission prefix_y="right" prefix_x="front" />
+        <xacro:wheel_transmission prefix_y="right" prefix_x="rear" />
+      </xacro:if>
     </xacro:if>
     <!-- ================================================================== -->
-    <xacro:if value="${enable_sensor_transmission}" >
-      <xacro:if value="${enable_kinect_sensor_transmission}" >
-        <xacro:sensor_transmission sensor="kinect" rotation="pitch" />
-        <xacro:sensor_transmission sensor="kinect" rotation="yaw" />
-      </xacro:if>
-      <!-- ================================================================ -->
-      <xacro:if value="${enable_laser_sensor_transmission}" >
-        <xacro:sensor_transmission sensor="laser" rotation="roll" />
-        <xacro:sensor_transmission sensor="laser" rotation="pitch" />
+    <xacro:if value="${enable_sensors}" >
+      <xacro:if value="${enable_sensor_transmission}" >
+        <!-- ============================================================== -->
+        <xacro:if value="${enable_kinect_sensor}" >
+          <xacro:if value="${enable_kinect_sensor_transmission}" >
+            <xacro:sensor_transmission sensor="kinect" rotation="pitch" />
+            <xacro:sensor_transmission sensor="kinect" rotation="yaw" />
+          </xacro:if>
+        </xacro:if>
+        <!-- ============================================================== -->
+        <xacro:if value="${enable_hokuyo_laser_sensor}" >
+          <xacro:if value="${enable_laser_sensor_transmission}" >
+            <xacro:sensor_transmission sensor="laser" rotation="roll" />
+            <xacro:sensor_transmission sensor="laser" rotation="pitch" />
+          </xacro:if>
+        </xacro:if>
+        <!-- ============================================================== -->
       </xacro:if>
     </xacro:if>

File: pandora_robots_description/urdf/pioneer3at/pioneer3at.urdf.xacro (robot description, xacro)
@@ -348,20 +348,22 @@
     </gazebo>
     <!-- Wheel Transmission =============================================== -->
-    <transmission name="p3at_front_${suffix}_wheel_transmission" >
-      <type>transmission_interface/SimpleTransmission</type>
-      <joint name="p3at_front_${suffix}_wheel_joint" />
-      <actuator name="p3at_front_${suffix}_motor" >
-        <hardwareInterface>EffortJointInterface</hardwareInterface>
-        <mechanicalReduction>1</mechanicalReduction>
-      </actuator>
-    </transmission>
-    <transmission name="p3at_back_${suffix}_wheel_transmission" >
-      <type>transmission_interface/SimpleTransmission</type>
-      <joint name="p3at_back_${suffix}_wheel_joint" />
-      <actuator name="p3at_back_${suffix}_motor" >
-        <hardwareInterface>EffortJointInterface</hardwareInterface>
-        <mechanicalReduction>1</mechanicalReduction>
-      </actuator>
-    </transmission>
+    <xacro:if value="$(arg control)" >
+      <transmission name="p3at_front_${suffix}_wheel_transmission" >
+        <type>transmission_interface/SimpleTransmission</type>
+        <joint name="p3at_front_${suffix}_wheel_joint" />
+        <actuator name="p3at_front_${suffix}_motor" >
+          <hardwareInterface>EffortJointInterface</hardwareInterface>
+          <mechanicalReduction>1</mechanicalReduction>
+        </actuator>
+      </transmission>
+      <transmission name="p3at_back_${suffix}_wheel_transmission" >
+        <type>transmission_interface/SimpleTransmission</type>
+        <joint name="p3at_back_${suffix}_wheel_joint" />
+        <actuator name="p3at_back_${suffix}_motor" >
+          <hardwareInterface>EffortJointInterface</hardwareInterface>
+          <mechanicalReduction>1</mechanicalReduction>
+        </actuator>
+      </transmission>
+    </xacro:if>
   </xacro:macro>
   <!-- Add Wheels ========================================================= -->
@@ -440,6 +442,8 @@
     <origin xyz="0.2 0 0.33" rpy="0 0 0" />
   </xacro:kinect_caster>
-  <xacro:sensor_transmission sensor="kinect" rotation="pitch" />
-  <xacro:sensor_transmission sensor="kinect" rotation="yaw" />
+  <xacro:if value="$(arg control)" >
+    <xacro:sensor_transmission sensor="kinect" rotation="pitch" />
+    <xacro:sensor_transmission sensor="kinect" rotation="yaw" />
+  </xacro:if>
   <!-- Hokuyo Laser ======================================================= -->
   <xacro:include filename="$(find pandora_sensors_description)/urdf/hokuyo_utm_30lx.urdf.xacro" />
@@ -447,6 +451,8 @@
     <origin xyz="0.25 0 0.15" rpy="0 0 0" />
   </xacro:hokuyo_caster>
-  <xacro:sensor_transmission sensor="laser" rotation="roll" />
-  <xacro:sensor_transmission sensor="laser" rotation="pitch" />
+  <xacro:if value="$(arg control)" >
+    <xacro:sensor_transmission sensor="laser" rotation="roll" />
+    <xacro:sensor_transmission sensor="laser" rotation="pitch" />
+  </xacro:if>
   <!-- Sonars ============================================================= -->
   <xacro:include filename="$(find pandora_sensors_description)/urdf/sonar_sensor.urdf.xacro" />

Commit message: Fix gears wheel joint limits and change side link gazebo color.

File: pandora_robots_description/urdf/gears/config/gears_configurations.xacro (robot description, xacro)
@@ -14,5 +14,5 @@
     <xacro:property name="enable_wheel_joints" value="true" />
   <!-- Sensors ============================================================ -->
-  <xacro:property name="enable_sensors" value="false" />
+  <xacro:property name="enable_sensors" value="true" />
     <xacro:property name="enable_kinect_sensor" value="true" />
     <xacro:property name="enable_hokuyo_laser_sensor" value="true" />

File: pandora_robots_description/urdf/gears/config/gears_physics.gazebo.xacro (robot description, xacro)
@@ -30,5 +30,5 @@
                params="prefix_y" >
     <gazebo reference="${prefix_y}_${side_link_name}_link" >
-      <material>Gazebo/White</material>
+      <material>Gazebo/FlatBlack</material>
       <!-- <gravity>false</gravity> -->
       <!-- <dampingFactor>0.0</dampingFactor> -->
@@ -119,6 +119,6 @@
     <!-- <dynamics damping="0.0"
                    friction="0.0" /> -->
-    <limit effort="100.0"
-           velocity="100.0" />
+    <limit effort="50.0"
+           velocity="50.0" />
       <!-- lower="-0.0" -->
       <!-- upper="0.0" -->

Commit message: Add pandora imu stabilizer plugin to available plugins, modify ros control plugin's namespace and modify gears' config.

File: pandora_robots_description/urdf/gears/config/gears_configurations.xacro (robot description, xacro)
@@ -31,4 +31,5 @@
     <xacro:property name="enable_pandora_p3d_plugin" value="false" />
     <xacro:property name="enable_ros_imu_plugin" value="false" />
+    <xacro:property name="enable_pandora_imu_stabilizer_plugin" value="false" />
     <xacro:property name="enable_ros_control_plugin" value="true" />
     <xacro:property name="enable_ros_skid_steer_drive_plugin" value="true" />

File: pandora_robots_description/urdf/gears/gazebo/plugins.gazebo.xacro (robot description, xacro)
@@ -43,9 +43,9 @@
     <!-- ================================================================== -->
   </xacro:macro>
-<!-- Imu ################################################################## -->
+<!-- Ros Imu ############################################################## -->
   <xacro:macro name="ros_imu_plugin" >
     <!-- ================================================================== -->
     <gazebo>
-      <plugin name="imu_en_ros"
+      <plugin name="RosImuPlugin"
               filename="libgazebo_ros_imu.so" >
         <updateRate>50.0</updateRate>
@@ -54,6 +54,24 @@
         <robotNamespace>${robot_namespace}</robotNamespace>
         <bodyName>${base_link_name}_link</bodyName>
-        <!-- <rollCorrectionJoint>laser_roll_joint</rollCorrectionJoint> -->
-        <!-- <pitchCorrectionJoint>laser_pitch_joint</pitchCorrectionJoint> -->
+        <gaussianNoise>0.0</gaussianNoise>
+        <xyzOffset>0 0 0</xyzOffset>
+        <rpyOffset>0 0 0</rpyOffset>
+      </plugin>
+    </gazebo>
+    <!-- ================================================================== -->
+  </xacro:macro>
+<!-- Pandora Imu ########################################################## -->
+  <xacro:macro name="pandora_imu_stabilizer_plugin" >
+    <!-- ================================================================== -->
+    <gazebo>
+      <plugin name="PandoraImuStabilizerPlugin"
+              filename="libpandora_imu_stabilizer_plugin.so" >
+        <updateRate>50.0</updateRate>
+        <topicName>/sensors/imu</topicName>
+        <serviceName>default_imu</serviceName>
+        <robotNamespace>${robot_namespace}</robotNamespace>
+        <bodyName>${base_link_name}_link</bodyName>
+        <rollCorrectionJoint>laser_roll_joint</rollCorrectionJoint>
+        <pitchCorrectionJoint>laser_pitch_joint</pitchCorrectionJoint>
         <gaussianNoise>0.0</gaussianNoise>
         <xyzOffset>0 0 0</xyzOffset>
@@ -64,10 +82,11 @@
   </xacro:macro>
 <!-- Ros Control ########################################################## -->
-  <xacro:macro name="ros_control_plugin" >
+  <xacro:macro name="gazebo_ros_control_plugin" >
     <!-- ================================================================== -->
     <gazebo>
-      <plugin name="gazebo_ros_control"
+      <plugin name="GazeboRosControl"
               filename="libgazebo_ros_control.so" >
-      <robotNamespace>${robot_namespace}</robotNamespace>
+      <!-- <robotNamespace>${robot_namespace}</robotNamespace> -->
+      <robotNamespace>gears</robotNamespace>
       <robotSimType>gazebo_ros_control/DefaultRobotHWSim</robotSimType>
       </plugin>

File: pandora_robots_description/urdf/gears/gears.urdf.xacro (robot description, xacro)
@@ -158,10 +158,18 @@
     <!-- ================================================================== -->
     <xacro:if value="${enable_ros_imu_plugin}" >
-      <xacro:ros_imu_plugin />
+      <xacro:unless value="${enable_pandora_imu_stabilizer_plugin}" >
+        <xacro:ros_imu_plugin />
+      </xacro:unless>
+    </xacro:if>
+    <!-- ================================================================== -->
+    <xacro:if value="${enable_pandora_imu_stabilizer_plugin}" >
+      <xacro:unless value="${enable_ros_imu_plugin}" >
+        <xacro:pandora_imu_stabilizer_plugin />
+      </xacro:unless>
     </xacro:if>
     <!-- ================================================================== -->
     <xacro:if value="$(arg control)" >
       <xacro:if value="${enable_ros_control_plugin}" >
-        <xacro:ros_control_plugin />
+        <xacro:gazebo_ros_control_plugin />
       </xacro:if>
     </xacro:if>

File: pandora_robots_description/urdf/pioneer3at/pioneer3at.urdf.xacro (robot description, xacro)
@@ -419,6 +419,4 @@
       <robotNamespace></robotNamespace>
       <bodyName>base_link</bodyName>
-      <!-- <rollCorrectionJoint>laser_roll_joint</rollCorrectionJoint> -->
-      <!-- <pitchCorrectionJoint>laser_pitch_joint</pitchCorrectionJoint> -->
       <gaussianNoise>0.0</gaussianNoise>
       <xyzOffset>0 0 0</xyzOffset>

Commit message: Fix kinect joint types when ros control is not enabled.

File: pandora_robots_description/urdf/gears/config/gears_configurations.xacro (robot description, xacro)
@@ -21,9 +21,4 @@
     <xacro:property name="enable_co2_sensor" value="false" />
     <xacro:property name="enable_microphone_sensor" value="false" />
-  <!-- Transmission ======================================================= -->
-  <xacro:property name="enable_sensor_transmission" value="true" />
-    <xacro:property name="enable_laser_sensor_transmission" value="true" />
-    <xacro:property name="enable_kinect_sensor_transmission" value="true" />
-  <xacro:property name="enable_wheel_transmission" value="true" />
   <!-- Plugins ============================================================ -->
   <xacro:property name="enable_plugins" value="true" />
@@ -31,7 +26,4 @@
     <xacro:property name="enable_pandora_p3d_plugin" value="false" />
     <xacro:property name="enable_ros_imu_plugin" value="false" />
-    <xacro:property name="enable_pandora_imu_stabilizer_plugin" value="false" />
-    <xacro:property name="enable_ros_control_plugin" value="true" />
-    <xacro:property name="enable_ros_skid_steer_drive_plugin" value="true" />
   <!-- SDF Physics ======================================================== -->
   <xacro:property name="enable_sdf_physics" value="true" />

File: pandora_robots_description/urdf/gears/gazebo/sensors.xacro (robot description, xacro)
@@ -16,7 +16,8 @@
   <!-- ==================================================================== -->
 <!-- Kinect ############################################################### -->
-  <xacro:macro name="kinect_sensor" >
+  <xacro:macro name="kinect_sensor"
+               params="control" >
     <!-- ================================================================== -->
-    <xacro:kinect_caster parent="${base_link_name}_link" >
+    <xacro:kinect_caster parent="${base_link_name}_link" control="${control}" >
       <origin xyz="0.156 0.0 0.526"
               rpy="${zero}" />

File: pandora_robots_description/urdf/gears/gears.urdf.xacro (robot description, xacro)
@@ -88,5 +88,5 @@
     <!-- ================================================================== -->
     <xacro:if value="${enable_kinect_sensor}" >
-      <xacro:kinect_sensor />
+      <xacro:kinect_sensor control="$(arg control)" />
     </xacro:if>
     <!-- ================================================================== -->
@@ -117,30 +117,22 @@
     <!-- ================================================================== -->
     <xacro:if value="${enable_wheel_links}" >
-      <xacro:if value="${enable_wheel_transmission}" >
-        <xacro:wheel_transmission prefix_y="left" prefix_x="front" />
-        <xacro:wheel_transmission prefix_y="left" prefix_x="rear" />
-        <xacro:wheel_transmission prefix_y="right" prefix_x="front" />
-        <xacro:wheel_transmission prefix_y="right" prefix_x="rear" />
-      </xacro:if>
+      <xacro:wheel_transmission prefix_y="left" prefix_x="front" />
+      <xacro:wheel_transmission prefix_y="left" prefix_x="rear" />
+      <xacro:wheel_transmission prefix_y="right" prefix_x="front" />
+      <xacro:wheel_transmission prefix_y="right" prefix_x="rear" />
     </xacro:if>
     <!-- ================================================================== -->
     <xacro:if value="${enable_sensors}" >
-      <xacro:if value="${enable_sensor_transmission}" >
-        <!-- ============================================================== -->
-        <xacro:if value="${enable_kinect_sensor}" >
-          <xacro:if value="${enable_kinect_sensor_transmission}" >
-            <xacro:sensor_transmission sensor="kinect" rotation="pitch" />
-            <xacro:sensor_transmission sensor="kinect" rotation="yaw" />
-          </xacro:if>
-        </xacro:if>
-        <!-- ============================================================== -->
-        <xacro:if value="${enable_hokuyo_laser_sensor}" >
-          <xacro:if value="${enable_laser_sensor_transmission}" >
-            <xacro:sensor_transmission sensor="laser" rotation="roll" />
-            <xacro:sensor_transmission sensor="laser" rotation="pitch" />
-          </xacro:if>
-        </xacro:if>
-        <!-- ============================================================== -->
+      <!-- ================================================================ -->
+      <xacro:if value="${enable_kinect_sensor}" >
+        <xacro:sensor_transmission sensor="kinect" rotation="pitch" />
+        <xacro:sensor_transmission sensor="kinect" rotation="yaw" />
       </xacro:if>
+      <!-- ================================================================ -->
+      <xacro:if value="${enable_hokuyo_laser_sensor}" >
+        <xacro:sensor_transmission sensor="laser" rotation="roll" />
+        <xacro:sensor_transmission sensor="laser" rotation="pitch" />
+      </xacro:if>
+      <!-- ================================================================ -->
     </xacro:if>
     <!-- ================================================================== -->
@@ -157,25 +149,25 @@
     </xacro:if>
     <!-- ================================================================== -->
-    <xacro:if value="${enable_ros_imu_plugin}" >
-      <xacro:unless value="${enable_pandora_imu_stabilizer_plugin}" >
-        <xacro:ros_imu_plugin />
-      </xacro:unless>
-    </xacro:if>
-    <!-- ================================================================== -->
-    <xacro:if value="${enable_pandora_imu_stabilizer_plugin}" >
-      <xacro:unless value="${enable_ros_imu_plugin}" >
-        <xacro:pandora_imu_stabilizer_plugin />
-      </xacro:unless>
+    <xacro:if value="$(arg control)" >
+      <xacro:gazebo_ros_control_plugin />
     </xacro:if>
     <!-- ================================================================== -->
     <xacro:if value="$(arg control)" >
-      <xacro:if value="${enable_ros_control_plugin}" >
-        <xacro:gazebo_ros_control_plugin />
+      <xacro:if value="${enable_ros_imu_plugin}" >
+        <xacro:ros_imu_plugin />
       </xacro:if>
     </xacro:if>
     <!-- ================================================================== -->
-    <xacro:if value="${enable_ros_skid_steer_drive_plugin}" >
+    <xacro:if value="${enable_sensors}" >
+      <xacro:if value="${enable_hokuyo_laser_sensor}" >
+        <xacro:unless value="$(arg control)" >
+          <xacro:pandora_imu_stabilizer_plugin />
+        </xacro:unless>
+      </xacro:if>
+    </xacro:if>
+    <!-- ================================================================== -->
+    <xacro:unless value="$(arg control)" >
       <xacro:ros_skid_steer_drive_plugin />
-    </xacro:if>
+    </xacro:unless>
   <!-- ==================================================================== -->
   </xacro:if>

File: pandora_sensors_description/urdf/kinect_camera.urdf.xacro (robot description, xacro)
@@ -2,5 +2,5 @@
 <robot xmlns:xacro="http://ros.org/wiki/xacro" >
   <xacro:macro name="kinect_caster"
-               params="parent *origin" >
+               params="parent control *origin" >
     <link name="kinect_link" >
       <inertial>
@@ -110,27 +110,48 @@
       </collision>
     </link>
-    <joint name="kinect_pitch_joint"
-           type="revolute" >
-      <parent link="${parent}" />
-      <child link="kinect_base_link" />
-      <xacro:insert_block name="origin" />
-      <axis xyz="0 1 0" />
-      <limit lower="-1.57"
-             upper="1.57"
-             effort="300"
-             velocity="100.0" />
-    </joint>
-    <joint name="kinect_yaw_joint"
-           type="revolute" >
-      <parent link="kinect_base_link" />
-      <child link="kinect_link" />
-      <origin xyz="0 0 0"
-              rpy="0 0 0" />
-      <axis xyz="0 0 1" />
-      <limit lower="-1.57"
-             upper="1.57"
-             effort="300"
-             velocity="100.0" />
-    </joint>
+    <xacro:if value="${control}" >
+      <joint name="kinect_pitch_joint"
+             type="revolute" >
+        <parent link="${parent}" />
+        <child link="kinect_base_link" />
+        <xacro:insert_block name="origin" />
+        <axis xyz="0 1 0" />
+        <limit lower="-1.57"
+               upper="1.57"
+               effort="300"
+               velocity="100.0" />
+      </joint>
+    </xacro:if>
+    <xacro:unless value="${control}" >
+      <joint name="kinect_pitch_joint"
+             type="fixed" >
+        <parent link="${parent}" />
+        <child link="kinect_base_link" />
+        <xacro:insert_block name="origin" />
+      </joint>
+    </xacro:unless>
+    <xacro:if value="${control}" >
+      <joint name="kinect_yaw_joint"
+             type="revolute" >
+        <parent link="kinect_base_link" />
+        <child link="kinect_link" />
+        <origin xyz="0 0 0"
+                rpy="0 0 0" />
+        <axis xyz="0 0 1" />
+        <limit lower="-1.57"
+               upper="1.57"
+               effort="300"
+               velocity="100.0" />
+      </joint>
+    </xacro:if>
+    <xacro:unless value="${control}" >
+      <joint name="kinect_yaw_joint"
+             type="fixed" >
+        <parent link="kinect_base_link" />
+        <child link="kinect_link" />
+        <origin xyz="0 0 0"
+                rpy="0 0 0" />
+      </joint>
+    </xacro:unless>
   </xacro:macro>
 </robot>
