Commit message: Add arg for ros control hardware interface.

File: pandora_robots_description/urdf/gears/config/gears_configurations.xacro (robot description, xacro)
@@ -26,4 +26,5 @@
     <xacro:property name="enable_pandora_p3d_plugin" value="false" />
     <xacro:property name="enable_ros_imu_plugin" value="false" />
+    <xacro:property name="enable_pandora_imu_stabilizer_plugin" value="true" />
   <!-- SDF Physics ======================================================== -->
   <xacro:property name="enable_sdf_physics" value="true" />

File: pandora_robots_description/urdf/gears/gazebo/plugins.gazebo.xacro (robot description, xacro)
@@ -82,5 +82,6 @@
   </xacro:macro>
 <!-- Ros Control ########################################################## -->
-  <xacro:macro name="gazebo_ros_control_plugin" >
+  <xacro:macro name="gazebo_ros_control_plugin"
+               params="hw_sim" >
     <!-- ================================================================== -->
     <gazebo>
@@ -89,5 +90,5 @@
       <!-- <robotNamespace>${robot_namespace}</robotNamespace> -->
       <robotNamespace>control</robotNamespace>
-      <robotSimType>pandora_gazebo_interface/GazeboInterface</robotSimType>
+      <robotSimType>${hw_sim}</robotSimType>
       </plugin>
     </gazebo>

File: pandora_robots_description/urdf/gears/gears.urdf.xacro (robot description, xacro)
@@ -150,5 +150,10 @@
     <!-- ================================================================== -->
     <xacro:if value="$(arg control)" >
-      <xacro:gazebo_ros_control_plugin />
+      <xacro:if value="$(arg hw_interface)" >
+        <xacro:gazebo_ros_control_plugin hw_sim="pandora_gazebo_interface/GazeboInterface" />
+      </xacro:if>
+      <xacro:unless value="$(arg hw_interface)" >
+        <xacro:gazebo_ros_control_plugin hw_sim="DefaultRobotHWSim" />
+      </xacro:unless>
     </xacro:if>
     <!-- ================================================================== -->
@@ -162,5 +167,7 @@
       <xacro:if value="${enable_hokuyo_laser_sensor}" >
         <xacro:unless value="$(arg control)" >
-          <xacro:pandora_imu_stabilizer_plugin />
+          <xacro:if value="${enable_pandora_imu_stabilizer_plugin}" >
+            <xacro:pandora_imu_stabilizer_plugin />
+          </xacro:if>
         </xacro:unless>
       </xacro:if>
