Commit message: Add linear elevator.

File: pandora_robots_description/urdf/gears/config/gears_configurations.xacro (robot description, xacro)
@@ -7,8 +7,10 @@
   <xacro:property name="enable_links" value="true" />
     <xacro:property name="enable_base_link" value="true" />
+    <xacro:property name="enable_linear_elevator_link" value="true" />
     <xacro:property name="enable_side_links" value="true" />
     <xacro:property name="enable_wheel_links" value="true" />
   <!-- Joints ============================================================= -->
   <xacro:property name="enable_joints" value="true" />
+    <xacro:property name="enable_linear_elevator_joint" value="true" />
     <xacro:property name="enable_side_joints" value="true" />
     <xacro:property name="enable_wheel_joints" value="true" />
@@ -30,6 +32,8 @@
   <xacro:property name="enable_sdf_physics" value="true" />
     <xacro:property name="enable_base_link_sdf_physics" value="false" />
+    <xacro:property name="enable_linear_elevator_link_sdf_physics" value="false" />
     <xacro:property name="enable_side_link_sdf_physics" value="false" />
     <xacro:property name="enable_wheel_link_sdf_physics" value="true" />
+    <xacro:property name="enable_linear_elevator_joint_sdf_physics" value="false" />
     <xacro:property name="enable_side_joint_sdf_physics" value="false" />
     <xacro:property name="enable_wheel_joint_sdf_physics" value="false" />
@@ -37,4 +41,5 @@
   <!-- TODO -->
   <xacro:property name="enable_simlified_visual_base_link_mesh" value="false" />
+  <xacro:property name="enable_simlified_visual_linear_elevator_link_mesh" value="false" />
   <xacro:property name="enable_simlified_visual_side_link_mesh" value="false" />
   <xacro:property name="enable_simlified_visual_wheel_link_mesh" value="false" />
@@ -44,4 +49,5 @@
   <xacro:property name="side_joint_type" value="revolute" />
   <xacro:property name="wheel_joint_type" value="continuous" />
+  <xacro:property name="linear_elevator_joint_type" value="prismatic" />
   <!-- ==================================================================== -->
 <!-- Gears Coefficients ################################################### -->
@@ -53,5 +59,6 @@
   <xacro:property name="wheel_min_depth" value="0.001" />
   <!-- ==================================================================== -->
-  <xacro:property name="side_joint_max_angle" value="0.785" />
+  <xacro:property name="linear_elevator_joint_max_limit" value="0.2" />
+  <xacro:property name="side_joint_max_limit" value="0.785" />
   <xacro:property name="side_joint_damping" value="0.0" />
   <!-- ==================================================================== -->

File: pandora_robots_description/urdf/gears/config/gears_physics.gazebo.xacro (robot description, xacro)
@@ -11,4 +11,22 @@
   <xacro:macro name="base_link_sdf_physics" >
     <gazebo reference="${base_link_name}_link" >
+      <!-- <material>Gazebo/Grey</material> -->
+      <!-- <gravity>false</gravity> -->
+      <!-- <dampingFactor>0.0</dampingFactor> -->
+      <!-- <maxVel>0.0</maxVel> -->
+      <!-- <minDepth>0.0</minDepth> -->
+      <!-- <mu1>0.0</mu1> -->
+      <!-- <mu2>0.0</mu2> -->
+      <!-- <fdir1>0 0 0</fdir1> -->
+      <!-- <kp>0.0</kp> -->
+      <!-- <kd>0.0</kd> -->
+      <!-- <selfCollide>false</selfCollide> -->
+      <!-- <maxContacts>1</maxContacts> -->
+      <!-- <laserRetro>0.0</laserRetro> -->
+    </gazebo>
+  </xacro:macro>
+  <!-- ==================================================================== -->
+  <xacro:macro name="linear_elevator_link_sdf_physics" >
+    <gazebo reference="${linear_elevator_link_name}_link" >
       <!-- <material>Gazebo/Grey</material> -->
       <!-- <gravity>false</gravity> -->
@@ -67,4 +85,17 @@
 <!-- Joints (SDF) ######################################################### -->
   <!-- ==================================================================== -->
+  <xacro:macro name="linear_elevator_joint_sdf_physics" >
+    <gazebo reference="${linear_elevator_name}_joint" >
+      <!-- <kp>0.0</kp> -->
+      <!-- <kd>0.0</kd> -->
+      <!-- <stopCfm>0.0</stopCfm> -->
+      <!-- <stopErp>0.0</stopErp> -->
+      <!-- <provideFeedback>false</provideFeedback> -->
+      <!-- <cfmDamping>true</cfmDamping> -->
+      <implicitSpringDamper>true</implicitSpringDamper>
+      <!-- <fudgeFactor>0.0</fudgeFactor> -->
+    </gazebo>
+  </xacro:macro>
+  <!-- ==================================================================== -->
   <xacro:macro name="side_joint_sdf_physics"
                params="prefix_y" >
@@ -97,4 +128,20 @@
 <!-- Joints (URDF) ######################################################## -->
   <!-- ==================================================================== -->
+  <xacro:macro name="linear_elevator_joint_urdf_physics" >
+    <axis xyz="0 0 1" />
+    <!-- <calibration rising="0.0"
+                      falling="0.0" /> -->
+    <dynamics damping="0.0" />
+         <!-- friction="0.0" /> -->
+    <limit lower="-${linear_elevator_joint_max_limit}"
+           upper="${linear_elevator_joint_max_limit}"
+           effort="100.0"
+           velocity="100.0" />
+    <!-- <safety_controller soft_lower_limit="0.0"
+                            soft_upper_limit="0.0"
+                            k_position="0.0"
+                            k_velocity="0.0" /> -->
+  </xacro:macro>
+  <!-- ==================================================================== -->
   <xacro:macro name="side_joint_urdf_physics" >
     <axis xyz="0 1 0" />
@@ -103,6 +150,6 @@
     <dynamics damping="${side_joint_damping}" />
          <!-- friction="0.0" /> -->
-    <limit lower="-${side_joint_max_angle}"
-           upper="${side_joint_max_angle}"
+    <limit lower="-${side_joint_max_limit}"
+           upper="${side_joint_max_limit}"
            effort="100.0"
            velocity="100.0" />

File: pandora_robots_description/urdf/gears/config/properties/inertia_tensors.xacro (robot description, xacro)
@@ -9,4 +9,13 @@
              iyz="0.022113"
              izz="0.126610" />
+  </xacro:macro>
+  <!-- ==================================================================== -->
+  <xacro:macro name="linear_elevator_link_inertia" >
+    <inertia ixx="0.001"
+             ixy="0.001"
+             ixz="0.001"
+             iyy="0.001"
+             iyz="0.001"
+             izz="0.001" />
   </xacro:macro>
   <!-- ==================================================================== -->

File: pandora_robots_description/urdf/gears/config/properties/joint_offsets.xacro (robot description, xacro)
@@ -1,4 +1,9 @@
 <?xml version="1.0"?>
 <robot xmlns:xacro="http://ros.org/wiki/xacro" >
+  <!-- ==================================================================== -->
+  <xacro:macro name="linear_elevator_joint_origin" >
+    <origin xyz="0.0 0.3 0.5"
+            rpy="${zero}" />
+  </xacro:macro>
   <!-- ==================================================================== -->
   <xacro:macro name="side_joint_origin"

File: pandora_robots_description/urdf/gears/config/properties/link_offsets.xacro (robot description, xacro)
@@ -6,4 +6,8 @@
     <origin xyz="-1.1543E-07 -1.3195E-07 0.23164"
             rpy="${zero}" />
+  </xacro:macro>
+  <!-- ==================================================================== -->
+  <xacro:macro name="linear_elevator_link_inertial_origin" >
+    <xacro:default_origin />
   </xacro:macro>
   <!-- ==================================================================== -->
@@ -23,4 +27,8 @@
   <!-- ==================================================================== -->
   <xacro:macro name="base_link_visual_origin" >
+    <xacro:default_origin />
+  </xacro:macro>
+  <!-- ==================================================================== -->
+  <xacro:macro name="linear_elevator_link_visual_origin" >
     <xacro:default_origin />
   </xacro:macro>
@@ -44,4 +52,8 @@
   </xacro:macro>
   <!-- ==================================================================== -->
+  <xacro:macro name="linear_elevator_link_collision_origin" >
+    <xacro:default_origin />
+  </xacro:macro>
+  <!-- ==================================================================== -->
   <xacro:macro name="side_link_collision_origin"
                params="reflect_y" >

File: pandora_robots_description/urdf/gears/config/properties/masses.xacro (robot description, xacro)
@@ -4,4 +4,8 @@
   <xacro:macro name="base_link_mass" >
     <mass value="9.3044" />
+  </xacro:macro>
+  <!-- ==================================================================== -->
+  <xacro:macro name="linear_elevator_link_mass" >
+    <mass value="0.001" />
   </xacro:macro>
   <!-- ==================================================================== -->

File: pandora_robots_description/urdf/gears/config/properties/materials.xacro (robot description, xacro)
@@ -112,4 +112,8 @@
   </material>
   <!-- ==================================================================== -->
+  <material name="linear_elevator" >
+    <color rgba="${190/255} ${190/255} ${190/255} 1.0" />
+  </material>
+  <!-- ==================================================================== -->
   <material name="side" >
     <color rgba="${190/255} ${190/255} ${190/255} 1.0" />

File: pandora_robots_description/urdf/gears/config/properties/meshes.xacro (robot description, xacro)
@@ -7,4 +7,11 @@
       <mesh filename="package://pandora_robots_description/meshes/gears/visual/base_link.dae" />
       <!-- <mesh filename="package://pandora_robots_description/meshes/gears/collision/base_link.stl" /> -->
+    </geometry>
+  </xacro:macro>
+  <!-- ==================================================================== -->
+  <xacro:macro name="linear_elevator_link_visual_mesh" >
+    <geometry>
+      <mesh filename="package://pandora_robots_description/meshes/gears/visual/linear_elevator_link.dae" />
+      <!-- <mesh filename="package://pandora_robots_description/meshes/gears/collision/linear_elevator_link.stl" /> -->
     </geometry>
   </xacro:macro>
@@ -33,4 +40,11 @@
   </xacro:macro>
   <!-- ==================================================================== -->
+  <xacro:macro name="linear_elevator_link_collision_mesh" >
+    <geometry>
+      <mesh filename="package://pandora_robots_description/meshes/gears/collision/linear_elevator_link.stl" />
+      <!-- <mesh filename="package://pandora_robots_description/meshes/gears/visual/linear_elevator_link.dae" /> -->
+    </geometry>
+  </xacro:macro>
+  <!-- ==================================================================== -->
   <xacro:macro name="side_link_collision_mesh" >
     <geometry>

File: pandora_robots_description/urdf/gears/config/properties/names.xacro (robot description, xacro)
@@ -9,4 +9,6 @@
   <xacro:property name="base_link_name" value="base" />
   <!-- ==================================================================== -->
+  <xacro:property name="linear_elevator_link_name" value="linear_elevator" />
+  <!-- ==================================================================== -->
   <xacro:property name="side_link_name" value="side" />
   <!-- ==================================================================== -->
@@ -15,10 +17,10 @@
 <!-- Joints ############################################################### -->
   <!-- ==================================================================== -->
+  <xacro:property name="linear_elevator_joint_name" value="linear_elevator" />
+  <!-- ==================================================================== -->
   <xacro:property name="side_joint_name" value="side" />
   <!-- ==================================================================== -->
   <xacro:property name="wheel_joint_name" value="wheel" />
   <!-- ==================================================================== -->
-  <xacro:property name="name" value="value" />
-  <!-- ==================================================================== -->
 <!-- ###################################################################### -->
 </robot>

File: pandora_robots_description/urdf/gears/gazebo/transmission.xacro (robot description, xacro)
@@ -1,4 +1,17 @@
 <?xml version="1.0"?>
 <robot xmlns:xacro="http://ros.org/wiki/xacro" >
+<!-- Linear Elevator ###################################################### -->
+  <xacro:macro name="linear_elevator_transmission" >
+    <!-- ================================================================== -->
+    <transmission name="${linear_elevatorlink_name}_transmission" >
+      <type>transmission_interface/SimpleTransmission</type>
+      <joint name="${linear_elevator_joint_name}_joint" />
+      <actuator name="linear_elevator_motor" >
+        <hardwareInterface>EffortJointInterface</hardwareInterface>
+        <mechanicalReduction>1.0</mechanicalReduction>
+      </actuator>
+    </transmission>
+    <!-- ================================================================== -->
+  </xacro:macro>
 <!-- Wheel ################################################################ -->
   <xacro:macro name="wheel_transmission"

File: pandora_robots_description/urdf/gears/gears.urdf.xacro (robot description, xacro)
@@ -20,4 +20,8 @@
     <xacro:if value="${enable_base_link}" >
       <xacro:base_link />
+    </xacro:if>
+    <!-- ================================================================== -->
+    <xacro:if value="${enable_linear_elevator_link}" >
+      <xacro:linear_elevator_link />
     </xacro:if>
     <!-- ================================================================== -->
@@ -38,4 +42,8 @@
   <xacro:if value="${enable_joints}" >
     <!-- ================================================================== -->
+    <xacro:if value="${enable_linear_elevator_joint}" >
+      <xacro:linear_elevator_joint />
+    </xacro:if>
+    <!-- ================================================================== -->
     <xacro:if value="${enable_side_joints}" >
       <xacro:side_joint prefix_y="left" reflect_y="1" />
@@ -55,14 +63,18 @@
     <xacro:robot_sdf_physics />
     <xacro:if value="${enable_sdf_physics}" >
-      <!-- ================================================================== -->
+      <!-- ================================================================ -->
       <xacro:if value="${enable_base_link_sdf_physics}" >
         <xacro:base_link_sdf_physics />
       </xacro:if>
-      <!-- ================================================================== -->
+      <!-- ================================================================ -->
+      <xacro:if value="${enable_linear_elevator_link_sdf_physics}" >
+        <xacro:linear_elevator_link_sdf_physics />
+      </xacro:if>
+      <!-- ================================================================ -->
       <xacro:if value="${enable_side_link_sdf_physics}" >
         <xacro:side_link_sdf_physics prefix_y="left" />
         <xacro:side_link_sdf_physics prefix_y="right" />
       </xacro:if>
-      <!-- ================================================================== -->
+      <!-- ================================================================ -->
       <xacro:if value="${enable_wheel_link_sdf_physics}" >
         <xacro:wheel_link_sdf_physics prefix_y="left" prefix_x="front" />
@@ -71,10 +83,14 @@
         <xacro:wheel_link_sdf_physics prefix_y="right" prefix_x="rear" />
       </xacro:if>
-      <!-- ================================================================== -->
+      <!-- ================================================================ -->
+      <xacro:if value="${enable_linear_elevator_joint_sdf_physics}" >
+        <xacro:linear_elevator_joint_sdf_physics />
+      </xacro:if>
+      <!-- ================================================================ -->
       <xacro:if value="${enable_side_joint_sdf_physics}" >
         <xacro:side_joint_sdf_physics prefix_y="left" />
         <xacro:side_joint_sdf_physics prefix_y="right" />
       </xacro:if>
-      <!-- ================================================================== -->
+      <!-- ================================================================ -->
       <xacro:if value="${enable_wheel_joint_sdf_physics}" >
         <xacro:wheel_joint_sdf_physics prefix_y="left" prefix_x="front" />
@@ -83,5 +99,5 @@
         <xacro:wheel_joint_sdf_physics prefix_y="right" prefix_x="rear" />
       </xacro:if>
-      <!-- ================================================================== -->
+      <!-- ================================================================ -->
     </xacro:if>
   </xacro:unless>
@@ -123,5 +139,5 @@
   <xacro:unless value="$(arg real)" >
     <xacro:if value="$(arg control)" >
-      <!-- ================================================================== -->
+      <!-- ================================================================ -->
       <xacro:if value="${enable_wheel_links}" >
         <xacro:wheel_transmission prefix_y="left" prefix_x="front" />
@@ -130,19 +146,23 @@
         <xacro:wheel_transmission prefix_y="right" prefix_x="rear" />
       </xacro:if>
-      <!-- ================================================================== -->
+      <!-- ================================================================ -->
+      <xacro:if value="${enable_linear_elevator_link}" >
+        <xacro:linear_elevator_transmission />
+      </xacro:if>
+      <!-- ================================================================ -->
       <xacro:if value="${enable_sensors}" >
-        <!-- ================================================================ -->
+        <!-- ============================================================== -->
         <xacro:if value="${enable_kinect_sensor}" >
           <xacro:sensor_transmission sensor="kinect" rotation="pitch" />
           <xacro:sensor_transmission sensor="kinect" rotation="yaw" />
         </xacro:if>
-        <!-- ================================================================ -->
+        <!-- ============================================================== -->
         <xacro:if value="${enable_hokuyo_laser_sensor}" >
           <xacro:sensor_transmission sensor="laser" rotation="roll" />
           <xacro:sensor_transmission sensor="laser" rotation="pitch" />
         </xacro:if>
-        <!-- ================================================================ -->
-      </xacro:if>
-      <!-- ================================================================== -->
+        <!-- ============================================================== -->
+      </xacro:if>
+      <!-- ================================================================ -->
     </xacro:if>
   </xacro:unless>
@@ -150,13 +170,13 @@
   <xacro:unless value="$(arg real)" >
     <xacro:if value="${enable_plugins}" >
-      <!-- ================================================================== -->
+      <!-- ================================================================ -->
       <xacro:if value="${enable_pandora_differential_plugin}" >
         <xacro:pandora_differential_plugin />
       </xacro:if>
-      <!-- ================================================================== -->
+      <!-- ================================================================ -->
       <xacro:if value="${enable_pandora_p3d_plugin}" >
         <xacro:pandora_p3d_plugin />
       </xacro:if>
-      <!-- ================================================================== -->
+      <!-- ================================================================ -->
       <xacro:if value="$(arg control)" >
         <xacro:if value="$(arg interface)" >
@@ -167,5 +187,5 @@
         </xacro:unless>
       </xacro:if>
-      <!-- ================================================================== -->
+      <!-- ================================================================ -->
       <xacro:if value="$(arg control)" >
         <xacro:if value="${enable_ros_imu_plugin}" >
@@ -173,5 +193,5 @@
         </xacro:if>
       </xacro:if>
-      <!-- ================================================================== -->
+      <!-- ================================================================ -->
       <xacro:if value="${enable_sensors}" >
         <xacro:if value="${enable_hokuyo_laser_sensor}" >
@@ -183,9 +203,9 @@
         </xacro:if>
       </xacro:if>
-      <!-- ================================================================== -->
+      <!-- ================================================================ -->
       <xacro:unless value="$(arg control)" >
         <xacro:ros_skid_steer_drive_plugin />
       </xacro:unless>
-    <!-- ==================================================================== -->
+    <!-- ================================================================== -->
     </xacro:if>
   </xacro:unless>

File: pandora_robots_description/urdf/gears/model/joints.urdf.xacro (robot description, xacro)
@@ -1,4 +1,16 @@
 <?xml version="1.0" ?>
 <robot xmlns:xacro="http://ros.org/wiki/xacro" >
+<!-- Linear Elevator ###################################################### -->
+  <xacro:macro name="linear_elevator_joint" >
+    <!-- ================================================================== -->
+    <joint name="${linear_elevator_joint_name}_joint"
+           type="${linear_elevator_joint_type}" >
+      <parent link="${base_link_name}_link" />
+      <child link="${linear_elevator_link_name}_link" />
+      <xacro:linear_elevator_joint_origin />
+      <xacro:linear_elevator_joint_urdf_physics />
+    </joint>
+    <!-- ================================================================== -->
+  </xacro:macro>
 <!-- Side ################################################################# -->
   <xacro:macro name="side_joint"

File: pandora_robots_description/urdf/gears/model/links.urdf.xacro (robot description, xacro)
@@ -18,4 +18,25 @@
         <xacro:base_link_collision_origin />
         <xacro:base_link_collision_mesh />
+      </collision>
+    </link>
+    <!-- ================================================================== -->
+  </xacro:macro>
+<!-- Linear Elevator ###################################################### -->
+  <xacro:macro name="linear_elevator_link" >
+    <!-- ================================================================== -->
+    <link name="${linear_elevator_link_name}_link" >
+      <inertial>
+        <xacro:linear_elevator_link_inertial_origin />
+        <xacro:linear_elevator_link_mass />
+        <xacro:linear_elevator_link_inertia />
+      </inertial>
+      <visual>
+        <xacro:linear_elevator_link_visual_origin />
+        <xacro:linear_elevator_link_visual_mesh />
+        <material name="linear_elevator" />
+      </visual>
+      <collision>
+        <xacro:linear_elevator_link_collision_origin />
+        <xacro:linear_elevator_link_collision_mesh />
       </collision>
     </link>
