Commit message: Fix linear elevator's joint limits.

File: pandora_robots_description/urdf/gears/config/gears_configurations.xacro (robot description, xacro)
@@ -59,5 +59,5 @@
   <xacro:property name="wheel_min_depth" value="0.001" />
   <!-- ==================================================================== -->
-  <xacro:property name="linear_elevator_joint_max_limit" value="0.2" />
+  <xacro:property name="linear_elevator_joint_max_limit" value="0.24" />
   <xacro:property name="side_joint_max_limit" value="0.785" />
   <xacro:property name="side_joint_damping" value="0.0" />

File: pandora_robots_description/urdf/gears/config/gears_physics.gazebo.xacro (robot description, xacro)
@@ -150,5 +150,5 @@
     <dynamics damping="${side_joint_damping}" />
          <!-- friction="0.0" /> -->
-    <limit lower="-${side_joint_max_limit}"
+    <limit lower="0"
            upper="${side_joint_max_limit}"
            effort="100.0"
@@ -166,6 +166,6 @@
     <!-- <dynamics damping="0.0"
                    friction="0.0" /> -->
-    <limit effort="50.0"
-           velocity="50.0" />
+    <limit effort="100.0"
+           velocity="100.0" />
       <!-- lower="-0.0" -->
       <!-- upper="0.0" -->

File: pandora_robots_description/urdf/gears/config/properties/joint_offsets.xacro (robot description, xacro)
@@ -3,6 +3,5 @@
   <!-- ==================================================================== -->
   <xacro:macro name="linear_elevator_joint_origin" >
-    <origin xyz="0.0 0.3 0.5"
-            rpy="${zero}" />
+    <xacro:default_origin />
   </xacro:macro>
   <!-- ==================================================================== -->

File: pandora_robots_description/urdf/gears/gazebo/plugins.gazebo.xacro (robot description, xacro)
@@ -15,5 +15,5 @@
         <leftSideJoint>left_${side_joint_name}_joint</leftSideJoint>
         <rightSideJoint>right_${side_joint_name}_joint</rightSideJoint>
-        <maxAngle>${side_joint_max_angle}</maxAngle>
+        <maxAngle>${side_joint_max_limit}</maxAngle>
         <sideJointDamping>${side_joint_damping}</sideJointDamping>
         <P>120.0</P>

Commit message: Add final meshes for base and linear and fix sensor poses.

File: pandora_robots_description/urdf/gears/config/gears_configurations.xacro (robot description, xacro)
@@ -40,14 +40,14 @@
   <!-- Meshes ============================================================= -->
   <!-- TODO -->
-  <xacro:property name="enable_simlified_visual_base_link_mesh" value="false" />
-  <xacro:property name="enable_simlified_visual_linear_elevator_link_mesh" value="false" />
-  <xacro:property name="enable_simlified_visual_side_link_mesh" value="false" />
-  <xacro:property name="enable_simlified_visual_wheel_link_mesh" value="false" />
+  <xacro:property name="enable_simplified_visual_base_link_mesh" value="false" />
+  <xacro:property name="enable_simplified_visual_linear_elevator_link_mesh" value="false" />
+  <xacro:property name="enable_simplified_visual_side_link_mesh" value="false" />
+  <xacro:property name="enable_simplified_visual_wheel_link_mesh" value="false" />
   <!-- ==================================================================== -->
 <!-- Gears Misc ########################################################### -->
   <!-- ==================================================================== -->
+  <xacro:property name="linear_elevator_joint_type" value="prismatic" />
   <xacro:property name="side_joint_type" value="revolute" />
   <xacro:property name="wheel_joint_type" value="continuous" />
-  <xacro:property name="linear_elevator_joint_type" value="prismatic" />
   <!-- ==================================================================== -->
 <!-- Gears Coefficients ################################################### -->

File: pandora_robots_description/urdf/gears/config/gears_physics.gazebo.xacro (robot description, xacro)
@@ -132,6 +132,6 @@
     <!-- <calibration rising="0.0"
                       falling="0.0" /> -->
-    <dynamics damping="0.0" />
-         <!-- friction="0.0" /> -->
+    <!-- <dynamics damping="0.0"
+                   friction="0.0" /> -->
     <limit lower="0"
            upper="${linear_elevator_joint_max_limit}"

File: pandora_robots_description/urdf/gears/config/properties/inertia_tensors.xacro (robot description, xacro)
@@ -3,19 +3,19 @@
   <!-- ==================================================================== -->
   <xacro:macro name="base_link_inertia" >
-    <inertia ixx="0.410690"
-             ixy="0.011589"
-             ixz="0.081825"
-             iyy="0.424490"
-             iyz="0.022113"
-             izz="0.126610" />
+    <inertia ixx="0.11754"
+             ixy="0.0039217"
+             ixz="0.0053416"
+             iyy="0.12773"
+             iyz="-0.0039963"
+             izz="0.10593" />
   </xacro:macro>
   <!-- ==================================================================== -->
   <xacro:macro name="linear_elevator_link_inertia" >
-    <inertia ixx="0.001"
-             ixy="0.001"
-             ixz="0.001"
-             iyy="0.001"
-             iyz="0.001"
-             izz="0.001" />
+    <inertia ixx="0.015755"
+             ixy="-0.00089486"
+             ixz="-0.0017447"
+             iyy="0.014259"
+             iyz="0.0037284"
+             izz="0.0035941" />
   </xacro:macro>
   <!-- ==================================================================== -->

File: pandora_robots_description/urdf/gears/config/properties/joint_offsets.xacro (robot description, xacro)
@@ -3,5 +3,6 @@
   <!-- ==================================================================== -->
   <xacro:macro name="linear_elevator_joint_origin" >
-    <xacro:default_origin />
+    <origin xyz="0.09368 -0.0005 0.19695"
+            rpy="${zero}" />
   </xacro:macro>
   <!-- ==================================================================== -->

File: pandora_robots_description/urdf/gears/config/properties/link_offsets.xacro (robot description, xacro)
@@ -4,10 +4,11 @@
   <!-- ==================================================================== -->
   <xacro:macro name="base_link_inertial_origin" >
-    <origin xyz="-1.1543E-07 -1.3195E-07 0.23164"
+    <origin xyz="-0.010032 -0.0067035 0.16451"
             rpy="${zero}" />
   </xacro:macro>
   <!-- ==================================================================== -->
   <xacro:macro name="linear_elevator_link_inertial_origin" >
-    <xacro:default_origin />
+    <origin xyz="0.01229 0.026011 0.26669"
+            rpy="${zero}" />
   </xacro:macro>
   <!-- ==================================================================== -->

File: pandora_robots_description/urdf/gears/config/properties/masses.xacro (robot description, xacro)
@@ -3,9 +3,9 @@
   <!-- ==================================================================== -->
   <xacro:macro name="base_link_mass" >
-    <mass value="9.3044" />
+    <mass value="8.6373" />
   </xacro:macro>
   <!-- ==================================================================== -->
   <xacro:macro name="linear_elevator_link_mass" >
-    <mass value="0.001" />
+    <mass value="1.0889" />
   </xacro:macro>
   <!-- ==================================================================== -->

File: pandora_robots_description/urdf/gears/gazebo/plugins.gazebo.xacro (robot description, xacro)
@@ -83,5 +83,5 @@
 <!-- Ros Control ########################################################## -->
   <xacro:macro name="gazebo_ros_control_plugin"
-               params="hw_sim" >
+               params="hw_sim ns" >
     <!-- ================================================================== -->
     <gazebo>
@@ -89,5 +89,5 @@
               filename="libgazebo_ros_control.so" >
       <!-- <robotNamespace>${robot_namespace}</robotNamespace> -->
-      <robotNamespace>control</robotNamespace>
+      <robotNamespace>${ns}</robotNamespace>
       <robotSimType>${hw_sim}</robotSimType>
       </plugin>

File: pandora_robots_description/urdf/gears/gazebo/sensors.xacro (robot description, xacro)
@@ -19,6 +19,7 @@
                params="control" >
     <!-- ================================================================== -->
-    <xacro:kinect_caster parent="${base_link_name}_link" control="${control}" >
-      <origin xyz="0.156 0.0 0.526"
+    <xacro:kinect_caster parent="${linear_elevator_link_name}_link"
+                         control="${control}" >
+      <origin xyz="0.12252 0.01239 0.24402"
               rpy="${zero}" />
     </xacro:kinect_caster>
@@ -40,6 +41,6 @@
     <xacro:sonar_caster name="${prefix_y}_rear"
                         parent="${base_link_name}_link" >
-      <origin xyz="-0.2 ${ reflect_y * ( 0.15 ) } 0.13"
-              rpy="0.0 0.0 ${PI}" />
+      <origin xyz="-0.15519 ${ reflect_y * ( 0.113 + ( - 1 ) * reflect_y * 0.00051 ) } 0.14305"
+              rpy="0.0 0.0 ${ PI + ( - 1 ) * refleft_y * PI_6 }" />
     </xacro:sonar_caster>
     <!-- ================================================================== -->
@@ -48,6 +49,6 @@
   <xacro:macro name="thermal_sensor" >
     <!-- ================================================================== -->
-    <xacro:thermal_caster parent="${base_link_name}_link" >
-      <origin xyz="0.2 -0.05 0.23"
+    <xacro:thermal_caster parent="${linear_elevator_link_name}_link" >
+      <origin xyz="-0.00411 0.10566 0.42419"
               rpy="${zero}" />
     </xacro:thermal_caster>
@@ -57,6 +58,6 @@
   <xacro:macro name="co2_sensor" >
     <!-- ================================================================== -->
-    <xacro:co2_caster parent="${base_link_name}_link" >
-      <origin xyz="0.2 0.0 0.36"
+    <xacro:co2_caster parent="${linear_elevator_link_name}_link" >
+      <origin xyz="-0.00411 0.09004 0.40273"
               rpy="${zero}" />
     </xacro:co2_caster>
@@ -66,6 +67,6 @@
   <xacro:macro name="microphone_sensor" >
     <!-- ================================================================== -->
-    <xacro:microphone_caster parent="${base_link_name}_link" >
-      <origin xyz="0.2 0.0 0.38"
+    <xacro:microphone_caster parent="${linear_elevator_link_name}_link" >
+      <origin xyz="-0.00411 0.1211 0.40273"
               rpy="${zero}" />
     </xacro:microphone_caster>

File: pandora_robots_description/urdf/gears/gazebo/transmission.xacro (robot description, xacro)
@@ -4,5 +4,5 @@
   <xacro:macro name="linear_elevator_transmission" >
     <!-- ================================================================== -->
-    <transmission name="${linear_elevatorlink_name}_transmission" >
+    <transmission name="${linear_elevator_link_name}_transmission" >
       <type>transmission_interface/SimpleTransmission</type>
       <joint name="${linear_elevator_joint_name}_joint" />

Commit message: Add argument to load description for real robot.

File: pandora_robots_description/urdf/gears/config/gears_configurations.xacro (robot description, xacro)
@@ -29,6 +29,6 @@
   <!-- SDF Physics ======================================================== -->
   <xacro:property name="enable_sdf_physics" value="true" />
-    <xacro:property name="enable_base_link_sdf_physics" value="true" />
-    <xacro:property name="enable_side_link_sdf_physics" value="true" />
+    <xacro:property name="enable_base_link_sdf_physics" value="false" />
+    <xacro:property name="enable_side_link_sdf_physics" value="false" />
     <xacro:property name="enable_wheel_link_sdf_physics" value="true" />
     <xacro:property name="enable_side_joint_sdf_physics" value="false" />

File: pandora_robots_description/urdf/gears/gears.urdf.xacro (robot description, xacro)
@@ -52,41 +52,48 @@
   </xacro:if>
 <!-- Load Physics ######################################################### -->
-  <xacro:robot_sdf_physics />
-  <xacro:if value="${enable_sdf_physics}" >
-    <!-- ================================================================== -->
-    <xacro:if value="${enable_base_link_sdf_physics}" >
-      <xacro:base_link_sdf_physics />
+  <xacro:unless value="$(arg real)" >
+    <xacro:robot_sdf_physics />
+    <xacro:if value="${enable_sdf_physics}" >
+      <!-- ================================================================== -->
+      <xacro:if value="${enable_base_link_sdf_physics}" >
+        <xacro:base_link_sdf_physics />
+      </xacro:if>
+      <!-- ================================================================== -->
+      <xacro:if value="${enable_side_link_sdf_physics}" >
+        <xacro:side_link_sdf_physics prefix_y="left" />
+        <xacro:side_link_sdf_physics prefix_y="right" />
+      </xacro:if>
+      <!-- ================================================================== -->
+      <xacro:if value="${enable_wheel_link_sdf_physics}" >
+        <xacro:wheel_link_sdf_physics prefix_y="left" prefix_x="front" />
+        <xacro:wheel_link_sdf_physics prefix_y="left" prefix_x="rear" />
+        <xacro:wheel_link_sdf_physics prefix_y="right" prefix_x="front" />
+        <xacro:wheel_link_sdf_physics prefix_y="right" prefix_x="rear" />
+      </xacro:if>
+      <!-- ================================================================== -->
+      <xacro:if value="${enable_side_joint_sdf_physics}" >
+        <xacro:side_joint_sdf_physics prefix_y="left" />
+        <xacro:side_joint_sdf_physics prefix_y="right" />
+      </xacro:if>
+      <!-- ================================================================== -->
+      <xacro:if value="${enable_wheel_joint_sdf_physics}" >
+        <xacro:wheel_joint_sdf_physics prefix_y="left" prefix_x="front" />
+        <xacro:wheel_joint_sdf_physics prefix_y="left" prefix_x="rear" />
+        <xacro:wheel_joint_sdf_physics prefix_y="right" prefix_x="front" />
+        <xacro:wheel_joint_sdf_physics prefix_y="right" prefix_x="rear" />
+      </xacro:if>
+      <!-- ================================================================== -->
     </xacro:if>
-    <!-- ================================================================== -->
-    <xacro:if value="${enable_side_link_sdf_physics}" >
-      <xacro:side_link_sdf_physics prefix_y="left" />
-      <xacro:side_link_sdf_physics prefix_y="right" />
-    </xacro:if>
-    <!-- ================================================================== -->
-    <xacro:if value="${enable_wheel_link_sdf_physics}" >
-      <xacro:wheel_link_sdf_physics prefix_y="left" prefix_x="front" />
-      <xacro:wheel_link_sdf_physics prefix_y="left" prefix_x="rear" />
-      <xacro:wheel_link_sdf_physics prefix_y="right" prefix_x="front" />
-      <xacro:wheel_link_sdf_physics prefix_y="right" prefix_x="rear" />
-    </xacro:if>
-    <!-- ================================================================== -->
-    <xacro:if value="${enable_side_joint_sdf_physics}" >
-      <xacro:side_joint_sdf_physics prefix_y="left" />
-      <xacro:side_joint_sdf_physics prefix_y="right" />
-    </xacro:if>
-    <!-- ================================================================== -->
-    <xacro:if value="${enable_wheel_joint_sdf_physics}" >
-      <xacro:wheel_joint_sdf_physics prefix_y="left" prefix_x="front" />
-      <xacro:wheel_joint_sdf_physics prefix_y="left" prefix_x="rear" />
-      <xacro:wheel_joint_sdf_physics prefix_y="right" prefix_x="front" />
-      <xacro:wheel_joint_sdf_physics prefix_y="right" prefix_x="rear" />
-    </xacro:if>
-    <!-- ================================================================== -->
-  </xacro:if>
+  </xacro:unless>
 <!-- Load Sensors ######################################################### -->
   <xacro:if value="${enable_sensors}" >
     <!-- ================================================================== -->
     <xacro:if value="${enable_kinect_sensor}" >
-      <xacro:kinect_sensor control="$(arg control)" />
+      <xacro:if value="$(arg real)" >
+        <xacro:kinect_sensor control="true" />
+      </xacro:if>
+      <xacro:unless value="$(arg real)" >
+        <xacro:kinect_sensor control="$(arg control)" />
+      </xacro:unless>
     </xacro:if>
     <!-- ================================================================== -->
@@ -114,69 +121,73 @@
   </xacro:if>
 <!-- Load Transmissions ################################################### -->
-  <xacro:if value="$(arg control)" >
-    <!-- ================================================================== -->
-    <xacro:if value="${enable_wheel_links}" >
-      <xacro:wheel_transmission prefix_y="left" prefix_x="front" />
-      <xacro:wheel_transmission prefix_y="left" prefix_x="rear" />
-      <xacro:wheel_transmission prefix_y="right" prefix_x="front" />
-      <xacro:wheel_transmission prefix_y="right" prefix_x="rear" />
+  <xacro:unless value="$(arg real)" >
+    <xacro:if value="$(arg control)" >
+      <!-- ================================================================== -->
+      <xacro:if value="${enable_wheel_links}" >
+        <xacro:wheel_transmission prefix_y="left" prefix_x="front" />
+        <xacro:wheel_transmission prefix_y="left" prefix_x="rear" />
+        <xacro:wheel_transmission prefix_y="right" prefix_x="front" />
+        <xacro:wheel_transmission prefix_y="right" prefix_x="rear" />
+      </xacro:if>
+      <!-- ================================================================== -->
+      <xacro:if value="${enable_sensors}" >
+        <!-- ================================================================ -->
+        <xacro:if value="${enable_kinect_sensor}" >
+          <xacro:sensor_transmission sensor="kinect" rotation="pitch" />
+          <xacro:sensor_transmission sensor="kinect" rotation="yaw" />
+        </xacro:if>
+        <!-- ================================================================ -->
+        <xacro:if value="${enable_hokuyo_laser_sensor}" >
+          <xacro:sensor_transmission sensor="laser" rotation="roll" />
+          <xacro:sensor_transmission sensor="laser" rotation="pitch" />
+        </xacro:if>
+        <!-- ================================================================ -->
+      </xacro:if>
+      <!-- ================================================================== -->
     </xacro:if>
-    <!-- ================================================================== -->
-    <xacro:if value="${enable_sensors}" >
-      <!-- ================================================================ -->
-      <xacro:if value="${enable_kinect_sensor}" >
-        <xacro:sensor_transmission sensor="kinect" rotation="pitch" />
-        <xacro:sensor_transmission sensor="kinect" rotation="yaw" />
+  </xacro:unless>
+<!-- Load Plugins ######################################################### -->
+  <xacro:unless value="$(arg real)" >
+    <xacro:if value="${enable_plugins}" >
+      <!-- ================================================================== -->
+      <xacro:if value="${enable_pandora_differential_plugin}" >
+        <xacro:pandora_differential_plugin />
       </xacro:if>
-      <!-- ================================================================ -->
-      <xacro:if value="${enable_hokuyo_laser_sensor}" >
-        <xacro:sensor_transmission sensor="laser" rotation="roll" />
-        <xacro:sensor_transmission sensor="laser" rotation="pitch" />
+      <!-- ================================================================== -->
+      <xacro:if value="${enable_pandora_p3d_plugin}" >
+        <xacro:pandora_p3d_plugin />
       </xacro:if>
-      <!-- ================================================================ -->
-    </xacro:if>
-    <!-- ================================================================== -->
-  </xacro:if>
-<!-- Load Plugins ######################################################### -->
-  <xacro:if value="${enable_plugins}" >
-    <!-- ================================================================== -->
-    <xacro:if value="${enable_pandora_differential_plugin}" >
-      <xacro:pandora_differential_plugin />
-    </xacro:if>
-    <!-- ================================================================== -->
-    <xacro:if value="${enable_pandora_p3d_plugin}" >
-      <xacro:pandora_p3d_plugin />
-    </xacro:if>
-    <!-- ================================================================== -->
-    <xacro:if value="$(arg control)" >
-      <xacro:if value="$(arg interface)" >
-        <xacro:gazebo_ros_control_plugin hw_sim="pandora_gazebo_interface/GazeboInterface" />
-      </xacro:if>
-      <xacro:unless value="$(arg interface)" >
-        <xacro:gazebo_ros_control_plugin hw_sim="gazebo_ros_control/DefaultRobotHWSim" />
-      </xacro:unless>
-    </xacro:if>
-    <!-- ================================================================== -->
-    <xacro:if value="$(arg control)" >
-      <xacro:if value="${enable_ros_imu_plugin}" >
-        <xacro:ros_imu_plugin />
-      </xacro:if>
-    </xacro:if>
-    <!-- ================================================================== -->
-    <xacro:if value="${enable_sensors}" >
-      <xacro:if value="${enable_hokuyo_laser_sensor}" >
-        <xacro:unless value="$(arg control)" >
-          <xacro:if value="${enable_pandora_imu_stabilizer_plugin}" >
-            <xacro:pandora_imu_stabilizer_plugin />
-          </xacro:if>
+      <!-- ================================================================== -->
+      <xacro:if value="$(arg control)" >
+        <xacro:if value="$(arg interface)" >
+          <xacro:gazebo_ros_control_plugin hw_sim="pandora_gazebo_interface/GazeboInterface" />
+        </xacro:if>
+        <xacro:unless value="$(arg interface)" >
+          <xacro:gazebo_ros_control_plugin hw_sim="gazebo_ros_control/DefaultRobotHWSim" />
         </xacro:unless>
       </xacro:if>
+      <!-- ================================================================== -->
+      <xacro:if value="$(arg control)" >
+        <xacro:if value="${enable_ros_imu_plugin}" >
+          <xacro:ros_imu_plugin />
+        </xacro:if>
+      </xacro:if>
+      <!-- ================================================================== -->
+      <xacro:if value="${enable_sensors}" >
+        <xacro:if value="${enable_hokuyo_laser_sensor}" >
+          <xacro:unless value="$(arg control)" >
+            <xacro:if value="${enable_pandora_imu_stabilizer_plugin}" >
+              <xacro:pandora_imu_stabilizer_plugin />
+            </xacro:if>
+          </xacro:unless>
+        </xacro:if>
+      </xacro:if>
+      <!-- ================================================================== -->
+      <xacro:unless value="$(arg control)" >
+        <xacro:ros_skid_steer_drive_plugin />
+      </xacro:unless>
+    <!-- ==================================================================== -->
     </xacro:if>
-    <!-- ================================================================== -->
-    <xacro:unless value="$(arg control)" >
-      <xacro:ros_skid_steer_drive_plugin />
-    </xacro:unless>
-  <!-- ==================================================================== -->
-  </xacro:if>
+  </xacro:unless>
 <!-- ###################################################################### -->
 </robot>
