Commit message: Fix linear joint and thermal macro.

File: pandora_robots_description/urdf/gears/config/gears_configurations.xacro (robot description, xacro)
@@ -19,8 +19,8 @@
     <xacro:property name="enable_kinect_sensor" value="true" />
     <xacro:property name="enable_hokuyo_laser_sensor" value="true" />
-    <xacro:property name="enable_sonar_sensor" value="false" />
-    <xacro:property name="enable_thermal_sensor" value="false" />
-    <xacro:property name="enable_co2_sensor" value="false" />
-    <xacro:property name="enable_microphone_sensor" value="false" />
+    <xacro:property name="enable_sonar_sensors" value="true" />
+    <xacro:property name="enable_thermal_sensors" value="true" />
+    <xacro:property name="enable_co2_sensor" value="true" />
+    <xacro:property name="enable_microphone_sensor" value="true" />
   <!-- Plugins ============================================================ -->
   <xacro:property name="enable_plugins" value="true" />
@@ -59,5 +59,5 @@
   <xacro:property name="wheel_min_depth" value="0.001" />
   <!-- ==================================================================== -->
-  <xacro:property name="linear_elevator_joint_max_limit" value="0.24" />
+  <xacro:property name="linear_elevator_joint_max_limit" value="0.23" />
   <xacro:property name="side_joint_max_limit" value="0.785" />
   <xacro:property name="side_joint_damping" value="0.0" />

File: pandora_robots_description/urdf/gears/config/gears_physics.gazebo.xacro (robot description, xacro)
@@ -136,6 +136,6 @@
     <limit lower="0"
            upper="${linear_elevator_joint_max_limit}"
-           effort="100.0"
-           velocity="100.0" />
+           effort="1000.0"
+           velocity="1000.0" />
     <!-- <safety_controller soft_lower_limit="0.0"
                             soft_upper_limit="0.0"

File: pandora_robots_description/urdf/gears/config/properties/joint_offsets.xacro (robot description, xacro)
@@ -3,5 +3,5 @@
   <!-- ==================================================================== -->
   <xacro:macro name="linear_elevator_joint_origin" >
-    <origin xyz="0.09368 -0.0005 0.19695"
+    <origin xyz="0.09368 -0.0005 0.23995"
             rpy="${zero}" />
   </xacro:macro>

File: pandora_robots_description/urdf/gears/gazebo/sensors.xacro (robot description, xacro)
@@ -42,13 +42,26 @@
                         parent="${base_link_name}_link" >
       <origin xyz="-0.15519 ${ reflect_y * ( 0.113 + ( - 1 ) * reflect_y * 0.00051 ) } 0.14305"
-              rpy="0.0 0.0 ${ PI + ( - 1 ) * refleft_y * PI_6 }" />
+              rpy="0.0 0.0 ${ PI + ( - 1 ) * reflect_y * PI_6 }" />
     </xacro:sonar_caster>
     <!-- ================================================================== -->
   </xacro:macro>
 <!-- Thermal ############################################################## -->
-  <xacro:macro name="thermal_sensor" >
+  <xacro:macro name="thermal_sensors" >
     <!-- ================================================================== -->
-    <xacro:thermal_caster parent="${linear_elevator_link_name}_link" >
+    <xacro:thermal_caster parent="${linear_elevator_link_name}_link"
+                          prefix_y="middle" >
       <origin xyz="-0.00411 0.10566 0.42419"
+              rpy="${zero}" />
+    </xacro:thermal_caster>
+    <!-- ================================================================== -->
+    <xacro:thermal_caster parent="${linear_elevator_link_name}_link"
+                          prefix_y="right" >
+      <origin xyz="-0.00411 0.08566 0.42419"
+              rpy="${zero}" />
+    </xacro:thermal_caster>
+    <!-- ================================================================== -->
+    <xacro:thermal_caster parent="${linear_elevator_link_name}_link"
+                          prefix_y="left" >
+      <origin xyz="-0.00411 0.12566 0.42419"
               rpy="${zero}" />
     </xacro:thermal_caster>

File: pandora_robots_description/urdf/gears/gears.urdf.xacro (robot description, xacro)
@@ -118,11 +118,11 @@
     </xacro:if>
     <!-- ================================================================== -->
-    <xacro:if value="${enable_sonar_sensor}" >
+    <xacro:if value="${enable_sonar_sensors}" >
       <xacro:sonar_sensor prefix_y="left" reflect_y="1" />
       <xacro:sonar_sensor prefix_y="right" reflect_y="-1" />
     </xacro:if>
     <!-- ================================================================== -->
-    <xacro:if value="${enable_thermal_sensor}" >
-       <xacro:thermal_sensor />
+    <xacro:if value="${enable_thermal_sensors}" >
+       <xacro:thermal_sensors />
     </xacro:if>
     <!-- ================================================================== -->

File: pandora_sensors_description/urdf/thermal_sensor.urdf.xacro (robot description, xacro)
@@ -2,6 +2,6 @@
 <robot xmlns:xacro="http://ros.org/wiki/xacro" >
   <xacro:macro name="thermal_caster"
-               params="parent *origin" >
-    <link name="thermal_link" >
+               params="parent prefix_y *origin" >
+    <link name="${prefix_y}_thermal_link" >
       <inertial>
         <origin xyz="0 0 0.186"
@@ -26,5 +26,5 @@
       </collision>
     </link>
-    <gazebo reference="thermal_link" >
+    <gazebo reference="${prefix_y}_thermal_link" >
       <sensor name="thermal"
               type="camera" >
@@ -50,8 +50,8 @@
       </sensor>
     </gazebo>
-    <joint name="thermal_joint"
+    <joint name="${prefix_y}_thermal_joint"
            type="fixed" >
       <parent link="${parent}" />
-      <child link="thermal_link" />
+      <child link="${prefix_y}_thermal_link" />
       <xacro:insert_block name="origin" />
     </joint>
