Commit message: Add linear head.

File: pandora_robots_description/urdf/gears/config/gears_configurations.xacro (robot description, xacro)
@@ -8,4 +8,5 @@
     <xacro:property name="enable_base_link" value="true" />
     <xacro:property name="enable_linear_elevator_link" value="true" />
+    <xacro:property name="enable_linear_head_link" value="true" />
     <xacro:property name="enable_side_links" value="true" />
     <xacro:property name="enable_wheel_links" value="true" />
@@ -13,4 +14,5 @@
   <xacro:property name="enable_joints" value="true" />
     <xacro:property name="enable_linear_elevator_joint" value="true" />
+    <xacro:property name="enable_linear_head_joints" value="true" />
     <xacro:property name="enable_side_joints" value="true" />
     <xacro:property name="enable_wheel_joints" value="true" />
@@ -33,7 +35,10 @@
     <xacro:property name="enable_base_link_sdf_physics" value="false" />
     <xacro:property name="enable_linear_elevator_link_sdf_physics" value="false" />
+    <xacro:property name="enable_linear_head_link_sdf_physics" value="false" />
     <xacro:property name="enable_side_link_sdf_physics" value="false" />
     <xacro:property name="enable_wheel_link_sdf_physics" value="true" />
     <xacro:property name="enable_linear_elevator_joint_sdf_physics" value="false" />
+    <xacro:property name="enable_linear_head_pitch_joint_sdf_physics" value="false" />
+    <xacro:property name="enable_linear_head_yaw_joint_sdf_physics" value="false" />
     <xacro:property name="enable_side_joint_sdf_physics" value="false" />
     <xacro:property name="enable_wheel_joint_sdf_physics" value="false" />
@@ -42,4 +47,5 @@
   <xacro:property name="enable_simplified_visual_base_link_mesh" value="false" />
   <xacro:property name="enable_simplified_visual_linear_elevator_link_mesh" value="false" />
+  <xacro:property name="enable_simplified_visual_linear_head_link_mesh" value="false" />
   <xacro:property name="enable_simplified_visual_side_link_mesh" value="false" />
   <xacro:property name="enable_simplified_visual_wheel_link_mesh" value="false" />
@@ -48,4 +54,6 @@
   <!-- ==================================================================== -->
   <xacro:property name="linear_elevator_joint_type" value="prismatic" />
+  <xacro:property name="linear_head_pitch_joint_type" value="revolute" />
+  <xacro:property name="linear_head_yaw_joint_type" value="revolute" />
   <xacro:property name="side_joint_type" value="revolute" />
   <xacro:property name="wheel_joint_type" value="continuous" />
@@ -60,4 +68,7 @@
   <!-- ==================================================================== -->
   <xacro:property name="linear_elevator_joint_max_limit" value="0.23" />
+  <xacro:property name="linear_head_pitch_joint_max_limit" value="1.57" /> <!-- FIXME -->
+  <xacro:property name="linear_head_yaw_joint_max_limit" value="1.57" /> <!-- FIXME -->
+  <!-- TODO : Add limits for sensors -->
   <xacro:property name="side_joint_max_limit" value="0.785" />
   <xacro:property name="side_joint_damping" value="0.0" />

File: pandora_robots_description/urdf/gears/config/gears_physics.gazebo.xacro (robot description, xacro)
@@ -29,4 +29,22 @@
   <xacro:macro name="linear_elevator_link_sdf_physics" >
     <gazebo reference="${linear_elevator_link_name}_link" >
+      <!-- <material>Gazebo/Grey</material> -->
+      <!-- <gravity>false</gravity> -->
+      <!-- <dampingFactor>0.0</dampingFactor> -->
+      <!-- <maxVel>0.0</maxVel> -->
+      <!-- <minDepth>0.0</minDepth> -->
+      <!-- <mu1>0.0</mu1> -->
+      <!-- <mu2>0.0</mu2> -->
+      <!-- <fdir1>0 0 0</fdir1> -->
+      <!-- <kp>0.0</kp> -->
+      <!-- <kd>0.0</kd> -->
+      <!-- <selfCollide>false</selfCollide> -->
+      <!-- <maxContacts>1</maxContacts> -->
+      <!-- <laserRetro>0.0</laserRetro> -->
+    </gazebo>
+  </xacro:macro>
+  <!-- ==================================================================== -->
+  <xacro:macro name="linear_head_link_sdf_physics" >
+    <gazebo reference="${linear_head_link_name}_link" >
       <!-- <material>Gazebo/Grey</material> -->
       <!-- <gravity>false</gravity> -->
@@ -86,5 +104,31 @@
   <!-- ==================================================================== -->
   <xacro:macro name="linear_elevator_joint_sdf_physics" >
-    <gazebo reference="${linear_elevator_name}_joint" >
+    <gazebo reference="${linear_elevator_joint_name}_joint" >
+      <!-- <kp>0.0</kp> -->
+      <!-- <kd>0.0</kd> -->
+      <!-- <stopCfm>0.0</stopCfm> -->
+      <!-- <stopErp>0.0</stopErp> -->
+      <!-- <provideFeedback>false</provideFeedback> -->
+      <!-- <cfmDamping>true</cfmDamping> -->
+      <implicitSpringDamper>true</implicitSpringDamper>
+      <!-- <fudgeFactor>0.0</fudgeFactor> -->
+    </gazebo>
+  </xacro:macro>
+  <!-- ==================================================================== -->
+  <xacro:macro name="linear_head_pitch_joint_sdf_physics" >
+    <gazebo reference="${linear_head_pitch_joint_name}_joint" >
+      <!-- <kp>0.0</kp> -->
+      <!-- <kd>0.0</kd> -->
+      <!-- <stopCfm>0.0</stopCfm> -->
+      <!-- <stopErp>0.0</stopErp> -->
+      <!-- <provideFeedback>false</provideFeedback> -->
+      <!-- <cfmDamping>true</cfmDamping> -->
+      <implicitSpringDamper>true</implicitSpringDamper>
+      <!-- <fudgeFactor>0.0</fudgeFactor> -->
+    </gazebo>
+  </xacro:macro>
+  <!-- ==================================================================== -->
+  <xacro:macro name="linear_head_yaw_joint_sdf_physics" >
+    <gazebo reference="${linear_head_yaw_joint_name}_joint" >
       <!-- <kp>0.0</kp> -->
       <!-- <kd>0.0</kd> -->
@@ -138,4 +182,36 @@
            effort="1000.0"
            velocity="1000.0" />
+    <!-- <safety_controller soft_lower_limit="0.0"
+                            soft_upper_limit="0.0"
+                            k_position="0.0"
+                            k_velocity="0.0" /> -->
+  </xacro:macro>
+  <!-- ==================================================================== -->
+  <xacro:macro name="linear_head_pitch_joint_urdf_physics" >
+    <axis xyz="0 1 0" />
+    <!-- <calibration rising="0.0"
+                      falling="0.0" /> -->
+    <!-- <dynamics damping="0.0"
+                   friction="0.0" /> -->
+    <limit lower="-${linear_head_pitch_joint_max_limit}"
+           upper="${linear_head_pitch_joint_max_limit}"
+           effort="300.0"
+           velocity="100.0" />
+    <!-- <safety_controller soft_lower_limit="0.0"
+                            soft_upper_limit="0.0"
+                            k_position="0.0"
+                            k_velocity="0.0" /> -->
+  </xacro:macro>
+  <!-- ==================================================================== -->
+  <xacro:macro name="linear_head_yaw_joint_urdf_physics" >
+    <axis xyz="0 0 1" />
+    <!-- <calibration rising="0.0"
+                      falling="0.0" /> -->
+    <!-- <dynamics damping="0.0"
+                   friction="0.0" /> -->
+    <limit lower="-${linear_head_yaw_joint_max_limit}"
+           upper="${linear_head_yaw_joint_max_limit}"
+           effort="300.0"
+           velocity="100.0" />
     <!-- <safety_controller soft_lower_limit="0.0"
                             soft_upper_limit="0.0"

File: pandora_robots_description/urdf/gears/config/properties/inertia_tensors.xacro (robot description, xacro)
@@ -17,5 +17,23 @@
              iyy="0.014259"
              iyz="0.0037284"
-             izz="0.0035941" />
+             izz="0.0035941" /><!--TODO-->
+  </xacro:macro>
+  <!-- ==================================================================== -->
+  <xacro:macro name="linear_head_base_link_inertia" >
+    <inertia ixx="0.00000001"
+             ixy="0.00000001"
+             ixz="0.00000001"
+             iyy="0.00000001"
+             iyz="0.00000001"
+             izz="0.00000001" /><!--TODO Reduce -->
+  </xacro:macro>
+  <!-- ==================================================================== -->
+  <xacro:macro name="linear_head_link_inertia" >
+    <inertia ixx="0.01"
+             ixy="0.01"
+             ixz="0.01"
+             iyy="0.01"
+             iyz="0.01"
+             izz="0.01" /><!--TODO-->
   </xacro:macro>
   <!-- ==================================================================== -->

File: pandora_robots_description/urdf/gears/config/properties/joint_offsets.xacro (robot description, xacro)
@@ -5,4 +5,14 @@
     <origin xyz="0.09368 -0.0005 0.23995"
             rpy="${zero}" />
+  </xacro:macro>
+  <!-- ==================================================================== -->
+  <xacro:macro name="linear_head_pitch_joint_origin" >
+    <origin xyz="0.0 0.0 0.0"
+            rpy="${zero}" /><!--TODO-->
+  </xacro:macro>
+  <!-- ==================================================================== -->
+  <xacro:macro name="linear_head_yaw_joint_origin" >
+    <origin xyz="0.0 0.0 0.0"
+            rpy="${zero}" /><!--TODO Translate because of second servo -->
   </xacro:macro>
   <!-- ==================================================================== -->

File: pandora_robots_description/urdf/gears/config/properties/link_offsets.xacro (robot description, xacro)
@@ -10,5 +10,14 @@
   <xacro:macro name="linear_elevator_link_inertial_origin" >
     <origin xyz="0.01229 0.026011 0.26669"
-            rpy="${zero}" />
+            rpy="${zero}" /><!--TODO-->
+  </xacro:macro>
+  <!-- ==================================================================== -->
+  <xacro:macro name="linear_head_base_link_inertial_origin" >
+    <xacro:default_origin />
+  </xacro:macro>
+  <!-- ==================================================================== -->
+  <xacro:macro name="linear_head_link_inertial_origin" >
+    <origin xyz="0.0 0.0 0.0"
+            rpy="${zero}" /><!--TODO-->
   </xacro:macro>
   <!-- ==================================================================== -->
@@ -32,4 +41,12 @@
   <!-- ==================================================================== -->
   <xacro:macro name="linear_elevator_link_visual_origin" >
+    <xacro:default_origin />
+  </xacro:macro>
+  <!-- ==================================================================== -->
+  <xacro:macro name="linear_head_base_link_visual_origin" >
+    <xacro:default_origin />
+  </xacro:macro>
+  <!-- ==================================================================== -->
+  <xacro:macro name="linear_head_link_visual_origin" >
     <xacro:default_origin />
   </xacro:macro>
@@ -57,4 +74,12 @@
   </xacro:macro>
   <!-- ==================================================================== -->
+  <xacro:macro name="linear_head_base_link_collision_origin" >
+    <xacro:default_origin />
+  </xacro:macro>
+  <!-- ==================================================================== -->
+  <xacro:macro name="linear_head_link_collision_origin" >
+    <xacro:default_origin />
+  </xacro:macro>
+  <!-- ==================================================================== -->
   <xacro:macro name="side_link_collision_origin"
                params="reflect_y" >

File: pandora_robots_description/urdf/gears/config/properties/masses.xacro (robot description, xacro)
@@ -7,5 +7,13 @@
   <!-- ==================================================================== -->
   <xacro:macro name="linear_elevator_link_mass" >
-    <mass value="1.0889" />
+    <mass value="1.0889" /><!--TODO-->
+  </xacro:macro>
+  <!-- ==================================================================== -->
+  <xacro:macro name="linear_head_base_link_mass" >
+    <mass value="0.001" /><!--TODO Reduce -->
+  </xacro:macro>
+  <!-- ==================================================================== -->
+  <xacro:macro name="linear_head_link_mass" >
+    <mass value="0.1" /><!--TODO-->
   </xacro:macro>
   <!-- ==================================================================== -->

File: pandora_robots_description/urdf/gears/config/properties/materials.xacro (robot description, xacro)
@@ -116,4 +116,8 @@
   </material>
   <!-- ==================================================================== -->
+  <material name="linear_head" >
+    <color rgba="${190/255} ${190/255} ${190/255} 1.0" />
+  </material>
+  <!-- ==================================================================== -->
   <material name="side" >
     <color rgba="${190/255} ${190/255} ${190/255} 1.0" />

File: pandora_robots_description/urdf/gears/config/properties/meshes.xacro (robot description, xacro)
@@ -14,4 +14,11 @@
       <mesh filename="package://pandora_robots_description/meshes/gears/visual/linear_elevator_link.dae" />
       <!-- <mesh filename="package://pandora_robots_description/meshes/gears/collision/linear_elevator_link.stl" /> -->
+    </geometry>
+  </xacro:macro>
+  <!-- ==================================================================== -->
+  <xacro:macro name="linear_head_link_visual_mesh" >
+    <geometry>
+      <mesh filename="package://pandora_robots_description/meshes/gears/visual/linear_head_link.dae" />
+      <!-- <mesh filename="package://pandora_robots_description/meshes/gears/collision/linear_head_link.stl" /> -->
     </geometry>
   </xacro:macro>
@@ -47,4 +54,11 @@
   </xacro:macro>
   <!-- ==================================================================== -->
+  <xacro:macro name="linear_head_link_collision_mesh" >
+    <geometry>
+      <mesh filename="package://pandora_robots_description/meshes/gears/collision/linear_head_link.stl" />
+      <!-- <mesh filename="package://pandora_robots_description/meshes/gears/visual/linear_head_link.dae" /> -->
+    </geometry>
+  </xacro:macro>
+  <!-- ==================================================================== -->
   <xacro:macro name="side_link_collision_mesh" >
     <geometry>

File: pandora_robots_description/urdf/gears/config/properties/names.xacro (robot description, xacro)
@@ -11,4 +11,6 @@
   <xacro:property name="linear_elevator_link_name" value="linear_elevator" />
   <!-- ==================================================================== -->
+  <xacro:property name="linear_head_link_name" value="linear_head" />
+  <!-- ==================================================================== -->
   <xacro:property name="side_link_name" value="side" />
   <!-- ==================================================================== -->
@@ -19,4 +21,8 @@
   <xacro:property name="linear_elevator_joint_name" value="linear_elevator" />
   <!-- ==================================================================== -->
+  <xacro:property name="linear_head_pitch_joint_name" value="linear_head_pitch" />
+  <!-- ==================================================================== -->
+  <xacro:property name="linear_head_yaw_joint_name" value="linear_head_yaw" />
+  <!-- ==================================================================== -->
   <xacro:property name="side_joint_name" value="side" />
   <!-- ==================================================================== -->

File: pandora_robots_description/urdf/gears/gazebo/sensors.xacro (robot description, xacro)
@@ -49,20 +49,20 @@
   <xacro:macro name="thermal_sensors" >
     <!-- ================================================================== -->
-    <xacro:thermal_caster parent="${linear_elevator_link_name}_link"
+    <xacro:thermal_caster parent="${linear_head_link_name}_link"
                           prefix_y="middle" >
-      <origin xyz="-0.00411 0.10566 0.42419"
-              rpy="${zero}" />
+      <origin xyz="0.0 0.0 0.0"
+              rpy="${zero}" /><!--TODO-->
     </xacro:thermal_caster>
     <!-- ================================================================== -->
-    <xacro:thermal_caster parent="${linear_elevator_link_name}_link"
+    <xacro:thermal_caster parent="${linear_head_link_name}_link"
                           prefix_y="right" >
-      <origin xyz="-0.00411 0.08566 0.42419"
-              rpy="${zero}" />
+      <origin xyz="0.0 -0.02 0.0"
+              rpy="${zero}" /><!--TODO-->
     </xacro:thermal_caster>
     <!-- ================================================================== -->
-    <xacro:thermal_caster parent="${linear_elevator_link_name}_link"
+    <xacro:thermal_caster parent="${linear_head_link_name}_link"
                           prefix_y="left" >
-      <origin xyz="-0.00411 0.12566 0.42419"
-              rpy="${zero}" />
+      <origin xyz="0.0 0.02 0.0"
+              rpy="${zero}" /><!--TODO-->
     </xacro:thermal_caster>
     <!-- ================================================================== -->
@@ -71,7 +71,7 @@
   <xacro:macro name="co2_sensor" >
     <!-- ================================================================== -->
-    <xacro:co2_caster parent="${linear_elevator_link_name}_link" >
-      <origin xyz="-0.00411 0.09004 0.40273"
-              rpy="${zero}" />
+    <xacro:co2_caster parent="${linear_head_link_name}_link" >
+      <origin xyz="0.0 0.02 -0.02"
+              rpy="${zero}" /><!--TODO-->
     </xacro:co2_caster>
     <!-- ================================================================== -->
@@ -80,7 +80,7 @@
   <xacro:macro name="microphone_sensor" >
     <!-- ================================================================== -->
-    <xacro:microphone_caster parent="${linear_elevator_link_name}_link" >
-      <origin xyz="-0.00411 0.1211 0.40273"
-              rpy="${zero}" />
+    <xacro:microphone_caster parent="${linear_head_link_name}_link" >
+      <origin xyz="0.0 -0.02 -0.02"
+              rpy="${zero}" /><!--TODO-->
     </xacro:microphone_caster>
     <!-- ================================================================== -->

File: pandora_robots_description/urdf/gears/gazebo/transmission.xacro (robot description, xacro)
@@ -8,4 +8,18 @@
       <joint name="${linear_elevator_joint_name}_joint" />
       <actuator name="linear_elevator_motor" >
+        <hardwareInterface>EffortJointInterface</hardwareInterface>
+        <mechanicalReduction>1.0</mechanicalReduction>
+      </actuator>
+    </transmission>
+    <!-- ================================================================== -->
+  </xacro:macro>
+<!-- Linear Head ########################################################## -->
+  <xacro:macro name="linear_head_transmission"
+               params="rotation" >
+    <!-- ================================================================== -->
+    <transmission name="${linear_head_link_name}_${rotation}_transmission" >
+      <type>transmission_interface/SimpleTransmission</type>
+      <joint name="${linear_head_link_name}_${rotation}_joint" />
+      <actuator name="${linear_head_link_name}_${rotation}_motor" >
         <hardwareInterface>EffortJointInterface</hardwareInterface>
         <mechanicalReduction>1.0</mechanicalReduction>

File: pandora_robots_description/urdf/gears/gears.urdf.xacro (robot description, xacro)
@@ -24,4 +24,8 @@
     <xacro:if value="${enable_linear_elevator_link}" >
       <xacro:linear_elevator_link />
+    </xacro:if>
+    <!-- ================================================================== -->
+    <xacro:if value="${enable_linear_head_link}" >
+      <xacro:linear_head_links />
     </xacro:if>
     <!-- ================================================================== -->
@@ -46,4 +50,8 @@
     </xacro:if>
     <!-- ================================================================== -->
+    <xacro:if value="${enable_linear_head_joints}" >
+      <xacro:linear_head_joints />
+    </xacro:if>
+    <!-- ================================================================== -->
     <xacro:if value="${enable_side_joints}" >
       <xacro:side_joint prefix_y="left" reflect_y="1" />
@@ -72,4 +80,8 @@
       </xacro:if>
       <!-- ================================================================ -->
+      <xacro:if value="${enable_linear_head_link_sdf_physics}" >
+        <xacro:linear_head_link_sdf_physics />
+      </xacro:if>
+      <!-- ================================================================ -->
       <xacro:if value="${enable_side_link_sdf_physics}" >
         <xacro:side_link_sdf_physics prefix_y="left" />
@@ -88,4 +100,12 @@
       </xacro:if>
       <!-- ================================================================ -->
+      <xacro:if value="${enable_linear_head_pitch_joint_sdf_physics}" >
+        <xacro:linear_head_pitch_joint_sdf_physics />
+      </xacro:if>
+      <!-- ================================================================ -->
+      <xacro:if value="${enable_linear_head_yaw_joint_sdf_physics}" >
+        <xacro:linear_head_yaw_joint_sdf_physics />
+      </xacro:if>
+      <!-- ================================================================ -->
       <xacro:if value="${enable_side_joint_sdf_physics}" >
         <xacro:side_joint_sdf_physics prefix_y="left" />
@@ -140,4 +160,13 @@
     <xacro:if value="$(arg control)" >
       <!-- ================================================================ -->
+      <xacro:if value="${enable_linear_elevator_link}" >
+        <xacro:linear_elevator_transmission />
+      </xacro:if>
+      <!-- ================================================================ -->
+      <xacro:if value="${enable_linear_head_link}" >
+        <xacro:linear_head_transmission rotation="pitch" />
+        <xacro:linear_head_transmission rotation="yaw" />
+      </xacro:if>
+      <!-- ================================================================ -->
       <xacro:if value="${enable_wheel_links}" >
         <xacro:wheel_transmission prefix_y="left" prefix_x="front" />
@@ -145,8 +174,4 @@
         <xacro:wheel_transmission prefix_y="right" prefix_x="front" />
         <xacro:wheel_transmission prefix_y="right" prefix_x="rear" />
-      </xacro:if>
-      <!-- ================================================================ -->
-      <xacro:if value="${enable_linear_elevator_link}" >
-        <xacro:linear_elevator_transmission />
       </xacro:if>
       <!-- ================================================================ -->
