Commit message: Add linear head.

File: pandora_robots_description/urdf/gears/model/joints.urdf.xacro (robot description, xacro)
@@ -10,4 +10,24 @@
       <xacro:linear_elevator_joint_origin />
       <xacro:linear_elevator_joint_urdf_physics />
+    </joint>
+    <!-- ================================================================== -->
+  </xacro:macro>
+<!-- Linear Head  ######################################################### -->
+  <xacro:macro name="linear_head_joints" >
+    <!-- ================================================================== -->
+    <joint name="${linear_head_pitch_joint_name}_joint"
+           type="${linear_head_pitch_joint_type}" >
+      <parent link="${linear_elevator_link_name}_link" />
+      <child link="${linear_head_link_name}_base_link" />
+      <xacro:linear_head_pitch_joint_origin />
+      <xacro:linear_head_pitch_joint_urdf_physics />
+    </joint>
+    <!-- ================================================================== -->
+    <joint name="${linear_head_yaw_joint_name}_joint"
+           type="${linear_head_yaw_joint_type}" >
+      <parent link="${linear_head_link_name}_base_link" />
+      <child link="${linear_head_link_name}_link" />
+      <xacro:linear_head_yaw_joint_origin />
+      <xacro:linear_head_yaw_joint_urdf_physics />
     </joint>
     <!-- ================================================================== -->

File: pandora_robots_description/urdf/gears/model/links.urdf.xacro (robot description, xacro)
@@ -39,4 +39,45 @@
         <xacro:linear_elevator_link_collision_origin />
         <xacro:linear_elevator_link_collision_mesh />
+      </collision>
+    </link>
+    <!-- ================================================================== -->
+  </xacro:macro>
+<!-- Linear Head ########################################################## -->
+  <xacro:macro name="linear_head_links" >
+    <!-- ================================================================== -->
+    <link name="${linear_head_link_name}_base_link" >
+      <inertial>
+        <xacro:linear_head_base_link_inertial_origin />
+        <xacro:linear_head_base_link_mass />
+        <xacro:linear_head_base_link_inertia />
+      </inertial>
+      <visual>
+        <xacro:linear_head_base_link_visual_origin />
+        <geometry>
+          <box size="0 0 0" />
+        </geometry>
+      </visual>
+      <collision>
+        <xacro:linear_head_base_link_collision_origin />
+        <geometry>
+          <box size="0 0 0" />
+        </geometry>
+      </collision>
+    </link>
+    <!-- ================================================================== -->
+    <link name="${linear_head_link_name}_link" >
+      <inertial>
+        <xacro:linear_head_link_inertial_origin />
+        <xacro:linear_head_link_mass />
+        <xacro:linear_head_link_inertia />
+      </inertial>
+      <visual>
+        <xacro:linear_head_link_visual_origin />
+        <xacro:linear_head_link_visual_mesh />
+        <material name="linear_head" />
+      </visual>
+      <collision>
+        <xacro:linear_head_link_collision_origin />
+        <xacro:linear_head_link_collision_mesh />
       </collision>
     </link>

Commit message: Update sensor inertia and meshes.

File: pandora_robots_description/urdf/gears/config/gears_configurations.xacro (robot description, xacro)
@@ -67,7 +67,7 @@
   <xacro:property name="wheel_min_depth" value="0.001" />
   <!-- ==================================================================== -->
-  <xacro:property name="linear_elevator_joint_max_limit" value="0.23" />
-  <xacro:property name="linear_head_pitch_joint_max_limit" value="1.57" /> <!-- FIXME -->
-  <xacro:property name="linear_head_yaw_joint_max_limit" value="1.57" /> <!-- FIXME -->
+  <xacro:property name="linear_elevator_joint_max_limit" value="0.0" />
+  <xacro:property name="linear_head_pitch_joint_max_limit" value="0.0" /> <!-- FIXME -->
+  <xacro:property name="linear_head_yaw_joint_max_limit" value="0.0" /> <!-- FIXME -->
   <!-- TODO : Add limits for sensors -->
   <xacro:property name="side_joint_max_limit" value="0.785" />

File: pandora_robots_description/urdf/gears/config/properties/inertia_tensors.xacro (robot description, xacro)
@@ -26,5 +26,5 @@
              iyy="0.00000001"
              iyz="0.00000001"
-             izz="0.00000001" /><!--TODO Reduce -->
+             izz="0.00000001" />
   </xacro:macro>
   <!-- ==================================================================== -->

File: pandora_robots_description/urdf/gears/config/properties/masses.xacro (robot description, xacro)
@@ -11,5 +11,5 @@
   <!-- ==================================================================== -->
   <xacro:macro name="linear_head_base_link_mass" >
-    <mass value="0.001" /><!--TODO Reduce -->
+    <mass value="0.0001" />
   </xacro:macro>
   <!-- ==================================================================== -->

File: pandora_robots_description/urdf/gears/gazebo/sensors.xacro (robot description, xacro)
@@ -21,5 +21,5 @@
     <xacro:kinect_caster parent="${linear_elevator_link_name}_link"
                          control="${control}" >
-      <origin xyz="0.09144 0.01239 0.19742"
+      <origin xyz="0.06744 0.01239 0.19742"
               rpy="${zero}" />
     </xacro:kinect_caster>

File: pandora_sensors_description/urdf/co2_sensor.urdf.xacro (robot description, xacro)
@@ -5,13 +5,13 @@
     <link name="co2_link" >
       <inertial>
-        <origin xyz="0.008 0.0 0.0"
+        <origin xyz="0.005 0.0 0.0"
                 rpy="0 0 0" />
-        <mass value="0.1" />
-        <inertia ixx="1"
+        <mass value="0.005" />
+        <inertia ixx="2.1208E-7"
                  ixy="0"
                  ixz="0"
-                 iyy="1"
+                 iyy="4.033E-7"
                  iyz="0"
-                 izz="1" /><!-- FIXME -->
+                 izz="2.1208E-7" />
       </inertial>
       <visual name="visual" >
@@ -23,8 +23,7 @@
       </visual>
       <collision name="collision" >
-        <origin xyz="0 0 0"
-                rpy="0 0 0" />
+        <origin xyz="0.007 0.0 0.0" />
         <geometry>
-          <box size="0.01 0.01 0.01" />
+          <box size="0.025 0.025 0.025" />
         </geometry>
       </collision>

File: pandora_sensors_description/urdf/hokuyo_utm_30lx.urdf.xacro (robot description, xacro)
@@ -5,5 +5,5 @@
     <link name="laser_link" >
       <inertial>
-        <mass value="0.01" />
+        <mass value="0.16" />
         <origin xyz="0 0 0" />
         <inertia ixx="0.0002632"
@@ -68,5 +68,5 @@
     <link name="hokuyo_base_link" >
       <inertial>
-        <mass value="0.001" />
+        <mass value="0.0001" />
         <origin xyz="0 0 0" />
         <inertia ixx="0.00000001"

File: pandora_sensors_description/urdf/kinect_camera.urdf.xacro (robot description, xacro)
@@ -5,17 +5,18 @@
     <link name="kinect_link" >
       <inertial>
-        <origin xyz="-0.02891 -0.00024 0.00037"
+        <origin xyz="0.0023 -0.00024 0.01818"
                 rpy="0 0 0" />
-        <mass value="0.1" />
-        <inertia ixx="0.0004075"
+        <mass value="0.226796185" />
+        <inertia ixx="1.4641E-3"
                  ixy="0.0"
                  ixz="0.0"
-                 iyy="0.0004075"
+                 iyy="9.2532E-5"
                  iyz="0.0"
-                 izz="0.0004075" /><!-- FIXME -->
+                 izz="1.5077E-3" /><!-- FIXME -->
       </inertial>
       <collision name="collision" >
+        <origin xyz="0.0 0.0 0.018" />
         <geometry>
-          <box size="0.073000 0.276000 0.072000" />
+          <box size="0.079 0.295 0.055" />
         </geometry>
       </collision>
@@ -106,5 +107,5 @@
         <parent link="kinect_base_link" />
         <child link="kinect_link" />
-        <origin xyz="0.0 0.0 0.02825"
+        <origin xyz="0.024 0.0 0.02825"
                 rpy="0.0 0.0 0.0" />
         <axis xyz="0 0 1" />
@@ -120,5 +121,5 @@
         <parent link="kinect_base_link" />
         <child link="kinect_link" />
-        <origin xyz="0.0 0.0 0.02825"
+        <origin xyz="0.024 0.0 0.02825"
                 rpy="0.0 0.0 0.0" />
       </joint>

File: pandora_sensors_description/urdf/microphone_sensor.urdf.xacro (robot description, xacro)
@@ -5,13 +5,13 @@
     <link name="microphone_link" >
       <inertial>
-        <origin xyz="0.008 0.0 0.0"
+        <origin xyz="0.005 0.0 0.0"
                 rpy="0 0 0" />
-        <mass value="0.1" />
-        <inertia ixx="1"
+        <mass value="0.005" />
+        <inertia ixx="2.1208E-7"
                  ixy="0"
                  ixz="0"
-                 iyy="1"
+                 iyy="4.033E-7"
                  iyz="0"
-                 izz="1" /><!-- FIXME -->
+                 izz="2.1208E-7" />
       </inertial>
       <visual name="visual" >
@@ -23,8 +23,7 @@
       </visual>
       <collision name="collision" >
-        <origin xyz="0 0 0"
-                rpy="0 0 0" />
+        <origin xyz="0.007 0.0 0.0" />
         <geometry>
-          <box size="0.01 0.01 0.01" />
+          <box size="0.025 0.025 0.025" />
         </geometry>
       </collision>

File: pandora_sensors_description/urdf/sonar_sensor.urdf.xacro (robot description, xacro)
@@ -11,13 +11,13 @@
     <link name="${name}_sonar_link" >
       <inertial>
-        <origin xyz="0.008 0.0 0.0"
+        <origin xyz="0.005 0.0 0.0"
                 rpy="0 0 0" />
-        <mass value="0.1" />
-        <inertia ixx="1.0"
+        <mass value="0.010" />
+        <inertia ixx="4.2416E-7"
                  ixy="0.0"
                  ixz="0.0"
-                 iyy="1.0"
+                 iyy="2.0166E-6"
                  iyz="0.0"
-                 izz="1.0" /><!-- FIXME -->
+                 izz="1.6341E-6" />
       </inertial>
       <visual name="visual" >
@@ -27,6 +27,7 @@
       </visual>
       <collision name="collision" >
+        <origin xyz="0.007 0.0 0.0" />
         <geometry>
-            <box size="0.01 0.01 0.01" />
+          <box size="0.025 0.05 0.025" />
         </geometry>
       </collision>

File: pandora_sensors_description/urdf/thermal_sensor.urdf.xacro (robot description, xacro)
@@ -5,13 +5,13 @@
     <link name="${prefix_y}_thermal_link" >
       <inertial>
-        <origin xyz="0.008 0.0 0.0"
+        <origin xyz="0.005 0.0 0.0"
                 rpy="0 0 0" />
-        <mass value="0.1" />
-        <inertia ixx="1.0"
-                 ixy="0.0"
-                 ixz="0.0"
-                 iyy="1.0"
-                 iyz="0.0"
-                 izz="1.0" /><!-- FIXME -->
+        <mass value="0.005" />
+        <inertia ixx="2.1208E-7"
+                 ixy="0"
+                 ixz="0"
+                 iyy="4.033E-7"
+                 iyz="0"
+                 izz="2.1208E-7" />
       </inertial>
       <visual name="visual" >
@@ -21,6 +21,7 @@
       </visual>
       <collision name="collision" >
+        <origin xyz="0.007 0.0 0.0" />
         <geometry>
-          <box size="0.01 0.01 0.01" />
+          <box size="0.025 0.025 0.025" />
         </geometry>
       </collision>

Commit message: Add all joint limits to config file.

File: pandora_robots_description/urdf/gears/config/gears_configurations.xacro (robot description, xacro)
@@ -67,10 +67,22 @@
   <xacro:property name="wheel_min_depth" value="0.001" />
   <!-- ==================================================================== -->
-  <xacro:property name="linear_elevator_joint_max_limit" value="0.0" />
-  <xacro:property name="linear_head_pitch_joint_max_limit" value="0.0" /> <!-- FIXME -->
-  <xacro:property name="linear_head_yaw_joint_max_limit" value="0.0" /> <!-- FIXME -->
-  <!-- TODO : Add limits for sensors -->
+  <xacro:property name="side_joint_damping" value="0.0" />
+  <!-- ==================================================================== -->
+  <xacro:property name="side_joint_min_limit" value="-0.785" />
   <xacro:property name="side_joint_max_limit" value="0.785" />
-  <xacro:property name="side_joint_damping" value="0.0" />
+  <xacro:property name="linear_elevator_joint_min_limit" value="0.0" />
+  <xacro:property name="linear_elevator_joint_max_limit" value="0.23" />
+  <xacro:property name="linear_head_pitch_joint_min_limit" value="-1.57" /> <!--FIXME-->
+  <xacro:property name="linear_head_pitch_joint_max_limit" value="1.57" /> <!--FIXME-->
+  <xacro:property name="linear_head_yaw_joint_min_limit" value="-1.57" /> <!--FIXME-->
+  <xacro:property name="linear_head_yaw_joint_max_limit" value="1.57" /> <!--FIXME-->
+  <xacro:property name="laser_roll_joint_min_limit" value="-1.57" /> <!--FIXME-->
+  <xacro:property name="laser_roll_joint_max_limit" value="1.57" /> <!--FIXME-->
+  <xacro:property name="laser_pitch_joint_min_limit" value="-1.57" /> <!--FIXME-->
+  <xacro:property name="laser_pitch_joint_max_limit" value="1.57" /> <!--FIXME-->
+  <xacro:property name="kinect_pitch_joint_min_limit" value="-1.57" /> <!--FIXME-->
+  <xacro:property name="kinect_pitch_joint_max_limit" value="1.57" /> <!--FIXME-->
+  <xacro:property name="kinect_yaw_joint_min_limit" value="-1.57" /> <!--FIXME-->
+  <xacro:property name="kinect_yaw_joint_max_limit" value="1.57" /> <!--FIXME-->
   <!-- ==================================================================== -->
   <xacro:property name="max_robot_linear_velocity" value="2.0" />

File: pandora_robots_description/urdf/gears/config/gears_physics.gazebo.xacro (robot description, xacro)
@@ -178,5 +178,5 @@
     <!-- <dynamics damping="0.0"
                    friction="0.0" /> -->
-    <limit lower="0"
+    <limit lower="${linear_elevator_joint_min_limit}"
            upper="${linear_elevator_joint_max_limit}"
            effort="1000.0"
@@ -194,5 +194,5 @@
     <!-- <dynamics damping="0.0"
                    friction="0.0" /> -->
-    <limit lower="-${linear_head_pitch_joint_max_limit}"
+    <limit lower="${linear_head_pitch_joint_min_limit}"
            upper="${linear_head_pitch_joint_max_limit}"
            effort="300.0"
@@ -210,5 +210,5 @@
     <!-- <dynamics damping="0.0"
                    friction="0.0" /> -->
-    <limit lower="-${linear_head_yaw_joint_max_limit}"
+    <limit lower="${linear_head_yaw_joint_min_limit}"
            upper="${linear_head_yaw_joint_max_limit}"
            effort="300.0"
@@ -226,5 +226,5 @@
     <dynamics damping="${side_joint_damping}" />
          <!-- friction="0.0" /> -->
-    <limit lower="-${side_joint_max_limit}"
+    <limit lower="${side_joint_min_limit}"
            upper="${side_joint_max_limit}"
            effort="100.0"

File: pandora_robots_description/urdf/gears/gazebo/sensors.xacro (robot description, xacro)
@@ -15,4 +15,17 @@
   <xacro:include filename="$(find pandora_sensors_description)/urdf/microphone_sensor.urdf.xacro" />
   <!-- ==================================================================== -->
+<!-- Hokuyo Laser ######################################################### -->
+  <xacro:macro name="hokuyo_laser_sensor" >
+    <!-- ================================================================== -->
+    <xacro:hokuyo_caster parent="${base_link_name}_link"
+                         roll_min_limit="${laser_roll_joint_min_limit}"
+                         roll_max_limit="${laser_roll_joint_max_limit}"
+                         pitch_min_limit="${laser_pitch_joint_min_limit}"
+                         pitch_max_limit="${laser_pitch_joint_max_limit}" >
+      <origin xyz="0.1894 0.0 0.09679"
+              rpy="${zero}" />
+    </xacro:hokuyo_caster>
+    <!-- ================================================================== -->
+  </xacro:macro>
 <!-- Kinect ############################################################### -->
   <xacro:macro name="kinect_sensor"
@@ -20,17 +33,12 @@
     <!-- ================================================================== -->
     <xacro:kinect_caster parent="${linear_elevator_link_name}_link"
-                         control="${control}" >
+                         control="${control}"
+                         pitch_min_limit="${kinect_pitch_joint_min_limit}"
+                         pitch_max_limit="${kinect_pitch_joint_max_limit}"
+                         yaw_min_limit="${kinect_yaw_joint_min_limit}"
+                         yaw_max_limit="${kinect_yaw_joint_max_limit}" >
       <origin xyz="0.05148 0.01239 0.19742"
               rpy="${zero}" />
     </xacro:kinect_caster>
-    <!-- ================================================================== -->
-  </xacro:macro>
-<!-- Hokuyo Laser ######################################################### -->
-  <xacro:macro name="hokuyo_laser_sensor" >
-    <!-- ================================================================== -->
-    <xacro:hokuyo_caster parent="${base_link_name}_link" >
-      <origin xyz="0.1894 0.0 0.09679"
-              rpy="${zero}" />
-    </xacro:hokuyo_caster>
     <!-- ================================================================== -->
   </xacro:macro>

File: pandora_robots_description/urdf/gears/gears.urdf.xacro (robot description, xacro)
@@ -144,5 +144,5 @@
     <!-- ================================================================== -->
     <xacro:if value="${enable_thermal_sensors}" >
-       <xacro:thermal_sensors />
+      <xacro:thermal_sensors />
     </xacro:if>
     <!-- ================================================================== -->

File: pandora_sensors_description/urdf/hokuyo_utm_30lx.urdf.xacro (robot description, xacro)
@@ -2,5 +2,10 @@
 <robot xmlns:xacro="http://ros.org/wiki/xacro" >
   <xacro:macro name="hokuyo_caster"
-               params="parent *origin" >
+               params="parent
+                       roll_min_limit
+                       roll_max_limit
+                       pitch_min_limit
+                       pitch_max_limit
+                       *origin" >
     <link name="laser_link" >
       <inertial>
@@ -90,8 +95,8 @@
       <xacro:insert_block name="origin" />
       <axis xyz="1 0 0" />
-      <limit lower="-1.57"
-             upper="1.57"
+      <limit lower="${roll_min_limit}"
+             upper="${roll_max_limit}"
              effort="300"
-             velocity="100.0" /><!--FIXME-->
+             velocity="100.0" />
     </joint>
     <joint name="laser_pitch_joint"
@@ -102,8 +107,8 @@
               rpy="0 0 0" />
       <axis xyz="0 1 0" />
-      <limit lower="-1.57"
-             upper="1.57"
+      <limit lower="${pitch_min_limit}"
+             upper="${pitch_max_limit}"
              effort="300"
-             velocity="100.0" /><!--FIXME-->
+             velocity="100.0" />
     </joint>
   </xacro:macro>

File: pandora_sensors_description/urdf/kinect_camera.urdf.xacro (robot description, xacro)
@@ -2,5 +2,11 @@
 <robot xmlns:xacro="http://ros.org/wiki/xacro" >
   <xacro:macro name="kinect_caster"
-               params="parent control *origin" >
+               params="parent
+                       control
+                       pitch_min_limit
+                       pitch_max_limit
+                       yaw_min_limit
+                       yaw_max_limit
+                       *origin" >
     <link name="kinect_link" >
       <inertial>
@@ -88,8 +94,8 @@
         <xacro:insert_block name="origin" />
         <axis xyz="0 1 0" />
-        <limit lower="-1.57"
-               upper="1.57"
+        <limit lower="${pitch_min_limit}"
+               upper="${pitch_max_limit}"
                effort="300"
-               velocity="100.0" /><!--FIXME-->
+               velocity="100.0" />
       </joint>
     </xacro:if>
@@ -110,8 +116,8 @@
                 rpy="0.0 0.0 0.0" />
         <axis xyz="0 0 1" />
-        <limit lower="-1.57"
-               upper="1.57"
+        <limit lower="${yaw_min_limit}"
+               upper="${yaw_max_limit}"
                effort="300"
-               velocity="100.0" /><!--FIXME-->
+               velocity="100.0" />
       </joint>
     </xacro:if>
