Commit message: Fix colors.

File: pandora_robots_description/urdf/gears/config/gears_configurations.xacro (robot description, xacro)
@@ -19,6 +19,6 @@
   <!-- Sensors ============================================================ -->
   <xacro:property name="enable_sensors" value="true" />
+    <xacro:property name="enable_hokuyo_laser_sensor" value="true" />
     <xacro:property name="enable_kinect_sensor" value="true" />
-    <xacro:property name="enable_hokuyo_laser_sensor" value="true" />
     <xacro:property name="enable_sonar_sensors" value="true" />
     <xacro:property name="enable_thermal_sensors" value="true" />
@@ -92,4 +92,5 @@
   <!-- ==================================================================== -->
   <xacro:property name="max_robot_linear_acceleration" value="1.0" />
+  <xacro:property name="max_robot_angular_acceleration" value="0.2" />
   <xacro:property name="max_kinect_angular_acceleration" value="0.0" />
   <xacro:property name="max_laser_angular_acceleration" value="0.0" />

File: pandora_robots_description/urdf/gears/gears.urdf.xacro (robot description, xacro)
@@ -125,4 +125,8 @@
   <xacro:if value="${enable_sensors}" >
     <!-- ================================================================== -->
+    <xacro:if value="${enable_hokuyo_laser_sensor}" >
+      <xacro:hokuyo_laser_sensor />
+    </xacro:if>
+    <!-- ================================================================== -->
     <xacro:if value="${enable_kinect_sensor}" >
       <xacro:if value="$(arg real)" >
@@ -132,8 +136,4 @@
         <xacro:kinect_sensor control="$(arg control)" />
       </xacro:unless>
-    </xacro:if>
-    <!-- ================================================================== -->
-    <xacro:if value="${enable_hokuyo_laser_sensor}" >
-      <xacro:hokuyo_laser_sensor />
     </xacro:if>
     <!-- ================================================================== -->
@@ -178,12 +178,12 @@
       <xacro:if value="${enable_sensors}" >
         <!-- ============================================================== -->
+        <xacro:if value="${enable_hokuyo_laser_sensor}" >
+          <xacro:sensor_transmission sensor="laser" rotation="roll" />
+          <xacro:sensor_transmission sensor="laser" rotation="pitch" />
+        </xacro:if>
+        <!-- ============================================================== -->
         <xacro:if value="${enable_kinect_sensor}" >
           <xacro:sensor_transmission sensor="kinect" rotation="pitch" />
           <xacro:sensor_transmission sensor="kinect" rotation="yaw" />
-        </xacro:if>
-        <!-- ============================================================== -->
-        <xacro:if value="${enable_hokuyo_laser_sensor}" >
-          <xacro:sensor_transmission sensor="laser" rotation="roll" />
-          <xacro:sensor_transmission sensor="laser" rotation="pitch" />
         </xacro:if>
         <!-- ============================================================== -->
@@ -205,8 +205,4 @@
       </xacro:if>
       <!-- ================================================================ -->
-      <xacro:if value="${enable_pandora_p3d_plugin}" >
-        <xacro:pandora_p3d_plugin />
-      </xacro:if>
-      <!-- ================================================================ -->
       <xacro:if value="$(arg control)" >
         <xacro:if value="$(arg interface)" >
@@ -218,4 +214,8 @@
                                            ns="control" />
         </xacro:unless>
+      </xacro:if>
+      <!-- ================================================================ -->
+      <xacro:if value="${enable_pandora_p3d_plugin}" >
+        <xacro:pandora_p3d_plugin />
       </xacro:if>
       <!-- ================================================================ -->

Commit message: Make all revolute joints fixed when ros control is not enabled.

File: pandora_robots_description/urdf/gears/config/gears_configurations.xacro (robot description, xacro)
@@ -30,5 +30,5 @@
     <xacro:property name="enable_pandora_p3d_plugin" value="false" />
     <xacro:property name="enable_ros_imu_plugin" value="false" />
-    <xacro:property name="enable_pandora_imu_stabilizer_plugin" value="true" />
+    <xacro:property name="enable_pandora_imu_stabilizer_plugin" value="false" />
   <!-- SDF Physics ======================================================== -->
   <xacro:property name="enable_sdf_physics" value="true" />

File: pandora_robots_description/urdf/gears/gazebo/sensors.xacro (robot description, xacro)
@@ -16,7 +16,9 @@
   <!-- ==================================================================== -->
 <!-- Hokuyo Laser ######################################################### -->
-  <xacro:macro name="hokuyo_laser_sensor" >
+  <xacro:macro name="hokuyo_laser_sensor"
+               params="control" >
     <!-- ================================================================== -->
     <xacro:hokuyo_caster parent="${base_link_name}_link"
+                         control="${control}"
                          roll_min_limit="${laser_roll_joint_min_limit}"
                          roll_max_limit="${laser_roll_joint_max_limit}"

File: pandora_robots_description/urdf/gears/gears.urdf.xacro (robot description, xacro)
@@ -47,9 +47,19 @@
     <!-- ================================================================== -->
     <xacro:if value="${enable_linear_elevator_joint}" >
-      <xacro:linear_elevator_joint />
+      <xacro:if value="$(arg real)" >
+        <xacro:linear_elevator_joint control="true" />
+      </xacro:if>
+      <xacro:unless value="$(arg real)" >
+        <xacro:linear_elevator_joint control="$(arg control)" />
+      </xacro:unless>
     </xacro:if>
     <!-- ================================================================== -->
     <xacro:if value="${enable_linear_head_joints}" >
-      <xacro:linear_head_joints />
+      <xacro:if value="$(arg real)" >
+        <xacro:linear_head_joints control="true" />
+      </xacro:if>
+      <xacro:unless value="$(arg real)" >
+        <xacro:linear_head_joints control="$(arg control)" />
+      </xacro:unless>
     </xacro:if>
     <!-- ================================================================== -->
@@ -126,5 +136,10 @@
     <!-- ================================================================== -->
     <xacro:if value="${enable_hokuyo_laser_sensor}" >
-      <xacro:hokuyo_laser_sensor />
+      <xacro:if value="$(arg real)" >
+        <xacro:hokuyo_laser_sensor control="true" />
+      </xacro:if>
+      <xacro:unless value="$(arg real)" >
+        <xacro:hokuyo_laser_sensor control="$(arg control)" />
+      </xacro:unless>
     </xacro:if>
     <!-- ================================================================== -->

File: pandora_robots_description/urdf/gears/model/joints.urdf.xacro (robot description, xacro)
@@ -2,34 +2,67 @@
 <robot xmlns:xacro="http://ros.org/wiki/xacro" >
 <!-- Linear Elevator ###################################################### -->
-  <xacro:macro name="linear_elevator_joint" >
-    <!-- ================================================================== -->
-    <joint name="${linear_elevator_joint_name}_joint"
-           type="${linear_elevator_joint_type}" >
-      <parent link="${base_link_name}_link" />
-      <child link="${linear_elevator_link_name}_link" />
-      <xacro:linear_elevator_joint_origin />
-      <xacro:linear_elevator_joint_urdf_physics />
-    </joint>
-    <!-- ================================================================== -->
+  <xacro:macro name="linear_elevator_joint"
+               params="control" >
+    <xacro:if value="${control}" >
+      <!-- ================================================================ -->
+      <joint name="${linear_elevator_joint_name}_joint"
+             type="${linear_elevator_joint_type}" >
+        <parent link="${base_link_name}_link" />
+        <child link="${linear_elevator_link_name}_link" />
+        <xacro:linear_elevator_joint_origin />
+        <xacro:linear_elevator_joint_urdf_physics />
+      </joint>
+      <!-- ================================================================ -->
+    </xacro:if>
+    <xacro:unless value="${control}" >
+      <!-- ================================================================ -->
+      <joint name="${linear_elevator_joint_name}_joint"
+             type="fixed" >
+        <parent link="${base_link_name}_link" />
+        <child link="${linear_elevator_link_name}_link" />
+        <xacro:linear_elevator_joint_origin />
+      </joint>
+      <!-- ================================================================ -->
+    </xacro:unless>
   </xacro:macro>
 <!-- Linear Head  ######################################################### -->
-  <xacro:macro name="linear_head_joints" >
-    <!-- ================================================================== -->
-    <joint name="${linear_head_pitch_joint_name}_joint"
-           type="${linear_head_pitch_joint_type}" >
-      <parent link="${linear_elevator_link_name}_link" />
-      <child link="${linear_head_link_name}_base_link" />
-      <xacro:linear_head_pitch_joint_origin />
-      <xacro:linear_head_pitch_joint_urdf_physics />
-    </joint>
-    <!-- ================================================================== -->
-    <joint name="${linear_head_yaw_joint_name}_joint"
-           type="${linear_head_yaw_joint_type}" >
-      <parent link="${linear_head_link_name}_base_link" />
-      <child link="${linear_head_link_name}_link" />
-      <xacro:linear_head_yaw_joint_origin />
-      <xacro:linear_head_yaw_joint_urdf_physics />
-    </joint>
-    <!-- ================================================================== -->
+  <xacro:macro name="linear_head_joints"
+               params="control" >
+    <xacro:if value="${control}" >
+      <!-- ================================================================ -->
+      <joint name="${linear_head_pitch_joint_name}_joint"
+             type="${linear_head_pitch_joint_type}" >
+        <parent link="${linear_elevator_link_name}_link" />
+        <child link="${linear_head_link_name}_base_link" />
+        <xacro:linear_head_pitch_joint_origin />
+        <xacro:linear_head_pitch_joint_urdf_physics />
+      </joint>
+      <!-- ================================================================ -->
+      <joint name="${linear_head_yaw_joint_name}_joint"
+             type="${linear_head_yaw_joint_type}" >
+        <parent link="${linear_head_link_name}_base_link" />
+        <child link="${linear_head_link_name}_link" />
+        <xacro:linear_head_yaw_joint_origin />
+        <xacro:linear_head_yaw_joint_urdf_physics />
+      </joint>
+      <!-- ================================================================ -->
+    </xacro:if>
+    <xacro:unless value="${control}" >
+      <!-- ================================================================ -->
+      <joint name="${linear_head_pitch_joint_name}_joint"
+             type="fixed" >
+        <parent link="${linear_elevator_link_name}_link" />
+        <child link="${linear_head_link_name}_base_link" />
+        <xacro:linear_head_pitch_joint_origin />
+      </joint>
+      <!-- ================================================================ -->
+      <joint name="${linear_head_yaw_joint_name}_joint"
+             type="fixed" >
+        <parent link="${linear_head_link_name}_base_link" />
+        <child link="${linear_head_link_name}_link" />
+        <xacro:linear_head_yaw_joint_origin />
+      </joint>
+      <!-- ================================================================ -->
+    </xacro:unless>
   </xacro:macro>
 <!-- Side ################################################################# -->

File: pandora_sensors_description/urdf/hokuyo_utm_30lx.urdf.xacro (robot description, xacro)
@@ -3,4 +3,5 @@
   <xacro:macro name="hokuyo_caster"
                params="parent
+                       control
                        roll_min_limit
                        roll_max_limit
@@ -89,27 +90,50 @@
       </collision>
     </link>
-    <joint name="laser_roll_joint"
-           type="revolute" >
-      <parent link="${parent}" />
-      <child link="hokuyo_base_link" />
-      <xacro:insert_block name="origin" />
-      <axis xyz="1 0 0" />
-      <limit lower="${roll_min_limit}"
-             upper="${roll_max_limit}"
-             effort="50"
-             velocity="50.0" />
-    </joint>
-    <joint name="laser_pitch_joint"
-           type="revolute" >
-      <parent link="hokuyo_base_link" />
-      <child link="laser_link" />
-      <origin xyz="0.013 0 0.02301"
-              rpy="0 0 0" />
-      <axis xyz="0 1 0" />
-      <limit lower="${pitch_min_limit}"
-             upper="${pitch_max_limit}"
-             effort="50"
-             velocity="50.0" />
-    </joint>
+    <!-- Roll Joint ########################################################-->
+    <xacro:if value="${control}" >
+      <joint name="laser_roll_joint"
+             type="revolute" >
+        <parent link="${parent}" />
+        <child link="hokuyo_base_link" />
+        <xacro:insert_block name="origin" />
+        <axis xyz="1 0 0" />
+        <limit lower="${roll_min_limit}"
+               upper="${roll_max_limit}"
+               effort="50"
+               velocity="50.0" />
+      </joint>
+    </xacro:if>
+    <xacro:unless value="${control}" >
+      <joint name="laser_roll_joint"
+             type="fixed" >
+        <parent link="${parent}" />
+        <child link="hokuyo_base_link" />
+        <xacro:insert_block name="origin" />
+      </joint>
+    </xacro:unless>
+    <!-- Pitch Joint #######################################################-->
+    <xacro:if value="${control}" >
+      <joint name="laser_pitch_joint"
+             type="revolute" >
+        <parent link="hokuyo_base_link" />
+        <child link="laser_link" />
+        <origin xyz="0.013 0 0.02301"
+                rpy="0 0 0" />
+        <axis xyz="0 1 0" />
+        <limit lower="${pitch_min_limit}"
+               upper="${pitch_max_limit}"
+               effort="50"
+               velocity="50.0" />
+      </joint>
+    </xacro:if>
+    <xacro:unless value="${control}" >
+      <joint name="laser_pitch_joint"
+             type="fixed" >
+        <parent link="hokuyo_base_link" />
+        <child link="laser_link" />
+        <origin xyz="0.013 0 0.02301"
+                rpy="0 0 0" />
+      </joint>
+    </xacro:unless>
   </xacro:macro>
 </robot>

File: pandora_sensors_description/urdf/kinect_camera.urdf.xacro (robot description, xacro)
@@ -87,4 +87,5 @@
       </collision>
     </link>
+    <!-- Pitch Joint #######################################################-->
     <xacro:if value="${control}" >
       <joint name="kinect_pitch_joint"
@@ -108,4 +109,5 @@
       </joint>
     </xacro:unless>
+    <!-- Yaw Joint #########################################################-->
     <xacro:if value="${control}" >
       <joint name="kinect_yaw_joint"
