Commit message: Update all origins and inertia of urdf elements.

File: pandora_robots_description/urdf/gears/config/properties/inertia_tensors.xacro (robot description, xacro)
@@ -12,10 +12,10 @@
   <!-- ==================================================================== -->
   <xacro:macro name="linear_elevator_link_inertia" >
-    <inertia ixx="0.015755"
-             ixy="-0.00089486"
-             ixz="-0.0017447"
-             iyy="0.014259"
-             iyz="0.0037284"
-             izz="0.0035941" /><!--TODO-->
+    <inertia ixx="0.0097139"
+             ixy="-0.00039516"
+             ixz="-0.00086264"
+             iyy="0.0095873"
+             iyz="0.0012764"
+             izz="0.0017829" />
   </xacro:macro>
   <!-- ==================================================================== -->
@@ -30,10 +30,10 @@
   <!-- ==================================================================== -->
   <xacro:macro name="linear_head_link_inertia" >
-    <inertia ixx="0.01"
-             ixy="0.01"
-             ixz="0.01"
-             iyy="0.01"
-             iyz="0.01"
-             izz="0.01" /><!--TODO-->
+    <inertia ixx="0.00030418"
+             ixy="-1.3735E-05"
+             ixz="-2.3947E-05"
+             iyy="0.00015881"
+             iyz="-7.9817E-06"
+             izz="0.00024855" />
   </xacro:macro>
   <!-- ==================================================================== -->

File: pandora_robots_description/urdf/gears/config/properties/joint_offsets.xacro (robot description, xacro)
@@ -8,11 +8,11 @@
   <!-- ==================================================================== -->
   <xacro:macro name="linear_head_pitch_joint_origin" >
-    <origin xyz="0.0 0.0 0.0"
-            rpy="${zero}" /><!--TODO-->
+    <origin xyz="-0.0145 0.1056 0.35787"
+            rpy="${zero}" />
   </xacro:macro>
   <!-- ==================================================================== -->
   <xacro:macro name="linear_head_yaw_joint_origin" >
-    <origin xyz="0.0 0.0 0.0"
-            rpy="${zero}" /><!--TODO Translate because of second servo -->
+    <origin xyz="0.0 0.0 0.021"
+            rpy="${zero}" />
   </xacro:macro>
   <!-- ==================================================================== -->

File: pandora_robots_description/urdf/gears/config/properties/link_offsets.xacro (robot description, xacro)
@@ -9,6 +9,6 @@
   <!-- ==================================================================== -->
   <xacro:macro name="linear_elevator_link_inertial_origin" >
-    <origin xyz="0.01229 0.026011 0.26669"
-            rpy="${zero}" /><!--TODO-->
+    <origin xyz="0.017561 0.0109 0.24001"
+            rpy="${zero}" />
   </xacro:macro>
   <!-- ==================================================================== -->
@@ -18,6 +18,6 @@
   <!-- ==================================================================== -->
   <xacro:macro name="linear_head_link_inertial_origin" >
-    <origin xyz="0.0 0.0 0.0"
-            rpy="${zero}" /><!--TODO-->
+    <origin xyz="-0.0027417 0.0050805 0.037323"
+            rpy="${zero}" />
   </xacro:macro>
   <!-- ==================================================================== -->

File: pandora_robots_description/urdf/gears/config/properties/masses.xacro (robot description, xacro)
@@ -7,5 +7,5 @@
   <!-- ==================================================================== -->
   <xacro:macro name="linear_elevator_link_mass" >
-    <mass value="1.0889" /><!--TODO-->
+    <mass value="0.92399" />
   </xacro:macro>
   <!-- ==================================================================== -->
@@ -15,5 +15,5 @@
   <!-- ==================================================================== -->
   <xacro:macro name="linear_head_link_mass" >
-    <mass value="0.1" /><!--TODO-->
+    <mass value="0.16491" />
   </xacro:macro>
   <!-- ==================================================================== -->

File: pandora_robots_description/urdf/gears/gazebo/sensors.xacro (robot description, xacro)
@@ -21,5 +21,5 @@
     <xacro:kinect_caster parent="${linear_elevator_link_name}_link"
                          control="${control}" >
-      <origin xyz="0.12252 0.01239 0.24402"
+      <origin xyz="0.09144 0.01239 0.19742"
               rpy="${zero}" />
     </xacro:kinect_caster>
@@ -31,5 +31,5 @@
     <xacro:hokuyo_caster parent="${base_link_name}_link" >
       <origin xyz="0.2 0.0 0.15"
-              rpy="${zero}" />
+              rpy="${zero}" /><!-- FIXME -->
     </xacro:hokuyo_caster>
     <!-- ================================================================== -->
@@ -51,18 +51,18 @@
     <xacro:thermal_caster parent="${linear_head_link_name}_link"
                           prefix_y="middle" >
-      <origin xyz="0.0 0.0 0.0"
-              rpy="${zero}" /><!--TODO-->
+      <origin xyz="0.01039 0.00007 0.04532"
+              rpy="${zero}" />
     </xacro:thermal_caster>
     <!-- ================================================================== -->
     <xacro:thermal_caster parent="${linear_head_link_name}_link"
                           prefix_y="right" >
-      <origin xyz="0.0 -0.02 0.0"
-              rpy="${zero}" /><!--TODO-->
+      <origin xyz="-0.00128 0.04774 0.03108"
+              rpy="0 0 ${PI_3}" />
     </xacro:thermal_caster>
     <!-- ================================================================== -->
     <xacro:thermal_caster parent="${linear_head_link_name}_link"
                           prefix_y="left" >
-      <origin xyz="0.0 0.02 0.0"
-              rpy="${zero}" /><!--TODO-->
+      <origin xyz="-0.00128 -0.04774 0.03108"
+              rpy="0 0 ${ - PI_3}" />
     </xacro:thermal_caster>
     <!-- ================================================================== -->
@@ -72,6 +72,6 @@
     <!-- ================================================================== -->
     <xacro:co2_caster parent="${linear_head_link_name}_link" >
-      <origin xyz="0.0 0.02 -0.02"
-              rpy="${zero}" /><!--TODO-->
+      <origin xyz="0.01039 -0.01556 0.02386"
+              rpy="${zero}" />
     </xacro:co2_caster>
     <!-- ================================================================== -->
@@ -81,6 +81,6 @@
     <!-- ================================================================== -->
     <xacro:microphone_caster parent="${linear_head_link_name}_link" >
-      <origin xyz="0.0 -0.02 -0.02"
-              rpy="${zero}" /><!--TODO-->
+      <origin xyz="0.01039 0.01556 0.02386"
+              rpy="${zero}" />
     </xacro:microphone_caster>
     <!-- ================================================================== -->

File: pandora_sensors_description/urdf/kinect_camera.urdf.xacro (robot description, xacro)
@@ -106,6 +106,6 @@
         <parent link="kinect_base_link" />
         <child link="kinect_link" />
-        <origin xyz="0 0 0"
-                rpy="0 0 0" />
+        <origin xyz="0.0 0.0 0.02825"
+                rpy="0.0 0.0 0.0" />
         <axis xyz="0 0 1" />
         <limit lower="-1.57"
@@ -120,6 +120,6 @@
         <parent link="kinect_base_link" />
         <child link="kinect_link" />
-        <origin xyz="0 0 0"
-                rpy="0 0 0" />
+        <origin xyz="0.0 0.0 0.02825"
+                rpy="0.0 0.0 0.0" />
       </joint>
     </xacro:unless>

Commit message: Add new meshes for laser and motors and fix all positions.

File: pandora_robots_description/urdf/gears/config/properties/inertia_tensors.xacro (robot description, xacro)
@@ -26,5 +26,5 @@
              iyy="0.00000001"
              iyz="0.00000001"
-             izz="0.00000001" />
+             izz="0.00000001" /><!--FIXME-->
   </xacro:macro>
   <!-- ==================================================================== -->

File: pandora_robots_description/urdf/gears/config/properties/joint_offsets.xacro (robot description, xacro)
@@ -8,10 +8,10 @@
   <!-- ==================================================================== -->
   <xacro:macro name="linear_head_pitch_joint_origin" >
-    <origin xyz="-0.0145 0.1056 0.35787"
+    <origin xyz="-0.0145 0.0686 0.35787"
             rpy="${zero}" />
   </xacro:macro>
   <!-- ==================================================================== -->
   <xacro:macro name="linear_head_yaw_joint_origin" >
-    <origin xyz="0.0 0.0 0.021"
+    <origin xyz="0.0 0.037 0.021"
             rpy="${zero}" />
   </xacro:macro>

File: pandora_robots_description/urdf/gears/config/properties/link_offsets.xacro (robot description, xacro)
@@ -4,32 +4,27 @@
   <!-- ==================================================================== -->
   <xacro:macro name="base_link_inertial_origin" >
-    <origin xyz="-0.010032 -0.0067035 0.16451"
-            rpy="${zero}" />
+    <origin xyz="-0.010032 -0.0067035 0.16451" />
   </xacro:macro>
   <!-- ==================================================================== -->
   <xacro:macro name="linear_elevator_link_inertial_origin" >
-    <origin xyz="0.017561 0.0109 0.24001"
-            rpy="${zero}" />
+    <origin xyz="0.017561 0.0109 0.24001" />
   </xacro:macro>
   <!-- ==================================================================== -->
   <xacro:macro name="linear_head_base_link_inertial_origin" >
-    <xacro:default_origin />
+    <origin xyz="0.02347 0.0 0.00124" />
   </xacro:macro>
   <!-- ==================================================================== -->
   <xacro:macro name="linear_head_link_inertial_origin" >
-    <origin xyz="-0.0027417 0.0050805 0.037323"
-            rpy="${zero}" />
+    <origin xyz="-0.0027417 0.0050805 0.037323" />
   </xacro:macro>
   <!-- ==================================================================== -->
   <xacro:macro name="side_link_inertial_origin"
                params="reflect_y" >
-    <origin xyz="${ reflect_y * ( -9.2074E-08 ) } ${ reflect_y * ( 0.010782 ) } -0.028501"
-            rpy="${zero}" />
+    <origin xyz="${ reflect_y * ( -9.2074E-08 ) } ${ reflect_y * ( 0.010782 ) } -0.028501" />
   </xacro:macro>
   <!-- ==================================================================== -->
   <xacro:macro name="wheel_link_inertial_origin"
                params="reflect_y" >
-    <origin xyz="${ reflect_y * ( -2.2235E-05 ) } ${ reflect_y * ( -0.00052624 ) } 2.4287E-05"
-            rpy="${zero}" />
+    <origin xyz="${ reflect_y * ( -2.2235E-05 ) } ${ reflect_y * ( -0.00052624 ) } 2.4287E-05" />
   </xacro:macro>
   <!-- ==================================================================== -->
@@ -45,5 +40,6 @@
   <!-- ==================================================================== -->
   <xacro:macro name="linear_head_base_link_visual_origin" >
-    <xacro:default_origin />
+    <origin xyz="${zero}"
+            rpy="0.0 0.0 ${PI_2}" />
   </xacro:macro>
   <!-- ==================================================================== -->
@@ -75,5 +71,6 @@
   <!-- ==================================================================== -->
   <xacro:macro name="linear_head_base_link_collision_origin" >
-    <xacro:default_origin />
+    <origin xyz="0.0 0.02347 0.00124"
+            rpy="0.0 0.0 ${PI_2}" />
   </xacro:macro>
   <!-- ==================================================================== -->

File: pandora_robots_description/urdf/gears/config/properties/masses.xacro (robot description, xacro)
@@ -11,5 +11,5 @@
   <!-- ==================================================================== -->
   <xacro:macro name="linear_head_base_link_mass" >
-    <mass value="0.0001" />
+    <mass value="0.0001" /><!--FIXME-->
   </xacro:macro>
   <!-- ==================================================================== -->

File: pandora_robots_description/urdf/gears/config/properties/materials.xacro (robot description, xacro)
@@ -109,9 +109,13 @@
   <!-- ==================================================================== -->
   <material name="base" >
-    <color rgba="${230/255} ${230/255} ${230/255} 0.8" />
+    <color rgba="${10/255} ${10/255} ${10/255} 0.8" />
   </material>
   <!-- ==================================================================== -->
   <material name="linear_elevator" >
     <color rgba="${190/255} ${190/255} ${190/255} 1.0" />
+  </material>
+  <!-- ==================================================================== -->
+  <material name="linear_head_base" >
+    <color rgba="${30/255} ${30/255} ${30/255} 1.0" />
   </material>
   <!-- ==================================================================== -->

File: pandora_robots_description/urdf/gears/config/properties/meshes.xacro (robot description, xacro)
@@ -14,4 +14,10 @@
       <mesh filename="package://pandora_robots_description/meshes/gears/visual/linear_elevator_link.dae" />
       <!-- <mesh filename="package://pandora_robots_description/meshes/gears/collision/linear_elevator_link.stl" /> -->
+    </geometry>
+  </xacro:macro>
+  <!-- ==================================================================== -->
+  <xacro:macro name="linear_head_base_link_visual_mesh" >
+    <geometry>
+      <mesh filename="package://pandora_robots_description/meshes/gears/visual/servo_motor.dae" />
     </geometry>
   </xacro:macro>
@@ -54,4 +60,10 @@
   </xacro:macro>
   <!-- ==================================================================== -->
+  <xacro:macro name="linear_head_base_link_collision_mesh" >
+    <geometry>
+      <box size="0.050 0.032 0.041" />
+    </geometry>
+  </xacro:macro>
+  <!-- ==================================================================== -->
   <xacro:macro name="linear_head_link_collision_mesh" >
     <geometry>

File: pandora_robots_description/urdf/gears/gazebo/sensors.xacro (robot description, xacro)
@@ -21,5 +21,5 @@
     <xacro:kinect_caster parent="${linear_elevator_link_name}_link"
                          control="${control}" >
-      <origin xyz="0.06744 0.01239 0.19742"
+      <origin xyz="0.05148 0.01239 0.19742"
               rpy="${zero}" />
     </xacro:kinect_caster>
@@ -30,6 +30,6 @@
     <!-- ================================================================== -->
     <xacro:hokuyo_caster parent="${base_link_name}_link" >
-      <origin xyz="0.2 0.0 0.15"
-              rpy="${zero}" /><!-- FIXME -->
+      <origin xyz="0.1894 0.0 0.09679"
+              rpy="${zero}" />
     </xacro:hokuyo_caster>
     <!-- ================================================================== -->

File: pandora_robots_description/urdf/gears/model/links.urdf.xacro (robot description, xacro)
@@ -54,13 +54,10 @@
       <visual>
         <xacro:linear_head_base_link_visual_origin />
-        <geometry>
-          <box size="0 0 0" />
-        </geometry>
+        <xacro:linear_head_base_link_visual_mesh />
+        <material name="linear_head_base" />
       </visual>
       <collision>
         <xacro:linear_head_base_link_collision_origin />
-        <geometry>
-          <box size="0 0 0" />
-        </geometry>
+        <xacro:linear_head_base_link_collision_mesh />
       </collision>
     </link>

File: pandora_sensors_description/urdf/hokuyo_utm_30lx.urdf.xacro (robot description, xacro)
@@ -14,22 +14,14 @@
                  izz="0.000162" />
       </inertial>
-      <visual name="visual" >
+      <visual>
         <geometry>
           <mesh filename="package://pandora_sensors_description/meshes/hokuyo_utm_30lx/hokuyo_utm_30lx.dae" />
         </geometry>
       </visual>
-      <collision name="collision-base" >
-        <origin xyz="0 0 -0.0145"
+      <collision>
+        <origin xyz="0 0 0.05299"
                 rpy="0 0 0" />
         <geometry>
-      <box size="0.05 0.05 0.041" />
-        </geometry>
-      </collision>
-      <collision name="collision-top" >
-        <origin xyz="0 0 0.0205"
-                rpy="0 0 0" />
-        <geometry>
-          <cylinder radius="0.021"
-                    length="0.029" />
+          <box size="0.062 0.063 0.116" />
         </geometry>
       </collision>
@@ -38,5 +30,5 @@
       <sensor name="laser"
               type="ray" >
-        <pose>0.01 0 0.0175 0 -0 0</pose>
+        <pose>0.0225 0 0.105 0 0 0</pose>
         <ray>
           <scan>
@@ -68,6 +60,6 @@
     <link name="hokuyo_base_link" >
       <inertial>
-        <mass value="0.0001" />
-        <origin xyz="0 0 0" />
+        <origin xyz="0.013 0.0 0.00951" />
+        <mass value="0.0001" /><!--FIXME-->
         <inertia ixx="0.00000001"
                  ixy="0"
@@ -75,5 +67,5 @@
                  iyy="0.00000001"
                  iyz="0"
-                 izz="0.00000001" />
+                 izz="0.00000001" /><!--FIXME-->
       </inertial>
       <visual>
@@ -81,12 +73,12 @@
                 rpy="0 0 0" />
         <geometry>
-          <box size="0 0 0" />
+          <mesh filename="package://pandora_sensors_description/meshes/hokuyo_utm_30lx/laser_pitch_servo.dae" />
         </geometry>
       </visual>
       <collision>
-        <origin xyz="0 0 0"
+        <origin xyz="0.01285 0.00018 0.00959"
                 rpy="0 0 0" />
         <geometry>
-          <box size="0 0 0" />
+          <box size="0.032 0.038 0.050" />
         </geometry>
       </collision>
@@ -107,5 +99,6 @@
       <parent link="hokuyo_base_link" />
       <child link="laser_link" />
-      <origin xyz="0 0 0" rpy="0 0 0" />
+      <origin xyz="0.013 0 0.02301"
+              rpy="0 0 0" />
       <axis xyz="0 1 0" />
       <limit lower="-1.57"

File: pandora_sensors_description/urdf/kinect_camera.urdf.xacro (robot description, xacro)
@@ -13,5 +13,5 @@
                  iyy="9.2532E-5"
                  iyz="0.0"
-                 izz="1.5077E-3" /><!-- FIXME -->
+                 izz="1.5077E-3" />
       </inertial>
       <collision name="collision" >
@@ -57,6 +57,6 @@
     <link name="kinect_base_link" >
       <inertial>
-        <mass value="0.001" />
-        <origin xyz="0 0 0" />
+        <origin xyz="0.02347 0.0 0.00124" />
+        <mass value="0.0001" /><!--FIXME-->
         <inertia ixx="0.00000001"
                  ixy="0"
@@ -64,5 +64,5 @@
                  iyy="0.00000001"
                  iyz="0"
-                 izz="0.00000001" />
+                 izz="0.00000001" /><!--FIXME-->
       </inertial>
       <visual>
@@ -70,12 +70,12 @@
                 rpy="0 0 0" />
         <geometry>
-          <box size="0 0 0" />
+          <mesh filename="package://pandora_robots_description/meshes/gears/visual/servo_motor.dae" />
         </geometry>
       </visual>
       <collision>
-        <origin xyz="0 0 0"
+        <origin xyz="0.02347 0.0 0.00124"
                 rpy="0 0 0" />
         <geometry>
-          <box size="0 0 0" />
+          <box size="0.050 0.032 0.041" />
         </geometry>
       </collision>
@@ -107,5 +107,5 @@
         <parent link="kinect_base_link" />
         <child link="kinect_link" />
-        <origin xyz="0.024 0.0 0.02825"
+        <origin xyz="0.037 0.0 0.021"
                 rpy="0.0 0.0 0.0" />
         <axis xyz="0 0 1" />
@@ -121,5 +121,5 @@
         <parent link="kinect_base_link" />
         <child link="kinect_link" />
-        <origin xyz="0.024 0.0 0.02825"
+        <origin xyz="0.037 0.0 0.021"
                 rpy="0.0 0.0 0.0" />
       </joint>
