Commit message: Add arg in differential plugin macro to enable joint state publishing.

File: pandora_robots_description/urdf/gears/gazebo/plugins.gazebo.xacro (robot description, xacro)
@@ -2,5 +2,6 @@
 <robot xmlns:xacro="http://ros.org/wiki/xacro" >
 <!-- Differential ######################################################### -->
-  <xacro:macro name="pandora_differential_plugin" >
+  <xacro:macro name="pandora_differential_plugin"
+               params="publish_joint_states" >
     <!-- ================================================================== -->
     <gazebo>
@@ -8,4 +9,5 @@
               filename="libpandora_differential_plugin.so" >
         <robotNamespace>${robot_namespace}</robotNamespace>
+        <publishJointStates>${publish_joint_states}</publishJointStates>
         <baseLink>${base_link_name}_link</baseLink>
         <leftFrontWheelLink>left_front_${wheel_link_name}_link</leftFrontWheelLink>

File: pandora_robots_description/urdf/gears/gears.urdf.xacro (robot description, xacro)
@@ -197,5 +197,10 @@
       <!-- ================================================================ -->
       <xacro:if value="${enable_pandora_differential_plugin}" >
-        <xacro:pandora_differential_plugin />
+        <xacro:if value="$(arg interface)" >
+          <xacro:pandora_differential_plugin publish_joint_states="false" />
+        </xacro:if>
+        <xacro:unless value="$(arg interface)" >
+          <xacro:pandora_differential_plugin publish_joint_states="true" />
+        </xacro:unless>
       </xacro:if>
       <!-- ================================================================ -->
@@ -206,8 +211,10 @@
       <xacro:if value="$(arg control)" >
         <xacro:if value="$(arg interface)" >
-          <xacro:gazebo_ros_control_plugin hw_sim="pandora_gazebo_interface/GazeboInterface" />
+          <xacro:gazebo_ros_control_plugin hw_sim="pandora_gazebo_interface/GazeboInterface"
+                                           ns="control" />
         </xacro:if>
         <xacro:unless value="$(arg interface)" >
-          <xacro:gazebo_ros_control_plugin hw_sim="gazebo_ros_control/DefaultRobotHWSim" />
+          <xacro:gazebo_ros_control_plugin hw_sim="gazebo_ros_control/DefaultRobotHWSim"
+                                           ns="control" />
         </xacro:unless>
       </xacro:if>
