Commit message: Fix meshes' paths.

File: pandora_robots_description/urdf/gears/links/linear/head/base/linear_head_base_link_config.xacro (robot description, xacro)
@@ -33,4 +33,5 @@
     <geometry>
       <mesh filename="package://pandora_robots_description/meshes/gears/visual/linear/head/servo_motor.dae" />
+      <!-- <box size="0.050 0.032 0.041" /> -->
     </geometry>
   </xacro:macro>
@@ -39,4 +40,5 @@
     <geometry>
       <box size="0.050 0.032 0.041" />
+      <!-- <mesh filename="package://pandora_robots_description/meshes/gears/visual/linear/head/servo_motor.dae" /> -->
     </geometry>
   </xacro:macro>

File: pandora_robots_description/urdf/gears/links/linear/head/main/linear_head_main_link_config.xacro (robot description, xacro)
@@ -31,5 +31,5 @@
     <geometry>
       <mesh filename="package://pandora_robots_description/meshes/gears/visual/linear/head/linear_head_main_link.dae" />
-      <!-- <mesh filename="package://pandora_robots_description/meshes/gears/collision/linear/head/linear_head_main_link.dae" /> -->
+      <!-- <mesh filename="package://pandora_robots_description/meshes/gears/collision/linear/head/linear_head_main_link.stl" /> -->
     </geometry>
   </xacro:macro>
@@ -37,5 +37,5 @@
   <xacro:macro name="linear_head_main_link_collision_mesh" >
     <geometry>
-      <mesh filename="package://pandora_robots_description/meshes/gears/collision/linear/head/linear_head_main_link.dae" />
+      <mesh filename="package://pandora_robots_description/meshes/gears/collision/linear/head/linear_head_main_link.stl" />
       <!-- <mesh filename="package://pandora_robots_description/meshes/gears/visual/linear/head/linear_head_main_link.dae" /> -->
     </geometry>

File: pandora_sensors_description/urdf/kinect_camera.urdf.xacro (robot description, xacro)
@@ -76,5 +76,5 @@
                 rpy="0 0 0" />
         <geometry>
-          <mesh filename="package://pandora_robots_description/meshes/gears/visual/servo_motor.dae" />
+          <mesh filename="package://pandora_robots_description/meshes/gears/visual/linear/head/servo_motor.dae" />
         </geometry>
       </visual>
