Commit message: Correct thermal sensors' names.

File: pandora_robots_description/urdf/gears/properties/materials.xacro (robot description, xacro)
@@ -108,5 +108,5 @@
   <!-- ==================================================================== -->
   <material name="base" >
-    <color rgba="${10/255} ${10/255} ${10/255} 0.8" />
+    <color rgba="${0/255} ${0/255} ${0/255} 1.0" />
   </material>
   <!-- ==================================================================== -->
@@ -124,9 +124,9 @@
   <!-- ==================================================================== -->
   <material name="side" >
-    <color rgba="${190/255} ${190/255} ${190/255} 1.0" />
+    <color rgba="${0/255} ${0/255} ${0/255} 1.0" />
   </material>
   <!-- ==================================================================== -->
   <material name="wheel" >
-    <color rgba="${20/255} ${20/255} ${0/255} 0.9" />
+    <color rgba="${5/255} ${5/255} ${0/255} 1.0" />
   </material>
   <!-- ==================================================================== -->

File: pandora_robots_description/urdf/gears/sensors/thermal_sensor.xacro (robot description, xacro)
@@ -17,6 +17,6 @@
     <xacro:thermal_caster parent="linear_head_main_link"
                           prefix_y="left" >
-      <origin xyz="-0.00128 -0.04774 0.03108"
-              rpy="0 0 ${-PI_3}" />
+      <origin xyz="-0.00128 0.04774 0.03108"
+              rpy="0 0 ${PI_3}" />
     </xacro:thermal_caster>
   </xacro:macro>
@@ -25,6 +25,6 @@
     <xacro:thermal_caster parent="linear_head_main_link"
                           prefix_y="right" >
-      <origin xyz="-0.00128 0.04774 0.03108"
-              rpy="0 0 ${PI_3}" />
+      <origin xyz="-0.00128 -0.04774 0.03108"
+              rpy="0 0 ${-PI_3}" />
     </xacro:thermal_caster>
   </xacro:macro>
