Commit message: Correct link meshes' dimensions and joint offsets.

File: pandora_robots_description/urdf/gears/joints/side_joint.urdf.xacro (robot description, xacro)
@@ -10,5 +10,5 @@
       <child link="${prefix_y}_side_link" />
       <!-- ================================================================ -->
-      <origin xyz="0.0 ${ reflect_y * ( 0.110 ) } 0.0"
+      <origin xyz="0.0 ${ reflect_y * ( 0.10314 ) } 0.0"
               rpy="${zero}" />
       <!-- ================================================================ -->

File: pandora_robots_description/urdf/gears/joints/wheel_joint.urdf.xacro (robot description, xacro)
@@ -10,5 +10,5 @@
       <child link="${prefix_y}_${prefix_x}_wheel_link" />
       <!-- ================================================================ -->
-      <origin xyz="${ reflect_x * ( 0.198785 ) } ${ reflect_y * ( 0.110545 ) } -0.052795"
+      <origin xyz="${ reflect_x * ( 0.198785 ) } ${ reflect_y * ( 0.06886 ) } -0.052795"
               rpy="${zero}" />
       <!-- ================================================================ -->

File: pandora_robots_description/urdf/gears/urdf_configurations.xacro (robot description, xacro)
@@ -105,9 +105,9 @@
   <!-- TODO -->
   <!-- Wheels ============================================================= -->
-  <xacro:property name="wheel_length" value="0.076" />
+  <xacro:property name="wheel_length" value="0.07985" />
   <!-- ==================================================================== -->
-  <xacro:property name="wheel_radius" value="0.088895" />
+  <xacro:property name="wheel_radius" value="0.09794" />
   <!-- ==================================================================== -->
-  <xacro:property name="wheel_separation" value="0.39757" />
+  <xacro:property name="wheel_separation" value="0.344" />
   <!-- ==================================================================== -->
 <!-- ###################################################################### -->
