Commit message: Adjust linear's head position.

File: pandora_robots_description/urdf/gears/joints/linear_head_pitch_joint.urdf.xacro (robot description, xacro)
@@ -12,5 +12,5 @@
         <child link="linear_head_base_link" />
         <!-- ============================================================== -->
-        <origin xyz="-0.0145 0.0686 0.35787"
+        <origin xyz="0.008 0.02049 0.4055"
                 rpy="${zero}" />
         <!-- ============================================================== -->
@@ -25,5 +25,5 @@
         <child link="linear_head_base_link" />
         <!-- ============================================================== -->
-        <origin xyz="-0.0145 0.0686 0.35787"
+        <origin xyz="0.008 0.02049 0.4055"
                 rpy="${zero}" />
         <!-- ============================================================== -->

File: pandora_robots_description/urdf/gears/joints/linear_head_yaw_joint.urdf.xacro (robot description, xacro)
@@ -12,5 +12,5 @@
         <child link="linear_head_main_link" />
         <!-- ============================================================== -->
-        <origin xyz="0.0 0.037 0.021"
+        <origin xyz="0.02107 0.0 0.021"
                 rpy="${zero}" />
         <!-- ============================================================== -->
@@ -25,5 +25,5 @@
         <child link="linear_head_main_link" />
         <!-- ============================================================== -->
-        <origin xyz="0.0 0.037 0.021"
+        <origin xyz="0.02107 0.0 0.021"
                 rpy="${zero}" />
         <!-- ============================================================== -->

File: pandora_robots_description/urdf/gears/links/base_link.urdf.xacro (robot description, xacro)
@@ -6,5 +6,5 @@
       <inertial>
         <!-- ============================================================== -->
-        <origin xyz="-0.010032 -0.0067035 0.16451" />
+        <origin xyz="-0.010032 -0.0067035 0.12451" />
         <!-- ============================================================== -->
         <mass value="8.6373" />

File: pandora_robots_description/urdf/gears/links/linear_head_base_link.urdf.xacro (robot description, xacro)
@@ -6,5 +6,5 @@
       <inertial>
         <!-- ============================================================== -->
-        <origin xyz="0.02347 0.0 0.00124" />
+        <origin xyz="0.00754 0.0 0.00124" />
         <!-- ============================================================== -->
         <mass value="0.0001" /><!--FIXME-->
@@ -20,6 +20,6 @@
       <visual>
         <!-- ============================================================== -->
-        <origin xyz="${zero}"
-                rpy="0.0 0.0 ${PI_2}" />
+        <origin xyz="-0.01593 0.0 0.0"
+                rpy="${zero}" />
         <!-- ============================================================== -->
         <geometry>
@@ -32,6 +32,6 @@
       <collision>
         <!-- ============================================================== -->
-        <origin xyz="0.0 0.02347 0.00124"
-                rpy="0.0 0.0 ${PI_2}" />
+        <origin xyz="0.00754 0.0 0.00124"
+                rpy="${zero}" />
         <!-- ============================================================== -->
         <geometry>

File: pandora_robots_description/urdf/gears/urdf_configurations.xacro (robot description, xacro)
@@ -50,5 +50,5 @@
   <!-- ==================================================================== -->
   <xacro:property name="linear_elevator_joint_min_limit" value="0.0" />
-  <xacro:property name="linear_elevator_joint_max_limit" value="0.23" /> <!--FIXME-->
+  <xacro:property name="linear_elevator_joint_max_limit" value="0.18" /> <!--FIXME-->
   <!-- ==================================================================== -->
   <xacro:property name="linear_head_pitch_joint_min_limit" value="-1.57" /> <!--FIXME-->

Commit message: Adjust head's position and fix meshes to fit servo motors.

File: pandora_robots_description/urdf/gears/joints/linear_head_pitch_joint.urdf.xacro (robot description, xacro)
@@ -9,8 +9,8 @@
              type="fixed" >
         <!-- ============================================================== -->
-        <parent link="linear_elevator_link" />
-        <child link="linear_head_base_link" />
+        <parent link="linear_head_base_link" />
+        <child link="linear_head_main_link" />
         <!-- ============================================================== -->
-        <origin xyz="-0.0145 0.0686 0.35787"
+        <origin xyz="0.0 0.00026 0.03689"
                 rpy="${zero}" />
         <!-- ============================================================== -->
@@ -22,8 +22,8 @@
              type="${linear_head_pitch_joint_type}" >
         <!-- ============================================================== -->
-        <parent link="linear_elevator_link" />
-        <child link="linear_head_base_link" />
+        <parent link="linear_head_base_link" />
+        <child link="linear_head_main_link" />
         <!-- ============================================================== -->
-        <origin xyz="-0.0145 0.0686 0.35787"
+        <origin xyz="0.0 0.00026 0.03689"
                 rpy="${zero}" />
         <!-- ============================================================== -->

File: pandora_robots_description/urdf/gears/joints/linear_head_yaw_joint.urdf.xacro (robot description, xacro)
@@ -9,8 +9,8 @@
              type="fixed" >
         <!-- ============================================================== -->
-        <parent link="linear_head_base_link" />
-        <child link="linear_head_main_link" />
+        <parent link="linear_elevator_link" />
+        <child link="linear_head_base_link" />
         <!-- ============================================================== -->
-        <origin xyz="0.0 0.037 0.021"
+        <origin xyz="-0.0035 0.06177 0.36617"
                 rpy="${zero}" />
         <!-- ============================================================== -->
@@ -22,8 +22,8 @@
              type="${linear_head_yaw_joint_type}" >
         <!-- ============================================================== -->
-        <parent link="linear_head_base_link" />
-        <child link="linear_head_main_link" />
+        <parent link="linear_elevator_link" />
+        <child link="linear_head_base_link" />
         <!-- ============================================================== -->
-        <origin xyz="0.0 0.037 0.021"
+        <origin xyz="-0.0035 0.06177 0.36617"
                 rpy="${zero}" />
         <!-- ============================================================== -->

File: pandora_robots_description/urdf/gears/links/linear_head_base_link.urdf.xacro (robot description, xacro)
@@ -6,5 +6,5 @@
       <inertial>
         <!-- ============================================================== -->
-        <origin xyz="0.02409 0.0 0.00124" />
+        <origin xyz="0.0 0.00152 0.02409" />
         <!-- ============================================================== -->
         <mass value="0.0001" /><!--FIXME-->
@@ -21,5 +21,5 @@
         <!-- ============================================================== -->
         <origin xyz="${zero}"
-                rpy="0.0 0.0 ${PI_2}" />
+                rpy="0.0 ${-PI_2} ${-PI_2}" />
         <!-- ============================================================== -->
         <geometry>
@@ -32,6 +32,6 @@
       <collision>
         <!-- ============================================================== -->
-        <origin xyz="0.0 0.02347 0.00124"
-                rpy="0.0 0.0 ${PI_2}" />
+        <origin xyz="0.0 0.00152 0.02409"
+                rpy="0.0 ${-PI_2} ${-PI_2}" />
         <!-- ============================================================== -->
         <geometry>

File: pandora_robots_description/urdf/gears/links/linear_head_main_link.urdf.xacro (robot description, xacro)
@@ -6,5 +6,5 @@
       <inertial>
         <!-- ============================================================== -->
-        <origin xyz="-0.0027417 0.0050805 0.037323" />
+        <origin xyz="-0.00329 -0.02726 0.05623" />
         <!-- ============================================================== -->
         <mass value="0.16491" />

File: pandora_robots_description/urdf/gears/sensors/co2_sensor.xacro (robot description, xacro)
@@ -7,5 +7,5 @@
   <xacro:macro name="co2_sensor" >
     <xacro:co2_caster parent="linear_head_main_link" >
-      <origin xyz="0.01039 -0.01556 0.02386"
+      <origin xyz="0.00915 -0.05293 0.05251"
               rpy="${zero}" />
     </xacro:co2_caster>

File: pandora_robots_description/urdf/gears/sensors/microphone_sensor.xacro (robot description, xacro)
@@ -7,5 +7,5 @@
   <xacro:macro name="microphone_sensor" >
     <xacro:microphone_caster parent="linear_head_main_link" >
-      <origin xyz="0.01039 0.01556 0.02386"
+      <origin xyz="0.00915 -0.02181 0.05251"
               rpy="${zero}" />
     </xacro:microphone_caster>

File: pandora_robots_description/urdf/gears/sensors/thermal_sensor.xacro (robot description, xacro)
@@ -9,5 +9,5 @@
     <xacro:thermal_caster parent="linear_head_main_link"
                           prefix_y="middle" >
-      <origin xyz="0.01039 0.00007 0.04532"
+      <origin xyz="0.00915 -0.0373 0.07397"
               rpy="${zero}" />
     </xacro:thermal_caster>
@@ -17,5 +17,5 @@
     <xacro:thermal_caster parent="linear_head_main_link"
                           prefix_y="left" >
-      <origin xyz="-0.00128 0.04774 0.03108"
+      <origin xyz="-0.00252 0.01037 0.05973"
               rpy="0 0 ${PI_3}" />
     </xacro:thermal_caster>
@@ -25,5 +25,5 @@
     <xacro:thermal_caster parent="linear_head_main_link"
                           prefix_y="right" >
-      <origin xyz="-0.00128 -0.04774 0.03108"
+      <origin xyz="-0.00252 -0.08511 0.05973"
               rpy="0 0 ${-PI_3}" />
     </xacro:thermal_caster>

File: pandora_sensors_description/urdf/hokuyo_urg_04lx.urdf.xacro (robot description, xacro)
@@ -32,5 +32,5 @@
         <!-- ============================================================== -->
         <geometry>
-          <mesh filename="package://pandora_sensors_description/meshes/hokuyo_utm_30lx/laser_pitch_servo.dae" />
+          <mesh filename="package://pandora_sensors_description/meshes/hokuyo_urg_04lx/laser_pitch_servo.dae" />
         </geometry>
         <!-- ============================================================== -->
@@ -69,5 +69,5 @@
         <!-- ============================================================== -->
         <geometry>
-          <mesh filename="package://pandora_sensors_description/meshes/hokuyo_utm_30lx/hokuyo_utm_30lx.dae" />
+          <mesh filename="package://pandora_sensors_description/meshes/hokuyo_urg_04lx/hokuyo_urg_04lx.dae" />
         </geometry>
         <!-- ============================================================== -->
@@ -75,9 +75,9 @@
       <collision>
         <!-- ============================================================== -->
-        <origin xyz="0 0 0.05299"
-                rpy="0 0 0" />
-        <!-- ============================================================== -->
-        <geometry>
-          <box size="0.062 0.063 0.116" />
+        <origin xyz="0 0 0.05099"
+                rpy="0 0 0" />
+        <!-- ============================================================== -->
+        <geometry>
+          <box size="0.062 0.063 0.12" />
         </geometry>
         <!-- ============================================================== -->
@@ -150,5 +150,5 @@
         <child link="laser_main_link" />
         <!-- ============================================================== -->
-        <origin xyz="0.013 0 0.02301"
+        <origin xyz="0.013 0.0 0.02301"
                 rpy="0 0 0" />
         <!-- ============================================================== -->
