Commit message: Update model.

File: pandora_robots_description/urdf/gears/joints/linear_elevator_joint.urdf.xacro (robot description, xacro)
@@ -12,5 +12,5 @@
         <child link="linear_elevator_link" />
         <!-- ============================================================== -->
-        <origin xyz="0.09368 -0.0005 0.23995"
+        <origin xyz="0.09377 -0.00176 0.18797"
                 rpy="${zero}" />
         <!-- ============================================================== -->
@@ -25,5 +25,5 @@
         <child link="linear_elevator_link" />
         <!-- ============================================================== -->
-        <origin xyz="0.09368 -0.0005 0.23995"
+        <origin xyz="0.09377 -0.00176 0.18797"
                 rpy="${zero}" />
         <!-- ============================================================== -->

File: pandora_robots_description/urdf/gears/joints/linear_head_pitch_joint.urdf.xacro (robot description, xacro)
@@ -12,5 +12,5 @@
         <child link="linear_head_base_link" />
         <!-- ============================================================== -->
-        <origin xyz="0.008 0.02049 0.4055"
+        <origin xyz="-0.0145 0.0686 0.35787"
                 rpy="${zero}" />
         <!-- ============================================================== -->
@@ -25,5 +25,5 @@
         <child link="linear_head_base_link" />
         <!-- ============================================================== -->
-        <origin xyz="0.008 0.02049 0.4055"
+        <origin xyz="-0.0145 0.0686 0.35787"
                 rpy="${zero}" />
         <!-- ============================================================== -->

File: pandora_robots_description/urdf/gears/joints/linear_head_yaw_joint.urdf.xacro (robot description, xacro)
@@ -12,5 +12,5 @@
         <child link="linear_head_main_link" />
         <!-- ============================================================== -->
-        <origin xyz="0.02107 0.0 0.021"
+        <origin xyz="0.0 0.037 0.021"
                 rpy="${zero}" />
         <!-- ============================================================== -->
@@ -25,5 +25,5 @@
         <child link="linear_head_main_link" />
         <!-- ============================================================== -->
-        <origin xyz="0.02107 0.0 0.021"
+        <origin xyz="0.0 0.037 0.021"
                 rpy="${zero}" />
         <!-- ============================================================== -->

File: pandora_robots_description/urdf/gears/links/base_link.urdf.xacro (robot description, xacro)
@@ -6,14 +6,14 @@
       <inertial>
         <!-- ============================================================== -->
-        <origin xyz="-0.010032 -0.0067035 0.12451" />
+        <origin xyz="-0.00968 -0.00122 0.17947" />
         <!-- ============================================================== -->
-        <mass value="8.6373" />
+        <mass value="8.25079" />
         <!-- ============================================================== -->
-        <inertia ixx="0.11754"
-                 ixy="0.0039217"
-                 ixz="0.0053416"
-                 iyy="0.12773"
-                 iyz="-0.0039963"
-                 izz="0.10593" />
+        <inertia ixx="0.112701442"
+                 ixy="-0.000233829"
+                 ixz="-0.014681510"
+                 iyy="0.096589855"
+                 iyz="-0.000177925"
+                 izz="0.083438037" />
         <!-- ============================================================== -->
       </inertial>

File: pandora_robots_description/urdf/gears/links/linear_head_base_link.urdf.xacro (robot description, xacro)
@@ -6,5 +6,5 @@
       <inertial>
         <!-- ============================================================== -->
-        <origin xyz="0.00754 0.0 0.00124" />
+        <origin xyz="0.02409 0.0 0.00124" />
         <!-- ============================================================== -->
         <mass value="0.0001" /><!--FIXME-->
@@ -20,6 +20,6 @@
       <visual>
         <!-- ============================================================== -->
-        <origin xyz="-0.01593 0.0 0.0"
-                rpy="${zero}" />
+        <origin xyz="${zero}"
+                rpy="0.0 0.0 ${PI_2}" />
         <!-- ============================================================== -->
         <geometry>
@@ -32,6 +32,6 @@
       <collision>
         <!-- ============================================================== -->
-        <origin xyz="0.00754 0.0 0.00124"
-                rpy="${zero}" />
+        <origin xyz="0.0 0.02347 0.00124"
+                rpy="0.0 0.0 ${PI_2}" />
         <!-- ============================================================== -->
         <geometry>

File: pandora_robots_description/urdf/gears/links/side_link.urdf.xacro (robot description, xacro)
@@ -7,14 +7,14 @@
       <inertial>
         <!-- ============================================================== -->
-        <origin xyz="${ reflect_y * ( -9.2074E-08 ) } ${ reflect_y * ( 0.010782 ) } -0.028501" />
+        <origin xyz="${ reflect_y * ( -8.21E-06 ) } ${ reflect_y * ( 0.00188403 ) } -0.04035954" />
         <!-- ============================================================== -->
-        <mass value="0.93539" />
+        <mass value="1.81542748" />
         <!-- ============================================================== -->
-        <inertia ixx="0.001211"
-                 ixy="-4.0495E-05"
-                 ixz="${ reflect_y * ( 1.0211E-06 ) }"
-                 iyy="0.026668"
-                 iyz="${ reflect_y * ( -0.00024586 ) }"
-                 izz="0.026454" />
+        <inertia ixx="0.000596450"
+                 ixy="-0.000025495"
+                 ixz="${ reflect_y * ( 0.000000573 ) }"
+                 iyy="0.016130501"
+                 iyz="${ reflect_y * ( -0.000066532 ) }"
+                 izz="0.015779275" />
         <!-- ============================================================== -->
       </inertial>

File: pandora_robots_description/urdf/gears/links/wheel_link.urdf.xacro (robot description, xacro)
@@ -9,12 +9,12 @@
         <origin xyz="${ reflect_y * ( -2.2235E-05 ) } ${ reflect_y * ( -0.00052624 ) } 2.4287E-05" />
         <!-- ============================================================== -->
-        <mass value="1.2128" />
+        <mass value="0.88" />
         <!-- ============================================================== -->
-        <inertia ixx="0.0032586"
-                 ixy="5.862E-08"
-                 ixz="${ reflect_y * ( 4.2142E-07 ) }"
-                 iyy="0.0054812"
-                 iyz="${ reflect_y * ( -6.4028E-08 ) }"
-                 izz="0.0032574" />
+        <inertia ixx="0.0023644"
+                 ixy="4.2534E-08"
+                 ixz="${ reflect_y * ( 3.0578E-07 ) }"
+                 iyy="0.0039771"
+                 iyz="${ reflect_y * ( -4.6458E-08 ) }"
+                 izz="0.0023635" />
         <!-- ============================================================== -->
       </inertial>

File: pandora_robots_description/urdf/gears/sensors/sonar_sensor.xacro (robot description, xacro)
@@ -9,5 +9,5 @@
     <xacro:sonar_caster name="left"
                         parent="base_link" >
-      <origin xyz="-0.15519 0.11249 0.14305"
+      <origin xyz="-0.15026 0.06429 0.39925"
               rpy="0.0 0.0 ${ 5 * PI_6 }" />
     </xacro:sonar_caster>
@@ -17,5 +17,5 @@
     <xacro:sonar_caster name="right"
                         parent="base_link" >
-      <origin xyz="-0.15519 -0.11351 0.14305"
+      <origin xyz="-0.15026 -0.06429 0.39925"
               rpy="0.0 0.0 ${ 7 * PI_6 }" />
     </xacro:sonar_caster>

Commit message: Fix linear's dimensions.

File: pandora_robots_description/urdf/gears/joints/linear_elevator_joint.urdf.xacro (robot description, xacro)
@@ -12,5 +12,5 @@
         <child link="linear_elevator_link" />
         <!-- ============================================================== -->
-        <origin xyz="0.09377 -0.00176 0.18797"
+        <origin xyz="0.09377 -0.00176 0.18497"
                 rpy="${zero}" />
         <!-- ============================================================== -->
@@ -25,5 +25,5 @@
         <child link="linear_elevator_link" />
         <!-- ============================================================== -->
-        <origin xyz="0.09377 -0.00176 0.18797"
+        <origin xyz="0.09377 -0.00176 0.18497"
                 rpy="${zero}" />
         <!-- ============================================================== -->

File: pandora_robots_description/urdf/gears/joints/linear_head_yaw_joint.urdf.xacro (robot description, xacro)
@@ -12,5 +12,5 @@
         <child link="linear_head_base_link" />
         <!-- ============================================================== -->
-        <origin xyz="-0.0035 0.06177 0.36617"
+        <origin xyz="-0.0035 0.06177 0.31517"
                 rpy="${zero}" />
         <!-- ============================================================== -->
@@ -25,5 +25,5 @@
         <child link="linear_head_base_link" />
         <!-- ============================================================== -->
-        <origin xyz="-0.0035 0.06177 0.36617"
+        <origin xyz="-0.0035 0.06177 0.31517"
                 rpy="${zero}" />
         <!-- ============================================================== -->

File: pandora_robots_description/urdf/gears/sensors/kinect_sensor.xacro (robot description, xacro)
@@ -13,5 +13,5 @@
                          yaw_min_limit="${kinect_yaw_joint_min_limit}"
                          yaw_max_limit="${kinect_yaw_joint_max_limit}" >
-      <origin xyz="0.06744 0.01239 0.19742"
+      <origin xyz="0.07044 0.01239 0.14642"
               rpy="${zero}" />
     </xacro:kinect_caster>

File: pandora_robots_description/urdf/gears/sensors/laser_sensor.xacro (robot description, xacro)
@@ -14,5 +14,5 @@
                          pitch_max_limit="${laser_pitch_joint_max_limit}" >
       <origin xyz="0.1894 0.0 0.09679"
-              rpy="${zero}" />
+              rpy="0.0436 0.0 0.0" />
     </xacro:hokuyo_caster>
   </xacro:macro>
