Commit message: Fix laser's center of mass and adjust kinect's links and joints.

File: pandora_robots_description/urdf/gears/sensors/kinect_sensor.xacro (robot description, xacro)
@@ -13,5 +13,5 @@
                          yaw_min_limit="${kinect_yaw_joint_min_limit}"
                          yaw_max_limit="${kinect_yaw_joint_max_limit}" >
-      <origin xyz="0.05148 0.01239 0.19742"
+      <origin xyz="0.06744 0.01239 0.19742"
               rpy="${zero}" />
     </xacro:kinect_caster>

File: pandora_robots_description/urdf/gears/sensors/laser_sensor.xacro (robot description, xacro)
@@ -2,5 +2,5 @@
 <robot xmlns:xacro="http://ros.org/wiki/xacro" >
   <!-- ==================================================================== -->
-  <xacro:include filename="$(find pandora_sensors_description)/urdf/hokuyo_utm_30lx.urdf.xacro" />
+  <xacro:include filename="$(find pandora_sensors_description)/urdf/hokuyo_urg_04lx.urdf.xacro" />
   <!-- ==================================================================== -->
 <!-- ###################################################################### -->

File: pandora_sensors_description/urdf/hokuyo_urg_04lx.urdf.xacro (robot description, xacro)
@@ -51,5 +51,5 @@
       <inertial>
         <!-- ============================================================== -->
-        <origin xyz="0 0 0" />
+        <origin xyz="0.0 0.0 0.06" />
         <!-- ============================================================== -->
         <mass value="0.16" />

File: pandora_sensors_description/urdf/kinect_camera.urdf.xacro (robot description, xacro)
@@ -14,5 +14,5 @@
       <inertial>
         <!-- ============================================================== -->
-        <origin xyz="0.02347 0.0 0.00124" />
+        <origin xyz="0.00754 0.0 0.00124" />
         <!-- ============================================================== -->
         <mass value="0.0001" /><!--FIXME-->
@@ -28,6 +28,6 @@
       <visual>
         <!-- ============================================================== -->
-        <origin xyz="0 0 0"
-                rpy="0 0 0" />
+        <origin xyz="-0.01593 0.0 0.0"
+                rpy="0.0 0.0 0.0" />
         <!-- ============================================================== -->
         <geometry>
@@ -38,5 +38,5 @@
       <collision>
         <!-- ============================================================== -->
-        <origin xyz="0.02347 0.0 0.00124"
+        <origin xyz="0.00754 0.0 0.00124"
                 rpy="0 0 0" />
         <!-- ============================================================== -->
@@ -272,5 +272,5 @@
         <child link="kinect_base_link" />
         <!-- ============================================================== -->
-        <origin xyz="0.037 0.0 0.021"
+        <origin xyz="0.02107 0.0 0.021"
                 rpy="0.0 0.0 0.0" />
         <!-- ============================================================== -->
@@ -284,5 +284,5 @@
         <child link="kinect_base_link" />
         <!-- ============================================================== -->
-        <origin xyz="0.037 0.0 0.021"
+        <origin xyz="0.02107 0.0 0.021"
                 rpy="0.0 0.0 0.0" />
         <!-- ============================================================== -->
@@ -346,5 +346,5 @@
       <child link="kinect_depth_frame" />
       <!-- ================================================================ -->
-      <origin xyz="0.0 -0.02 0.0"
+      <origin xyz="0.0 0.044 0.0"
               rpy="0.0 0.0 0.0" />
       <!-- ================================================================ -->
@@ -367,5 +367,5 @@
       <child link="kinect_rgb_frame" />
       <!-- ================================================================ -->
-      <origin xyz="0.0 -0.045 0.0"
+      <origin xyz="0.0 0.019 0.0"
               rpy="0.0 0.0 0.0" />
       <!-- ================================================================ -->

Commit message: Fix laser's dimensions and position.

File: pandora_robots_description/urdf/gears/sensors/kinect_sensor.xacro (robot description, xacro)
@@ -14,5 +14,5 @@
                          yaw_max_limit="${kinect_yaw_joint_max_limit}" >
       <origin xyz="0.07044 0.01239 0.14642"
-              rpy="${zero}" />
+              rpy="-0.0436 0.0 0.0" />
     </xacro:kinect_caster>
   </xacro:macro>

File: pandora_robots_description/urdf/gears/sensors/laser_sensor.xacro (robot description, xacro)
@@ -13,6 +13,6 @@
                          pitch_min_limit="${laser_pitch_joint_min_limit}"
                          pitch_max_limit="${laser_pitch_joint_max_limit}" >
-      <origin xyz="0.1894 0.0 0.09679"
-              rpy="0.0436 0.0 0.0" />
+      <origin xyz="0.1974 0.0 0.09679"
+              rpy="${zero}" />
     </xacro:hokuyo_caster>
   </xacro:macro>

File: pandora_sensors_description/urdf/hokuyo_urg_04lx.urdf.xacro (robot description, xacro)
@@ -75,9 +75,9 @@
       <collision>
         <!-- ============================================================== -->
-        <origin xyz="0 0 0.05099"
-                rpy="0 0 0" />
-        <!-- ============================================================== -->
-        <geometry>
-          <box size="0.062 0.063 0.12" />
+        <origin xyz="0 0 0.04822"
+                rpy="0 0 0" />
+        <!-- ============================================================== -->
+        <geometry>
+          <box size="0.050 0.050 0.114" />
         </geometry>
         <!-- ============================================================== -->
@@ -192,5 +192,5 @@
       <child link="laser_link" />
       <!-- ================================================================ -->
-      <origin xyz="0.0225 0.0 0.105"
+      <origin xyz="0.0 0.0 0.08893"
               rpy="0 0 0" />
       <!-- ================================================================ -->
