Commit message: Update sensor meshes and fix their positions.

File: pandora_robots_description/urdf/gears/sensors/microphone_sensor.xacro (robot description, xacro)
@@ -7,5 +7,5 @@
   <xacro:macro name="microphone_sensor" >
     <xacro:microphone_caster parent="linear_head_main_link" >
-      <origin xyz="0.00915 -0.02181 0.05251"
+      <origin xyz="-0.02175 -0.0374 0.09643"
               rpy="${zero}" />
     </xacro:microphone_caster>

File: pandora_robots_description/urdf/gears/sensors/sonar_sensor.xacro (robot description, xacro)
@@ -7,5 +7,5 @@
   <!-- ==================================================================== -->
   <xacro:macro name="left_sonar_sensor" >
-    <xacro:sonar_caster name="left"
+    <xacro:sonar_caster prefix_y="left"
                         parent="base_link" >
       <origin xyz="-0.15026 0.06429 0.39925"
@@ -15,5 +15,5 @@
   <!-- ==================================================================== -->
   <xacro:macro name="right_sonar_sensor" >
-    <xacro:sonar_caster name="right"
+    <xacro:sonar_caster prefix_y="right"
                         parent="base_link" >
       <origin xyz="-0.15026 -0.06429 0.39925"

File: pandora_robots_description/urdf/gears/sensors/thermal_sensor.xacro (robot description, xacro)
@@ -9,6 +9,6 @@
     <xacro:thermal_caster parent="linear_head_main_link"
                           prefix_y="middle" >
-      <origin xyz="0.00915 -0.0373 0.07397"
-              rpy="${zero}" />
+      <origin xyz="0.01575 -0.0614 0.08243"
+              rpy="${-PI_2} 0 0" />
     </xacro:thermal_caster>
   </xacro:macro>
@@ -17,5 +17,5 @@
     <xacro:thermal_caster parent="linear_head_main_link"
                           prefix_y="left" >
-      <origin xyz="-0.00252 0.01037 0.05973"
+      <origin xyz="0.00076 0.01607 0.05800"
               rpy="0 0 ${PI_3}" />
     </xacro:thermal_caster>
@@ -25,5 +25,5 @@
     <xacro:thermal_caster parent="linear_head_main_link"
                           prefix_y="right" >
-      <origin xyz="-0.00252 -0.08511 0.05973"
+      <origin xyz="0.00076 -0.09086 0.05800"
               rpy="0 0 ${-PI_3}" />
     </xacro:thermal_caster>

File: pandora_sensors_description/urdf/co2.urdf.xacro (robot description, xacro)
@@ -26,5 +26,5 @@
         <!-- ============================================================== -->
         <geometry>
-          <mesh filename="package://pandora_sensors_description/meshes/co2/co2.dae" />
+          <mesh filename="package://pandora_sensors_description/meshes/co2/dynament.dae" />
         </geometry>
         <!-- ============================================================== -->
@@ -32,9 +32,9 @@
       <collision>
         <!-- ============================================================== -->
-        <origin xyz="0.007 0.0 0.0"
+        <origin xyz="0.0075 0.0 0.0"
                 rpy="0 0 0" />
         <!-- ============================================================== -->
         <geometry>
-          <box size="0.025 0.025 0.025" />
+          <box size="0.015 0.022 0.022" />
         </geometry>
         <!-- ============================================================== -->
@@ -42,5 +42,22 @@
     </link>
     <!-- ################################################################## -->
-    <joint name="co2_joint"
+    <link name="co2_frame" >
+      <inertial>
+        <!-- ============================================================== -->
+        <origin xyz="0.0 0.0 0.0" />
+        <!-- ============================================================== -->
+        <mass value="0.0001" />
+        <!-- ============================================================== -->
+        <inertia ixx="0.00000001"
+                 ixy="0"
+                 ixz="0"
+                 iyy="0.00000001"
+                 iyz="0"
+                 izz="0.00000001" />
+        <!-- ============================================================== -->
+      </inertial>
+    </link>
+    <!-- ################################################################## -->
+    <joint name="co2_main_joint"
            type="fixed" >
       <!-- ================================================================ -->
@@ -51,4 +68,16 @@
       <!-- ================================================================ -->
     </joint>
+    <!-- ################################################################## -->
+    <joint name="co2_joint"
+           type="fixed" >
+      <!-- ================================================================ -->
+      <parent link="co2_link" />
+      <child link="co2_frame" />
+      <!-- ================================================================ -->
+      <origin xyz="0.015 0.0 0.0"
+              rpy="0.0 0.0 0.0" />
+      <!-- ================================================================ -->
+    </joint>
+    <!-- ################################################################## -->
   </xacro:macro>
 <!-- ###################################################################### -->

File: pandora_sensors_description/urdf/kinect.urdf.xacro (robot description, xacro)
@@ -381,4 +381,5 @@
       <!-- ================================================================ -->
     </joint>
+    <!-- ################################################################## -->
   </xacro:macro>
 <!-- ###################################################################### -->

File: pandora_sensors_description/urdf/laser.urdf.xacro (robot description, xacro)
@@ -196,4 +196,5 @@
       <!-- ================================================================ -->
     </joint>
+    <!-- ################################################################## -->
   </xacro:macro>
 <!-- ###################################################################### -->

File: pandora_sensors_description/urdf/microphone.urdf.xacro (robot description, xacro)
@@ -8,5 +8,5 @@
       <inertial>
         <!-- ============================================================== -->
-        <origin xyz="0.005 0.0 0.0" />
+        <origin xyz="0.01177 0.0 0.0" />
         <!-- ============================================================== -->
         <mass value="0.005" />
@@ -26,5 +26,5 @@
         <!-- ============================================================== -->
         <geometry>
-          <mesh filename="package://pandora_sensors_description/meshes/microphone/microphone.dae" />
+          <mesh filename="package://pandora_sensors_description/meshes/microphone/kinect_array.dae" />
         </geometry>
         <!-- ============================================================== -->
@@ -32,9 +32,9 @@
       <collision>
         <!-- ============================================================== -->
-        <origin xyz="0.007 0.0 0.0"
+        <origin xyz="0.0 0.0 0.01"
                 rpy="0 0 0" />
         <!-- ============================================================== -->
         <geometry>
-          <box size="0.025 0.025 0.025" />
+          <box size="0.053 0.055 0.020" />
         </geometry>
         <!-- ============================================================== -->
@@ -42,5 +42,23 @@
     </link>
     <!-- ################################################################## -->
-    <joint name="microphone_joint" type="fixed" >
+    <link name="microphone_frame" >
+      <inertial>
+        <!-- ============================================================== -->
+        <origin xyz="0.0 0.0 0.0" />
+        <!-- ============================================================== -->
+        <mass value="0.0001" />
+        <!-- ============================================================== -->
+        <inertia ixx="0.00000001"
+                 ixy="0"
+                 ixz="0"
+                 iyy="0.00000001"
+                 iyz="0"
+                 izz="0.00000001" />
+        <!-- ============================================================== -->
+      </inertial>
+    </link>
+    <!-- ################################################################## -->
+    <joint name="microphone_main_joint"
+           type="fixed" >
       <!-- ================================================================ -->
       <parent link="${parent}" />
@@ -50,4 +68,16 @@
       <!-- ================================================================ -->
     </joint>
+    <!-- ################################################################## -->
+    <joint name="microphone_joint"
+           type="fixed" >
+      <!-- ================================================================ -->
+      <parent link="microphone_link" />
+      <child link="microphone_frame" />
+      <!-- ================================================================ -->
+      <origin xyz="0.0 0.0 0.0125"
+              rpy="0.0 0.0 0.0" />
+      <!-- ================================================================ -->
+    </joint>
+    <!-- ################################################################## -->
   </xacro:macro>
 <!-- ###################################################################### -->

File: pandora_sensors_description/urdf/sonar.urdf.xacro (robot description, xacro)
@@ -3,7 +3,7 @@
 <!-- ###################################################################### -->
   <xacro:macro name="sonar_caster"
-               params="name parent *origin" >
+               params="parent prefix_y *origin" >
     <!-- ################################################################## -->
-    <link name="${name}_sonar_link" >
+    <link name="${prefix_y}_sonar_link" >
       <inertial>
         <!-- ============================================================== -->
@@ -26,5 +26,5 @@
         <!-- ============================================================== -->
         <geometry>
-          <mesh filename="package://pandora_sensors_description/meshes/sonar/max_sonar_ez4.dae" />
+          <mesh filename="package://pandora_sensors_description/meshes/sonar/max_ez4.dae" />
         </geometry>
         <!-- ============================================================== -->
@@ -32,9 +32,9 @@
       <collision>
         <!-- ============================================================== -->
-        <origin xyz="0.007 0.0 0.0"
+        <origin xyz="0.0075 0.0 0.0"
                 rpy="0 0 0" />
         <!-- ============================================================== -->
         <geometry>
-          <box size="0.025 0.05 0.025" />
+          <box size="0.015 0.044 0.022" />
         </geometry>
         <!-- ============================================================== -->
@@ -42,13 +42,42 @@
     </link>
     <!-- ################################################################## -->
-    <joint name="${name}_sonar_joint"
+    <link name="${prefix_y}_sonar_frame" >
+      <inertial>
+        <!-- ============================================================== -->
+        <origin xyz="0.0 0.0 0.0" />
+        <!-- ============================================================== -->
+        <mass value="0.0001" />
+        <!-- ============================================================== -->
+        <inertia ixx="0.00000001"
+                 ixy="0"
+                 ixz="0"
+                 iyy="0.00000001"
+                 iyz="0"
+                 izz="0.00000001" />
+        <!-- ============================================================== -->
+      </inertial>
+    </link>
+    <!-- ################################################################## -->
+    <joint name="${prefix_y}_sonar_main_joint"
            type="fixed" >
       <!-- ================================================================ -->
       <parent link="${parent}" />
-      <child link="${name}_sonar_link" />
+      <child link="${prefix_y}_sonar_link" />
       <!-- ================================================================ -->
       <xacro:insert_block name="origin" />
       <!-- ================================================================ -->
     </joint>
+    <!-- ################################################################## -->
+    <joint name="${prefix_y}_sonar_joint"
+           type="fixed" >
+      <!-- ================================================================ -->
+      <parent link="${prefix_y}_sonar_link" />
+      <child link="${prefix_y}_sonar_frame" />
+      <!-- ================================================================ -->
+      <origin xyz="0.015 0.0 0.0"
+              rpy="0.0 0.0 0.0" />
+      <!-- ================================================================ -->
+    </joint>
+    <!-- ################################################################## -->
   </xacro:macro>
 <!-- ###################################################################### -->

File: pandora_sensors_description/urdf/thermal.urdf.xacro (robot description, xacro)
@@ -5,8 +5,8 @@
                params="parent prefix_y *origin" >
     <!-- ################################################################## -->
-    <link name="${prefix_y}_thermal_link" >
+    <link name="${prefix_y}_thermal_main_link" >
       <inertial>
         <!-- ============================================================== -->
-        <origin xyz="0.005 0.0 0.0" />
+        <origin xyz="0.00126 0.0 0.0" />
         <!-- ============================================================== -->
         <mass value="0.005" />
@@ -32,9 +32,9 @@
       <collision>
         <!-- ============================================================== -->
-        <origin xyz="0.007 0.0 0.0"
+        <origin xyz="0.00225 0.0 0.0"
                 rpy="0 0 0" />
         <!-- ============================================================== -->
         <geometry>
-          <box size="0.025 0.025 0.025" />
+          <box size="0.004 0.020 0.037" />
         </geometry>
         <!-- ============================================================== -->
@@ -42,13 +42,70 @@
     </link>
     <!-- ################################################################## -->
-    <joint name="${prefix_y}_thermal_joint"
+    <link name="${prefix_y}_thermal_frame" >
+      <inertial>
+        <!-- ============================================================== -->
+        <origin xyz="0.0 0.0 0.0" />
+        <!-- ============================================================== -->
+        <mass value="0.0001" />
+        <!-- ============================================================== -->
+        <inertia ixx="0.00000001"
+                 ixy="0"
+                 ixz="0"
+                 iyy="0.00000001"
+                 iyz="0"
+                 izz="0.00000001" />
+        <!-- ============================================================== -->
+      </inertial>
+    </link>
+    <!-- ################################################################## -->
+    <link name="${prefix_y}_thermal_optical_frame" >
+      <inertial>
+        <!-- ============================================================== -->
+        <origin xyz="0.0 0.0 0.0" />
+        <!-- ============================================================== -->
+        <mass value="0.0001" />
+        <!-- ============================================================== -->
+        <inertia ixx="0.00000001"
+                 ixy="0"
+                 ixz="0"
+                 iyy="0.00000001"
+                 iyz="0"
+                 izz="0.00000001" />
+        <!-- ============================================================== -->
+      </inertial>
+    </link>
+    <!-- ################################################################## -->
+    <joint name="${prefix_y}_thermal_main_joint"
            type="fixed" >
       <!-- ================================================================ -->
       <parent link="${parent}" />
-      <child link="${prefix_y}_thermal_link" />
+      <child link="${prefix_y}_thermal_main_link" />
       <!-- ================================================================ -->
       <xacro:insert_block name="origin" />
       <!-- ================================================================ -->
     </joint>
+    <!-- ################################################################## -->
+    <joint name="${prefix_y}_thermal_joint"
+           type="fixed" >
+      <!-- ================================================================ -->
+      <parent link="${prefix_y}_thermal_main_link" />
+      <child link="${prefix_y}_thermal_frame" />
+      <!-- ================================================================ -->
+      <origin xyz="0.0045 0.0 0.00125"
+              rpy="0.0 0.0 0.0" />
+      <!-- ================================================================ -->
+    </joint>
+    <!-- ################################################################## -->
+    <joint name="${prefix_y}_thermal_optical_joint"
+           type="fixed" >
+      <!-- ================================================================ -->
+      <parent link="${prefix_y}_thermal_frame" />
+      <child link="${prefix_y}_thermal_optical_frame" />
+      <!-- ================================================================ -->
+      <origin xyz="0.0 0.0 0.0"
+              rpy="-1.5708 0.0 -1.5708" />
+      <!-- ================================================================ -->
+    </joint>
+    <!-- ################################################################## -->
   </xacro:macro>
 <!-- ###################################################################### -->
