Commit message: Fix linear sonar position.

File: pandora_robots_description/urdf/gears/sensors/sonar_sensor.xacro (robot description, xacro)
@@ -9,5 +9,5 @@
     <xacro:sonar_caster name="linear"
                         parent="linear_elevator_link" >
-      <origin xyz="0.01195 0.0 0.32700"
+      <origin xyz="0.0195 -0.0051 0.3270"
               rpy="${zero}" />
     </xacro:sonar_caster>
