Commit message: Adjust robot's inertia.

File: pandora_robots_description/urdf/gears/links/base_link.urdf.xacro (robot description, xacro)
@@ -10,10 +10,10 @@
         <mass value="8.25079" />
         <!-- ============================================================== -->
-        <inertia ixx="0.112701442"
-                 ixy="-0.000233829"
-                 ixz="-0.014681510"
-                 iyy="0.096589855"
-                 iyz="-0.000177925"
-                 izz="0.083438037" />
+        <inertia ixx="0.00845260815"
+                 ixy="-0.00001753717"
+                 ixz="-0.00110111325"
+                 iyy="0.00724423912"
+                 iyz="-0.00001334437"
+                 izz="0.006257852775" />
         <!-- ============================================================== -->
       </inertial>

File: pandora_robots_description/urdf/gears/links/wheel_link.urdf.xacro (robot description, xacro)
@@ -9,12 +9,12 @@
         <origin xyz="${ reflect_y * ( -2.2235E-05 ) } ${ reflect_y * ( -0.00052624 ) } 2.4287E-05" />
         <!-- ============================================================== -->
-        <mass value="1.5" />
+        <mass value="6.90375" />
         <!-- ============================================================== -->
-        <inertia ixx="0.0040302"
-                 ixy="7.250E-08"
-                 ixz="${ reflect_y * ( 5.2121E-07 ) }"
-                 iyy="0.0067791"
-                 iyz="${ reflect_y * ( -7.9189E-08 ) }"
-                 izz="0.0040286" />
+        <inertia ixx="0.0201150"
+                 ixy="36.2014E-08"
+                 ixz="${ reflect_y * ( 24.6150E-07 ) }"
+                 iyy="0.0326038"
+                 iyz="${ reflect_y * ( -4.0050E-07 ) }"
+                 izz="0.0201129" />
         <!-- ============================================================== -->
       </inertial>

Commit message: Revert base and wheel inertia changes.

File: pandora_robots_description/urdf/gears/links/base_link.urdf.xacro (robot description, xacro)
@@ -10,10 +10,10 @@
         <mass value="8.25079" />
         <!-- ============================================================== -->
-        <inertia ixx="0.00845260815"
-                 ixy="-0.00001753717"
-                 ixz="-0.00110111325"
-                 iyy="0.00724423912"
-                 iyz="-0.00001334437"
-                 izz="0.006257852775" />
+        <inertia ixx="0.112701442"
+                 ixy="-0.000233829"
+                 ixz="-0.014681510"
+                 iyy="0.096589855"
+                 iyz="-0.000177925"
+                 izz="0.083438037" />
         <!-- ============================================================== -->
       </inertial>

File: pandora_robots_description/urdf/gears/links/wheel_link.urdf.xacro (robot description, xacro)
@@ -9,14 +9,15 @@
         <origin xyz="${ reflect_y * ( -2.2235E-05 ) } ${ reflect_y * ( -0.00052624 ) } 2.4287E-05" />
         <!-- ============================================================== -->
-        <mass value="6.90375" />
+        <mass value="1.5" />
         <!-- ============================================================== -->
-        <inertia ixx="0.0201150"
-                 ixy="36.2014E-08"
-                 ixz="${ reflect_y * ( 24.6150E-07 ) }"
-                 iyy="0.0326038"
-                 iyz="${ reflect_y * ( -4.0050E-07 ) }"
-                 izz="0.0201129" />
+        <inertia ixx="0.0040302"
+                 ixy="7.250E-08"
+                 ixz="${ reflect_y * ( 5.2121E-07 ) }"
+                 iyy="0.0067791"
+                 iyz="${ reflect_y * ( -7.9189E-08 ) }"
+                 izz="0.0040286" />
         <!-- ============================================================== -->
       </inertial>
+Z
       <visual>
         <!-- ============================================================== -->
