Commit message: Increase wheel mass.

File: pandora_robots_description/urdf/gears/links/wheel_link.urdf.xacro (robot description, xacro)
@@ -9,12 +9,12 @@
         <origin xyz="${ reflect_y * ( -2.2235E-05 ) } ${ reflect_y * ( -0.00052624 ) } 2.4287E-05" />
         <!-- ============================================================== -->
-        <mass value="0.88" />
+        <mass value="1.5" />
         <!-- ============================================================== -->
-        <inertia ixx="0.0023644"
-                 ixy="4.2534E-08"
-                 ixz="${ reflect_y * ( 3.0578E-07 ) }"
-                 iyy="0.0039771"
-                 iyz="${ reflect_y * ( -4.6458E-08 ) }"
-                 izz="0.0023635" />
+        <inertia ixx="0.0040302"
+                 ixy="7.250E-08"
+                 ixz="${ reflect_y * ( 5.2121E-07 ) }"
+                 iyy="0.0067791"
+                 iyz="${ reflect_y * ( -7.9189E-08 ) }"
+                 izz="0.0040286" />
         <!-- ============================================================== -->
       </inertial>

Commit message: Fix kinect's position and rename sensors.

File: pandora_robots_description/urdf/gears/links/wheel_link.urdf.xacro (robot description, xacro)
@@ -19,5 +19,4 @@
         <!-- ============================================================== -->
       </inertial>
-Z
       <visual>
         <!-- ============================================================== -->

File: pandora_robots_description/urdf/gears/sensors/camera_sensor.xacro (robot description, xacro)
@@ -2,5 +2,5 @@
 <robot xmlns:xacro="http://ros.org/wiki/xacro" >
   <!-- ==================================================================== -->
-  <xacro:include filename="$(find pandora_sensors_description)/urdf/logitech_camera.urdf.xacro" />
+  <xacro:include filename="$(find pandora_sensors_description)/urdf/camera.urdf.xacro" />
   <!-- ==================================================================== -->
 <!-- ###################################################################### -->

File: pandora_robots_description/urdf/gears/sensors/co2_sensor.xacro (robot description, xacro)
@@ -2,5 +2,5 @@
 <robot xmlns:xacro="http://ros.org/wiki/xacro" >
   <!-- ==================================================================== -->
-  <xacro:include filename="$(find pandora_sensors_description)/urdf/co2_sensor.urdf.xacro" />
+  <xacro:include filename="$(find pandora_sensors_description)/urdf/co2.urdf.xacro" />
   <!-- ==================================================================== -->
 <!-- ###################################################################### -->

File: pandora_robots_description/urdf/gears/sensors/kinect_sensor.xacro (robot description, xacro)
@@ -2,5 +2,5 @@
 <robot xmlns:xacro="http://ros.org/wiki/xacro" >
   <!-- ==================================================================== -->
-  <xacro:include filename="$(find pandora_sensors_description)/urdf/kinect_camera.urdf.xacro" />
+  <xacro:include filename="$(find pandora_sensors_description)/urdf/kinect.urdf.xacro" />
   <!-- ==================================================================== -->
 <!-- ###################################################################### -->
@@ -13,5 +13,5 @@
                          yaw_min_limit="${kinect_yaw_joint_min_limit}"
                          yaw_max_limit="${kinect_yaw_joint_max_limit}" >
-      <origin xyz="0.07044 0.01239 0.14642"
+      <origin xyz="0.07353 0.01239 0.14642"
               rpy="-0.0436 0.0 0.0" />
     </xacro:kinect_caster>

File: pandora_robots_description/urdf/gears/sensors/laser_sensor.xacro (robot description, xacro)
@@ -2,10 +2,10 @@
 <robot xmlns:xacro="http://ros.org/wiki/xacro" >
   <!-- ==================================================================== -->
-  <xacro:include filename="$(find pandora_sensors_description)/urdf/hokuyo_urg_04lx.urdf.xacro" />
+  <xacro:include filename="$(find pandora_sensors_description)/urdf/laser.urdf.xacro" />
   <!-- ==================================================================== -->
 <!-- ###################################################################### -->
   <xacro:macro name="laser_sensor"
                params="fixed" >
-    <xacro:hokuyo_caster parent="base_link"
+    <xacro:laser_caster parent="base_link"
                          fixed="${fixed}"
                          roll_min_limit="${laser_roll_joint_min_limit}"
@@ -15,5 +15,5 @@
       <origin xyz="0.1974 0.0 0.09679"
               rpy="${zero}" />
-    </xacro:hokuyo_caster>
+    </xacro:laser_caster>
   </xacro:macro>
 <!-- ###################################################################### -->

File: pandora_robots_description/urdf/gears/sensors/microphone_sensor.xacro (robot description, xacro)
@@ -2,5 +2,5 @@
 <robot xmlns:xacro="http://ros.org/wiki/xacro" >
   <!-- ==================================================================== -->
-  <xacro:include filename="$(find pandora_sensors_description)/urdf/microphone_sensor.urdf.xacro" />
+  <xacro:include filename="$(find pandora_sensors_description)/urdf/microphone.urdf.xacro" />
   <!-- ==================================================================== -->
 <!-- ###################################################################### -->

File: pandora_robots_description/urdf/gears/sensors/sonar_sensor.xacro (robot description, xacro)
@@ -2,5 +2,5 @@
 <robot xmlns:xacro="http://ros.org/wiki/xacro" >
   <!-- ==================================================================== -->
-  <xacro:include filename="$(find pandora_sensors_description)/urdf/sonar_sensor.urdf.xacro" />
+  <xacro:include filename="$(find pandora_sensors_description)/urdf/sonar.urdf.xacro" />
   <!-- ==================================================================== -->
 <!-- ###################################################################### -->

File: pandora_robots_description/urdf/gears/sensors/thermal_sensor.xacro (robot description, xacro)
@@ -2,5 +2,5 @@
 <robot xmlns:xacro="http://ros.org/wiki/xacro" >
   <!-- ==================================================================== -->
-  <xacro:include filename="$(find pandora_sensors_description)/urdf/thermal_sensor.urdf.xacro" />
+  <xacro:include filename="$(find pandora_sensors_description)/urdf/thermal.urdf.xacro" />
   <!-- ==================================================================== -->
 <!-- ###################################################################### -->

File: pandora_sensors_description/urdf/camera.urdf.xacro (robot description, xacro)
@@ -26,5 +26,5 @@
         <!-- ============================================================== -->
         <geometry>
-          <mesh filename="package://pandora_sensors_description/meshes/logitech_camera/logitech_camera.dae" />
+          <mesh filename="package://pandora_sensors_description/meshes/camera/logitech.dae" />
         </geometry>
         <!-- ============================================================== -->

File: pandora_sensors_description/urdf/co2.urdf.xacro (robot description, xacro)
@@ -2,8 +2,8 @@
 <robot xmlns:xacro="http://ros.org/wiki/xacro" >
 <!-- ###################################################################### -->
-  <xacro:macro name="microphone_caster"
+  <xacro:macro name="co2_caster"
                params="parent *origin" >
     <!-- ################################################################## -->
-    <link name="microphone_link" >
+    <link name="co2_link" >
       <inertial>
         <!-- ============================================================== -->
@@ -26,5 +26,5 @@
         <!-- ============================================================== -->
         <geometry>
-          <mesh filename="package://pandora_sensors_description/meshes/microphone_sensor/microphone_small.dae" />
+          <mesh filename="package://pandora_sensors_description/meshes/co2/co2.dae" />
         </geometry>
         <!-- ============================================================== -->
@@ -42,8 +42,9 @@
     </link>
     <!-- ################################################################## -->
-    <joint name="microphone_joint" type="fixed" >
+    <joint name="co2_joint"
+           type="fixed" >
       <!-- ================================================================ -->
       <parent link="${parent}" />
-      <child link="microphone_link" />
+      <child link="co2_link" />
       <!-- ================================================================ -->
       <xacro:insert_block name="origin" />

File: pandora_sensors_description/urdf/kinect.urdf.xacro (robot description, xacro)
@@ -69,5 +69,5 @@
         <!-- ============================================================== -->
         <geometry>
-          <mesh filename="package://pandora_sensors_description/meshes/kinect_camera/kinect_base.dae" />
+          <mesh filename="package://pandora_sensors_description/meshes/kinect/base.dae" />
         </geometry>
         <!-- ============================================================== -->
@@ -106,5 +106,5 @@
         <!-- ============================================================== -->
         <geometry>
-          <mesh filename="package://pandora_sensors_description/meshes/kinect_camera/asus_xtion_pro.dae" />
+          <mesh filename="package://pandora_sensors_description/meshes/kinect/asus_xtion_pro.dae" />
         </geometry>
         <!-- ============================================================== -->

File: pandora_sensors_description/urdf/laser.urdf.xacro (robot description, xacro)
@@ -2,5 +2,5 @@
 <robot xmlns:xacro="http://ros.org/wiki/xacro" >
 <!-- ###################################################################### -->
-  <xacro:macro name="hokuyo_caster"
+  <xacro:macro name="laser_caster"
                params="parent
                        fixed
@@ -32,5 +32,5 @@
         <!-- ============================================================== -->
         <geometry>
-          <mesh filename="package://pandora_sensors_description/meshes/hokuyo_urg_04lx/laser_pitch_servo.dae" />
+          <mesh filename="package://pandora_sensors_description/meshes/laser/pitch_servo_motor.dae" />
         </geometry>
         <!-- ============================================================== -->
@@ -69,5 +69,5 @@
         <!-- ============================================================== -->
         <geometry>
-          <mesh filename="package://pandora_sensors_description/meshes/hokuyo_urg_04lx/hokuyo_urg_04lx.dae" />
+          <mesh filename="package://pandora_sensors_description/meshes/laser/hokuyo_urg_04lx.dae" />
         </geometry>
         <!-- ============================================================== -->

File: pandora_sensors_description/urdf/microphone.urdf.xacro (robot description, xacro)
@@ -2,8 +2,8 @@
 <robot xmlns:xacro="http://ros.org/wiki/xacro" >
 <!-- ###################################################################### -->
-  <xacro:macro name="thermal_caster"
-               params="parent prefix_y *origin" >
+  <xacro:macro name="microphone_caster"
+               params="parent *origin" >
     <!-- ################################################################## -->
-    <link name="${prefix_y}_thermal_link" >
+    <link name="microphone_link" >
       <inertial>
         <!-- ============================================================== -->
@@ -26,5 +26,5 @@
         <!-- ============================================================== -->
         <geometry>
-          <mesh filename="package://pandora_sensors_description/meshes/thermal_sensor/thermal_small.dae" />
+          <mesh filename="package://pandora_sensors_description/meshes/microphone/microphone.dae" />
         </geometry>
         <!-- ============================================================== -->
@@ -42,9 +42,8 @@
     </link>
     <!-- ################################################################## -->
-    <joint name="${prefix_y}_thermal_joint"
-           type="fixed" >
+    <joint name="microphone_joint" type="fixed" >
       <!-- ================================================================ -->
       <parent link="${parent}" />
-      <child link="${prefix_y}_thermal_link" />
+      <child link="microphone_link" />
       <!-- ================================================================ -->
       <xacro:insert_block name="origin" />

File: pandora_sensors_description/urdf/sonar.urdf.xacro (robot description, xacro)
@@ -2,20 +2,20 @@
 <robot xmlns:xacro="http://ros.org/wiki/xacro" >
 <!-- ###################################################################### -->
-  <xacro:macro name="co2_caster"
-               params="parent *origin" >
+  <xacro:macro name="sonar_caster"
+               params="name parent *origin" >
     <!-- ################################################################## -->
-    <link name="co2_link" >
+    <link name="${name}_sonar_link" >
       <inertial>
         <!-- ============================================================== -->
         <origin xyz="0.005 0.0 0.0" />
         <!-- ============================================================== -->
-        <mass value="0.005" />
+        <mass value="0.010" />
         <!-- ============================================================== -->
-        <inertia ixx="2.1208E-7"
-                 ixy="0"
-                 ixz="0"
-                 iyy="4.033E-7"
-                 iyz="0"
-                 izz="2.1208E-7" />
+        <inertia ixx="4.2416E-7"
+                 ixy="0.0"
+                 ixz="0.0"
+                 iyy="2.0166E-6"
+                 iyz="0.0"
+                 izz="1.6341E-6" />
         <!-- ============================================================== -->
       </inertial>
@@ -26,5 +26,5 @@
         <!-- ============================================================== -->
         <geometry>
-          <mesh filename="package://pandora_sensors_description/meshes/co2_sensor/co2_small.dae" />
+          <mesh filename="package://pandora_sensors_description/meshes/sonar/max_sonar_ez4.dae" />
         </geometry>
         <!-- ============================================================== -->
@@ -36,5 +36,5 @@
         <!-- ============================================================== -->
         <geometry>
-          <box size="0.025 0.025 0.025" />
+          <box size="0.025 0.05 0.025" />
         </geometry>
         <!-- ============================================================== -->
@@ -42,9 +42,9 @@
     </link>
     <!-- ################################################################## -->
-    <joint name="co2_joint"
+    <joint name="${name}_sonar_joint"
            type="fixed" >
       <!-- ================================================================ -->
       <parent link="${parent}" />
-      <child link="co2_link" />
+      <child link="${name}_sonar_link" />
       <!-- ================================================================ -->
       <xacro:insert_block name="origin" />

File: pandora_sensors_description/urdf/thermal.urdf.xacro (robot description, xacro)
@@ -2,20 +2,20 @@
 <robot xmlns:xacro="http://ros.org/wiki/xacro" >
 <!-- ###################################################################### -->
-  <xacro:macro name="sonar_caster"
-               params="name parent *origin" >
+  <xacro:macro name="thermal_caster"
+               params="parent prefix_y *origin" >
     <!-- ################################################################## -->
-    <link name="${name}_sonar_link" >
+    <link name="${prefix_y}_thermal_link" >
       <inertial>
         <!-- ============================================================== -->
         <origin xyz="0.005 0.0 0.0" />
         <!-- ============================================================== -->
-        <mass value="0.010" />
+        <mass value="0.005" />
         <!-- ============================================================== -->
-        <inertia ixx="4.2416E-7"
-                 ixy="0.0"
-                 ixz="0.0"
-                 iyy="2.0166E-6"
-                 iyz="0.0"
-                 izz="1.6341E-6" />
+        <inertia ixx="2.1208E-7"
+                 ixy="0"
+                 ixz="0"
+                 iyy="4.033E-7"
+                 iyz="0"
+                 izz="2.1208E-7" />
         <!-- ============================================================== -->
       </inertial>
@@ -26,5 +26,5 @@
         <!-- ============================================================== -->
         <geometry>
-          <mesh filename="package://pandora_sensors_description/meshes/sonar_sensor/max_sonar_ez4.dae" />
+          <mesh filename="package://pandora_sensors_description/meshes/thermal/grid_eye.dae" />
         </geometry>
         <!-- ============================================================== -->
@@ -36,5 +36,5 @@
         <!-- ============================================================== -->
         <geometry>
-          <box size="0.025 0.05 0.025" />
+          <box size="0.025 0.025 0.025" />
         </geometry>
         <!-- ============================================================== -->
@@ -42,9 +42,9 @@
     </link>
     <!-- ################################################################## -->
-    <joint name="${name}_sonar_joint"
+    <joint name="${prefix_y}_thermal_joint"
            type="fixed" >
       <!-- ================================================================ -->
       <parent link="${parent}" />
-      <child link="${name}_sonar_link" />
+      <child link="${prefix_y}_thermal_link" />
       <!-- ================================================================ -->
       <xacro:insert_block name="origin" />
