Commit message: Add damping to linear elevator joint for better control.

File: pandora_robots_description/urdf/gears/urdf_configurations.xacro (robot description, xacro)
@@ -52,5 +52,5 @@
   <xacro:property name="wheel_joint_damping" value="0.0" />
   <!-- ==================================================================== -->
-  <xacro:property name="linear_elevator_joint_damping" value="0.0" />
+  <xacro:property name="linear_elevator_joint_damping" value="5800.0" />
   <!-- ==================================================================== -->
   <xacro:property name="linear_head_pitch_joint_damping" value="0.0" />

Commit message: Add base link visual mesh and remove unecessary elements [ci skip]

File: pandora_robots_description/urdf/gears/urdf_configurations.xacro (robot description, xacro)
@@ -101,5 +101,7 @@
   <xacro:property name="wheel_radius" value="0.09794" />
   <!-- ==================================================================== -->
+  <xacro:property name="wheelbase" value="0.405" />
   <xacro:property name="wheel_separation" value="0.344" />
+  <xacro:property name="track" value="0.344" />
   <!-- ==================================================================== -->
 <!-- ###################################################################### -->

File: pandora_robots_description/urdf/woody/sensors/sonar_sensor.xacro (robot description, xacro)
@@ -5,12 +5,4 @@
   <!-- ==================================================================== -->
 <!-- ###################################################################### -->
-  <!-- ==================================================================== -->
-  <xacro:macro name="linear_sonar_sensor" >
-    <xacro:sonar_caster name="linear"
-                        parent="linear_elevator_link" >
-      <origin xyz="0.0195 -0.0051 0.3270"
-              rpy="${zero}" />
-    </xacro:sonar_caster>
-  </xacro:macro>
   <!-- ==================================================================== -->
   <xacro:macro name="left_sonar_sensor" >

File: pandora_robots_description/urdf/woody/sensors/thermal_sensor.xacro (robot description, xacro)
@@ -7,5 +7,5 @@
   <!-- ==================================================================== -->
   <xacro:macro name="middle_thermal_sensor" >
-    <xacro:thermal_caster parent="linear_head_main_link"
+    <xacro:thermal_caster parent="base_link"
                           prefix_y="middle" >
       <origin xyz="0.01575 -0.0614 0.08243"
@@ -13,21 +13,4 @@
     </xacro:thermal_caster>
   </xacro:macro>
-  <!-- ==================================================================== -->
-  <xacro:macro name="left_thermal_sensor" >
-    <xacro:thermal_caster parent="linear_head_main_link"
-                          prefix_y="left" >
-      <origin xyz="0.00076 0.01607 0.05800"
-              rpy="0 0 ${PI_3}" />
-    </xacro:thermal_caster>
-  </xacro:macro>
-  <!-- ==================================================================== -->
-  <xacro:macro name="right_thermal_sensor" >
-    <xacro:thermal_caster parent="linear_head_main_link"
-                          prefix_y="right" >
-      <origin xyz="0.00076 -0.09086 0.05800"
-              rpy="0 0 ${-PI_3}" />
-    </xacro:thermal_caster>
-  </xacro:macro>
-  <!-- ==================================================================== -->
 <!-- ###################################################################### -->
 </robot>

File: pandora_robots_description/urdf/woody/urdf_configurations.xacro (robot description, xacro)
@@ -3,5 +3,5 @@
 <!-- Elements' Status ##################################################### -->
   <!-- Sensors ============================================================ -->
-  <xacro:property name="enable_sensors" value="true" />
+  <xacro:property name="enable_sensors" value="false" />
     <!-- ================================================================== -->
     <xacro:property name="enable_laser_sensor" value="true" />
@@ -9,21 +9,17 @@
     <xacro:property name="enable_kinect_sensor" value="true" />
     <!-- ================================================================== -->
-    <xacro:property name="enable_camera_sensors" value="true" />
+    <xacro:property name="enable_camera_sensors" value="false" />
       <xacro:property name="enable_left_camera_sensor" value="true" />
       <xacro:property name="enable_right_camera_sensor" value="true" />
     <!-- ================================================================== -->
-    <xacro:property name="enable_sonar_sensors" value="true" />
-      <xacro:property name="enable_linear_sonar_sensor" value="true" />
+    <xacro:property name="enable_sonar_sensors" value="false" />
       <xacro:property name="enable_left_sonar_sensor" value="true" />
       <xacro:property name="enable_right_sonar_sensor" value="true" />
     <!-- ================================================================== -->
-    <xacro:property name="enable_thermal_sensors" value="true" />
-      <xacro:property name="enable_middle_thermal_sensor" value="true" />
-      <xacro:property name="enable_left_thermal_sensor" value="true" />
-      <xacro:property name="enable_right_thermal_sensor" value="true" />
+    <xacro:property name="enable_thermal_sensor" value="false" />
     <!-- ================================================================== -->
-    <xacro:property name="enable_co2_sensor" value="true" />
+    <xacro:property name="enable_co2_sensor" value="false" />
     <!-- ================================================================== -->
-    <xacro:property name="enable_microphone_sensor" value="true" />
+    <xacro:property name="enable_microphone_sensor" value="false" />
   <!-- ==================================================================== -->
 <!-- Joint Physics ######################################################## -->
@@ -33,10 +29,4 @@
   <xacro:property name="wheel_joint_type" value="continuous" />
   <!-- ==================================================================== -->
-  <xacro:property name="linear_elevator_joint_type" value="prismatic" />
-  <!-- ==================================================================== -->
-  <xacro:property name="linear_head_yaw_joint_type" value="revolute" />
-  <!-- ==================================================================== -->
-  <xacro:property name="linear_head_pitch_joint_type" value="revolute" />
-  <!-- ==================================================================== -->
   <!-- Joint Damping ====================================================== -->
   <xacro:property name="side_joint_damping" value="0.0" />
@@ -44,22 +34,7 @@
   <xacro:property name="wheel_joint_damping" value="0.0" />
   <!-- ==================================================================== -->
-  <xacro:property name="linear_elevator_joint_damping" value="5800.0" />
-  <!-- ==================================================================== -->
-  <xacro:property name="linear_head_pitch_joint_damping" value="0.0" />
-  <!-- ==================================================================== -->
-  <xacro:property name="linear_head_yaw_joint_damping" value="0.0" />
-  <!-- ==================================================================== -->
   <!-- Joint Limits ======================================================= -->
   <xacro:property name="side_joint_min_limit" value="-0.785" /> <!--FIXME-->
   <xacro:property name="side_joint_max_limit" value="0.785" /> <!--FIXME-->
-  <!-- ==================================================================== -->
-  <xacro:property name="linear_elevator_joint_min_limit" value="0.0" />
-  <xacro:property name="linear_elevator_joint_max_limit" value="0.18" /> <!--FIXME-->
-  <!-- ==================================================================== -->
-  <xacro:property name="linear_head_yaw_joint_min_limit" value="-1.57" /> <!--FIXME-->
-  <xacro:property name="linear_head_yaw_joint_max_limit" value="1.57" /> <!--FIXME-->
-  <!-- ==================================================================== -->
-  <xacro:property name="linear_head_pitch_joint_min_limit" value="-1.57" /> <!--FIXME-->
-  <xacro:property name="linear_head_pitch_joint_max_limit" value="1.57" /> <!--FIXME-->
   <!-- ==================================================================== -->
   <xacro:property name="laser_roll_joint_min_limit" value="-1.57" /> <!--FIXME-->
@@ -76,4 +51,5 @@
   <!-- ==================================================================== -->
 <!-- Coefficients ######################################################### -->
+  <!-- TODO -->
   <!-- Velocities ========================================================= -->
   <xacro:property name="max_robot_linear_velocity" value="2.0" />
@@ -101,5 +77,7 @@
   <xacro:property name="wheel_radius" value="0.09794" />
   <!-- ==================================================================== -->
-  <xacro:property name="wheel_separation" value="0.344" />
+  <xacro:property name="track" value="0.344" />
+  <!-- ==================================================================== -->
+  <xacro:property name="wheelbase" value="0.34678" />
   <!-- ==================================================================== -->
 <!-- ###################################################################### -->

File: pandora_robots_description/urdf/woody/woody.urdf.xacro (robot description, xacro)
@@ -12,13 +12,7 @@
   <xacro:include filename="$(find pandora_robots_description)/urdf/woody/links/side_link.urdf.xacro" />
   <xacro:include filename="$(find pandora_robots_description)/urdf/woody/links/wheel_link.urdf.xacro" />
-  <xacro:include filename="$(find pandora_robots_description)/urdf/woody/links/linear_elevator_link.urdf.xacro" />
-  <xacro:include filename="$(find pandora_robots_description)/urdf/woody/links/linear_head_base_link.urdf.xacro" />
-  <xacro:include filename="$(find pandora_robots_description)/urdf/woody/links/linear_head_main_link.urdf.xacro" />
   <!-- ==================================================================== -->
   <xacro:include filename="$(find pandora_robots_description)/urdf/woody/joints/side_joint.urdf.xacro" />
   <xacro:include filename="$(find pandora_robots_description)/urdf/woody/joints/wheel_joint.urdf.xacro" />
-  <xacro:include filename="$(find pandora_robots_description)/urdf/woody/joints/linear_elevator_joint.urdf.xacro" />
-  <xacro:include filename="$(find pandora_robots_description)/urdf/woody/joints/linear_head_pitch_joint.urdf.xacro" />
-  <xacro:include filename="$(find pandora_robots_description)/urdf/woody/joints/linear_head_yaw_joint.urdf.xacro" />
   <!-- ==================================================================== -->
   <xacro:include filename="$(find pandora_robots_description)/urdf/woody/sensors/laser_sensor.xacro" />
@@ -56,14 +50,4 @@
   <xacro:wheel_joint prefix_y="right" prefix_x="rear" reflect_y="-1" reflect_x="-1" />
   <!-- ================================================================== -->
-  <!-- ================================================================== -->
-  <xacro:linear_elevator_link />
-  <xacro:linear_elevator_joint fixed="${fixed}" />
-  <!-- ================================================================== -->
-  <xacro:linear_head_base_link />
-  <xacro:linear_head_yaw_joint fixed="${fixed}" />
-  <!-- ================================================================== -->
-  <xacro:linear_head_main_link />
-  <xacro:linear_head_pitch_joint fixed="${fixed}" />
-  <!-- ================================================================== -->
 <!-- Load Sensors ######################################################### -->
   <xacro:if value="${enable_sensors}" >
@@ -87,8 +71,4 @@
     <xacro:if value="${enable_sonar_sensors}" >
       <!-- ================================================================ -->
-      <xacro:if value="${enable_linear_sonar_sensor}" >
-        <xacro:linear_sonar_sensor />
-      </xacro:if>
-      <!-- ================================================================ -->
       <xacro:if value="${enable_left_sonar_sensor}" >
         <xacro:left_sonar_sensor />
@@ -100,18 +80,6 @@
       <!-- ================================================================ -->
     </xacro:if>
-    <xacro:if value="${enable_thermal_sensors}" >
-      <!-- ================================================================ -->
-      <xacro:if value="${enable_middle_thermal_sensor}" >
+    <xacro:if value="${enable_thermal_sensor}" >
         <xacro:middle_thermal_sensor />
-      </xacro:if>
-      <!-- ================================================================ -->
-      <xacro:if value="${enable_left_thermal_sensor}" >
-        <xacro:left_thermal_sensor />
-      </xacro:if>
-      <!-- ================================================================ -->
-      <xacro:if value="${enable_right_thermal_sensor}" >
-        <xacro:right_thermal_sensor />
-      </xacro:if>
-      <!-- ================================================================ -->
     </xacro:if>
     <xacro:if value="${enable_co2_sensor}" >
