Commit message: Refactor gears description.

File: pandora_robots_description/urdf/gears/gears.urdf.xacro (robot description, xacro)
@@ -4,160 +4,113 @@
 <!-- Import Files ######################################################### -->
   <!-- ==================================================================== -->
-  <xacro:include filename="$(find pandora_robots_description)/urdf/gears/config/gears_properties.xacro" />
-  <xacro:include filename="$(find pandora_robots_description)/urdf/gears/config/gears_configurations.xacro" />
-  <xacro:include filename="$(find pandora_robots_description)/urdf/gears/config/gears_physics.gazebo.xacro" />
+  <xacro:include filename="$(find pandora_robots_description)/urdf/gears/gears_configurations.xacro" />
+  <xacro:include filename="$(find pandora_robots_description)/urdf/gears/properties/constants.xacro" />
+  <xacro:include filename="$(find pandora_robots_description)/urdf/gears/properties/defaults.xacro" />
+  <xacro:include filename="$(find pandora_robots_description)/urdf/gears/properties/materials.xacro" />
   <!-- ==================================================================== -->
-  <xacro:include filename="$(find pandora_robots_description)/urdf/gears/model/links.urdf.xacro" />
-  <xacro:include filename="$(find pandora_robots_description)/urdf/gears/model/joints.urdf.xacro" />
+  <xacro:include filename="$(find pandora_robots_description)/urdf/gears/links/base/base_link.urdf.xacro" />
+  <xacro:include filename="$(find pandora_robots_description)/urdf/gears/links/side/side_link.urdf.xacro" />
+  <xacro:include filename="$(find pandora_robots_description)/urdf/gears/links/wheel/wheel_link.urdf.xacro" />
+  <xacro:include filename="$(find pandora_robots_description)/urdf/gears/links/linear/elevator/linear_elevator_link.urdf.xacro" />
+  <xacro:include filename="$(find pandora_robots_description)/urdf/gears/links/linear/head/base/linear_head_base_link.urdf.xacro" />
+  <xacro:include filename="$(find pandora_robots_description)/urdf/gears/links/linear/head/main/linear_head_main_link.urdf.xacro" />
   <!-- ==================================================================== -->
-  <xacro:include filename="$(find pandora_robots_description)/urdf/gears/gazebo/sensors.xacro" />
-  <xacro:include filename="$(find pandora_robots_description)/urdf/gears/gazebo/transmission.xacro" />
-  <xacro:include filename="$(find pandora_robots_description)/urdf/gears/gazebo/plugins.gazebo.xacro" />
+  <xacro:include filename="$(find pandora_robots_description)/urdf/gears/joints/side/side_joint.urdf.xacro" />
+  <xacro:include filename="$(find pandora_robots_description)/urdf/gears/joints/wheel/wheel_joint.urdf.xacro" />
+  <xacro:include filename="$(find pandora_robots_description)/urdf/gears/joints/linear/elevator/linear_elevator_joint.urdf.xacro" />
+  <xacro:include filename="$(find pandora_robots_description)/urdf/gears/joints/linear/head/base/linear_head_pitch_joint.urdf.xacro" />
+  <xacro:include filename="$(find pandora_robots_description)/urdf/gears/joints/linear/head/main/linear_head_yaw_joint.urdf.xacro" />
   <!-- ==================================================================== -->
-<!-- Load Links ########################################################### -->
-  <xacro:if value="${enable_links}" >
-    <!-- ================================================================== -->
-    <xacro:if value="${enable_base_link}" >
-      <xacro:base_link />
-    </xacro:if>
+  <xacro:include filename="$(find pandora_robots_description)/urdf/gears/sensors/laser/laser.xacro" />
+  <xacro:include filename="$(find pandora_robots_description)/urdf/gears/sensors/kinect/kinect.xacro" />
+  <xacro:include filename="$(find pandora_robots_description)/urdf/gears/sensors/sonar/sonar.xacro" />
+  <xacro:include filename="$(find pandora_robots_description)/urdf/gears/sensors/thermal/thermal.xacro" />
+  <xacro:include filename="$(find pandora_robots_description)/urdf/gears/sensors/co2/co2.xacro" />
+  <xacro:include filename="$(find pandora_robots_description)/urdf/gears/sensors/microphone/microphone.xacro" />
+  <!-- ==================================================================== -->
+<!-- Load Links & Joints ################################################## -->
+  <!-- ==================================================================== -->
+  <xacro:if value="${enable_base_link}" >
+    <xacro:base_link />
+  </xacro:if>
+  <!-- ==================================================================== -->
+  <xacro:if value="${enable_side_links}" >
+    <xacro:side_link prefix_y="left" reflect_y="1" />
+    <xacro:side_link prefix_y="right" reflect_y="-1" />
+    <xacro:side_joint prefix_y="left" reflect_y="1" />
+    <xacro:side_joint prefix_y="right" reflect_y="-1" />
+  </xacro:if>
+  <!-- ==================================================================== -->
+  <xacro:if value="${enable_wheel_links}" >
+    <xacro:wheel_link prefix_y="left" prefix_x="front" reflect_y="1" reflect_x="1" />
+    <xacro:wheel_link prefix_y="left" prefix_x="rear" reflect_y="1" reflect_x="-1" />
+    <xacro:wheel_link prefix_y="right" prefix_x="front" reflect_y="-1" reflect_x="1" />
+    <xacro:wheel_link prefix_y="right" prefix_x="rear" reflect_y="-1" reflect_x="-1" />
+    <xacro:wheel_joint prefix_y="left" prefix_x="front" reflect_y="1" reflect_x="1" />
+    <xacro:wheel_joint prefix_y="left" prefix_x="rear" reflect_y="1" reflect_x="-1" />
+    <xacro:wheel_joint prefix_y="right" prefix_x="front" reflect_y="-1" reflect_x="1" />
+    <xacro:wheel_joint prefix_y="right" prefix_x="rear" reflect_y="-1" reflect_x="-1" />
+  </xacro:if>
+  <!-- ==================================================================== -->
+  <xacro:if value="${enable_linear_links}" >
     <!-- ================================================================== -->
     <xacro:if value="${enable_linear_elevator_link}" >
       <xacro:linear_elevator_link />
+      <xacro:linear_elevator_joint fixed="$(arg fixed)" />
     </xacro:if>
     <!-- ================================================================== -->
-    <xacro:if value="${enable_linear_head_link}" >
-      <xacro:linear_head_links />
-    </xacro:if>
-    <!-- ================================================================== -->
-    <xacro:if value="${enable_side_links}" >
-      <xacro:side_link prefix_y="left" reflect_y="1" />
-      <xacro:side_link prefix_y="right" reflect_y="-1" />
-    </xacro:if>
-    <!-- ================================================================== -->
-    <xacro:if value="${enable_wheel_links}" >
-      <xacro:wheel_link prefix_y="left" prefix_x="front" reflect_y="1" reflect_x="1" />
-      <xacro:wheel_link prefix_y="left" prefix_x="rear" reflect_y="1" reflect_x="-1" />
-      <xacro:wheel_link prefix_y="right" prefix_x="front" reflect_y="-1" reflect_x="1" />
-      <xacro:wheel_link prefix_y="right" prefix_x="rear" reflect_y="-1" reflect_x="-1" />
+    <xacro:if value="${enable_linear_head_links}" >
+      <!-- ================================================================ -->
+      <xacro:if value="${enable_linear_head_base_link}" >
+        <xacro:linear_head_base_link />
+        <xacro:linear_head_pitch_joint fixed="$(arg fixed)" />
+      </xacro:if>
+      <!-- ================================================================ -->
+      <xacro:if value="${enable_linear_head_main_link}" >
+        <xacro:linear_head_main_link />
+        <xacro:linear_head_yaw_joint fixed="$(arg fixed)" />
+      </xacro:if>
+      <!-- ================================================================ -->
     </xacro:if>
     <!-- ================================================================== -->
   </xacro:if>
-<!-- Load Joints ########################################################## -->
-  <xacro:if value="${enable_joints}" >
+  <!-- ==================================================================== -->
+<!-- Load Sensors ######################################################### -->
+  <xacro:if value="${enable_sensors}" >
     <!-- ================================================================== -->
-    <xacro:if value="${enable_linear_elevator_joint}" >
-      <xacro:if value="$(arg real)" >
-        <xacro:linear_elevator_joint control="true" />
-      </xacro:if>
-      <xacro:unless value="$(arg real)" >
-        <xacro:linear_elevator_joint control="$(arg control)" />
-      </xacro:unless>
+    <xacro:if value="${enable_laser_sensor}" >
+      <xacro:laser_sensor fixed="$(arg fixed)" />
     </xacro:if>
     <!-- ================================================================== -->
-    <xacro:if value="${enable_linear_head_joints}" >
-      <xacro:if value="$(arg real)" >
-        <xacro:linear_head_joints control="true" />
-      </xacro:if>
-      <xacro:unless value="$(arg real)" >
-        <xacro:linear_head_joints control="$(arg control)" />
-      </xacro:unless>
+    <xacro:if value="${enable_kinect_sensor}" >
+      <xacro:kinect_sensor fixed="$(arg fixed)" />
     </xacro:if>
     <!-- ================================================================== -->
-    <xacro:if value="${enable_side_joints}" >
-      <xacro:side_joint prefix_y="left" reflect_y="1" />
-      <xacro:side_joint prefix_y="right" reflect_y="-1" />
-    </xacro:if>
-    <!-- ================================================================== -->
-    <xacro:if value="${enable_wheel_joints}" >
-      <xacro:wheel_joint prefix_y="left" prefix_x="front" reflect_y="1" reflect_x="1" />
-      <xacro:wheel_joint prefix_y="left" prefix_x="rear" reflect_y="1" reflect_x="-1" />
-      <xacro:wheel_joint prefix_y="right" prefix_x="front" reflect_y="-1" reflect_x="1" />
-      <xacro:wheel_joint prefix_y="right" prefix_x="rear" reflect_y="-1" reflect_x="-1" />
-    </xacro:if>
-    <!-- ================================================================== -->
-  </xacro:if>
-<!-- Load Physics ######################################################### -->
-  <xacro:unless value="$(arg real)" >
-    <xacro:robot_sdf_physics />
-    <xacro:if value="${enable_sdf_physics}" >
+    <xacro:if value="${enable_sonar_sensors}" >
       <!-- ================================================================ -->
-      <xacro:if value="${enable_base_link_sdf_physics}" >
-        <xacro:base_link_sdf_physics />
+      <xacro:if value="${enable_left_sonar_sensor}" >
+        <xacro:sonar_sensor prefix_y="left" reflect_y="1" />
       </xacro:if>
       <!-- ================================================================ -->
-      <xacro:if value="${enable_linear_elevator_link_sdf_physics}" >
-        <xacro:linear_elevator_link_sdf_physics />
-      </xacro:if>
-      <!-- ================================================================ -->
-      <xacro:if value="${enable_linear_head_link_sdf_physics}" >
-        <xacro:linear_head_link_sdf_physics />
-      </xacro:if>
-      <!-- ================================================================ -->
-      <xacro:if value="${enable_side_link_sdf_physics}" >
-        <xacro:side_link_sdf_physics prefix_y="left" />
-        <xacro:side_link_sdf_physics prefix_y="right" />
-      </xacro:if>
-      <!-- ================================================================ -->
-      <xacro:if value="${enable_wheel_link_sdf_physics}" >
-        <xacro:wheel_link_sdf_physics prefix_y="left" prefix_x="front" />
-        <xacro:wheel_link_sdf_physics prefix_y="left" prefix_x="rear" />
-        <xacro:wheel_link_sdf_physics prefix_y="right" prefix_x="front" />
-        <xacro:wheel_link_sdf_physics prefix_y="right" prefix_x="rear" />
-      </xacro:if>
-      <!-- ================================================================ -->
-      <xacro:if value="${enable_linear_elevator_joint_sdf_physics}" >
-        <xacro:linear_elevator_joint_sdf_physics />
-      </xacro:if>
-      <!-- ================================================================ -->
-      <xacro:if value="${enable_linear_head_pitch_joint_sdf_physics}" >
-        <xacro:linear_head_pitch_joint_sdf_physics />
-      </xacro:if>
-      <!-- ================================================================ -->
-      <xacro:if value="${enable_linear_head_yaw_joint_sdf_physics}" >
-        <xacro:linear_head_yaw_joint_sdf_physics />
-      </xacro:if>
-      <!-- ================================================================ -->
-      <xacro:if value="${enable_side_joint_sdf_physics}" >
-        <xacro:side_joint_sdf_physics prefix_y="left" />
-        <xacro:side_joint_sdf_physics prefix_y="right" />
-      </xacro:if>
-      <!-- ================================================================ -->
-      <xacro:if value="${enable_wheel_joint_sdf_physics}" >
-        <xacro:wheel_joint_sdf_physics prefix_y="left" prefix_x="front" />
-        <xacro:wheel_joint_sdf_physics prefix_y="left" prefix_x="rear" />
-        <xacro:wheel_joint_sdf_physics prefix_y="right" prefix_x="front" />
-        <xacro:wheel_joint_sdf_physics prefix_y="right" prefix_x="rear" />
+      <xacro:if value="${enable_right_sonar_sensor}" >
+        <xacro:sonar_sensor prefix_y="right" reflect_y="-1" />
       </xacro:if>
       <!-- ================================================================ -->
     </xacro:if>
-  </xacro:unless>
-<!-- Load Sensors ######################################################### -->
-  <xacro:if value="${enable_sensors}" >
-    <!-- ================================================================== -->
-    <xacro:if value="${enable_hokuyo_laser_sensor}" >
-      <xacro:if value="$(arg real)" >
-        <xacro:hokuyo_laser_sensor control="true" />
-      </xacro:if>
-      <xacro:unless value="$(arg real)" >
-        <xacro:hokuyo_laser_sensor control="$(arg control)" />
-      </xacro:unless>
-    </xacro:if>
-    <!-- ================================================================== -->
-    <xacro:if value="${enable_kinect_sensor}" >
-      <xacro:if value="$(arg real)" >
-        <xacro:kinect_sensor control="true" />
-      </xacro:if>
-      <xacro:unless value="$(arg real)" >
-        <xacro:kinect_sensor control="$(arg control)" />
-      </xacro:unless>
-    </xacro:if>
-    <!-- ================================================================== -->
-    <xacro:if value="${enable_sonar_sensors}" >
-      <xacro:sonar_sensor prefix_y="left" reflect_y="1" />
-      <xacro:sonar_sensor prefix_y="right" reflect_y="-1" />
-    </xacro:if>
     <!-- ================================================================== -->
     <xacro:if value="${enable_thermal_sensors}" >
-      <xacro:thermal_sensors />
+      <!-- ================================================================ -->
+      <xacro:if value="${enable_middle_thermal_sensor}" >
+        <xacro:middle_thermal_sensor />
+      </xacro:if>
+      <!-- ================================================================ -->
+      <xacro:if value="${enable_left_thermal_sensor}" >
+        <xacro:left_thermal_sensor />
+      </xacro:if>
+      <!-- ================================================================ -->
+      <xacro:if value="${enable_right_thermal_sensor}" >
+        <xacro:right_thermal_sensor />
+      </xacro:if>
+      <!-- ================================================================ -->
     </xacro:if>
     <!-- ================================================================== -->
@@ -171,90 +124,4 @@
     <!-- ================================================================== -->
   </xacro:if>
-<!-- Load Transmissions ################################################### -->
-  <xacro:unless value="$(arg real)" >
-    <xacro:if value="$(arg control)" >
-      <!-- ================================================================ -->
-      <xacro:if value="${enable_linear_elevator_link}" >
-        <xacro:linear_elevator_transmission />
-      </xacro:if>
-      <!-- ================================================================ -->
-      <xacro:if value="${enable_linear_head_link}" >
-        <xacro:linear_head_transmission rotation="pitch" />
-        <xacro:linear_head_transmission rotation="yaw" />
-      </xacro:if>
-      <!-- ================================================================ -->
-      <xacro:if value="${enable_wheel_links}" >
-        <xacro:wheel_transmission prefix_y="left" prefix_x="front" />
-        <xacro:wheel_transmission prefix_y="left" prefix_x="rear" />
-        <xacro:wheel_transmission prefix_y="right" prefix_x="front" />
-        <xacro:wheel_transmission prefix_y="right" prefix_x="rear" />
-      </xacro:if>
-      <!-- ================================================================ -->
-      <xacro:if value="${enable_sensors}" >
-        <!-- ============================================================== -->
-        <xacro:if value="${enable_hokuyo_laser_sensor}" >
-          <xacro:sensor_transmission sensor="laser" rotation="roll" />
-          <xacro:sensor_transmission sensor="laser" rotation="pitch" />
-        </xacro:if>
-        <!-- ============================================================== -->
-        <xacro:if value="${enable_kinect_sensor}" >
-          <xacro:sensor_transmission sensor="kinect" rotation="pitch" />
-          <xacro:sensor_transmission sensor="kinect" rotation="yaw" />
-        </xacro:if>
-        <!-- ============================================================== -->
-      </xacro:if>
-      <!-- ================================================================ -->
-    </xacro:if>
-  </xacro:unless>
-<!-- Load Plugins ######################################################### -->
-  <xacro:unless value="$(arg real)" >
-    <xacro:if value="${enable_plugins}" >
-      <!-- ================================================================ -->
-      <xacro:if value="${enable_pandora_differential_plugin}" >
-        <xacro:if value="$(arg interface)" >
-          <xacro:pandora_differential_plugin publish_joint_states="false" />
-        </xacro:if>
-        <xacro:unless value="$(arg interface)" >
-          <xacro:pandora_differential_plugin publish_joint_states="true" />
-        </xacro:unless>
-      </xacro:if>
-      <!-- ================================================================ -->
-      <xacro:if value="$(arg control)" >
-        <xacro:if value="$(arg interface)" >
-          <xacro:gazebo_ros_control_plugin hw_sim="pandora_gazebo_interface/GazeboInterface"
-                                           ns="control" />
-        </xacro:if>
-        <xacro:unless value="$(arg interface)" >
-          <xacro:gazebo_ros_control_plugin hw_sim="gazebo_ros_control/DefaultRobotHWSim"
-                                           ns="control" />
-        </xacro:unless>
-      </xacro:if>
-      <!-- ================================================================ -->
-      <xacro:if value="${enable_pandora_p3d_plugin}" >
-        <xacro:pandora_p3d_plugin />
-      </xacro:if>
-      <!-- ================================================================ -->
-      <xacro:if value="$(arg control)" >
-        <xacro:if value="${enable_ros_imu_plugin}" >
-          <xacro:ros_imu_plugin />
-        </xacro:if>
-      </xacro:if>
-      <!-- ================================================================ -->
-      <xacro:if value="${enable_sensors}" >
-        <xacro:if value="${enable_hokuyo_laser_sensor}" >
-          <xacro:unless value="$(arg control)" >
-            <xacro:if value="${enable_pandora_imu_stabilizer_plugin}" >
-              <xacro:pandora_imu_stabilizer_plugin />
-            </xacro:if>
-          </xacro:unless>
-        </xacro:if>
-      </xacro:if>
-      <!-- ================================================================ -->
-      <xacro:unless value="$(arg control)" >
-        <xacro:ros_skid_steer_drive_plugin />
-      </xacro:unless>
-    <!-- ================================================================== -->
-    </xacro:if>
-  </xacro:unless>
 <!-- ###################################################################### -->
 </robot>

File: pandora_sensors_description/urdf/hokuyo_utm_30lx.urdf.xacro (robot description, xacro)
@@ -3,5 +3,5 @@
   <xacro:macro name="hokuyo_caster"
                params="parent
-                       control
+                       fixed
                        roll_min_limit
                        roll_max_limit
@@ -91,5 +91,13 @@
     </link>
     <!-- Roll Joint ########################################################-->
-    <xacro:if value="${control}" >
+    <xacro:if value="${fixed}" >
+      <joint name="laser_roll_joint"
+             type="fixed" >
+        <parent link="${parent}" />
+        <child link="hokuyo_base_link" />
+        <xacro:insert_block name="origin" />
+      </joint>
+    </xacro:if>
+    <xacro:unless value="${fixed}" >
       <joint name="laser_roll_joint"
              type="revolute" >
@@ -103,15 +111,16 @@
                velocity="50.0" />
       </joint>
-    </xacro:if>
-    <xacro:unless value="${control}" >
-      <joint name="laser_roll_joint"
-             type="fixed" >
-        <parent link="${parent}" />
-        <child link="hokuyo_base_link" />
-        <xacro:insert_block name="origin" />
-      </joint>
     </xacro:unless>
     <!-- Pitch Joint #######################################################-->
-    <xacro:if value="${control}" >
+    <xacro:if value="${fixed}" >
+      <joint name="laser_pitch_joint"
+             type="fixed" >
+        <parent link="hokuyo_base_link" />
+        <child link="laser_link" />
+        <origin xyz="0.013 0 0.02301"
+                rpy="0 0 0" />
+      </joint>
+    </xacro:if>
+    <xacro:unless value="${fixed}" >
       <joint name="laser_pitch_joint"
              type="revolute" >
@@ -126,13 +135,4 @@
                velocity="50.0" />
       </joint>
-    </xacro:if>
-    <xacro:unless value="${control}" >
-      <joint name="laser_pitch_joint"
-             type="fixed" >
-        <parent link="hokuyo_base_link" />
-        <child link="laser_link" />
-        <origin xyz="0.013 0 0.02301"
-                rpy="0 0 0" />
-      </joint>
     </xacro:unless>
   </xacro:macro>
