Commit message: Refactor gears description.

File: pandora_sensors_description/urdf/kinect_camera.urdf.xacro (robot description, xacro)
@@ -3,5 +3,5 @@
   <xacro:macro name="kinect_caster"
                params="parent
-                       control
+                       fixed
                        pitch_min_limit
                        pitch_max_limit
@@ -52,5 +52,5 @@
                 filename="libgazebo_ros_openni_kinect.so" >
           <pointCloudTopicName>point_cloud</pointCloudTopicName>
-          <frameName>kinect_camera</frameName>
+          <frameName>kinect_link</frameName>
           <cameraName>kinect</cameraName>
           <imageTopicName>image</imageTopicName>
@@ -88,5 +88,13 @@
     </link>
     <!-- Pitch Joint #######################################################-->
-    <xacro:if value="${control}" >
+    <xacro:if value="${fixed}" >
+      <joint name="kinect_pitch_joint"
+             type="fixed" >
+        <parent link="${parent}" />
+        <child link="kinect_base_link" />
+        <xacro:insert_block name="origin" />
+      </joint>
+    </xacro:if>
+    <xacro:unless value="${fixed}" >
       <joint name="kinect_pitch_joint"
              type="revolute" >
@@ -100,15 +108,16 @@
                velocity="50.0" />
       </joint>
-    </xacro:if>
-    <xacro:unless value="${control}" >
-      <joint name="kinect_pitch_joint"
-             type="fixed" >
-        <parent link="${parent}" />
-        <child link="kinect_base_link" />
-        <xacro:insert_block name="origin" />
-      </joint>
     </xacro:unless>
     <!-- Yaw Joint #########################################################-->
-    <xacro:if value="${control}" >
+    <xacro:if value="${fixed}" >
+      <joint name="kinect_yaw_joint"
+             type="fixed" >
+        <parent link="kinect_base_link" />
+        <child link="kinect_link" />
+        <origin xyz="0.037 0.0 0.021"
+                rpy="0.0 0.0 0.0" />
+      </joint>
+    </xacro:if>
+    <xacro:unless value="${fixed}" >
       <joint name="kinect_yaw_joint"
              type="revolute" >
@@ -123,13 +132,4 @@
                velocity="50.0" />
       </joint>
-    </xacro:if>
-    <xacro:unless value="${control}" >
-      <joint name="kinect_yaw_joint"
-             type="fixed" >
-        <parent link="kinect_base_link" />
-        <child link="kinect_link" />
-        <origin xyz="0.037 0.0 0.021"
-                rpy="0.0 0.0 0.0" />
-      </joint>
     </xacro:unless>
   </xacro:macro>

Commit message: Add macro for robot bringup and update description launcher.

File: pandora_robots_description/urdf/gears/gears.urdf.xacro (robot description, xacro)
@@ -1,5 +1,4 @@
 <?xml version="1.0"?>
-<robot name="gears"
-       xmlns:xacro="http://ros.org/wiki/xacro" >
+<robot xmlns:xacro="http://ros.org/wiki/xacro" >
 <!-- Import Files ######################################################### -->
   <!-- ==================================================================== -->
@@ -30,4 +29,6 @@
   <xacro:include filename="$(find pandora_robots_description)/urdf/gears/sensors/microphone_sensor.xacro" />
   <!-- ==================================================================== -->
+<xacro:macro name="gears_urdf"
+             params="fixed" >
 <!-- Load Links & Joints ################################################## -->
   <xacro:if value="${enable_base_link}" >
@@ -62,5 +63,5 @@
     <xacro:if value="${enable_linear_elevator_link}" >
       <xacro:linear_elevator_link />
-      <xacro:linear_elevator_joint fixed="$(arg fixed)" />
+      <xacro:linear_elevator_joint fixed="${fixed}" />
     </xacro:if>
     <!-- ================================================================== -->
@@ -69,10 +70,10 @@
       <xacro:if value="${enable_linear_head_base_link}" >
         <xacro:linear_head_base_link />
-        <xacro:linear_head_pitch_joint fixed="$(arg fixed)" />
+        <xacro:linear_head_pitch_joint fixed="${fixed}" />
       </xacro:if>
       <!-- ================================================================ -->
       <xacro:if value="${enable_linear_head_main_link}" >
         <xacro:linear_head_main_link />
-        <xacro:linear_head_yaw_joint fixed="$(arg fixed)" />
+        <xacro:linear_head_yaw_joint fixed="${fixed}" />
       </xacro:if>
       <!-- ================================================================ -->
@@ -83,8 +84,8 @@
   <xacro:if value="${enable_sensors}" >
     <xacro:if value="${enable_laser_sensor}" >
-      <xacro:laser_sensor fixed="$(arg fixed)" />
+      <xacro:laser_sensor fixed="${fixed}" />
     </xacro:if>
     <xacro:if value="${enable_kinect_sensor}" >
-      <xacro:kinect_sensor fixed="$(arg fixed)" />
+      <xacro:kinect_sensor fixed="${fixed}" />
     </xacro:if>
     <xacro:if value="${enable_sonar_sensors}" >
@@ -121,4 +122,5 @@
     </xacro:if>
   </xacro:if>
+</xacro:macro>
 <!-- ###################################################################### -->
 </robot>

Commit message: Add optical frame links to kinect.

File: pandora_robots_description/urdf/gears/gears.urdf.xacro (robot description, xacro)
@@ -91,10 +91,10 @@
     <xacro:if value="${enable_sonar_sensors}" >
       <!-- ================================================================ -->
-      <xacro:if value="${enable_left_rear_sonar_sensor}" >
-        <xacro:left_rear_sonar_sensor />
+      <xacro:if value="${enable_left_sonar_sensor}" >
+        <xacro:left_sonar_sensor />
       </xacro:if>
       <!-- ================================================================ -->
-      <xacro:if value="${enable_right_rear_sonar_sensor}" >
-        <xacro:right_rear_sonar_sensor />
+      <xacro:if value="${enable_right_sonar_sensor}" >
+        <xacro:right_sonar_sensor />
       </xacro:if>
       <!-- ================================================================ -->

File: pandora_robots_description/urdf/gears/sensors/sonar_sensor.xacro (robot description, xacro)
@@ -6,6 +6,6 @@
 <!-- ###################################################################### -->
   <!-- ==================================================================== -->
-  <xacro:macro name="left_rear_sonar_sensor" >
-    <xacro:sonar_caster name="left_rear"
+  <xacro:macro name="left_sonar_sensor" >
+    <xacro:sonar_caster name="left"
                         parent="base_link" >
       <origin xyz="-0.15519 0.11249 0.14305"
@@ -14,6 +14,6 @@
   </xacro:macro>
   <!-- ==================================================================== -->
-  <xacro:macro name="right_rear_sonar_sensor" >
-    <xacro:sonar_caster name="right_rear"
+  <xacro:macro name="right_sonar_sensor" >
+    <xacro:sonar_caster name="right"
                         parent="base_link" >
       <origin xyz="-0.15519 -0.11351 0.14305"

File: pandora_robots_description/urdf/gears/urdf_configurations.xacro (robot description, xacro)
@@ -23,6 +23,6 @@
     <!-- ================================================================== -->
     <xacro:property name="enable_sonar_sensors" value="true" />
-      <xacro:property name="enable_left_rear_sonar_sensor" value="true" />
-      <xacro:property name="enable_right_rear_sonar_sensor" value="true" />
+      <xacro:property name="enable_left_sonar_sensor" value="true" />
+      <xacro:property name="enable_right_sonar_sensor" value="true" />
     <!-- ================================================================== -->
     <xacro:property name="enable_thermal_sensors" value="true" />

File: pandora_sensors_description/urdf/hokuyo_utm_30lx.urdf.xacro (robot description, xacro)
@@ -84,5 +84,22 @@
       </collision>
     </link>
-    <!-- Roll Joint ########################################################-->
+    <!-- ################################################################## -->
+    <link name="laser_link" >
+      <inertial>
+        <!-- ============================================================== -->
+        <origin xyz="0.0 0.0 0.0" />
+        <!-- ============================================================== -->
+        <mass value="0.0001" /><!--FIXME-->
+        <!-- ============================================================== -->
+        <inertia ixx="0.00000001"
+                 ixy="0"
+                 ixz="0"
+                 iyy="0.00000001"
+                 iyz="0"
+                 izz="0.00000001" /><!--FIXME-->
+        <!-- ============================================================== -->
+      </inertial>
+    </link>
+    <!-- Roll Joint ####################################################### -->
     <xacro:if value="${fixed}" >
       <joint name="laser_roll_joint"
@@ -125,5 +142,5 @@
       </joint>
     </xacro:unless>
-    <!-- Pitch Joint #######################################################-->
+    <!-- Pitch Joint ###################################################### -->
     <xacro:if value="${fixed}" >
       <joint name="laser_pitch_joint"
@@ -168,4 +185,15 @@
       </joint>
     </xacro:unless>
+    <!-- Ray Joint ######################################################## -->
+    <joint name="laser_joint"
+           type="fixed" >
+      <!-- ================================================================ -->
+      <parent link="laser_main_link" />
+      <child link="laser_link" />
+      <!-- ================================================================ -->
+      <origin xyz="0.0225 0.0 0.105"
+              rpy="0 0 0" />
+      <!-- ================================================================ -->
+    </joint>
   </xacro:macro>
 <!-- ###################################################################### -->

File: pandora_sensors_description/urdf/kinect_camera.urdf.xacro (robot description, xacro)
@@ -84,4 +84,106 @@
       </collision>
     </link>
+    <!-- ################################################################## -->
+    <link name="kinect_frame" >
+      <inertial>
+        <!-- ============================================================== -->
+        <origin xyz="0.0 0.0 0.0" />
+        <!-- ============================================================== -->
+        <mass value="0.0001" /><!--FIXME-->
+        <!-- ============================================================== -->
+        <inertia ixx="0.00000001"
+                 ixy="0"
+                 ixz="0"
+                 iyy="0.00000001"
+                 iyz="0"
+                 izz="0.00000001" /><!--FIXME-->
+        <!-- ============================================================== -->
+      </inertial>
+    </link>
+    <!-- ################################################################## -->
+    <link name="kinect_optical_frame" >
+      <inertial>
+        <!-- ============================================================== -->
+        <origin xyz="0.0 0.0 0.0" />
+        <!-- ============================================================== -->
+        <mass value="0.0001" /><!--FIXME-->
+        <!-- ============================================================== -->
+        <inertia ixx="0.00000001"
+                 ixy="0"
+                 ixz="0"
+                 iyy="0.00000001"
+                 iyz="0"
+                 izz="0.00000001" /><!--FIXME-->
+        <!-- ============================================================== -->
+      </inertial>
+    </link>
+    <!-- ################################################################## -->
+    <link name="kinect_depth_frame" >
+      <inertial>
+        <!-- ============================================================== -->
+        <origin xyz="0.0 0.0 0.0" />
+        <!-- ============================================================== -->
+        <mass value="0.0001" /><!--FIXME-->
+        <!-- ============================================================== -->
+        <inertia ixx="0.00000001"
+                 ixy="0"
+                 ixz="0"
+                 iyy="0.00000001"
+                 iyz="0"
+                 izz="0.00000001" /><!--FIXME-->
+        <!-- ============================================================== -->
+      </inertial>
+    </link>
+    <!-- ################################################################## -->
+    <link name="kinect_depth_optical_frame" >
+      <inertial>
+        <!-- ============================================================== -->
+        <origin xyz="0.0 0.0 0.0" />
+        <!-- ============================================================== -->
+        <mass value="0.0001" /><!--FIXME-->
+        <!-- ============================================================== -->
+        <inertia ixx="0.00000001"
+                 ixy="0"
+                 ixz="0"
+                 iyy="0.00000001"
+                 iyz="0"
+                 izz="0.00000001" /><!--FIXME-->
+        <!-- ============================================================== -->
+      </inertial>
+    </link>
+    <!-- ################################################################## -->
+    <link name="kinect_rgb_frame" >
+      <inertial>
+        <!-- ============================================================== -->
+        <origin xyz="0.0 0.0 0.0" />
+        <!-- ============================================================== -->
+        <mass value="0.0001" /><!--FIXME-->
+        <!-- ============================================================== -->
+        <inertia ixx="0.00000001"
+                 ixy="0"
+                 ixz="0"
+                 iyy="0.00000001"
+                 iyz="0"
+                 izz="0.00000001" /><!--FIXME-->
+        <!-- ============================================================== -->
+      </inertial>
+    </link>
+    <!-- ################################################################## -->
+    <link name="kinect_rgb_optical_frame" >
+      <inertial>
+        <!-- ============================================================== -->
+        <origin xyz="0.0 0.0 0.0" />
+        <!-- ============================================================== -->
+        <mass value="0.0001" /><!--FIXME-->
+        <!-- ============================================================== -->
+        <inertia ixx="0.00000001"
+                 ixy="0"
+                 ixz="0"
+                 iyy="0.00000001"
+                 iyz="0"
+                 izz="0.00000001" /><!--FIXME-->
+        <!-- ============================================================== -->
+      </inertial>
+    </link>
     <!-- Pitch Joint #######################################################-->
     <xacro:if value="${fixed}" >
@@ -168,4 +270,67 @@
       </joint>
     </xacro:unless>
+    <!-- Camera Joint ##################################################### -->
+    <joint name="kinect_joint"
+           type="fixed" >
+      <!-- ================================================================ -->
+      <parent link="kinect_main_link" />
+      <child link="kinect_frame" />
+      <!-- ================================================================ -->
+      <origin xyz="0.03016 0.0 0.01781"
+              rpy="0.0 0.0 0.0" />
+      <!-- ================================================================ -->
+    </joint>
+    <joint name="kinect_optical_joint"
+           type="fixed" >
+      <!-- ================================================================ -->
+      <parent link="kinect_frame" />
+      <child link="kinect_optical_frame" />
+      <!-- ================================================================ -->
+      <origin xyz="0.0 0.0 0.0"
+              rpy="-1.5708 0.0 -1.5708" />
+      <!-- ================================================================ -->
+    </joint>
+    <!-- Depth Joint ###################################################### -->
+    <joint name="kinect_depth_joint"
+           type="fixed" >
+      <!-- ================================================================ -->
+      <parent link="kinect_frame" />
+      <child link="kinect_depth_frame" />
+      <!-- ================================================================ -->
+      <origin xyz="0.0 -0.02 0.0"
+              rpy="0.0 0.0 0.0" />
+      <!-- ================================================================ -->
+    </joint>
+    <joint name="kinect_depth_optical_joint"
+           type="fixed" >
+      <!-- ================================================================ -->
+      <parent link="kinect_depth_frame" />
+      <child link="kinect_depth_optical_frame" />
+      <!-- ================================================================ -->
+      <origin xyz="0.0 0.0 0.0"
+              rpy="-1.5708 0.0 -1.5708" />
+      <!-- ================================================================ -->
+    </joint>
+    <!-- RGB Joint ######################################################## -->
+    <joint name="kinect_rgb_joint"
+           type="fixed" >
+      <!-- ================================================================ -->
+      <parent link="kinect_frame" />
+      <child link="kinect_rgb_frame" />
+      <!-- ================================================================ -->
+      <origin xyz="0.0 -0.045 0.0"
+              rpy="0.0 0.0 0.0" />
+      <!-- ================================================================ -->
+    </joint>
+    <joint name="kinect_rgb_optical_joint"
+           type="fixed" >
+      <!-- ================================================================ -->
+      <parent link="kinect_rgb_frame" />
+      <child link="kinect_rgb_optical_frame" />
+      <!-- ================================================================ -->
+      <origin xyz="0.0 0.0 0.0"
+              rpy="-1.5708 0.0 -1.5708" />
+      <!-- ================================================================ -->
+    </joint>
   </xacro:macro>
 <!-- ###################################################################### -->
