Commit message: Remove redundant properties and conditionals from gears' description.

File: pandora_robots_description/urdf/gears/gears.urdf.xacro (robot description, xacro)
@@ -32,53 +32,37 @@
              params="fixed" >
 <!-- Load Links & Joints ################################################## -->
-  <xacro:if value="${enable_base_link}" >
-    <xacro:base_link />
-  </xacro:if>
-  <xacro:if value="${enable_side_links}" >
-    <!-- ================================================================== -->
-    <xacro:side_link prefix_y="left" reflect_y="1" />
-    <xacro:side_joint prefix_y="left" reflect_y="1" />
-    <!-- ================================================================== -->
-    <xacro:side_link prefix_y="right" reflect_y="-1" />
-    <xacro:side_joint prefix_y="right" reflect_y="-1" />
-    <!-- ================================================================== -->
-  </xacro:if>
-  <xacro:if value="${enable_wheel_links}" >
-    <!-- ================================================================== -->
-    <xacro:wheel_link prefix_y="left" prefix_x="front" reflect_y="1" reflect_x="1" />
-    <xacro:wheel_joint prefix_y="left" prefix_x="front" reflect_y="1" reflect_x="1" />
-    <!-- ================================================================== -->
-    <xacro:wheel_link prefix_y="left" prefix_x="rear" reflect_y="1" reflect_x="-1" />
-    <xacro:wheel_joint prefix_y="left" prefix_x="rear" reflect_y="1" reflect_x="-1" />
-    <!-- ================================================================== -->
-    <xacro:wheel_link prefix_y="right" prefix_x="front" reflect_y="-1" reflect_x="1" />
-    <xacro:wheel_joint prefix_y="right" prefix_x="front" reflect_y="-1" reflect_x="1" />
-    <!-- ================================================================== -->
-    <xacro:wheel_link prefix_y="right" prefix_x="rear" reflect_y="-1" reflect_x="-1" />
-    <xacro:wheel_joint prefix_y="right" prefix_x="rear" reflect_y="-1" reflect_x="-1" />
-    <!-- ================================================================== -->
-  </xacro:if>
-  <xacro:if value="${enable_linear_links}" >
-    <!-- ================================================================== -->
-    <xacro:if value="${enable_linear_elevator_link}" >
-      <xacro:linear_elevator_link />
-      <xacro:linear_elevator_joint fixed="${fixed}" />
-    </xacro:if>
-    <!-- ================================================================== -->
-    <xacro:if value="${enable_linear_head_links}" >
-      <!-- ================================================================ -->
-      <xacro:if value="${enable_linear_head_base_link}" >
-        <xacro:linear_head_base_link />
-        <xacro:linear_head_pitch_joint fixed="${fixed}" />
-      </xacro:if>
-      <!-- ================================================================ -->
-      <xacro:if value="${enable_linear_head_main_link}" >
-        <xacro:linear_head_main_link />
-        <xacro:linear_head_yaw_joint fixed="${fixed}" />
-      </xacro:if>
-      <!-- ================================================================ -->
-    </xacro:if>
-    <!-- ================================================================== -->
-  </xacro:if>
+  <!-- ================================================================== -->
+  <xacro:base_link />
+  <!-- ================================================================== -->
+  <!-- ================================================================== -->
+  <xacro:side_link prefix_y="left" reflect_y="1" />
+  <xacro:side_joint prefix_y="left" reflect_y="1" />
+  <!-- ================================================================== -->
+  <xacro:side_link prefix_y="right" reflect_y="-1" />
+  <xacro:side_joint prefix_y="right" reflect_y="-1" />
+  <!-- ================================================================== -->
+  <!-- ================================================================== -->
+  <xacro:wheel_link prefix_y="left" prefix_x="front" reflect_y="1" reflect_x="1" />
+  <xacro:wheel_joint prefix_y="left" prefix_x="front" reflect_y="1" reflect_x="1" />
+  <!-- ================================================================== -->
+  <xacro:wheel_link prefix_y="left" prefix_x="rear" reflect_y="1" reflect_x="-1" />
+  <xacro:wheel_joint prefix_y="left" prefix_x="rear" reflect_y="1" reflect_x="-1" />
+  <!-- ================================================================== -->
+  <xacro:wheel_link prefix_y="right" prefix_x="front" reflect_y="-1" reflect_x="1" />
+  <xacro:wheel_joint prefix_y="right" prefix_x="front" reflect_y="-1" reflect_x="1" />
+  <!-- ================================================================== -->
+  <xacro:wheel_link prefix_y="right" prefix_x="rear" reflect_y="-1" reflect_x="-1" />
+  <xacro:wheel_joint prefix_y="right" prefix_x="rear" reflect_y="-1" reflect_x="-1" />
+  <!-- ================================================================== -->
+  <!-- ================================================================== -->
+  <xacro:linear_elevator_link />
+  <xacro:linear_elevator_joint fixed="${fixed}" />
+  <!-- ================================================================== -->
+  <xacro:linear_head_base_link />
+  <xacro:linear_head_pitch_joint fixed="${fixed}" />
+  <!-- ================================================================== -->
+  <xacro:linear_head_main_link />
+  <xacro:linear_head_yaw_joint fixed="${fixed}" />
+  <!-- ================================================================== -->
 <!-- Load Sensors ######################################################### -->
   <xacro:if value="${enable_sensors}" >

File: pandora_robots_description/urdf/gears/urdf_configurations.xacro (robot description, xacro)
@@ -2,17 +2,4 @@
 <robot xmlns:xacro="http://ros.org/wiki/xacro" >
 <!-- Elements' Status ##################################################### -->
-  <!-- Links ============================================================== -->
-  <xacro:property name="enable_base_link" value="true" />
-    <!-- ================================================================== -->
-  <xacro:property name="enable_side_links" value="true" />
-    <!-- ================================================================== -->
-  <xacro:property name="enable_wheel_links" value="true" />
-    <!-- ================================================================== -->
-  <xacro:property name="enable_linear_links" value="true" />
-    <xacro:property name="enable_linear_elevator_link" value="true" />
-    <xacro:property name="enable_linear_head_links" value="true" />
-      <xacro:property name="enable_linear_head_base_link" value="true" />
-      <xacro:property name="enable_linear_head_main_link" value="true" />
-  <!-- ==================================================================== -->
   <!-- Sensors ============================================================ -->
   <xacro:property name="enable_sensors" value="true" />

Commit message: Add cameras to urdf.

File: pandora_robots_description/urdf/gears/gears.urdf.xacro (robot description, xacro)
@@ -24,4 +24,5 @@
   <xacro:include filename="$(find pandora_robots_description)/urdf/gears/sensors/laser_sensor.xacro" />
   <xacro:include filename="$(find pandora_robots_description)/urdf/gears/sensors/kinect_sensor.xacro" />
+  <xacro:include filename="$(find pandora_robots_description)/urdf/gears/sensors/camera_sensor.xacro" />
   <xacro:include filename="$(find pandora_robots_description)/urdf/gears/sensors/sonar_sensor.xacro" />
   <xacro:include filename="$(find pandora_robots_description)/urdf/gears/sensors/thermal_sensor.xacro" />
@@ -73,4 +74,15 @@
       <xacro:kinect_sensor fixed="${fixed}" />
     </xacro:if>
+    <xacro:if value="${enable_camera_sensors}" >
+      <!-- ================================================================ -->
+      <xacro:if value="${enable_left_camera_sensor}" >
+        <xacro:left_camera_sensor />
+      </xacro:if>
+      <!-- ================================================================ -->
+      <xacro:if value="${enable_right_camera_sensor}" >
+        <xacro:right_camera_sensor />
+      </xacro:if>
+      <!-- ================================================================ -->
+    </xacro:if>
     <xacro:if value="${enable_sonar_sensors}" >
       <!-- ================================================================ -->

File: pandora_robots_description/urdf/gears/sensors/camera_sensor.xacro (robot description, xacro)
@@ -8,7 +8,7 @@
   <xacro:macro name="left_camera_sensor" >
     <xacro:camera_caster parent="base_link"
-                           prefix_y="left" >
-      <origin xyz=""
-              rpy="" />
+                         prefix_y="left" >
+      <origin xyz="-0.10874 0.0754 0.38825"
+              rpy="0.0 0.0 ${ 3 * PI_4 }" />
     </xacro:camera_caster>
   </xacro:macro>
@@ -16,7 +16,7 @@
   <xacro:macro name="right_camera_sensor" >
     <xacro:camera_caster parent="base_link"
-                           prefix_y="right" >
-      <origin xyz=""
-              rpy="" />
+                         prefix_y="right" >
+      <origin xyz="-0.10874 -0.0754 0.38825"
+              rpy="0.0 0.0 ${ 5 * PI_4 }" />
     </xacro:camera_caster>
   </xacro:macro>

File: pandora_robots_description/urdf/gears/urdf_configurations.xacro (robot description, xacro)
@@ -8,4 +8,8 @@
     <!-- ================================================================== -->
     <xacro:property name="enable_kinect_sensor" value="true" />
+    <!-- ================================================================== -->
+    <xacro:property name="enable_camera_sensors" value="true" />
+      <xacro:property name="enable_left_camera_sensor" value="true" />
+      <xacro:property name="enable_right_camera_sensor" value="true" />
     <!-- ================================================================== -->
     <xacro:property name="enable_sonar_sensors" value="true" />

File: pandora_sensors_description/urdf/logitech_camera.urdf.xacro (robot description, xacro)
@@ -5,5 +5,5 @@
                params="parent prefix_y *origin" >
     <!-- ################################################################## -->
-    <link name="${prefix_y}_camera_link" >
+    <link name="${prefix_y}_camera_main_link" >
       <inertial>
         <!-- ============================================================== -->
@@ -42,13 +42,70 @@
     </link>
     <!-- ################################################################## -->
-    <joint name="${prefix_y}_camera_joint"
+    <link name="${prefix_y}_camera_frame" >
+      <inertial>
+        <!-- ============================================================== -->
+        <origin xyz="0.0 0.0 0.0" />
+        <!-- ============================================================== -->
+        <mass value="0.0001" />
+        <!-- ============================================================== -->
+        <inertia ixx="0.00000001"
+                 ixy="0"
+                 ixz="0"
+                 iyy="0.00000001"
+                 iyz="0"
+                 izz="0.00000001" />
+        <!-- ============================================================== -->
+      </inertial>
+    </link>
+    <!-- ################################################################## -->
+    <link name="${prefix_y}_camera_optical_frame" >
+      <inertial>
+        <!-- ============================================================== -->
+        <origin xyz="0.0 0.0 0.0" />
+        <!-- ============================================================== -->
+        <mass value="0.0001" />
+        <!-- ============================================================== -->
+        <inertia ixx="0.00000001"
+                 ixy="0"
+                 ixz="0"
+                 iyy="0.00000001"
+                 iyz="0"
+                 izz="0.00000001" />
+        <!-- ============================================================== -->
+      </inertial>
+    </link>
+    <!-- ################################################################## -->
+    <joint name="${prefix_y}_camera_main_joint"
            type="fixed" >
       <!-- ================================================================ -->
       <parent link="${parent}" />
-      <child link="${prefix_y}_camera_link" />
+      <child link="${prefix_y}_camera_main_link" />
       <!-- ================================================================ -->
       <xacro:insert_block name="origin" />
       <!-- ================================================================ -->
     </joint>
+    <!-- ################################################################## -->
+    <joint name="${prefix_y}_camera_joint"
+           type="fixed" >
+      <!-- ================================================================ -->
+      <parent link="${prefix_y}_camera_main_link" />
+      <child link="${prefix_y}_camera_frame" />
+      <!-- ================================================================ -->
+      <origin xyz="0.02499 0.0 0.05704"
+              rpy="0.0 -0.2792 0.0" />
+      <!-- ================================================================ -->
+    </joint>
+    <!-- ################################################################## -->
+    <joint name="${prefix_y}_camera_optical_joint"
+           type="fixed" >
+      <!-- ================================================================ -->
+      <parent link="${prefix_y}_camera_frame" />
+      <child link="${prefix_y}_camera_optical_frame" />
+      <!-- ================================================================ -->
+      <origin xyz="0.0 0.0 0.0"
+              rpy="-1.5708 0.0 -1.5708" />
+      <!-- ================================================================ -->
+    </joint>
+    <!-- ################################################################## -->
   </xacro:macro>
 <!-- ###################################################################### -->

Commit message: Add linear sonar link.

File: pandora_robots_description/urdf/gears/gears.urdf.xacro (robot description, xacro)
@@ -87,4 +87,8 @@
     <xacro:if value="${enable_sonar_sensors}" >
       <!-- ================================================================ -->
+      <xacro:if value="${enable_linear_sonar_sensor}" >
+        <xacro:linear_sonar_sensor />
+      </xacro:if>
+      <!-- ================================================================ -->
       <xacro:if value="${enable_left_sonar_sensor}" >
         <xacro:left_sonar_sensor />

File: pandora_robots_description/urdf/gears/sensors/sonar_sensor.xacro (robot description, xacro)
@@ -6,6 +6,14 @@
 <!-- ###################################################################### -->
   <!-- ==================================================================== -->
+  <xacro:macro name="linear_sonar_sensor" >
+    <xacro:sonar_caster name="linear"
+                        parent="linear_elevator_link" >
+      <origin xyz="0.01195 0.0 0.32700"
+              rpy="${zero}" />
+    </xacro:sonar_caster>
+  </xacro:macro>
+  <!-- ==================================================================== -->
   <xacro:macro name="left_sonar_sensor" >
-    <xacro:sonar_caster prefix_y="left"
+    <xacro:sonar_caster name="left"
                         parent="base_link" >
       <origin xyz="-0.15026 0.06429 0.39925"
@@ -15,5 +23,5 @@
   <!-- ==================================================================== -->
   <xacro:macro name="right_sonar_sensor" >
-    <xacro:sonar_caster prefix_y="right"
+    <xacro:sonar_caster name="right"
                         parent="base_link" >
       <origin xyz="-0.15026 -0.06429 0.39925"

File: pandora_robots_description/urdf/gears/urdf_configurations.xacro (robot description, xacro)
@@ -14,4 +14,5 @@
     <!-- ================================================================== -->
     <xacro:property name="enable_sonar_sensors" value="true" />
+      <xacro:property name="enable_linear_sonar_sensor" value="true" />
       <xacro:property name="enable_left_sonar_sensor" value="true" />
       <xacro:property name="enable_right_sonar_sensor" value="true" />

File: pandora_sensors_description/urdf/sonar.urdf.xacro (robot description, xacro)
@@ -3,7 +3,7 @@
 <!-- ###################################################################### -->
   <xacro:macro name="sonar_caster"
-               params="parent prefix_y *origin" >
+               params="parent name *origin" >
     <!-- ################################################################## -->
-    <link name="${prefix_y}_sonar_link" >
+    <link name="${name}_sonar_link" >
       <inertial>
         <!-- ============================================================== -->
@@ -42,5 +42,5 @@
     </link>
     <!-- ################################################################## -->
-    <link name="${prefix_y}_sonar_frame" >
+    <link name="${name}_sonar_frame" >
       <inertial>
         <!-- ============================================================== -->
@@ -59,9 +59,9 @@
     </link>
     <!-- ################################################################## -->
-    <joint name="${prefix_y}_sonar_main_joint"
+    <joint name="${name}_sonar_main_joint"
            type="fixed" >
       <!-- ================================================================ -->
       <parent link="${parent}" />
-      <child link="${prefix_y}_sonar_link" />
+      <child link="${name}_sonar_link" />
       <!-- ================================================================ -->
       <xacro:insert_block name="origin" />
@@ -69,9 +69,9 @@
     </joint>
     <!-- ################################################################## -->
-    <joint name="${prefix_y}_sonar_joint"
+    <joint name="${name}_sonar_joint"
            type="fixed" >
       <!-- ================================================================ -->
-      <parent link="${prefix_y}_sonar_link" />
-      <child link="${prefix_y}_sonar_frame" />
+      <parent link="${name}_sonar_link" />
+      <child link="${name}_sonar_frame" />
       <!-- ================================================================ -->
       <origin xyz="0.015 0.0 0.0"
