Commit message: Adjust link inertia and masses to fix gazebo-1.9.6 bug.

File: pandora_robots_description/urdf/gears/gears.urdf.xacro (robot description, xacro)
@@ -61,8 +61,8 @@
   <!-- ================================================================== -->
   <xacro:linear_head_base_link />
-  <xacro:linear_head_pitch_joint fixed="${fixed}" />
+  <xacro:linear_head_yaw_joint fixed="${fixed}" />
   <!-- ================================================================== -->
   <xacro:linear_head_main_link />
-  <xacro:linear_head_yaw_joint fixed="${fixed}" />
+  <xacro:linear_head_pitch_joint fixed="${fixed}" />
   <!-- ================================================================== -->
 <!-- Load Sensors ######################################################### -->

File: pandora_robots_description/urdf/gears/links/linear_head_base_link.urdf.xacro (robot description, xacro)
@@ -8,12 +8,12 @@
         <origin xyz="0.0 0.00152 0.02409" />
         <!-- ============================================================== -->
-        <mass value="0.0001" /><!--FIXME-->
+        <mass value="0.005" /><!--FIXME-->
         <!-- ============================================================== -->
-        <inertia ixx="0.00000001"
-                 ixy="0.00000001"
-                 ixz="0.00000001"
-                 iyy="0.00000001"
-                 iyz="0.00000001"
-                 izz="0.00000001" /><!--FIXME-->
+        <inertia ixx="1.0E-6"
+                 ixy="0"
+                 ixz="0"
+                 iyy="1.0E-6"
+                 iyz="0"
+                 izz="1.0E-6" /><!--FIXME-->
         <!-- ============================================================== -->
       </inertial>

File: pandora_robots_description/urdf/gears/urdf_configurations.xacro (robot description, xacro)
@@ -35,7 +35,7 @@
   <xacro:property name="linear_elevator_joint_type" value="prismatic" />
   <!-- ==================================================================== -->
+  <xacro:property name="linear_head_yaw_joint_type" value="revolute" />
+  <!-- ==================================================================== -->
   <xacro:property name="linear_head_pitch_joint_type" value="revolute" />
-  <!-- ==================================================================== -->
-  <xacro:property name="linear_head_yaw_joint_type" value="revolute" />
   <!-- ==================================================================== -->
   <!-- Joint Damping ====================================================== -->
@@ -57,9 +57,9 @@
   <xacro:property name="linear_elevator_joint_max_limit" value="0.18" /> <!--FIXME-->
   <!-- ==================================================================== -->
+  <xacro:property name="linear_head_yaw_joint_min_limit" value="-1.57" /> <!--FIXME-->
+  <xacro:property name="linear_head_yaw_joint_max_limit" value="1.57" /> <!--FIXME-->
+  <!-- ==================================================================== -->
   <xacro:property name="linear_head_pitch_joint_min_limit" value="-1.57" /> <!--FIXME-->
   <xacro:property name="linear_head_pitch_joint_max_limit" value="1.57" /> <!--FIXME-->
-  <!-- ==================================================================== -->
-  <xacro:property name="linear_head_yaw_joint_min_limit" value="-1.57" /> <!--FIXME-->
-  <xacro:property name="linear_head_yaw_joint_max_limit" value="1.57" /> <!--FIXME-->
   <!-- ==================================================================== -->
   <xacro:property name="laser_roll_joint_min_limit" value="-1.57" /> <!--FIXME-->

File: pandora_sensors_description/urdf/camera.urdf.xacro (robot description, xacro)
@@ -47,12 +47,12 @@
         <origin xyz="0.0 0.0 0.0" />
         <!-- ============================================================== -->
-        <mass value="0.0001" />
+        <mass value="0.005" />
         <!-- ============================================================== -->
-        <inertia ixx="0.00000001"
+        <inertia ixx="1.0E-6"
                  ixy="0"
                  ixz="0"
-                 iyy="0.00000001"
+                 iyy="1.0E-6"
                  iyz="0"
-                 izz="0.00000001" />
+                 izz="1.0E-6" />
         <!-- ============================================================== -->
       </inertial>
@@ -64,12 +64,12 @@
         <origin xyz="0.0 0.0 0.0" />
         <!-- ============================================================== -->
-        <mass value="0.0001" />
+        <mass value="0.005" />
         <!-- ============================================================== -->
-        <inertia ixx="0.00000001"
+        <inertia ixx="1.0E-6"
                  ixy="0"
                  ixz="0"
-                 iyy="0.00000001"
+                 iyy="1.0E-6"
                  iyz="0"
-                 izz="0.00000001" />
+                 izz="1.0E-6" />
         <!-- ============================================================== -->
       </inertial>

File: pandora_sensors_description/urdf/co2.urdf.xacro (robot description, xacro)
@@ -47,12 +47,12 @@
         <origin xyz="0.0 0.0 0.0" />
         <!-- ============================================================== -->
-        <mass value="0.0001" />
+        <mass value="0.005" />
         <!-- ============================================================== -->
-        <inertia ixx="0.00000001"
+        <inertia ixx="1.0E-6"
                  ixy="0"
                  ixz="0"
-                 iyy="0.00000001"
+                 iyy="1.0E-6"
                  iyz="0"
-                 izz="0.00000001" />
+                 izz="1.0E-6" />
         <!-- ============================================================== -->
       </inertial>

File: pandora_sensors_description/urdf/kinect.urdf.xacro (robot description, xacro)
@@ -16,12 +16,12 @@
         <origin xyz="0.00754 0.0 0.00124" />
         <!-- ============================================================== -->
-        <mass value="0.0001" /><!--FIXME-->
-        <!-- ============================================================== -->
-        <inertia ixx="0.00000001"
-                 ixy="0"
-                 ixz="0"
-                 iyy="0.00000001"
-                 iyz="0"
-                 izz="0.00000001" /><!--FIXME-->
+        <mass value="0.005" /><!--FIXME-->
+        <!-- ============================================================== -->
+        <inertia ixx="1.0E-6"
+                 ixy="0"
+                 ixz="0"
+                 iyy="1.0E-6"
+                 iyz="0"
+                 izz="1.0E-6" /><!--FIXME-->
         <!-- ============================================================== -->
       </inertial>
@@ -53,12 +53,12 @@
         <origin xyz="0.03416 0.0 0.01146" />
         <!-- ============================================================== -->
-        <mass value="0.0001" /><!--FIXME-->
-        <!-- ============================================================== -->
-        <inertia ixx="0.00000001"
-                 ixy="0"
-                 ixz="0"
-                 iyy="0.00000001"
-                 iyz="0"
-                 izz="0.00000001" /><!--FIXME-->
+        <mass value="0.005" /><!--FIXME-->
+        <!-- ============================================================== -->
+        <inertia ixx="1.0E-6"
+                 ixy="0"
+                 ixz="0"
+                 iyy="1.0E-6"
+                 iyz="0"
+                 izz="1.0E-6" /><!--FIXME-->
         <!-- ============================================================== -->
       </inertial>
@@ -127,12 +127,12 @@
         <origin xyz="0.0 0.0 0.0" />
         <!-- ============================================================== -->
-        <mass value="0.0001" /><!--FIXME-->
-        <!-- ============================================================== -->
-        <inertia ixx="0.00000001"
-                 ixy="0"
-                 ixz="0"
-                 iyy="0.00000001"
-                 iyz="0"
-                 izz="0.00000001" /><!--FIXME-->
+        <mass value="0.005" /><!--FIXME-->
+        <!-- ============================================================== -->
+        <inertia ixx="1.0E-6"
+                 ixy="0"
+                 ixz="0"
+                 iyy="1.0E-6"
+                 iyz="0"
+                 izz="1.0E-6" /><!--FIXME-->
         <!-- ============================================================== -->
       </inertial>
@@ -144,12 +144,12 @@
         <origin xyz="0.0 0.0 0.0" />
         <!-- ============================================================== -->
-        <mass value="0.0001" /><!--FIXME-->
-        <!-- ============================================================== -->
-        <inertia ixx="0.00000001"
-                 ixy="0"
-                 ixz="0"
-                 iyy="0.00000001"
-                 iyz="0"
-                 izz="0.00000001" /><!--FIXME-->
+        <mass value="0.005" /><!--FIXME-->
+        <!-- ============================================================== -->
+        <inertia ixx="1.0E-6"
+                 ixy="0"
+                 ixz="0"
+                 iyy="1.0E-6"
+                 iyz="0"
+                 izz="1.0E-6" /><!--FIXME-->
         <!-- ============================================================== -->
       </inertial>
@@ -161,12 +161,12 @@
         <origin xyz="0.0 0.0 0.0" />
         <!-- ============================================================== -->
-        <mass value="0.0001" /><!--FIXME-->
-        <!-- ============================================================== -->
-        <inertia ixx="0.00000001"
-                 ixy="0"
-                 ixz="0"
-                 iyy="0.00000001"
-                 iyz="0"
-                 izz="0.00000001" /><!--FIXME-->
+        <mass value="0.005" /><!--FIXME-->
+        <!-- ============================================================== -->
+        <inertia ixx="1.0E-6"
+                 ixy="0"
+                 ixz="0"
+                 iyy="1.0E-6"
+                 iyz="0"
+                 izz="1.0E-6" /><!--FIXME-->
         <!-- ============================================================== -->
       </inertial>
@@ -178,12 +178,12 @@
         <origin xyz="0.0 0.0 0.0" />
         <!-- ============================================================== -->
-        <mass value="0.0001" /><!--FIXME-->
-        <!-- ============================================================== -->
-        <inertia ixx="0.00000001"
-                 ixy="0"
-                 ixz="0"
-                 iyy="0.00000001"
-                 iyz="0"
-                 izz="0.00000001" /><!--FIXME-->
+        <mass value="0.005" /><!--FIXME-->
+        <!-- ============================================================== -->
+        <inertia ixx="1.0E-6"
+                 ixy="0"
+                 ixz="0"
+                 iyy="1.0E-6"
+                 iyz="0"
+                 izz="1.0E-6" /><!--FIXME-->
         <!-- ============================================================== -->
       </inertial>
@@ -195,12 +195,12 @@
         <origin xyz="0.0 0.0 0.0" />
         <!-- ============================================================== -->
-        <mass value="0.0001" /><!--FIXME-->
-        <!-- ============================================================== -->
-        <inertia ixx="0.00000001"
-                 ixy="0"
-                 ixz="0"
-                 iyy="0.00000001"
-                 iyz="0"
-                 izz="0.00000001" /><!--FIXME-->
+        <mass value="0.005" /><!--FIXME-->
+        <!-- ============================================================== -->
+        <inertia ixx="1.0E-6"
+                 ixy="0"
+                 ixz="0"
+                 iyy="1.0E-6"
+                 iyz="0"
+                 izz="1.0E-6" /><!--FIXME-->
         <!-- ============================================================== -->
       </inertial>
@@ -212,12 +212,12 @@
         <origin xyz="0.0 0.0 0.0" />
         <!-- ============================================================== -->
-        <mass value="0.0001" /><!--FIXME-->
-        <!-- ============================================================== -->
-        <inertia ixx="0.00000001"
-                 ixy="0"
-                 ixz="0"
-                 iyy="0.00000001"
-                 iyz="0"
-                 izz="0.00000001" /><!--FIXME-->
+        <mass value="0.005" /><!--FIXME-->
+        <!-- ============================================================== -->
+        <inertia ixx="1.0E-6"
+                 ixy="0"
+                 ixz="0"
+                 iyy="1.0E-6"
+                 iyz="0"
+                 izz="1.0E-6" /><!--FIXME-->
         <!-- ============================================================== -->
       </inertial>

File: pandora_sensors_description/urdf/laser.urdf.xacro (robot description, xacro)
@@ -16,12 +16,12 @@
         <origin xyz="0.013 0.0 0.00951" />
         <!-- ============================================================== -->
-        <mass value="0.0001" /><!--FIXME-->
-        <!-- ============================================================== -->
-        <inertia ixx="0.00000001"
+        <mass value="0.005" /><!--FIXME-->
+        <!-- ============================================================== -->
+        <inertia ixx="1.0E-6"
                  ixy="0"
                  ixz="0"
-                 iyy="0.00000001"
+                 iyy="1.0E-6"
                  iyz="0"
-                 izz="0.00000001" /><!--FIXME-->
+                 izz="1.0E-6" /><!--FIXME-->
         <!-- ============================================================== -->
       </inertial>
@@ -90,12 +90,12 @@
         <origin xyz="0.0 0.0 0.0" />
         <!-- ============================================================== -->
-        <mass value="0.0001" /><!--FIXME-->
-        <!-- ============================================================== -->
-        <inertia ixx="0.00000001"
+        <mass value="0.005" /><!--FIXME-->
+        <!-- ============================================================== -->
+        <inertia ixx="1.0E-6"
                  ixy="0"
                  ixz="0"
-                 iyy="0.00000001"
+                 iyy="1.0E-6"
                  iyz="0"
-                 izz="0.00000001" /><!--FIXME-->
+                 izz="1.0E-6" /><!--FIXME-->
         <!-- ============================================================== -->
       </inertial>

File: pandora_sensors_description/urdf/microphone.urdf.xacro (robot description, xacro)
@@ -47,12 +47,12 @@
         <origin xyz="0.0 0.0 0.0" />
         <!-- ============================================================== -->
-        <mass value="0.0001" />
+        <mass value="0.005" />
         <!-- ============================================================== -->
-        <inertia ixx="0.00000001"
+        <inertia ixx="1.0E-6"
                  ixy="0"
                  ixz="0"
-                 iyy="0.00000001"
+                 iyy="1.0E-6"
                  iyz="0"
-                 izz="0.00000001" />
+                 izz="1.0E-6" />
         <!-- ============================================================== -->
       </inertial>

File: pandora_sensors_description/urdf/sonar.urdf.xacro (robot description, xacro)
@@ -47,12 +47,12 @@
         <origin xyz="0.0 0.0 0.0" />
         <!-- ============================================================== -->
-        <mass value="0.0001" />
+        <mass value="0.005" />
         <!-- ============================================================== -->
-        <inertia ixx="0.00000001"
+        <inertia ixx="1.0E-6"
                  ixy="0"
                  ixz="0"
-                 iyy="0.00000001"
+                 iyy="1.0E-6"
                  iyz="0"
-                 izz="0.00000001" />
+                 izz="1.0E-6" />
         <!-- ============================================================== -->
       </inertial>

File: pandora_sensors_description/urdf/thermal.urdf.xacro (robot description, xacro)
@@ -47,12 +47,12 @@
         <origin xyz="0.0 0.0 0.0" />
         <!-- ============================================================== -->
-        <mass value="0.0001" />
+        <mass value="0.005" />
         <!-- ============================================================== -->
-        <inertia ixx="0.00000001"
+        <inertia ixx="1.0E-6"
                  ixy="0"
                  ixz="0"
-                 iyy="0.00000001"
+                 iyy="1.0E-6"
                  iyz="0"
-                 izz="0.00000001" />
+                 izz="1.0E-6" />
         <!-- ============================================================== -->
       </inertial>
@@ -64,12 +64,12 @@
         <origin xyz="0.0 0.0 0.0" />
         <!-- ============================================================== -->
-        <mass value="0.0001" />
+        <mass value="0.005" />
         <!-- ============================================================== -->
-        <inertia ixx="0.00000001"
+        <inertia ixx="1.0E-6"
                  ixy="0"
                  ixz="0"
-                 iyy="0.00000001"
+                 iyy="1.0E-6"
                  iyz="0"
-                 izz="0.00000001" />
+                 izz="1.0E-6" />
         <!-- ============================================================== -->
       </inertial>

Commit message: Updated gears

File: pandora_robots_description/urdf/gears/gears.urdf.xacro (robot description, xacro)
@@ -15,4 +15,6 @@
   <xacro:include filename="$(find pandora_robots_description)/urdf/gears/links/linear_head_base_link.urdf.xacro" />
   <xacro:include filename="$(find pandora_robots_description)/urdf/gears/links/linear_head_main_link.urdf.xacro" />
+  <xacro:include filename="$(find pandora_robots_description)/urdf/gears/links/differential_link.urdf.xacro" />
+  <xacro:include filename="$(find pandora_robots_description)/urdf/gears/links/differential_pin.urdf.xacro" />
   <!-- ==================================================================== -->
   <xacro:include filename="$(find pandora_robots_description)/urdf/gears/joints/side_joint.urdf.xacro" />
@@ -21,4 +23,5 @@
   <xacro:include filename="$(find pandora_robots_description)/urdf/gears/joints/linear_head_pitch_joint.urdf.xacro" />
   <xacro:include filename="$(find pandora_robots_description)/urdf/gears/joints/linear_head_yaw_joint.urdf.xacro" />
+  <xacro:include filename="$(find pandora_robots_description)/urdf/gears/joints/differential_joint.urdf.xacro" />
   <!-- ==================================================================== -->
   <xacro:include filename="$(find pandora_robots_description)/urdf/gears/sensors/laser_sensor.xacro" />
@@ -66,4 +69,8 @@
   <xacro:linear_head_pitch_joint fixed="${fixed}" />
   <!-- ================================================================== -->
+  <xacro:differential_link/>
+  <xacro:differential_joint/>
+  <xacro:differential_pin prefix_y="left" reflect_y="1"/>
+  <xacro:differential_pin prefix_y="right" reflect_y="-1"/>
 <!-- Load Sensors ######################################################### -->
   <xacro:if value="${enable_sensors}" >

File: pandora_robots_description/urdf/gears/urdf_configurations.xacro (robot description, xacro)
@@ -40,5 +40,5 @@
   <!-- ==================================================================== -->
   <!-- Joint Damping ====================================================== -->
-  <xacro:property name="side_joint_damping" value="0.0" />
+  <xacro:property name="side_joint_damping" value="60.0" />
   <!-- ==================================================================== -->
   <xacro:property name="wheel_joint_damping" value="0.0" />
