Commit message: Add kinect link

File: pandora_robots_description/urdf/woody/sensors/kinect_sensor.xacro (robot description, xacro)
@@ -7,5 +7,5 @@
   <xacro:macro name="kinect_sensor"
                params="fixed" >
-    <xacro:kinect_caster parent="linear_elevator_link"
+    <xacro:kinect_caster parent="base_link"
                          fixed="${fixed}"
                          pitch_min_limit="${kinect_pitch_joint_min_limit}"
@@ -13,6 +13,6 @@
                          yaw_min_limit="${kinect_yaw_joint_min_limit}"
                          yaw_max_limit="${kinect_yaw_joint_max_limit}" >
-      <origin xyz="0.07353 0.01239 0.14642"
-              rpy="-0.0436 0.0 0.0" />
+      <origin xyz="0.08085 0.02998 0.26749"
+              rpy="0.0 0.0 0.0" />
     </xacro:kinect_caster>
   </xacro:macro>

File: pandora_robots_description/urdf/woody/urdf_configurations.xacro (robot description, xacro)
@@ -7,5 +7,5 @@
     <xacro:property name="enable_laser_sensor" value="true" />
     <!-- ================================================================== -->
-    <xacro:property name="enable_kinect_sensor" value="false" />
+    <xacro:property name="enable_kinect_sensor" value="true" />
     <!-- ================================================================== -->
     <xacro:property name="enable_camera_sensors" value="false" />

File: pandora_sensors_description/urdf/kinect.urdf.xacro (robot description, xacro)
@@ -32,5 +32,5 @@
         <!-- ============================================================== -->
         <geometry>
-          <mesh filename="package://pandora_robots_description/meshes/woody/visual/linear/head/servo_motor.dae" />
+          <mesh filename="package://pandora_sensors_description/meshes/laser/pitch_servo_motor.dae" />
         </geometry>
         <!-- ============================================================== -->
