Commit message: Add flir and logitech sensors [skip ci]

File: pandora_robots_description/urdf/woody/sensors/camera_sensor.xacro (robot description, xacro)
@@ -9,5 +9,5 @@
     <xacro:camera_caster parent="base_link"
                          prefix_y="left" >
-      <origin xyz="-0.10874 0.0754 0.38825"
+      <origin xyz="-0.08308 0.08308 0.23081"
               rpy="0.0 0.0 ${ 3 * PI_4 }" />
     </xacro:camera_caster>
@@ -17,5 +17,5 @@
     <xacro:camera_caster parent="base_link"
                          prefix_y="right" >
-      <origin xyz="-0.10874 -0.0754 0.38825"
+      <origin xyz="-0.08308 -0.08308 0.23081"
               rpy="0.0 0.0 ${ 5 * PI_4 }" />
     </xacro:camera_caster>

File: pandora_robots_description/urdf/woody/sensors/flir_sensor.xacro (robot description, xacro)
@@ -2,13 +2,13 @@
 <robot xmlns:xacro="http://ros.org/wiki/xacro" >
   <!-- ==================================================================== -->
-  <xacro:include filename="$(find pandora_sensors_description)/urdf/thermal.urdf.xacro" />
+  <xacro:include filename="$(find pandora_sensors_description)/urdf/flir.urdf.xacro" />
   <!-- ==================================================================== -->
 <!-- ###################################################################### -->
   <!-- ==================================================================== -->
-  <xacro:macro name="thermal_sensor" >
-    <xacro:thermal_caster parent="base_link" >
-      <origin xyz="0.01575 -0.0614 0.08243"
-              rpy="${-PI_2} 0 0" />
-    </xacro:thermal_caster>
+  <xacro:macro name="flir_sensor" >
+    <xacro:flir_caster parent="kinect_main_link" >
+      <origin xyz="0.01732 0.07882 0.02341"
+              rpy="0 0 0" />
+    </xacro:flir_caster>
   </xacro:macro>
 <!-- ###################################################################### -->

File: pandora_robots_description/urdf/woody/urdf_configurations.xacro (robot description, xacro)
@@ -9,5 +9,7 @@
     <xacro:property name="enable_kinect_sensor" value="true" />
     <!-- ================================================================== -->
-    <xacro:property name="enable_camera_sensors" value="false" />
+    <xacro:property name="enable_flir_sensor" value="true" />
+    <!-- ================================================================== -->
+    <xacro:property name="enable_camera_sensors" value="true" />
       <xacro:property name="enable_left_camera_sensor" value="true" />
       <xacro:property name="enable_right_camera_sensor" value="true" />

File: pandora_robots_description/urdf/woody/woody.urdf.xacro (robot description, xacro)
@@ -18,4 +18,5 @@
   <xacro:include filename="$(find pandora_robots_description)/urdf/woody/sensors/laser_sensor.xacro" />
   <xacro:include filename="$(find pandora_robots_description)/urdf/woody/sensors/kinect_sensor.xacro" />
+  <xacro:include filename="$(find pandora_robots_description)/urdf/woody/sensors/flir_sensor.xacro" />
   <xacro:include filename="$(find pandora_robots_description)/urdf/woody/sensors/camera_sensor.xacro" />
   <xacro:include filename="$(find pandora_robots_description)/urdf/woody/sensors/sonar_sensor.xacro" />
@@ -58,4 +59,7 @@
       <xacro:kinect_sensor fixed="${fixed}" />
     </xacro:if>
+    <xacro:if value="${enable_flir_sensor}" >
+      <xacro:flir_sensor />
+    </xacro:if>
     <xacro:if value="${enable_camera_sensors}" >
       <!-- ================================================================ -->
@@ -81,5 +85,5 @@
     </xacro:if>
     <xacro:if value="${enable_thermal_sensor}" >
-        <xacro:middle_thermal_sensor />
+        <xacro:thermal_sensor />
     </xacro:if>
     <xacro:if value="${enable_co2_sensor}" >

File: pandora_sensors_description/urdf/flir.urdf.xacro (robot description, xacro)
@@ -2,8 +2,8 @@
 <robot xmlns:xacro="http://ros.org/wiki/xacro" >
 <!-- ###################################################################### -->
-  <xacro:macro name="thermal_caster"
+  <xacro:macro name="flir_caster"
                params="parent *origin" >
     <!-- ################################################################## -->
-    <link name="thermal_main_link" >
+    <link name="flir_main_link" >
       <inertial>
         <!-- ============================================================== -->
@@ -26,5 +26,5 @@
         <!-- ============================================================== -->
         <geometry>
-          <mesh filename="package://pandora_sensors_description/meshes/thermal/grid_eye.dae" />
+          <mesh filename="package://pandora_sensors_description/meshes/co2/dynament.dae" />
         </geometry>
         <!-- ============================================================== -->
@@ -42,5 +42,5 @@
     </link>
     <!-- ################################################################## -->
-    <link name="thermal_frame" >
+    <link name="flir_frame" >
       <inertial>
         <!-- ============================================================== -->
@@ -59,5 +59,5 @@
     </link>
     <!-- ################################################################## -->
-    <link name="thermal_optical_frame" >
+    <link name="flir_optical_frame" >
       <inertial>
         <!-- ============================================================== -->
@@ -76,9 +76,9 @@
     </link>
     <!-- ################################################################## -->
-    <joint name="thermal_main_joint"
+    <joint name="flir_main_joint"
            type="fixed" >
       <!-- ================================================================ -->
       <parent link="${parent}" />
-      <child link="thermal_main_link" />
+      <child link="flir_main_link" />
       <!-- ================================================================ -->
       <xacro:insert_block name="origin" />
@@ -86,9 +86,9 @@
     </joint>
     <!-- ################################################################## -->
-    <joint name="thermal_joint"
+    <joint name="flir_joint"
            type="fixed" >
       <!-- ================================================================ -->
-      <parent link="thermal_main_link" />
-      <child link="thermal_frame" />
+      <parent link="flir_main_link" />
+      <child link="flir_frame" />
       <!-- ================================================================ -->
       <origin xyz="0.0045 0.0 0.00125"
@@ -97,9 +97,9 @@
     </joint>
     <!-- ################################################################## -->
-    <joint name="thermal_optical_joint"
+    <joint name="flir_optical_joint"
            type="fixed" >
       <!-- ================================================================ -->
-      <parent link="thermal_frame" />
-      <child link="thermal_optical_frame" />
+      <parent link="flir_frame" />
+      <child link="flir_optical_frame" />
       <!-- ================================================================ -->
       <origin xyz="0.0 0.0 0.0"
