Commit message: Fix thermal macro name to be compatible with gears [skip ci]

File: pandora_robots_description/urdf/woody/sensors/thermal_sensor.xacro (robot description, xacro)
@@ -7,5 +7,6 @@
   <!-- ==================================================================== -->
   <xacro:macro name="thermal_sensor" >
-    <xacro:thermal_caster parent="base_link" >
+    <xacro:thermal_caster parent="base_link"
+                          prefix_y="middle" >
       <origin xyz="0.01575 -0.0614 0.08243"
               rpy="${-PI_2} 0 0" />

File: pandora_sensors_description/urdf/thermal.urdf.xacro (robot description, xacro)
@@ -3,7 +3,7 @@
 <!-- ###################################################################### -->
   <xacro:macro name="thermal_caster"
-               params="parent *origin" >
+               params="parent prefix_y *origin" >
     <!-- ################################################################## -->
-    <link name="thermal_main_link" >
+    <link name="${prefix_y}_thermal_main_link" >
       <inertial>
         <!-- ============================================================== -->
@@ -42,5 +42,5 @@
     </link>
     <!-- ################################################################## -->
-    <link name="thermal_frame" >
+    <link name="${prefix_y}_thermal_frame" >
       <inertial>
         <!-- ============================================================== -->
@@ -59,5 +59,5 @@
     </link>
     <!-- ################################################################## -->
-    <link name="thermal_optical_frame" >
+    <link name="${prefix_y}_thermal_optical_frame" >
       <inertial>
         <!-- ============================================================== -->
@@ -76,9 +76,9 @@
     </link>
     <!-- ################################################################## -->
-    <joint name="thermal_main_joint"
+    <joint name="${prefix_y}_thermal_main_joint"
            type="fixed" >
       <!-- ================================================================ -->
       <parent link="${parent}" />
-      <child link="thermal_main_link" />
+      <child link="${prefix_y}_thermal_main_link" />
       <!-- ================================================================ -->
       <xacro:insert_block name="origin" />
@@ -86,9 +86,9 @@
     </joint>
     <!-- ################################################################## -->
-    <joint name="thermal_joint"
+    <joint name="${prefix_y}_thermal_joint"
            type="fixed" >
       <!-- ================================================================ -->
-      <parent link="thermal_main_link" />
-      <child link="thermal_frame" />
+      <parent link="${prefix_y}_thermal_main_link" />
+      <child link="${prefix_y}_thermal_frame" />
       <!-- ================================================================ -->
       <origin xyz="0.0045 0.0 0.00125"
@@ -97,9 +97,9 @@
     </joint>
     <!-- ################################################################## -->
-    <joint name="thermal_optical_joint"
+    <joint name="${prefix_y}_thermal_optical_joint"
            type="fixed" >
       <!-- ================================================================ -->
-      <parent link="thermal_frame" />
-      <child link="thermal_optical_frame" />
+      <parent link="${prefix_y}_thermal_frame" />
+      <child link="${prefix_y}_thermal_optical_frame" />
       <!-- ================================================================ -->
       <origin xyz="0.0 0.0 0.0"
