Commit message: Added sonar new mesh (both mesh and urdf)

File: pandora_robots_description/urdf/woody/sensors/sonar_sensor.xacro (robot description, xacro)
@@ -9,6 +9,6 @@
     <xacro:sonar_caster name="left"
                         parent="base_link" >
-      <origin xyz="-0.15026 0.06429 0.39925"
-              rpy="0.0 0.0 ${ 5 * PI_6 }" />
+      <origin xyz="-0.146 0.1376 0.21406"
+              rpy="0.0 0.0 ${- PI_6 }" />
     </xacro:sonar_caster>
   </xacro:macro>
@@ -17,6 +17,6 @@
     <xacro:sonar_caster name="right"
                         parent="base_link" >
-      <origin xyz="-0.15026 -0.06429 0.39925"
-              rpy="0.0 0.0 ${ 7 * PI_6 }" />
+      <origin xyz="-0.146 -0.1376 0.21406"
+              rpy="0.0 0.0 ${ PI_6 }" />
     </xacro:sonar_caster>
   </xacro:macro>

File: pandora_robots_description/urdf/woody/urdf_configurations.xacro (robot description, xacro)
@@ -15,5 +15,5 @@
       <xacro:property name="enable_right_camera_sensor" value="true" />
     <!-- ================================================================== -->
-    <xacro:property name="enable_sonar_sensors" value="false" />
+    <xacro:property name="enable_sonar_sensors" value="true" />
       <xacro:property name="enable_left_sonar_sensor" value="true" />
       <xacro:property name="enable_right_sonar_sensor" value="true" />
