Commit message: Fixed c02 , thermal and flir in urdf and added flir mesh

File: pandora_robots_description/urdf/woody/sensors/co2_sensor.xacro (robot description, xacro)
@@ -6,6 +6,6 @@
 <!-- ###################################################################### -->
   <xacro:macro name="co2_sensor" >
-    <xacro:co2_caster parent="linear_head_main_link" >
-      <origin xyz="0.00915 -0.05293 0.05251"
+    <xacro:co2_caster parent="kinect_main_link" >
+      <origin xyz="0.0173 -0.0495 0.022"
               rpy="${zero}" />
     </xacro:co2_caster>

File: pandora_robots_description/urdf/woody/sensors/flir_sensor.xacro (robot description, xacro)
@@ -8,5 +8,5 @@
   <xacro:macro name="flir_sensor" >
     <xacro:flir_caster parent="kinect_main_link" >
-      <origin xyz="0.01732 0.07882 0.02341"
+      <origin xyz="0.0173 0.0747 0.022"
               rpy="0 0 0" />
     </xacro:flir_caster>

File: pandora_robots_description/urdf/woody/sensors/thermal_sensor.xacro (robot description, xacro)
@@ -7,8 +7,8 @@
   <!-- ==================================================================== -->
   <xacro:macro name="thermal_sensor" >
-    <xacro:thermal_caster parent="base_link"
+    <xacro:thermal_caster parent="kinect_main_link"
                           prefix_y="middle" >
-      <origin xyz="0.01575 -0.0614 0.08243"
-              rpy="${-PI_2} 0 0" />
+      <origin xyz="0.0173 0.0949 0.022"
+              rpy="0 0 0" />
     </xacro:thermal_caster>
   </xacro:macro>

File: pandora_robots_description/urdf/woody/urdf_configurations.xacro (robot description, xacro)
@@ -19,7 +19,7 @@
       <xacro:property name="enable_right_sonar_sensor" value="true" />
     <!-- ================================================================== -->
-    <xacro:property name="enable_thermal_sensor" value="false" />
+    <xacro:property name="enable_thermal_sensor" value="true" />
     <!-- ================================================================== -->
-    <xacro:property name="enable_co2_sensor" value="false" />
+    <xacro:property name="enable_co2_sensor" value="true" />
     <!-- ================================================================== -->
     <xacro:property name="enable_microphone_sensor" value="false" />

Commit message: Fix co2_link position [ci skip]

File: pandora_robots_description/urdf/woody/sensors/co2_sensor.xacro (robot description, xacro)
@@ -7,5 +7,5 @@
   <xacro:macro name="co2_sensor" >
     <xacro:co2_caster parent="kinect_main_link" >
-      <origin xyz="0.0173 -0.0495 0.022"
+      <origin xyz="0.0173 -0.0595 0.022"
               rpy="${zero}" />
     </xacro:co2_caster>
