Commit message: Modified side joint damping

File: pandora_robots_description/urdf/woody/urdf_configurations.xacro (robot description, xacro)
@@ -32,5 +32,5 @@
   <!-- ==================================================================== -->
   <!-- Joint Damping ====================================================== -->
-  <xacro:property name="side_joint_damping" value="0.0" />
+  <xacro:property name="side_joint_damping" value="60.0" />
   <!-- ==================================================================== -->
   <xacro:property name="wheel_joint_damping" value="0.0" />

Commit message: Refactor main urdf and config files [ci skip]

File: pandora_robots_description/urdf/woody/urdf_configurations.xacro (robot description, xacro)
@@ -1,86 +1,43 @@
 <?xml version="1.0"?>
 <robot xmlns:xacro="http://ros.org/wiki/xacro" >
-<!-- Elements' Status ##################################################### -->
-  <!-- Sensors ============================================================ -->
-  <xacro:property name="enable_sensors" value="true" />
-    <!-- ================================================================== -->
-    <xacro:property name="enable_laser_sensor" value="true" />
-    <!-- ================================================================== -->
-    <xacro:property name="enable_kinect_sensor" value="true" />
-    <!-- ================================================================== -->
-    <xacro:property name="enable_flir_sensor" value="true" />
-    <!-- ================================================================== -->
-    <xacro:property name="enable_camera_sensors" value="true" />
-      <xacro:property name="enable_left_camera_sensor" value="true" />
-      <xacro:property name="enable_right_camera_sensor" value="true" />
-    <!-- ================================================================== -->
-    <xacro:property name="enable_sonar_sensors" value="true" />
-      <xacro:property name="enable_left_sonar_sensor" value="true" />
-      <xacro:property name="enable_right_sonar_sensor" value="true" />
-    <!-- ================================================================== -->
-    <xacro:property name="enable_thermal_sensor" value="true" />
-    <!-- ================================================================== -->
-    <xacro:property name="enable_co2_sensor" value="true" />
-    <!-- ================================================================== -->
-    <xacro:property name="enable_microphone_sensor" value="false" />
-  <!-- ==================================================================== -->
+<!-- Sensors ############################################################## -->
+  <xacro:property name="enable_laser_sensor" value="true" />
+  <xacro:property name="enable_kinect_sensor" value="true" />
+  <xacro:property name="enable_flir_sensor" value="true" />
+  <xacro:property name="enable_left_camera_sensor" value="true" />
+  <xacro:property name="enable_right_camera_sensor" value="true" />
+  <xacro:property name="enable_left_sonar_sensor" value="true" />
+  <xacro:property name="enable_right_sonar_sensor" value="true" />
+  <xacro:property name="enable_thermal_sensor" value="true" />
+  <xacro:property name="enable_co2_sensor" value="true" />
+  <xacro:property name="enable_microphone_sensor" value="false" />
 <!-- Joint Physics ######################################################## -->
-  <!-- Joint Types ======================================================== -->
   <xacro:property name="side_joint_type" value="revolute" />
-  <!-- ==================================================================== -->
   <xacro:property name="wheel_joint_type" value="continuous" />
-  <!-- ==================================================================== -->
-  <!-- Joint Damping ====================================================== -->
   <xacro:property name="side_joint_damping" value="0.0" />
-  <!-- ==================================================================== -->
   <xacro:property name="wheel_joint_damping" value="0.0" />
-  <!-- ==================================================================== -->
-  <!-- Joint Limits ======================================================= -->
-  <xacro:property name="side_joint_min_limit" value="-0.785" /> <!--FIXME-->
-  <xacro:property name="side_joint_max_limit" value="0.785" /> <!--FIXME-->
-  <!-- ==================================================================== -->
-  <xacro:property name="laser_roll_joint_min_limit" value="-1.57" /> <!--FIXME-->
-  <xacro:property name="laser_roll_joint_max_limit" value="1.57" /> <!--FIXME-->
-  <!-- ==================================================================== -->
-  <xacro:property name="laser_pitch_joint_min_limit" value="-1.57" /> <!--FIXME-->
-  <xacro:property name="laser_pitch_joint_max_limit" value="1.57" /> <!--FIXME-->
-  <!-- ==================================================================== -->
-  <xacro:property name="kinect_pitch_joint_min_limit" value="-1.57" /> <!--FIXME-->
-  <xacro:property name="kinect_pitch_joint_max_limit" value="1.57" /> <!--FIXME-->
-  <!-- ==================================================================== -->
-  <xacro:property name="kinect_yaw_joint_min_limit" value="-1.57" /> <!--FIXME-->
-  <xacro:property name="kinect_yaw_joint_max_limit" value="1.57" /> <!--FIXME-->
-  <!-- ==================================================================== -->
-<!-- Coefficients ######################################################### -->
-  <!-- TODO -->
-  <!-- Velocities ========================================================= -->
+  <xacro:property name="side_joint_min_limit" value="-0.785" />
+  <xacro:property name="side_joint_max_limit" value="0.785" />
+  <xacro:property name="laser_roll_joint_min_limit" value="-0.523" />
+  <xacro:property name="laser_roll_joint_max_limit" value="0.523" />
+  <xacro:property name="laser_pitch_joint_min_limit" value="-0.523" />
+  <xacro:property name="laser_pitch_joint_max_limit" value="0.523" />
+  <xacro:property name="kinect_pitch_joint_min_limit" value="-0.785" />
+  <xacro:property name="kinect_pitch_joint_max_limit" value="0.785" />
+  <xacro:property name="kinect_yaw_joint_min_limit" value="-1.308" />
+  <xacro:property name="kinect_yaw_joint_max_limit" value="1.308" />
+<!-- TODO: Coefficients ################################################### -->
   <xacro:property name="max_robot_linear_velocity" value="2.0" />
-  <!-- ==================================================================== -->
   <xacro:property name="max_robot_angular_velocity" value="2.0" />
-  <!-- ==================================================================== -->
   <xacro:property name="max_kinect_angular_velocity" value="2.5" />
-  <!-- ==================================================================== -->
   <xacro:property name="max_laser_angular_velocity" value="2.5" />
-  <!-- ==================================================================== -->
-  <!-- Accelerations ====================================================== -->
   <xacro:property name="max_robot_linear_acceleration" value="1.0" />
-  <!-- ==================================================================== -->
   <xacro:property name="max_robot_angular_acceleration" value="0.2" />
-  <!-- ==================================================================== -->
   <xacro:property name="max_kinect_angular_acceleration" value="0.0" />
-  <!-- ==================================================================== -->
   <xacro:property name="max_laser_angular_acceleration" value="0.0" />
-  <!-- ==================================================================== -->
 <!-- Dimensions ########################################################### -->
-  <!-- TODO -->
-  <!-- Wheels ============================================================= -->
   <xacro:property name="wheel_length" value="0.07985" />
-  <!-- ==================================================================== -->
   <xacro:property name="wheel_radius" value="0.09794" />
-  <!-- ==================================================================== -->
   <xacro:property name="track" value="0.344" />
-  <!-- ==================================================================== -->
   <xacro:property name="wheelbase" value="0.34678" />
-  <!-- ==================================================================== -->
-<!-- ###################################################################### -->
 </robot>

File: pandora_robots_description/urdf/woody/woody.urdf.xacro (robot description, xacro)
@@ -2,18 +2,13 @@
 <robot xmlns:xacro="http://ros.org/wiki/xacro" >
 <!-- Import Files ######################################################### -->
-  <!-- ==================================================================== -->
   <xacro:include filename="$(find pandora_robots_description)/urdf/woody/urdf_configurations.xacro" />
-  <!-- ==================================================================== -->
   <xacro:include filename="$(find pandora_robots_description)/urdf/woody/properties/constants.xacro" />
   <xacro:include filename="$(find pandora_robots_description)/urdf/woody/properties/defaults.xacro" />
   <xacro:include filename="$(find pandora_robots_description)/urdf/woody/properties/materials.xacro" />
-  <!-- ==================================================================== -->
   <xacro:include filename="$(find pandora_robots_description)/urdf/woody/links/base_link.urdf.xacro" />
   <xacro:include filename="$(find pandora_robots_description)/urdf/woody/links/side_link.urdf.xacro" />
   <xacro:include filename="$(find pandora_robots_description)/urdf/woody/links/wheel_link.urdf.xacro" />
-  <!-- ==================================================================== -->
   <xacro:include filename="$(find pandora_robots_description)/urdf/woody/joints/side_joint.urdf.xacro" />
   <xacro:include filename="$(find pandora_robots_description)/urdf/woody/joints/wheel_joint.urdf.xacro" />
-  <!-- ==================================================================== -->
   <xacro:include filename="$(find pandora_robots_description)/urdf/woody/sensors/laser_sensor.xacro" />
   <xacro:include filename="$(find pandora_robots_description)/urdf/woody/sensors/kinect_sensor.xacro" />
@@ -24,75 +19,51 @@
   <xacro:include filename="$(find pandora_robots_description)/urdf/woody/sensors/co2_sensor.xacro" />
   <xacro:include filename="$(find pandora_robots_description)/urdf/woody/sensors/microphone_sensor.xacro" />
-  <!-- ==================================================================== -->
 <xacro:macro name="woody_urdf"
              params="fixed" >
 <!-- Load Links & Joints ################################################## -->
-  <!-- ================================================================== -->
   <xacro:base_link />
-  <!-- ================================================================== -->
-  <!-- ================================================================== -->
   <xacro:side_link prefix_y="left" reflect_y="1" />
   <xacro:side_joint prefix_y="left" reflect_y="1" />
-  <!-- ================================================================== -->
   <xacro:side_link prefix_y="right" reflect_y="-1" />
   <xacro:side_joint prefix_y="right" reflect_y="-1" />
-  <!-- ================================================================== -->
-  <!-- ================================================================== -->
   <xacro:wheel_link prefix_y="left" prefix_x="front" reflect_y="1" reflect_x="1" />
   <xacro:wheel_joint prefix_y="left" prefix_x="front" reflect_y="1" reflect_x="1" />
-  <!-- ================================================================== -->
   <xacro:wheel_link prefix_y="left" prefix_x="rear" reflect_y="1" reflect_x="-1" />
   <xacro:wheel_joint prefix_y="left" prefix_x="rear" reflect_y="1" reflect_x="-1" />
-  <!-- ================================================================== -->
   <xacro:wheel_link prefix_y="right" prefix_x="front" reflect_y="-1" reflect_x="1" />
   <xacro:wheel_joint prefix_y="right" prefix_x="front" reflect_y="-1" reflect_x="1" />
-  <!-- ================================================================== -->
   <xacro:wheel_link prefix_y="right" prefix_x="rear" reflect_y="-1" reflect_x="-1" />
   <xacro:wheel_joint prefix_y="right" prefix_x="rear" reflect_y="-1" reflect_x="-1" />
-  <!-- ================================================================== -->
 <!-- Load Sensors ######################################################### -->
-  <xacro:if value="${enable_sensors}" >
-    <xacro:if value="${enable_laser_sensor}" >
-      <xacro:laser_sensor fixed="${fixed}" />
-    </xacro:if>
-    <xacro:if value="${enable_kinect_sensor}" >
-      <xacro:kinect_sensor fixed="${fixed}" />
-    </xacro:if>
-    <xacro:if value="${enable_flir_sensor}" >
-      <xacro:flir_sensor />
-    </xacro:if>
-    <xacro:if value="${enable_camera_sensors}" >
-      <!-- ================================================================ -->
-      <xacro:if value="${enable_left_camera_sensor}" >
-        <xacro:left_camera_sensor />
-      </xacro:if>
-      <!-- ================================================================ -->
-      <xacro:if value="${enable_right_camera_sensor}" >
-        <xacro:right_camera_sensor />
-      </xacro:if>
-      <!-- ================================================================ -->
-    </xacro:if>
-    <xacro:if value="${enable_sonar_sensors}" >
-      <!-- ================================================================ -->
-      <xacro:if value="${enable_left_sonar_sensor}" >
-        <xacro:left_sonar_sensor />
-      </xacro:if>
-      <!-- ================================================================ -->
-      <xacro:if value="${enable_right_sonar_sensor}" >
-        <xacro:right_sonar_sensor />
-      </xacro:if>
-      <!-- ================================================================ -->
-    </xacro:if>
-    <xacro:if value="${enable_thermal_sensor}" >
-        <xacro:thermal_sensor />
-    </xacro:if>
-    <xacro:if value="${enable_co2_sensor}" >
-      <xacro:co2_sensor />
-    </xacro:if>
-    <xacro:if value="${enable_microphone_sensor}" >
-      <xacro:microphone_sensor />
-    </xacro:if>
+  <xacro:if value="${enable_laser_sensor}" >
+    <xacro:laser_sensor fixed="${fixed}" />
+  </xacro:if>
+  <xacro:if value="${enable_kinect_sensor}" >
+    <xacro:kinect_sensor fixed="${fixed}" />
+  </xacro:if>
+  <xacro:if value="${enable_flir_sensor}" >
+    <xacro:flir_sensor />
+  </xacro:if>
+  <xacro:if value="${enable_left_camera_sensor}" >
+    <xacro:left_camera_sensor />
+  </xacro:if>
+  <xacro:if value="${enable_right_camera_sensor}" >
+    <xacro:right_camera_sensor />
+  </xacro:if>
+  <xacro:if value="${enable_left_sonar_sensor}" >
+    <xacro:left_sonar_sensor />
+  </xacro:if>
+  <xacro:if value="${enable_right_sonar_sensor}" >
+    <xacro:right_sonar_sensor />
+  </xacro:if>
+  <xacro:if value="${enable_thermal_sensor}" >
+      <xacro:thermal_sensor />
+  </xacro:if>
+  <xacro:if value="${enable_co2_sensor}" >
+    <xacro:co2_sensor />
+  </xacro:if>
+  <xacro:if value="${enable_microphone_sensor}" >
+    <xacro:microphone_sensor />
   </xacro:if>
 </xacro:macro>
-<!-- ###################################################################### -->
 </robot>
