Commit message: Fix path names [ci skip]

File: pandora_robots_description/urdf/woody/links/base_link.urdf.xacro (robot description, xacro)
@@ -23,5 +23,5 @@
         <!-- ============================================================== -->
         <geometry>
-          <mesh filename="package://pandora_robots_description/meshes/gears/visual/base/base_link.dae" />
+          <mesh filename="package://pandora_robots_description/meshes/woody/visual/base/base_link.dae" />
         </geometry>
         <!-- ============================================================== -->
@@ -34,5 +34,5 @@
         <!-- ============================================================== -->
         <geometry>
-          <mesh filename="package://pandora_robots_description/meshes/gears/collision/base/base_link.stl" />
+          <mesh filename="package://pandora_robots_description/meshes/woody/collision/base/base_link.stl" />
         </geometry>
         <!-- ============================================================== -->

File: pandora_robots_description/urdf/woody/links/linear_elevator_link.urdf.xacro (robot description, xacro)
@@ -23,5 +23,5 @@
         <!-- ============================================================== -->
         <geometry>
-          <mesh filename="package://pandora_robots_description/meshes/gears/visual/linear/elevator/linear_elevator_link.dae" />
+          <mesh filename="package://pandora_robots_description/meshes/woody/visual/linear/elevator/linear_elevator_link.dae" />
         </geometry>
         <!-- ============================================================== -->
@@ -34,5 +34,5 @@
         <!-- ============================================================== -->
         <geometry>
-          <mesh filename="package://pandora_robots_description/meshes/gears/collision/linear/elevator/linear_elevator_link.stl" />
+          <mesh filename="package://pandora_robots_description/meshes/woody/collision/linear/elevator/linear_elevator_link.stl" />
         </geometry>
         <!-- ============================================================== -->

File: pandora_robots_description/urdf/woody/links/linear_head_base_link.urdf.xacro (robot description, xacro)
@@ -24,5 +24,5 @@
         <!-- ============================================================== -->
         <geometry>
-          <mesh filename="package://pandora_robots_description/meshes/gears/visual/linear/head/servo_motor.dae" />
+          <mesh filename="package://pandora_robots_description/meshes/woody/visual/linear/head/servo_motor.dae" />
         </geometry>
         <!-- ============================================================== -->

File: pandora_robots_description/urdf/woody/links/linear_head_main_link.urdf.xacro (robot description, xacro)
@@ -23,5 +23,5 @@
         <!-- ============================================================== -->
         <geometry>
-          <mesh filename="package://pandora_robots_description/meshes/gears/visual/linear/head/linear_head_main_link.dae" />
+          <mesh filename="package://pandora_robots_description/meshes/woody/visual/linear/head/linear_head_main_link.dae" />
         </geometry>
         <!-- ============================================================== -->
@@ -34,5 +34,5 @@
         <!-- ============================================================== -->
         <geometry>
-          <mesh filename="package://pandora_robots_description/meshes/gears/collision/linear/head/linear_head_main_link.stl" />
+          <mesh filename="package://pandora_robots_description/meshes/woody/collision/linear/head/linear_head_main_link.stl" />
         </geometry>
         <!-- ============================================================== -->

File: pandora_robots_description/urdf/woody/links/side_link.urdf.xacro (robot description, xacro)
@@ -25,5 +25,5 @@
         <!-- ============================================================== -->
         <geometry>
-          <mesh filename="package://pandora_robots_description/meshes/gears/visual/side/side_link.dae" />
+          <mesh filename="package://pandora_robots_description/meshes/woody/visual/side/side_link.dae" />
         </geometry>
         <!-- ============================================================== -->
@@ -37,5 +37,5 @@
         <!-- ============================================================== -->
         <geometry>
-          <mesh filename="package://pandora_robots_description/meshes/gears/collision/side/side_link.stl" />
+          <mesh filename="package://pandora_robots_description/meshes/woody/collision/side/side_link.stl" />
         </geometry>
         <!-- ============================================================== -->

File: pandora_robots_description/urdf/woody/links/wheel_link.urdf.xacro (robot description, xacro)
@@ -25,5 +25,5 @@
         <!-- ============================================================== -->
         <geometry>
-          <mesh filename="package://pandora_robots_description/meshes/gears/visual/wheel/wheel_link.dae" />
+          <mesh filename="package://pandora_robots_description/meshes/woody/visual/wheel/wheel_link.dae" />
         </geometry>
         <!-- ============================================================== -->
@@ -37,5 +37,5 @@
         <!-- ============================================================== -->
         <geometry>
-          <mesh filename="package://pandora_robots_description/meshes/gears/collision/wheel/wheel_link.stl" />
+          <mesh filename="package://pandora_robots_description/meshes/woody/collision/wheel/wheel_link.stl" />
         </geometry>
         <!-- ============================================================== -->

File: pandora_robots_description/urdf/woody/properties/materials.xacro (robot description, xacro)
@@ -101,5 +101,5 @@
   </material>
   <!-- ==================================================================== -->
-<!-- Gears Colors ######################################################### -->
+<!-- woody Colors ######################################################### -->
   <!-- ==================================================================== -->
   <material name="solidworks_default" >

File: pandora_sensors_description/urdf/kinect.urdf.xacro (robot description, xacro)
@@ -32,5 +32,5 @@
         <!-- ============================================================== -->
         <geometry>
-          <mesh filename="package://pandora_robots_description/meshes/gears/visual/linear/head/servo_motor.dae" />
+          <mesh filename="package://pandora_robots_description/meshes/woody/visual/linear/head/servo_motor.dae" />
         </geometry>
         <!-- ============================================================== -->

Commit message: temp

File: pandora_robots_description/urdf/woody/links/base_link.urdf.xacro (robot description, xacro)
@@ -6,5 +6,5 @@
       <inertial>
         <!-- ============================================================== -->
-        <origin xyz="-0.00968 -0.00122 0.17947" />
+        <origin xyz="-0.00968 -0.00122 0.19369" />
         <!-- ============================================================== -->
         <mass value="8.25079" />
@@ -39,4 +39,175 @@
       </collision>
     </link>
+    <link name="miniitx" >
+      <inertial>
+        <origin xyz="0.0 0.0 0.0" />
+        <mass value="0.589" />
+        <inertia ixx="0.0014381417"
+                 ixy="0.0"
+                 ixz="0.0"
+                 iyy="0.0019829667"
+                 iyz="0.0"
+                 izz="0.0033818417" />
+      </inertial>
+    </link>
+    <joint name="miniitx_joint"
+           type="fixed" >
+      <parent link="base_link" />
+      <child link="miniitx" />
+      <origin xyz="0.03895 0.0 0.16181"
+              rpy="0.0 0.0 0.0" />
+    </joint>
+    <link name="ssd" >
+      <inertial>
+        <origin xyz="0.0 0.0 0.0" />
+        <mass value="0.078" />
+        <inertia ixx="0.0000325"
+                 ixy="0.0"
+                 ixz="0.0"
+                 iyy="0.00006565"
+                 iyz="0.0"
+                 izz="0.00009685" />
+      </inertial>
+    </link>
+    <joint name="ssd_joint"
+           type="fixed" >
+      <parent link="base_link" />
+      <child link="ssd" />
+      <origin xyz="-0.06872 0.03699 0.07022"
+              rpy="0.0 0.0 0.0" />
+    </joint>
+    <link name="epos" >
+      <inertial>
+        <origin xyz="0.0 0.0 0.0" />
+        <mass value="0.136" />
+        <inertia ixx="0.0002266667"
+                 ixy="0.0"
+                 ixz="0.0"
+                 iyy="6.8283E-005"
+                 iyz="0.0"
+                 izz="0.0002858833" /> <!-- XXX -->
+      </inertial>
+    </link>
+    <joint name="epos_joint"
+           type="fixed" >
+      <parent link="base_link" />
+      <child link="epos" />
+      <origin xyz="-0.08263 0.0 0.03222"
+              rpy="0.0 0.0 0.0" />
+    </joint>
+    <link name="psu" >
+      <inertial>
+        <origin xyz="0.0 0.0 0.0" />
+        <mass value="0.178" />
+        <inertia ixx="0.0002241168"
+                 ixy="0.0"
+                 ixz="0.0"
+                 iyy="0.0001828208"
+                 iyz="0.0"
+                 izz="0.0004002627" />
+      </inertial>
+    </link>
+    <joint name="psu_joint"
+           type="fixed" >
+      <parent link="base_link" />
+      <child link="psu" />
+      <origin xyz="0.073 0.0 0.11023"
+              rpy="0.0 0.0 0.0" />
+    </joint>
+    <link name="battery1" >
+      <inertial>
+        <origin xyz="0.0 0.0 0.0" />
+        <mass value="0.8" />
+        <inertia ixx="0.0003576"
+                 ixy="0.0"
+                 ixz="0.0"
+                 iyy="0.0016806"
+                 iyz="0.0"
+                 izz="0.0015582" />
+      </inertial>
+    </link>
+    <joint name="battery1_joint"
+           type="fixed" >
+      <parent link="base_link" />
+      <child link="battery1" />
+      <origin xyz="0.10395 0.027 0.04822"
+              rpy="0.0 0.0 0.0" />
+    </joint>
+    <link name="battery2" >
+      <inertial>
+        <origin xyz="0.0 0.0 0.0" />
+        <mass value="0.8" />
+        <inertia ixx="0.0003576"
+                 ixy="0.0"
+                 ixz="0.0"
+                 iyy="0.0016806"
+                 iyz="0.0"
+                 izz="0.0015582" />
+      </inertial>
+    </link>
+    <joint name="battery2_joint"
+           type="fixed" >
+      <parent link="base_link" />
+      <child link="battery2" />
+      <origin xyz="0.10395 -0.027 0.04822"
+              rpy="0.0 0.0 0.0" />
+    </joint>
+    <link name="cables" >
+      <inertial>
+        <origin xyz="0.0 0.0 0.0" />
+        <mass value="0.6" />
+        <inertia ixx=""
+                 ixy="0.0"
+                 ixz="0.0"
+                 iyy=""
+                 iyz="0.0"
+                 izz="" />
+      </inertial>
+    </link>
+    <joint name="cables_joint"
+           type="fixed" >
+      <parent link="base_link" />
+      <child link="cables" />
+      <origin xyz="0.0 0.0 0.1"
+              rpy="0.0 0.0 0.0" />
+    </joint>
+    <link name="axis" >
+      <inertial>
+        <origin xyz="0.0 0.0 0.0" />
+        <mass value="0.446" />
+        <inertia ixx=""
+                 ixy="0.0"
+                 ixz="0.0"
+                 iyy=""
+                 iyz="0.0"
+                 izz="" />
+      </inertial>
+    </link>
+    <joint name="axis_joint"
+           type="fixed" >
+      <parent link="base_link" />
+      <child link="axis" />
+      <origin xyz="0.0 0.0 0.0"
+              rpy="0.0 0.0 0.0" />
+    </joint>
+    <link name="differential" >
+      <inertial>
+        <origin xyz="0.0 0.0 0.0" />
+        <mass value="0.31" />
+        <inertia ixx=""
+                 ixy="0.0"
+                 ixz="0.0"
+                 iyy=""
+                 iyz="0.0"
+                 izz="" />
+      </inertial>
+    </link>
+    <joint name="differential_joint"
+           type="fixed" >
+      <parent link="base_link" />
+      <child link="differential" />
+      <origin xyz="-0.15 0.0 0.09031"
+              rpy="0.0 0.0 0.0" />
+    </joint>
   </xacro:macro>
 <!-- ###################################################################### -->

Commit message: Add laser link

File: pandora_robots_description/urdf/woody/links/base_link.urdf.xacro (robot description, xacro)
@@ -157,10 +157,11 @@
         <origin xyz="0.0 0.0 0.0" />
         <mass value="0.6" />
-        <inertia ixx=""
-                 ixy="0.0"
-                 ixz="0.0"
-                 iyy=""
-                 iyz="0.0"
-                 izz="" />
+        <!-- TODO -->
+        <inertia ixx="0.0001"
+                 ixy="0.0"
+                 ixz="0.0"
+                 iyy="0.0001"
+                 iyz="0.0"
+                 izz="0.0001" />
       </inertial>
     </link>
@@ -176,10 +177,11 @@
         <origin xyz="0.0 0.0 0.0" />
         <mass value="0.446" />
-        <inertia ixx=""
-                 ixy="0.0"
-                 ixz="0.0"
-                 iyy=""
-                 iyz="0.0"
-                 izz="" />
+        <!-- TODO -->
+        <inertia ixx="0.0001"
+                 ixy="0.0"
+                 ixz="0.0"
+                 iyy="0.0001"
+                 iyz="0.0"
+                 izz="0.0001" />
       </inertial>
     </link>
@@ -195,10 +197,11 @@
         <origin xyz="0.0 0.0 0.0" />
         <mass value="0.31" />
-        <inertia ixx=""
-                 ixy="0.0"
-                 ixz="0.0"
-                 iyy=""
-                 iyz="0.0"
-                 izz="" />
+        <!-- TODO -->
+        <inertia ixx="0.0001"
+                 ixy="0.0"
+                 ixz="0.0"
+                 iyy="0.0001"
+                 iyz="0.0"
+                 izz="0.0001" />
       </inertial>
     </link>

File: pandora_robots_description/urdf/woody/sensors/laser_sensor.xacro (robot description, xacro)
@@ -13,5 +13,5 @@
                          pitch_min_limit="${laser_pitch_joint_min_limit}"
                          pitch_max_limit="${laser_pitch_joint_max_limit}" >
-      <origin xyz="0.1974 0.0 0.09679"
+      <origin xyz="0.2185 -0.00219 0.12885"
               rpy="${zero}" />
     </xacro:laser_caster>

File: pandora_robots_description/urdf/woody/urdf_configurations.xacro (robot description, xacro)
@@ -3,9 +3,9 @@
 <!-- Elements' Status ##################################################### -->
   <!-- Sensors ============================================================ -->
-  <xacro:property name="enable_sensors" value="false" />
+  <xacro:property name="enable_sensors" value="true" />
     <!-- ================================================================== -->
     <xacro:property name="enable_laser_sensor" value="true" />
     <!-- ================================================================== -->
-    <xacro:property name="enable_kinect_sensor" value="true" />
+    <xacro:property name="enable_kinect_sensor" value="false" />
     <!-- ================================================================== -->
     <xacro:property name="enable_camera_sensors" value="false" />

Commit message: Seperated differential link from base

File: pandora_robots_description/urdf/woody/links/base_link.urdf.xacro (robot description, xacro)
@@ -193,24 +193,4 @@
               rpy="0.0 0.0 0.0" />
     </joint>
-    <link name="differential" >
-      <inertial>
-        <origin xyz="0.0 0.0 0.0" />
-        <mass value="0.31" />
-        <!-- TODO -->
-        <inertia ixx="0.0001"
-                 ixy="0.0"
-                 ixz="0.0"
-                 iyy="0.0001"
-                 iyz="0.0"
-                 izz="0.0001" />
-      </inertial>
-    </link>
-    <joint name="differential_joint"
-           type="fixed" >
-      <parent link="base_link" />
-      <child link="differential" />
-      <origin xyz="-0.15 0.0 0.09031"
-              rpy="0.0 0.0 0.0" />
-    </joint>
   </xacro:macro>
 <!-- ###################################################################### -->

Commit message: Added raspberry , arm and imu to base_link.urdf

File: pandora_robots_description/urdf/woody/links/base_link.urdf.xacro (robot description, xacro)
@@ -74,6 +74,26 @@
       <parent link="base_link" />
       <child link="ssd" />
-      <origin xyz="-0.06872 0.03699 0.07022"
-              rpy="0.0 0.0 0.0" />
+      <origin xyz="0.059 -0.097 0.181"
+              rpy="${PI_2} 0.0 0.0" />
+    </joint>
+    <link name="raspberry" >
+      <xacro:solid_cuboid_inertial mass="0.062" width="0.070" height="0.025" depth="0.095" />
+    </link>
+    <joint name="raspberry_joint"
+           type="fixed" >
+      <parent link="base_link" />
+      <child link="raspberry" />
+      <origin xyz="0.071 0.076 0.24"
+              rpy="0.0 0.0 0.0" />
+    </joint>
+    <link name="arm" >
+      <xacro:solid_cuboid_inertial mass="0.050" width="0.064" height="0.03" depth="0.104" />
+    </link>
+    <joint name="arm_joint"
+           type="fixed" >
+      <parent link="base_link" />
+      <child link="arm" />
+      <origin xyz="-0.052 0.002 0.245"
+              rpy="0.0 0.0 ${PI_2}" />
     </joint>
     <link name="epos" >
@@ -213,4 +233,14 @@
               rpy="0.0 0.0 0.0" />
     </joint>
+    <link name="imu" >
+      <xacro:solid_cuboid_inertial mass="0.05" width="0.045" height="0.024" depth="0.057" />
+    </link>/
+    <joint name="imu_joint"
+           type="fixed" >
+      <parent link="base_link" />
+      <child link="imu" />
+      <origin xyz="0.09013 -0.08006 0.24281"
+              rpy="0.0 0.0 0.0" />
+    </joint>
   </xacro:macro>
 <!-- ###################################################################### -->

Commit message: Disable differential_link and fix inertia values [ci skip]

File: pandora_robots_description/urdf/woody/links/base_link.urdf.xacro (robot description, xacro)
@@ -177,11 +177,10 @@
         <origin xyz="0.0 0.0 0.0" />
         <mass value="0.6" />
-        <!-- TODO -->
-        <inertia ixx="0.0001"
-                 ixy="0.0"
-                 ixz="0.0"
-                 iyy="0.0001"
-                 iyz="0.0"
-                 izz="0.0001" />
+        <inertia ixx="0.00001"
+                 ixy="0.0"
+                 ixz="0.0"
+                 iyy="0.00001"
+                 iyz="0.0"
+                 izz="0.00001" />
       </inertial>
     </link>
@@ -194,15 +193,5 @@
     </joint>
     <link name="axis" >
-      <inertial>
-        <origin xyz="0.0 0.0 0.0" />
-        <mass value="0.446" />
-        <!-- TODO -->
-        <inertia ixx="0.0001"
-                 ixy="0.0"
-                 ixz="0.0"
-                 iyy="0.0001"
-                 iyz="0.0"
-                 izz="0.0001" />
-      </inertial>
+      <xacro:solid_cylinder_inertial mass="0.446" radius="0.03" height="0.267" />
     </link>
     <joint name="axis_joint"
@@ -211,24 +200,4 @@
       <child link="axis" />
       <origin xyz="0.0 0.0 0.0"
-              rpy="0.0 0.0 0.0" />
-    </joint>
-    <link name="differential" >
-      <inertial>
-        <origin xyz="0.0 0.0 0.0" />
-        <mass value="0.31" />
-        <!-- TODO -->
-        <inertia ixx="0.0001"
-                 ixy="0.0"
-                 ixz="0.0"
-                 iyy="0.0001"
-                 iyz="0.0"
-                 izz="0.0001" />
-      </inertial>
-    </link>
-    <joint name="differential_joint"
-           type="fixed" >
-      <parent link="base_link" />
-      <child link="differential" />
-      <origin xyz="-0.15 0.0 0.09031"
               rpy="0.0 0.0 0.0" />
     </joint>
@@ -243,4 +212,23 @@
               rpy="0.0 0.0 0.0" />
     </joint>
+<!--    <link name="differential" >-->
+<!--      <inertial>-->
+<!--        <origin xyz="0.0 0.0 0.0" />-->
+<!--        <mass value="0.31" />-->
+<!--        <inertia ixx="0.0001"-->
+<!--                 ixy="0.0"-->
+<!--                 ixz="0.0"-->
+<!--                 iyy="0.0001"-->
+<!--                 iyz="0.0"-->
+<!--                 izz="0.0001" />-->
+<!--      </inertial>-->
+<!--    </link>-->
+<!--    <joint name="differential_joint"-->
+<!--           type="fixed" >-->
+<!--      <parent link="base_link" />-->
+<!--      <child link="differential" />-->
+<!--      <origin xyz="-0.15 0.0 0.09031"-->
+<!--              rpy="0.0 0.0 0.0" />-->
+<!--    </joint>-->
   </xacro:macro>
 <!-- ###################################################################### -->
