Commit message: Refactor woody's link and joint files [ci skip]

File: pandora_robots_description/urdf/woody/links/base_link.urdf.xacro (robot description, xacro)
@@ -1,13 +1,9 @@
 <?xml version="1.0" ?>
 <robot xmlns:xacro="http://ros.org/wiki/xacro" >
-<!-- ###################################################################### -->
   <xacro:macro name="base_link" >
     <link name="base_link" >
       <inertial>
-        <!-- ============================================================== -->
         <origin xyz="-0.00968 -0.00122 0.19369" />
-        <!-- ============================================================== -->
         <mass value="8.25079" />
-        <!-- ============================================================== -->
         <inertia ixx="0.112701442"
                  ixy="-0.000233829"
@@ -16,25 +12,17 @@
                  iyz="-0.000177925"
                  izz="0.083438037" />
-        <!-- ============================================================== -->
       </inertial>
       <visual>
-        <!-- ============================================================== -->
         <xacro:default_origin />
-        <!-- ============================================================== -->
         <geometry>
           <mesh filename="package://pandora_robots_description/meshes/woody/visual/base/base_link.dae" />
         </geometry>
-        <!-- ============================================================== -->
         <material name="base" />
-        <!-- ============================================================== -->
       </visual>
       <collision>
-        <!-- ============================================================== -->
         <xacro:default_origin />
-        <!-- ============================================================== -->
         <geometry>
           <mesh filename="package://pandora_robots_description/meshes/woody/collision/base/base_link.stl" />
         </geometry>
-        <!-- ============================================================== -->
       </collision>
     </link>
@@ -135,5 +123,5 @@
               rpy="0.0 0.0 0.0" />
     </joint>
-    <link name="battery1" >
+    <link name="motor_battery" >
       <inertial>
         <origin xyz="0.0 0.0 0.0" />
@@ -147,12 +135,12 @@
       </inertial>
     </link>
-    <joint name="battery1_joint"
-           type="fixed" >
-      <parent link="base_link" />
-      <child link="battery1" />
+    <joint name="motor_battery_joint"
+           type="fixed" >
+      <parent link="base_link" />
+      <child link="motor_battery" />
       <origin xyz="0.10395 0.027 0.04822"
               rpy="0.0 0.0 0.0" />
     </joint>
-    <link name="battery2" >
+    <link name="pc_battery" >
       <inertial>
         <origin xyz="0.0 0.0 0.0" />
@@ -166,8 +154,8 @@
       </inertial>
     </link>
-    <joint name="battery2_joint"
-           type="fixed" >
-      <parent link="base_link" />
-      <child link="battery2" />
+    <joint name="pc_battery_joint"
+           type="fixed" >
+      <parent link="base_link" />
+      <child link="pc_battery" />
       <origin xyz="0.10395 -0.027 0.04822"
               rpy="0.0 0.0 0.0" />
@@ -232,4 +220,3 @@
 <!--    </joint>-->
   </xacro:macro>
-<!-- ###################################################################### -->
 </robot>
