Commit message: Remove redundant properties

File: pandora_robots_description/woody/urdf/joints/side_joint.urdf.xacro (robot description, xacro)
@@ -4,5 +4,5 @@
                params="prefix_y reflect_y" >
     <joint name="${prefix_y}_side_joint"
-           type="${side_joint_type}" >
+           type="revolute" >
       <parent link="base_link" />
       <child link="${prefix_y}_side_link" />

File: pandora_robots_description/woody/urdf/joints/wheel_joint.urdf.xacro (robot description, xacro)
@@ -4,5 +4,5 @@
                params="prefix_y prefix_x reflect_y reflect_x" >
     <joint name="${prefix_y}_${prefix_x}_wheel_joint"
-           type="${wheel_joint_type}" >
+           type="continuous" >
       <parent link="${prefix_y}_side_link" />
       <child link="${prefix_y}_${prefix_x}_wheel_link" />

File: pandora_robots_description/woody/urdf/links/base_link.urdf.xacro (robot description, xacro)
@@ -98,5 +98,5 @@
                  iyy="6.8283E-005"
                  iyz="0.0"
-                 izz="0.0002858833" /> <!-- XXX -->
+                 izz="0.0002858833" />
       </inertial>
     </link>

File: pandora_robots_description/woody/urdf/urdf_configurations.xacro (robot description, xacro)
@@ -13,6 +13,4 @@
   <xacro:property name="enable_microphone_sensor" value="false" />
   <!-- Joint Physics ###################################################### -->
-  <xacro:property name="side_joint_type" value="revolute" />
-  <xacro:property name="wheel_joint_type" value="continuous" />
   <xacro:property name="side_joint_damping" value="0.0" />
   <xacro:property name="wheel_joint_damping" value="0.0" />
