Commit message: Remove arguement in urdf for fixed joints

File: pandora_robots_description/woody/urdf/bringup.urdf.xacro (robot description, xacro)
@@ -3,4 +3,4 @@
        xmlns:xacro="http://ros.org/wiki/xacro" >
   <xacro:include filename="$(find pandora_robots_description)/urdf/woody/woody.urdf.xacro" />
-  <xacro:woody_urdf fixed="false" />
+  <xacro:woody_urdf />
 </robot>

File: pandora_robots_description/woody/urdf/woody.urdf.xacro (robot description, xacro)
@@ -19,51 +19,50 @@
   <xacro:include filename="$(find pandora_robots_description)/urdf/woody/sensors/co2_sensor.xacro" />
   <xacro:include filename="$(find pandora_robots_description)/urdf/woody/sensors/microphone_sensor.xacro" />
-<xacro:macro name="woody_urdf"
-             params="fixed" >
-  <!-- Load Links & Joints ################################################ -->
-  <xacro:base_link />
-  <xacro:side_link prefix_y="left" reflect_y="1" />
-  <xacro:side_joint prefix_y="left" reflect_y="1" />
-  <xacro:side_link prefix_y="right" reflect_y="-1" />
-  <xacro:side_joint prefix_y="right" reflect_y="-1" />
-  <xacro:wheel_link prefix_y="left" prefix_x="front" reflect_y="1" reflect_x="1" />
-  <xacro:wheel_joint prefix_y="left" prefix_x="front" reflect_y="1" reflect_x="1" />
-  <xacro:wheel_link prefix_y="left" prefix_x="rear" reflect_y="1" reflect_x="-1" />
-  <xacro:wheel_joint prefix_y="left" prefix_x="rear" reflect_y="1" reflect_x="-1" />
-  <xacro:wheel_link prefix_y="right" prefix_x="front" reflect_y="-1" reflect_x="1" />
-  <xacro:wheel_joint prefix_y="right" prefix_x="front" reflect_y="-1" reflect_x="1" />
-  <xacro:wheel_link prefix_y="right" prefix_x="rear" reflect_y="-1" reflect_x="-1" />
-  <xacro:wheel_joint prefix_y="right" prefix_x="rear" reflect_y="-1" reflect_x="-1" />
-  <!-- Load Sensors ####################################################### -->
-  <xacro:if value="${enable_laser_sensor}" >
-    <xacro:laser_sensor fixed="${fixed}" />
-  </xacro:if>
-  <xacro:if value="${enable_kinect_sensor}" >
-    <xacro:kinect_sensor fixed="${fixed}" />
-  </xacro:if>
-  <xacro:if value="${enable_flir_sensor}" >
-    <xacro:flir_sensor />
-  </xacro:if>
-  <xacro:if value="${enable_left_camera_sensor}" >
-    <xacro:left_camera_sensor />
-  </xacro:if>
-  <xacro:if value="${enable_right_camera_sensor}" >
-    <xacro:right_camera_sensor />
-  </xacro:if>
-  <xacro:if value="${enable_left_sonar_sensor}" >
-    <xacro:left_sonar_sensor />
-  </xacro:if>
-  <xacro:if value="${enable_right_sonar_sensor}" >
-    <xacro:right_sonar_sensor />
-  </xacro:if>
-  <xacro:if value="${enable_thermal_sensor}" >
-      <xacro:thermal_sensor />
-  </xacro:if>
-  <xacro:if value="${enable_co2_sensor}" >
-    <xacro:co2_sensor />
-  </xacro:if>
-  <xacro:if value="${enable_microphone_sensor}" >
-    <xacro:microphone_sensor />
-  </xacro:if>
-</xacro:macro>
+  <xacro:macro name="woody_urdf" >
+    <!-- Load Links & Joints ################################################ -->
+    <xacro:base_link />
+    <xacro:side_link prefix_y="left" reflect_y="1" />
+    <xacro:side_joint prefix_y="left" reflect_y="1" />
+    <xacro:side_link prefix_y="right" reflect_y="-1" />
+    <xacro:side_joint prefix_y="right" reflect_y="-1" />
+    <xacro:wheel_link prefix_y="left" prefix_x="front" reflect_y="1" reflect_x="1" />
+    <xacro:wheel_joint prefix_y="left" prefix_x="front" reflect_y="1" reflect_x="1" />
+    <xacro:wheel_link prefix_y="left" prefix_x="rear" reflect_y="1" reflect_x="-1" />
+    <xacro:wheel_joint prefix_y="left" prefix_x="rear" reflect_y="1" reflect_x="-1" />
+    <xacro:wheel_link prefix_y="right" prefix_x="front" reflect_y="-1" reflect_x="1" />
+    <xacro:wheel_joint prefix_y="right" prefix_x="front" reflect_y="-1" reflect_x="1" />
+    <xacro:wheel_link prefix_y="right" prefix_x="rear" reflect_y="-1" reflect_x="-1" />
+    <xacro:wheel_joint prefix_y="right" prefix_x="rear" reflect_y="-1" reflect_x="-1" />
+    <!-- Load Sensors ####################################################### -->
+    <xacro:if value="${enable_laser_sensor}" >
+      <xacro:laser_sensor fixed="${fixed}" />
+    </xacro:if>
+    <xacro:if value="${enable_kinect_sensor}" >
+      <xacro:kinect_sensor fixed="${fixed}" />
+    </xacro:if>
+    <xacro:if value="${enable_flir_sensor}" >
+      <xacro:flir_sensor />
+    </xacro:if>
+    <xacro:if value="${enable_left_camera_sensor}" >
+      <xacro:left_camera_sensor />
+    </xacro:if>
+    <xacro:if value="${enable_right_camera_sensor}" >
+      <xacro:right_camera_sensor />
+    </xacro:if>
+    <xacro:if value="${enable_left_sonar_sensor}" >
+      <xacro:left_sonar_sensor />
+    </xacro:if>
+    <xacro:if value="${enable_right_sonar_sensor}" >
+      <xacro:right_sonar_sensor />
+    </xacro:if>
+    <xacro:if value="${enable_thermal_sensor}" >
+        <xacro:thermal_sensor />
+    </xacro:if>
+    <xacro:if value="${enable_co2_sensor}" >
+      <xacro:co2_sensor />
+    </xacro:if>
+    <xacro:if value="${enable_microphone_sensor}" >
+      <xacro:microphone_sensor />
+    </xacro:if>
+  </xacro:macro>
 </robot>

Commit message: Rearrange mesh files

File: pandora_robots_description/woody/urdf/bringup.urdf.xacro (robot description, xacro)
@@ -2,5 +2,5 @@
 <robot name="woody"
        xmlns:xacro="http://ros.org/wiki/xacro" >
-  <xacro:include filename="$(find pandora_robots_description)/urdf/woody/woody.urdf.xacro" />
+  <xacro:include filename="$(find pandora_robots_description)/woody/urdf/woody.urdf.xacro" />
   <xacro:woody_urdf />
 </robot>

File: pandora_robots_description/woody/urdf/links/base_link.urdf.xacro (robot description, xacro)
@@ -16,5 +16,5 @@
         <xacro:default_origin />
         <geometry>
-          <mesh filename="package://pandora_robots_description/meshes/woody/visual/base/base_link.dae" />
+          <mesh filename="package://pandora_robots_description/woody/meshes/base_link.dae" />
         </geometry>
         <material name="base" />
@@ -23,5 +23,5 @@
         <xacro:default_origin />
         <geometry>
-          <mesh filename="package://pandora_robots_description/meshes/woody/collision/base/base_link.stl" />
+          <mesh filename="package://pandora_robots_description/woody/meshes/base_link.stl" />
         </geometry>
       </collision>

File: pandora_robots_description/woody/urdf/links/side_link.urdf.xacro (robot description, xacro)
@@ -18,5 +18,5 @@
                 rpy="0.0 0.0 ${ ( 1 - reflect_y ) * PI_2 }" />
         <geometry>
-          <mesh filename="package://pandora_robots_description/meshes/woody/visual/side/side_link.dae" />
+          <mesh filename="package://pandora_robots_description/woody/meshes/side_link.dae" />
         </geometry>
         <material name="side" />
@@ -26,5 +26,5 @@
                 rpy="0.0 0.0 ${ ( 1 - reflect_y ) * PI_2 }" />
         <geometry>
-          <mesh filename="package://pandora_robots_description/meshes/woody/collision/side/side_link.stl" />
+          <mesh filename="package://pandora_robots_description/woody/meshes/side_link.stl" />
         </geometry>
       </collision>

File: pandora_robots_description/woody/urdf/links/wheel_link.urdf.xacro (robot description, xacro)
@@ -18,5 +18,5 @@
                 rpy="0.0 0.0 ${ ( 1 - reflect_y ) * PI_2 }" />
         <geometry>
-          <mesh filename="package://pandora_robots_description/meshes/woody/visual/wheel/wheel_link.dae" />
+          <mesh filename="package://pandora_robots_description/woody/meshes/wheel_link.dae" />
         </geometry>
         <material name="wheel" />
@@ -26,5 +26,5 @@
                 rpy="0.0 0.0 ${ ( 1 - reflect_y ) * PI_2 }" />
         <geometry>
-          <mesh filename="package://pandora_robots_description/meshes/woody/collision/wheel/wheel_link.stl" />
+          <mesh filename="package://pandora_robots_description/woody/meshes/wheel_link.stl" />
         </geometry>
       </collision>

File: pandora_robots_description/woody/urdf/woody.urdf.xacro (robot description, xacro)
@@ -2,23 +2,23 @@
 <robot xmlns:xacro="http://ros.org/wiki/xacro" >
   <!-- Import Files ####################################################### -->
-  <xacro:include filename="$(find pandora_robots_description)/urdf/woody/urdf_configurations.xacro" />
-  <xacro:include filename="$(find pandora_robots_description)/urdf/woody/properties/constants.xacro" />
-  <xacro:include filename="$(find pandora_robots_description)/urdf/woody/properties/defaults.xacro" />
-  <xacro:include filename="$(find pandora_robots_description)/urdf/woody/properties/materials.xacro" />
-  <xacro:include filename="$(find pandora_robots_description)/urdf/woody/links/base_link.urdf.xacro" />
-  <xacro:include filename="$(find pandora_robots_description)/urdf/woody/links/side_link.urdf.xacro" />
-  <xacro:include filename="$(find pandora_robots_description)/urdf/woody/links/wheel_link.urdf.xacro" />
-  <xacro:include filename="$(find pandora_robots_description)/urdf/woody/joints/side_joint.urdf.xacro" />
-  <xacro:include filename="$(find pandora_robots_description)/urdf/woody/joints/wheel_joint.urdf.xacro" />
-  <xacro:include filename="$(find pandora_robots_description)/urdf/woody/sensors/laser_sensor.xacro" />
-  <xacro:include filename="$(find pandora_robots_description)/urdf/woody/sensors/kinect_sensor.xacro" />
-  <xacro:include filename="$(find pandora_robots_description)/urdf/woody/sensors/flir_sensor.xacro" />
-  <xacro:include filename="$(find pandora_robots_description)/urdf/woody/sensors/camera_sensor.xacro" />
-  <xacro:include filename="$(find pandora_robots_description)/urdf/woody/sensors/sonar_sensor.xacro" />
-  <xacro:include filename="$(find pandora_robots_description)/urdf/woody/sensors/thermal_sensor.xacro" />
-  <xacro:include filename="$(find pandora_robots_description)/urdf/woody/sensors/co2_sensor.xacro" />
-  <xacro:include filename="$(find pandora_robots_description)/urdf/woody/sensors/microphone_sensor.xacro" />
+  <xacro:include filename="$(find pandora_robots_description)/woody/urdf/urdf_configurations.xacro" />
+  <xacro:include filename="$(find pandora_robots_description)/woody/urdf/properties/constants.xacro" />
+  <xacro:include filename="$(find pandora_robots_description)/woody/urdf/properties/defaults.xacro" />
+  <xacro:include filename="$(find pandora_robots_description)/woody/urdf/properties/materials.xacro" />
+  <xacro:include filename="$(find pandora_robots_description)/woody/urdf/links/base_link.urdf.xacro" />
+  <xacro:include filename="$(find pandora_robots_description)/woody/urdf/links/side_link.urdf.xacro" />
+  <xacro:include filename="$(find pandora_robots_description)/woody/urdf/links/wheel_link.urdf.xacro" />
+  <xacro:include filename="$(find pandora_robots_description)/woody/urdf/joints/side_joint.urdf.xacro" />
+  <xacro:include filename="$(find pandora_robots_description)/woody/urdf/joints/wheel_joint.urdf.xacro" />
+  <xacro:include filename="$(find pandora_robots_description)/woody/urdf/sensors/laser_sensor.xacro" />
+  <xacro:include filename="$(find pandora_robots_description)/woody/urdf/sensors/kinect_sensor.xacro" />
+  <xacro:include filename="$(find pandora_robots_description)/woody/urdf/sensors/flir_sensor.xacro" />
+  <xacro:include filename="$(find pandora_robots_description)/woody/urdf/sensors/camera_sensor.xacro" />
+  <xacro:include filename="$(find pandora_robots_description)/woody/urdf/sensors/sonar_sensor.xacro" />
+  <xacro:include filename="$(find pandora_robots_description)/woody/urdf/sensors/thermal_sensor.xacro" />
+  <xacro:include filename="$(find pandora_robots_description)/woody/urdf/sensors/co2_sensor.xacro" />
+  <xacro:include filename="$(find pandora_robots_description)/woody/urdf/sensors/microphone_sensor.xacro" />
   <xacro:macro name="woody_urdf" >
-    <!-- Load Links & Joints ################################################ -->
+    <!-- Load Links & Joints ############################################## -->
     <xacro:base_link />
     <xacro:side_link prefix_y="left" reflect_y="1" />
@@ -34,5 +34,5 @@
     <xacro:wheel_link prefix_y="right" prefix_x="rear" reflect_y="-1" reflect_x="-1" />
     <xacro:wheel_joint prefix_y="right" prefix_x="rear" reflect_y="-1" reflect_x="-1" />
-    <!-- Load Sensors ####################################################### -->
+    <!-- Load Sensors ##################################################### -->
     <xacro:if value="${enable_laser_sensor}" >
       <xacro:laser_sensor fixed="${fixed}" />
