Commit message: Remove main urdf macro and delete bringup file

File: pandora_robots_description/woody/urdf/woody.urdf.xacro (robot description, xacro)
@@ -1,4 +1,5 @@
 <?xml version="1.0"?>
-<robot xmlns:xacro="http://ros.org/wiki/xacro" >
+<robot name="woody"
+       xmlns:xacro="http://ros.org/wiki/xacro" >
   <!-- Import Files ####################################################### -->
   <xacro:include filename="$(find pandora_urdf_properties)/xacro/constants.xacro" />
@@ -19,50 +20,48 @@
   <xacro:include filename="$(find pandora_robots_description)/woody/urdf/sensors/co2_sensor.xacro" />
   <xacro:include filename="$(find pandora_robots_description)/woody/urdf/sensors/microphone_sensor.xacro" />
-  <xacro:macro name="woody_urdf" >
-    <!-- Load Links & Joints ############################################## -->
-    <xacro:base_link />
-    <xacro:side_link prefix_y="left" reflect_y="1" />
-    <xacro:side_joint prefix_y="left" reflect_y="1" />
-    <xacro:side_link prefix_y="right" reflect_y="-1" />
-    <xacro:side_joint prefix_y="right" reflect_y="-1" />
-    <xacro:wheel_link prefix_y="left" prefix_x="front" reflect_y="1" reflect_x="1" />
-    <xacro:wheel_joint prefix_y="left" prefix_x="front" reflect_y="1" reflect_x="1" />
-    <xacro:wheel_link prefix_y="left" prefix_x="rear" reflect_y="1" reflect_x="-1" />
-    <xacro:wheel_joint prefix_y="left" prefix_x="rear" reflect_y="1" reflect_x="-1" />
-    <xacro:wheel_link prefix_y="right" prefix_x="front" reflect_y="-1" reflect_x="1" />
-    <xacro:wheel_joint prefix_y="right" prefix_x="front" reflect_y="-1" reflect_x="1" />
-    <xacro:wheel_link prefix_y="right" prefix_x="rear" reflect_y="-1" reflect_x="-1" />
-    <xacro:wheel_joint prefix_y="right" prefix_x="rear" reflect_y="-1" reflect_x="-1" />
-    <!-- Load Sensors ##################################################### -->
-    <xacro:if value="${enable_laser_sensor}" >
-      <xacro:laser_sensor />
-    </xacro:if>
-    <xacro:if value="${enable_kinect_sensor}" >
-      <xacro:kinect_sensor />
-    </xacro:if>
-    <xacro:if value="${enable_flir_sensor}" >
-      <xacro:flir_sensor />
-    </xacro:if>
-    <xacro:if value="${enable_left_camera_sensor}" >
-      <xacro:left_camera_sensor />
-    </xacro:if>
-    <xacro:if value="${enable_right_camera_sensor}" >
-      <xacro:right_camera_sensor />
-    </xacro:if>
-    <xacro:if value="${enable_left_sonar_sensor}" >
-      <xacro:left_sonar_sensor />
-    </xacro:if>
-    <xacro:if value="${enable_right_sonar_sensor}" >
-      <xacro:right_sonar_sensor />
-    </xacro:if>
-    <xacro:if value="${enable_thermal_sensor}" >
-      <xacro:thermal_sensor />
-    </xacro:if>
-    <xacro:if value="${enable_co2_sensor}" >
-      <xacro:co2_sensor />
-    </xacro:if>
-    <xacro:if value="${enable_microphone_sensor}" >
-      <xacro:microphone_sensor />
-    </xacro:if>
-  </xacro:macro>
+  <!-- Load Links & Joints ################################################ -->
+  <xacro:base_link />
+  <xacro:side_link prefix_y="left" reflect_y="1" />
+  <xacro:side_joint prefix_y="left" reflect_y="1" />
+  <xacro:side_link prefix_y="right" reflect_y="-1" />
+  <xacro:side_joint prefix_y="right" reflect_y="-1" />
+  <xacro:wheel_link prefix_y="left" prefix_x="front" reflect_y="1" reflect_x="1" />
+  <xacro:wheel_joint prefix_y="left" prefix_x="front" reflect_y="1" reflect_x="1" />
+  <xacro:wheel_link prefix_y="left" prefix_x="rear" reflect_y="1" reflect_x="-1" />
+  <xacro:wheel_joint prefix_y="left" prefix_x="rear" reflect_y="1" reflect_x="-1" />
+  <xacro:wheel_link prefix_y="right" prefix_x="front" reflect_y="-1" reflect_x="1" />
+  <xacro:wheel_joint prefix_y="right" prefix_x="front" reflect_y="-1" reflect_x="1" />
+  <xacro:wheel_link prefix_y="right" prefix_x="rear" reflect_y="-1" reflect_x="-1" />
+  <xacro:wheel_joint prefix_y="right" prefix_x="rear" reflect_y="-1" reflect_x="-1" />
+  <!-- Load Sensors ####################################################### -->
+  <xacro:if value="${enable_laser_sensor}" >
+    <xacro:laser_sensor />
+  </xacro:if>
+  <xacro:if value="${enable_kinect_sensor}" >
+    <xacro:kinect_sensor />
+  </xacro:if>
+  <xacro:if value="${enable_flir_sensor}" >
+    <xacro:flir_sensor />
+  </xacro:if>
+  <xacro:if value="${enable_left_camera_sensor}" >
+    <xacro:left_camera_sensor />
+  </xacro:if>
+  <xacro:if value="${enable_right_camera_sensor}" >
+    <xacro:right_camera_sensor />
+  </xacro:if>
+  <xacro:if value="${enable_left_sonar_sensor}" >
+    <xacro:left_sonar_sensor />
+  </xacro:if>
+  <xacro:if value="${enable_right_sonar_sensor}" >
+    <xacro:right_sonar_sensor />
+  </xacro:if>
+  <xacro:if value="${enable_thermal_sensor}" >
+    <xacro:thermal_sensor />
+  </xacro:if>
+  <xacro:if value="${enable_co2_sensor}" >
+    <xacro:co2_sensor />
+  </xacro:if>
+  <xacro:if value="${enable_microphone_sensor}" >
+    <xacro:microphone_sensor />
+  </xacro:if>
 </robot>
