Commit message: Delete args in urdf_configurations that enable/disable sensors

File: pandora_robots_description/woody/urdf/urdf_configurations.xacro (robot description, xacro)
@@ -1,16 +1,5 @@
 <?xml version="1.0"?>
 <robot xmlns:xacro="http://ros.org/wiki/xacro" >
-  <!-- Sensors ############################################################ -->
-  <xacro:property name="enable_laser_sensor" value="true" />
-  <xacro:property name="enable_kinect_sensor" value="true" />
-  <xacro:property name="enable_flir_sensor" value="true" />
-  <xacro:property name="enable_left_camera_sensor" value="true" />
-  <xacro:property name="enable_right_camera_sensor" value="true" />
-  <xacro:property name="enable_left_sonar_sensor" value="true" />
-  <xacro:property name="enable_right_sonar_sensor" value="true" />
-  <xacro:property name="enable_thermal_sensor" value="true" />
-  <xacro:property name="enable_co2_sensor" value="true" />
-  <xacro:property name="enable_microphone_sensor" value="false" />
-  <!-- Joint Physics ###################################################### -->
+  <!-- Joints ############################################################# -->
   <xacro:property name="side_joint_damping" value="0.0" />
   <xacro:property name="wheel_joint_damping" value="0.0" />

File: pandora_robots_description/woody/urdf/woody.urdf.xacro (robot description, xacro)
@@ -35,33 +35,13 @@
   <xacro:wheel_joint prefix_y="right" prefix_x="rear" reflect_y="-1" reflect_x="-1" />
   <!-- Load Sensors ####################################################### -->
-  <xacro:if value="${enable_laser_sensor}" >
-    <xacro:laser_sensor />
-  </xacro:if>
-  <xacro:if value="${enable_kinect_sensor}" >
-    <xacro:kinect_sensor />
-  </xacro:if>
-  <xacro:if value="${enable_flir_sensor}" >
-    <xacro:flir_sensor />
-  </xacro:if>
-  <xacro:if value="${enable_left_camera_sensor}" >
-    <xacro:left_camera_sensor />
-  </xacro:if>
-  <xacro:if value="${enable_right_camera_sensor}" >
-    <xacro:right_camera_sensor />
-  </xacro:if>
-  <xacro:if value="${enable_left_sonar_sensor}" >
-    <xacro:left_sonar_sensor />
-  </xacro:if>
-  <xacro:if value="${enable_right_sonar_sensor}" >
-    <xacro:right_sonar_sensor />
-  </xacro:if>
-  <xacro:if value="${enable_thermal_sensor}" >
-    <xacro:thermal_sensor />
-  </xacro:if>
-  <xacro:if value="${enable_co2_sensor}" >
-    <xacro:co2_sensor />
-  </xacro:if>
-  <xacro:if value="${enable_microphone_sensor}" >
-    <xacro:microphone_sensor />
-  </xacro:if>
+  <xacro:laser_sensor />
+  <xacro:kinect_sensor />
+  <xacro:flir_sensor />
+  <xacro:left_camera_sensor />
+  <xacro:right_camera_sensor />
+  <xacro:left_sonar_sensor />
+  <xacro:right_sonar_sensor />
+  <xacro:thermal_sensor />
+  <xacro:co2_sensor />
+  <!--<xacro:microphone_sensor />-->
 </robot>
