Commit message: Add pandora_urdf_properties package

File: pandora_robots_description/woody/urdf/links/base_link.urdf.xacro (robot description, xacro)
@@ -14,5 +14,4 @@
       </inertial>
       <visual>
-        <xacro:default_origin />
         <geometry>
           <mesh filename="package://pandora_robots_description/woody/meshes/base_link.dae" />
@@ -21,5 +20,4 @@
       </visual>
       <collision>
-        <xacro:default_origin />
         <geometry>
           <mesh filename="package://pandora_robots_description/woody/meshes/base_link.stl" />

File: pandora_robots_description/woody/urdf/woody.urdf.xacro (robot description, xacro)
@@ -2,8 +2,8 @@
 <robot xmlns:xacro="http://ros.org/wiki/xacro" >
   <!-- Import Files ####################################################### -->
+  <xacro:include filename="$(find pandora_urdf_properties)/xacro/constants.xacro" />
+  <xacro:include filename="$(find pandora_urdf_properties)/xacro/defaults.xacro" />
+  <xacro:include filename="$(find pandora_urdf_properties)/xacro/materials.xacro" />
   <xacro:include filename="$(find pandora_robots_description)/woody/urdf/urdf_configurations.xacro" />
-  <xacro:include filename="$(find pandora_robots_description)/woody/urdf/properties/constants.xacro" />
-  <xacro:include filename="$(find pandora_robots_description)/woody/urdf/properties/defaults.xacro" />
-  <xacro:include filename="$(find pandora_robots_description)/woody/urdf/properties/materials.xacro" />
   <xacro:include filename="$(find pandora_robots_description)/woody/urdf/links/base_link.urdf.xacro" />
   <xacro:include filename="$(find pandora_robots_description)/woody/urdf/links/side_link.urdf.xacro" />

File: pandora_sensors_description/urdf/camera.urdf.xacro (robot description, xacro)
@@ -1,4 +1,6 @@
 <?xml version="1.0" ?>
 <robot xmlns:xacro="http://ros.org/wiki/xacro" >
+  <xacro:include filename="$(find pandora_urdf_properties)/xacro/constants.xacro" />
+  <xacro:include filename="$(find pandora_urdf_properties)/xacro/defaults.xacro" />
 <!-- ###################################################################### -->
   <xacro:macro name="camera_caster"

File: pandora_sensors_description/urdf/co2.urdf.xacro (robot description, xacro)
@@ -1,4 +1,6 @@
 <?xml version="1.0" ?>
 <robot xmlns:xacro="http://ros.org/wiki/xacro" >
+  <xacro:include filename="$(find pandora_urdf_properties)/xacro/constants.xacro" />
+  <xacro:include filename="$(find pandora_urdf_properties)/xacro/defaults.xacro" />
 <!-- ###################################################################### -->
   <xacro:macro name="co2_caster"

File: pandora_sensors_description/urdf/flir.urdf.xacro (robot description, xacro)
@@ -1,4 +1,6 @@
 <?xml version="1.0" ?>
 <robot xmlns:xacro="http://ros.org/wiki/xacro" >
+  <xacro:include filename="$(find pandora_urdf_properties)/xacro/constants.xacro" />
+  <xacro:include filename="$(find pandora_urdf_properties)/xacro/defaults.xacro" />
 <!-- ###################################################################### -->
   <xacro:macro name="flir_caster"

File: pandora_sensors_description/urdf/kinect.urdf.xacro (robot description, xacro)
@@ -1,6 +1,6 @@
 <?xml version="1.0" ?>
 <robot xmlns:xacro="http://ros.org/wiki/xacro" >
-  <xacro:include filename="$(find pandora_robots_description)/urdf/woody/properties/constants.xacro" />
-  <xacro:include filename="$(find pandora_robots_description)/urdf/woody/properties/defaults.xacro" />
+  <xacro:include filename="$(find pandora_urdf_properties)/xacro/constants.xacro" />
+  <xacro:include filename="$(find pandora_urdf_properties)/xacro/defaults.xacro" />
   <xacro:macro name="kinect_caster"
                params="parent

File: pandora_sensors_description/urdf/laser.urdf.xacro (robot description, xacro)
@@ -1,6 +1,6 @@
 <?xml version="1.0" ?>
 <robot xmlns:xacro="http://ros.org/wiki/xacro" >
-  <xacro:include filename="$(find pandora_robots_description)/urdf/woody/properties/constants.xacro" />
-  <xacro:include filename="$(find pandora_robots_description)/urdf/woody/properties/defaults.xacro" />
+  <xacro:include filename="$(find pandora_urdf_properties)/xacro/constants.xacro" />
+  <xacro:include filename="$(find pandora_urdf_properties)/xacro/defaults.xacro" />
   <xacro:macro name="laser_caster"
                params="parent

File: pandora_sensors_description/urdf/microphone.urdf.xacro (robot description, xacro)
@@ -1,4 +1,6 @@
 <?xml version="1.0" ?>
 <robot xmlns:xacro="http://ros.org/wiki/xacro" >
+  <xacro:include filename="$(find pandora_urdf_properties)/xacro/constants.xacro" />
+  <xacro:include filename="$(find pandora_urdf_properties)/xacro/defaults.xacro" />
 <!-- ###################################################################### -->
   <xacro:macro name="microphone_caster"

File: pandora_sensors_description/urdf/sonar.urdf.xacro (robot description, xacro)
@@ -1,4 +1,6 @@
 <?xml version="1.0" ?>
 <robot xmlns:xacro="http://ros.org/wiki/xacro" >
+  <xacro:include filename="$(find pandora_urdf_properties)/xacro/constants.xacro" />
+  <xacro:include filename="$(find pandora_urdf_properties)/xacro/defaults.xacro" />
 <!-- ###################################################################### -->
   <xacro:macro name="sonar_caster"

File: pandora_sensors_description/urdf/thermal.urdf.xacro (robot description, xacro)
@@ -1,4 +1,6 @@
 <?xml version="1.0" ?>
 <robot xmlns:xacro="http://ros.org/wiki/xacro" >
+  <xacro:include filename="$(find pandora_urdf_properties)/xacro/constants.xacro" />
+  <xacro:include filename="$(find pandora_urdf_properties)/xacro/defaults.xacro" />
 <!-- ###################################################################### -->
   <xacro:macro name="thermal_caster"

File: pandora_urdf_properties/xacro/defaults.xacro (robot description, xacro)
@@ -42,49 +42,41 @@
   </xacro:macro>
   <xacro:macro name="solid_sphere_inertial"
-               params="mass
-                       radius
+               params="mass radius *origin" >
+    <inertial>
+      <xacro:insert_block name="origin" />
+      <mass value="${mass}" />
+      <inertia ixx="${(2 / 5) * mass * (radius * radius)}"
+               ixy="0.0"
+               ixz="0.0"
+               iyy="${(2 / 5) * mass * (radius * radius)}"
+               iyz="0.0"
+               izz="${(2 / 5) * mass * (radius * radius)}" />
+    </inertial>
+  </xacro:macro>
+  <xacro:macro name="solid_cuboid_inertial"
+               params="mass x y z
                        *origin" >
     <inertial>
       <xacro:insert_block name="origin" />
       <mass value="${mass}" />
-      <inertia ixx="${ ( 2 / 5 ) * mass * ( radius * radius ) }"
+      <inertia ixx="${(1 / 12) * mass * ((y * y) + (z * z))}"
                ixy="0.0"
                ixz="0.0"
-               iyy="${ ( 2 / 5 ) * mass * ( radius * radius ) }"
+               iyy="${(1 / 12) * mass * ((x * x) + (z * z))}"
                iyz="0.0"
-               izz="${ ( 2 / 5 ) * mass * ( radius * radius ) }" />
+               izz="${(1 / 12) * mass * ((x * x) + (y * y))}" />
     </inertial>
   </xacro:macro>
-  <xacro:macro name="solid_cuboid_inertial"
-               params="mass
-                       x
-                       y
-                       z
-                       *origin" >
+  <xacro:macro name="solid_cylinder_inertial"
+               params="mass radius height *origin" >
     <inertial>
       <xacro:insert_block name="origin" />
       <mass value="${mass}" />
-      <inertia ixx="${ ( 1 / 12 ) * mass * ( ( y * y ) + ( z * z ) ) }"
+      <inertia ixx="${(1 / 12) * mass * (3 * (radius * radius) + (height * height))}"
                ixy="0.0"
                ixz="0.0"
-               iyy="${ ( 1 / 12 ) * mass * ( ( x * x ) + ( z * z ) ) }"
+               iyy="${(1 / 12) * mass * (3 * (radius * radius) + (height * height))}"
                iyz="0.0"
-               izz="${ ( 1 / 12 ) * mass * ( ( x * x ) + ( y * y ) ) }" />
-    </inertial>
-  </xacro:macro>
-  <xacro:macro name="solid_cylinder_inertial"
-               params="mass
-                       radius
-                       height
-                       *origin" >
-    <inertial>
-      <xacro:insert_block name="origin" />
-      <mass value="${mass}" />
-      <inertia ixx="${ ( 1 / 12 ) * mass * ( 3 * ( radius * radius ) + ( height * height ) ) }"
-               ixy="0.0"
-               ixz="0.0"
-               iyy="${ ( 1 / 12 ) * mass * ( 3 * ( radius * radius ) + ( height * height ) ) }"
-               iyz="0.0"
-               izz="${ ( 1 / 2 ) * mass * ( radius * radius ) }" />
+               izz="${(1 / 2) * mass * (radius * radius)}" />
     </inertial>
   </xacro:macro>
