Commit message: Remove fixed args from laser and kinect description

File: pandora_robots_description/woody/urdf/sensors/kinect_sensor.xacro (robot description, xacro)
@@ -2,8 +2,6 @@
 <robot xmlns:xacro="http://ros.org/wiki/xacro" >
   <xacro:include filename="$(find pandora_sensors_description)/urdf/kinect.urdf.xacro" />
-  <xacro:macro name="kinect_sensor"
-               params="fixed" >
+  <xacro:macro name="kinect_sensor" >
     <xacro:kinect_caster parent="base_link"
-                         fixed="${fixed}"
                          pitch_min_limit="${kinect_pitch_joint_min_limit}"
                          pitch_max_limit="${kinect_pitch_joint_max_limit}"

File: pandora_robots_description/woody/urdf/sensors/laser_sensor.xacro (robot description, xacro)
@@ -2,8 +2,6 @@
 <robot xmlns:xacro="http://ros.org/wiki/xacro" >
   <xacro:include filename="$(find pandora_sensors_description)/urdf/laser.urdf.xacro" />
-  <xacro:macro name="laser_sensor"
-               params="fixed" >
+  <xacro:macro name="laser_sensor" >
     <xacro:laser_caster parent="base_link"
-                        fixed="${fixed}"
                         roll_min_limit="${laser_roll_joint_min_limit}"
                         roll_max_limit="${laser_roll_joint_max_limit}"

File: pandora_robots_description/woody/urdf/woody.urdf.xacro (robot description, xacro)
@@ -36,8 +36,8 @@
     <!-- Load Sensors ##################################################### -->
     <xacro:if value="${enable_laser_sensor}" >
-      <xacro:laser_sensor fixed="${fixed}" />
+      <xacro:laser_sensor />
     </xacro:if>
     <xacro:if value="${enable_kinect_sensor}" >
-      <xacro:kinect_sensor fixed="${fixed}" />
+      <xacro:kinect_sensor />
     </xacro:if>
     <xacro:if value="${enable_flir_sensor}" >
@@ -57,5 +57,5 @@
     </xacro:if>
     <xacro:if value="${enable_thermal_sensor}" >
-        <xacro:thermal_sensor />
+      <xacro:thermal_sensor />
     </xacro:if>
     <xacro:if value="${enable_co2_sensor}" >

File: pandora_sensors_description/urdf/kinect.urdf.xacro (robot description, xacro)
@@ -4,11 +4,7 @@
   <xacro:include filename="$(find pandora_urdf_properties)/xacro/defaults.xacro" />
   <xacro:macro name="kinect_caster"
-               params="parent
-                       fixed
-                       pitch_min_limit
-                       pitch_max_limit
-                       yaw_min_limit
-                       yaw_max_limit
-                       *origin" >
+               params="parent *origin
+                       pitch_min_limit pitch_max_limit
+                       yaw_min_limit yaw_max_limit" >
     <!-- Links ############################################################ -->
     <link name="kinect_yaw_servo_link" >
@@ -78,4 +74,41 @@
       </collision>
     </link>
+    <!-- Joints ########################################################### -->
+    <joint name="kinect_servo_parent_joint"
+           type="fixed" >
+      <parent link="${parent}" />
+      <child link="kinect_yaw_servo_link" />
+      <xacro:insert_block name="origin" />
+    </joint>
+    <joint name="kinect_yaw_joint"
+           type="revolute" >
+      <parent link="kinect_yaw_servo_link" />
+      <child link="kinect_pitch_servo_link" />
+      <origin xyz="0.0 0.0 0.06749"
+              rpy="0.0 0.0 0.0" />
+      <axis xyz="0 0 1" />
+      <limit lower="${yaw_min_limit}"
+             upper="${yaw_max_limit}"
+             effort="50"
+             velocity="50.0" />
+    </joint>
+    <joint name="kinect_pitch_joint"
+           type="revolute" >
+      <parent link="kinect_pitch_servo_link" />
+      <child link="kinect_platform_link" />
+      <axis xyz="0 1 0" />
+      <limit lower="${pitch_min_limit}"
+             upper="${pitch_max_limit}"
+             effort="50"
+             velocity="50.0" />
+    </joint>
+    <joint name="kinect_platform_joint"
+           type="fixed" >
+      <parent link="kinect_platform_link" />
+      <child link="kinect_link" />
+      <origin xyz="0.03261 -0.00101 0.04261"
+              rpy="0.0 0.0 0.0" />
+    </joint>
+    <!-- Frames ########################################################### -->
     <link name="kinect_frame" >
       <xacro:point_mass_inertial />
@@ -96,57 +129,4 @@
       <xacro:point_mass_inertial />
     </link>
-    <!-- Joints ########################################################### -->
-    <joint name="kinect_servo_base_joint"
-           type="fixed" >
-      <parent link="${parent}" />
-      <child link="kinect_yaw_servo_link" />
-      <xacro:insert_block name="origin" />
-    </joint>
-    <xacro:if value="${fixed}" >
-      <joint name="kinect_yaw_joint"
-             type="fixed" >
-        <parent link="kinect_yaw_servo_link" />
-        <child link="kinect_pitch_servo_link" />
-        <origin xyz="0.0 0.0 0.06749"
-                rpy="0.0 0.0 0.0" />
-      </joint>
-      <joint name="kinect_pitch_joint"
-             type="fixed" >
-        <parent link="kinect_pitch_servo_link" />
-        <child link="kinect_platform_link" />
-      </joint>
-    </xacro:if>
-    <xacro:unless value="${fixed}" >
-      <joint name="kinect_yaw_joint"
-             type="revolute" >
-        <parent link="kinect_yaw_servo_link" />
-        <child link="kinect_pitch_servo_link" />
-        <origin xyz="0.0 0.0 0.06749"
-                rpy="0.0 0.0 0.0" />
-        <axis xyz="0 0 1" />
-        <limit lower="${yaw_min_limit}"
-               upper="${yaw_max_limit}"
-               effort="50"
-               velocity="50.0" />
-      </joint>
-      <joint name="kinect_pitch_joint"
-             type="revolute" >
-        <parent link="kinect_pitch_servo_link" />
-        <child link="kinect_platform_link" />
-        <axis xyz="0 1 0" />
-        <limit lower="${pitch_min_limit}"
-               upper="${pitch_max_limit}"
-               effort="50"
-               velocity="50.0" />
-      </joint>
-    </xacro:unless>
-    <joint name="kinect_platform_joint"
-           type="fixed" >
-      <parent link="kinect_platform_link" />
-      <child link="kinect_link" />
-      <origin xyz="0.03261 -0.00101 0.04261"
-              rpy="0.0 0.0 0.0" />
-    </joint>
-    <!-- Frames ########################################################### -->
     <joint name="kinect_joint"
            type="fixed" >

File: pandora_sensors_description/urdf/laser.urdf.xacro (robot description, xacro)
@@ -4,11 +4,7 @@
   <xacro:include filename="$(find pandora_urdf_properties)/xacro/defaults.xacro" />
   <xacro:macro name="laser_caster"
-               params="parent
-                       fixed
-                       roll_min_limit
-                       roll_max_limit
-                       pitch_min_limit
-                       pitch_max_limit
-                       *origin" >
+               params="parent *origin
+                       roll_min_limit roll_max_limit
+                       pitch_min_limit pitch_max_limit" >
     <!-- Links ############################################################ -->
     <link name="laser_roll_servo_link" >
@@ -63,9 +59,6 @@
       </collision>
     </link>
-    <link name="laser_link" >
-      <xacro:point_mass_inertial />
-    </link>
     <!-- Joints ########################################################### -->
-    <joint name="laser_servo_base_joint"
+    <joint name="laser_servo_parent_joint"
            type="fixed" >
       <parent link="${parent}" />
@@ -73,46 +66,32 @@
       <xacro:insert_block name="origin" />
     </joint>
-    <xacro:if value="${fixed}" >
-      <joint name="laser_roll_joint"
-             type="fixed" >
-        <parent link="laser_roll_servo_link" />
-        <child link="laser_pitch_servo_link" />
-        <origin xyz="0.03999 0.0 0.0"
-                rpy="0 0 0" />
-      </joint>
-      <joint name="laser_pitch_joint"
-             type="fixed" >
-        <parent link="laser_pitch_servo_link" />
-        <child link="laser_main_link" />
-        <origin xyz="0.0 0.0 0.02276"
-                rpy="0 0 0" />
-      </joint>
-    </xacro:if>
-    <xacro:unless value="${fixed}" >
-      <joint name="laser_roll_joint"
-             type="revolute" >
-        <parent link="laser_roll_servo_link" />
-        <child link="laser_pitch_servo_link" />
-        <origin xyz="0.03999 0.0 0.0"
-                rpy="0 0 0" />
-        <axis xyz="1 0 0" />
-        <limit lower="${roll_min_limit}"
-               upper="${roll_max_limit}"
-               effort="50"
-               velocity="50.0" />
-      </joint>
-      <joint name="laser_pitch_joint"
-             type="revolute" >
-        <parent link="laser_pitch_servo_link" />
-        <child link="laser_main_link" />
-        <origin xyz="0.0 0.0 0.02276"
-                rpy="0 0 0" />
-        <axis xyz="0 1 0" />
-        <limit lower="${pitch_min_limit}"
-               upper="${pitch_max_limit}"
-               effort="50"
-               velocity="50.0" />
-      </joint>
-    </xacro:unless>
+    <joint name="laser_roll_joint"
+           type="revolute" >
+      <parent link="laser_roll_servo_link" />
+      <child link="laser_pitch_servo_link" />
+      <origin xyz="0.03999 0.0 0.0"
+              rpy="0 0 0" />
+      <axis xyz="1 0 0" />
+      <limit lower="${roll_min_limit}"
+             upper="${roll_max_limit}"
+             effort="50"
+             velocity="50.0" />
+    </joint>
+    <joint name="laser_pitch_joint"
+           type="revolute" >
+      <parent link="laser_pitch_servo_link" />
+      <child link="laser_main_link" />
+      <origin xyz="0.0 0.0 0.02276"
+              rpy="0 0 0" />
+      <axis xyz="0 1 0" />
+      <limit lower="${pitch_min_limit}"
+             upper="${pitch_max_limit}"
+             effort="50"
+             velocity="50.0" />
+    </joint>
+    <!-- Frames ########################################################### -->
+    <link name="laser_link" >
+      <xacro:point_mass_inertial />
+    </link>
     <joint name="laser_joint"
            type="fixed" >
