Commit message: Fix flir's position [ci skip]

File: pandora_robots_description/woody/urdf/sensors/thermal.xacro (robot description, xacro)
@@ -4,5 +4,5 @@
   <xacro:macro name="thermal" >
     <xacro:flir_lepton parent="kinect_platform_link" >
-      <origin xyz="0.0575 0.07522 0.05166"
+      <origin xyz="0.0575 0.07522 0.04716"
               rpy="0 0 0" />
     </xacro:flir_lepton>
