Commit message: Fix gears' sensor poses

File: pandora_robots_description/gears/urdf/sensors/camera_sensor.xacro (robot description, xacro)
@@ -1,9 +1,5 @@
 <?xml version="1.0"?>
 <robot xmlns:xacro="http://ros.org/wiki/xacro" >
-  <!-- ==================================================================== -->
   <xacro:include filename="$(find pandora_sensors_description)/urdf/camera.urdf.xacro" />
-  <!-- ==================================================================== -->
-<!-- ###################################################################### -->
-  <!-- ==================================================================== -->
   <xacro:macro name="left_camera_sensor" >
     <xacro:camera_caster parent="base_link"
@@ -13,5 +9,4 @@
     </xacro:camera_caster>
   </xacro:macro>
-  <!-- ==================================================================== -->
   <xacro:macro name="right_camera_sensor" >
     <xacro:camera_caster parent="base_link"
@@ -21,5 +16,3 @@
     </xacro:camera_caster>
   </xacro:macro>
-  <!-- ==================================================================== -->
-<!-- ###################################################################### -->
 </robot>

File: pandora_robots_description/gears/urdf/sensors/co2_sensor.xacro (robot description, xacro)
@@ -1,8 +1,5 @@
 <?xml version="1.0"?>
 <robot xmlns:xacro="http://ros.org/wiki/xacro" >
-  <!-- ==================================================================== -->
   <xacro:include filename="$(find pandora_sensors_description)/urdf/co2.urdf.xacro" />
-  <!-- ==================================================================== -->
-<!-- ###################################################################### -->
   <xacro:macro name="co2_sensor" >
     <xacro:co2_caster parent="linear_head_main_link" >
@@ -11,4 +8,3 @@
     </xacro:co2_caster>
   </xacro:macro>
-<!-- ###################################################################### -->
 </robot>

File: pandora_robots_description/gears/urdf/sensors/kinect_sensor.xacro (robot description, xacro)
@@ -1,12 +1,7 @@
 <?xml version="1.0"?>
 <robot xmlns:xacro="http://ros.org/wiki/xacro" >
-  <!-- ==================================================================== -->
   <xacro:include filename="$(find pandora_sensors_description)/urdf/kinect.urdf.xacro" />
-  <!-- ==================================================================== -->
-<!-- ###################################################################### -->
-  <xacro:macro name="kinect_sensor"
-               params="fixed" >
+  <xacro:macro name="kinect_sensor" >
     <xacro:kinect_caster parent="linear_elevator_link"
-                         fixed="${fixed}"
                          pitch_min_limit="${kinect_pitch_joint_min_limit}"
                          pitch_max_limit="${kinect_pitch_joint_max_limit}"
@@ -17,4 +12,3 @@
     </xacro:kinect_caster>
   </xacro:macro>
-<!-- ###################################################################### -->
 </robot>

File: pandora_robots_description/gears/urdf/sensors/laser_sensor.xacro (robot description, xacro)
@@ -1,20 +1,14 @@
 <?xml version="1.0"?>
 <robot xmlns:xacro="http://ros.org/wiki/xacro" >
-  <!-- ==================================================================== -->
   <xacro:include filename="$(find pandora_sensors_description)/urdf/laser.urdf.xacro" />
-  <!-- ==================================================================== -->
-<!-- ###################################################################### -->
-  <xacro:macro name="laser_sensor"
-               params="fixed" >
+  <xacro:macro name="laser_sensor" >
     <xacro:laser_caster parent="base_link"
-                         fixed="${fixed}"
-                         roll_min_limit="${laser_roll_joint_min_limit}"
-                         roll_max_limit="${laser_roll_joint_max_limit}"
-                         pitch_min_limit="${laser_pitch_joint_min_limit}"
-                         pitch_max_limit="${laser_pitch_joint_max_limit}" >
+                        roll_min_limit="${laser_roll_joint_min_limit}"
+                        roll_max_limit="${laser_roll_joint_max_limit}"
+                        pitch_min_limit="${laser_pitch_joint_min_limit}"
+                        pitch_max_limit="${laser_pitch_joint_max_limit}" >
       <origin xyz="0.1974 0.0 0.09679"
               rpy="${zero}" />
     </xacro:laser_caster>
   </xacro:macro>
-<!-- ###################################################################### -->
 </robot>

File: pandora_robots_description/gears/urdf/sensors/sonar_sensor.xacro (robot description, xacro)
@@ -1,9 +1,5 @@
 <?xml version="1.0"?>
 <robot xmlns:xacro="http://ros.org/wiki/xacro" >
-  <!-- ==================================================================== -->
   <xacro:include filename="$(find pandora_sensors_description)/urdf/sonar.urdf.xacro" />
-  <!-- ==================================================================== -->
-<!-- ###################################################################### -->
-  <!-- ==================================================================== -->
   <xacro:macro name="linear_sonar_sensor" >
     <xacro:sonar_caster name="linear"
@@ -13,5 +9,4 @@
     </xacro:sonar_caster>
   </xacro:macro>
-  <!-- ==================================================================== -->
   <xacro:macro name="left_sonar_sensor" >
     <xacro:sonar_caster name="left"
@@ -21,5 +16,4 @@
     </xacro:sonar_caster>
   </xacro:macro>
-  <!-- ==================================================================== -->
   <xacro:macro name="right_sonar_sensor" >
     <xacro:sonar_caster name="right"
@@ -29,5 +23,3 @@
     </xacro:sonar_caster>
   </xacro:macro>
-  <!-- ==================================================================== -->
-<!-- ###################################################################### -->
 </robot>

File: pandora_robots_description/gears/urdf/sensors/thermal_sensor.xacro (robot description, xacro)
@@ -1,9 +1,5 @@
 <?xml version="1.0"?>
 <robot xmlns:xacro="http://ros.org/wiki/xacro" >
-  <!-- ==================================================================== -->
   <xacro:include filename="$(find pandora_sensors_description)/urdf/thermal.urdf.xacro" />
-  <!-- ==================================================================== -->
-<!-- ###################################################################### -->
-  <!-- ==================================================================== -->
   <xacro:macro name="middle_thermal_sensor" >
     <xacro:thermal_caster parent="linear_head_main_link"
@@ -13,5 +9,4 @@
     </xacro:thermal_caster>
   </xacro:macro>
-  <!-- ==================================================================== -->
   <xacro:macro name="left_thermal_sensor" >
     <xacro:thermal_caster parent="linear_head_main_link"
@@ -21,5 +16,4 @@
     </xacro:thermal_caster>
   </xacro:macro>
-  <!-- ==================================================================== -->
   <xacro:macro name="right_thermal_sensor" >
     <xacro:thermal_caster parent="linear_head_main_link"
@@ -29,5 +23,3 @@
     </xacro:thermal_caster>
   </xacro:macro>
-  <!-- ==================================================================== -->
-<!-- ###################################################################### -->
 </robot>
