Commit message: Merge gears' links and joints to parts

File: pandora_robots_description/gears/urdf/gears.urdf.xacro (robot description, xacro)
@@ -1,126 +1,32 @@
 <?xml version="1.0"?>
-<robot xmlns:xacro="http://ros.org/wiki/xacro" >
-<!-- Import Files ######################################################### -->
-  <!-- ==================================================================== -->
-  <xacro:include filename="$(find pandora_robots_description)/urdf/gears/urdf_configurations.xacro" />
-  <!-- ==================================================================== -->
-  <xacro:include filename="$(find pandora_robots_description)/urdf/gears/properties/constants.xacro" />
-  <xacro:include filename="$(find pandora_robots_description)/urdf/gears/properties/defaults.xacro" />
-  <xacro:include filename="$(find pandora_robots_description)/urdf/gears/properties/materials.xacro" />
-  <!-- ==================================================================== -->
-  <xacro:include filename="$(find pandora_robots_description)/urdf/gears/links/base_link.urdf.xacro" />
-  <xacro:include filename="$(find pandora_robots_description)/urdf/gears/links/side_link.urdf.xacro" />
-  <xacro:include filename="$(find pandora_robots_description)/urdf/gears/links/wheel_link.urdf.xacro" />
-  <xacro:include filename="$(find pandora_robots_description)/urdf/gears/links/linear_elevator_link.urdf.xacro" />
-  <xacro:include filename="$(find pandora_robots_description)/urdf/gears/links/linear_head_base_link.urdf.xacro" />
-  <xacro:include filename="$(find pandora_robots_description)/urdf/gears/links/linear_head_main_link.urdf.xacro" />
-  <!-- ==================================================================== -->
-  <xacro:include filename="$(find pandora_robots_description)/urdf/gears/joints/side_joint.urdf.xacro" />
-  <xacro:include filename="$(find pandora_robots_description)/urdf/gears/joints/wheel_joint.urdf.xacro" />
-  <xacro:include filename="$(find pandora_robots_description)/urdf/gears/joints/linear_elevator_joint.urdf.xacro" />
-  <xacro:include filename="$(find pandora_robots_description)/urdf/gears/joints/linear_head_pitch_joint.urdf.xacro" />
-  <xacro:include filename="$(find pandora_robots_description)/urdf/gears/joints/linear_head_yaw_joint.urdf.xacro" />
-  <!-- ==================================================================== -->
-  <xacro:include filename="$(find pandora_robots_description)/urdf/gears/sensors/laser_sensor.xacro" />
-  <xacro:include filename="$(find pandora_robots_description)/urdf/gears/sensors/kinect_sensor.xacro" />
-  <xacro:include filename="$(find pandora_robots_description)/urdf/gears/sensors/camera_sensor.xacro" />
-  <xacro:include filename="$(find pandora_robots_description)/urdf/gears/sensors/sonar_sensor.xacro" />
-  <xacro:include filename="$(find pandora_robots_description)/urdf/gears/sensors/thermal_sensor.xacro" />
-  <xacro:include filename="$(find pandora_robots_description)/urdf/gears/sensors/co2_sensor.xacro" />
-  <xacro:include filename="$(find pandora_robots_description)/urdf/gears/sensors/microphone_sensor.xacro" />
-  <!-- ==================================================================== -->
-<xacro:macro name="gears_urdf"
-             params="fixed" >
-<!-- Load Links & Joints ################################################## -->
-  <!-- ================================================================== -->
-  <xacro:base_link />
-  <!-- ================================================================== -->
-  <!-- ================================================================== -->
-  <xacro:side_link prefix_y="left" reflect_y="1" />
-  <xacro:side_joint prefix_y="left" reflect_y="1" />
-  <!-- ================================================================== -->
-  <xacro:side_link prefix_y="right" reflect_y="-1" />
-  <xacro:side_joint prefix_y="right" reflect_y="-1" />
-  <!-- ================================================================== -->
-  <!-- ================================================================== -->
-  <xacro:wheel_link prefix_y="left" prefix_x="front" reflect_y="1" reflect_x="1" />
-  <xacro:wheel_joint prefix_y="left" prefix_x="front" reflect_y="1" reflect_x="1" />
-  <!-- ================================================================== -->
-  <xacro:wheel_link prefix_y="left" prefix_x="rear" reflect_y="1" reflect_x="-1" />
-  <xacro:wheel_joint prefix_y="left" prefix_x="rear" reflect_y="1" reflect_x="-1" />
-  <!-- ================================================================== -->
-  <xacro:wheel_link prefix_y="right" prefix_x="front" reflect_y="-1" reflect_x="1" />
-  <xacro:wheel_joint prefix_y="right" prefix_x="front" reflect_y="-1" reflect_x="1" />
-  <!-- ================================================================== -->
-  <xacro:wheel_link prefix_y="right" prefix_x="rear" reflect_y="-1" reflect_x="-1" />
-  <xacro:wheel_joint prefix_y="right" prefix_x="rear" reflect_y="-1" reflect_x="-1" />
-  <!-- ================================================================== -->
-  <!-- ================================================================== -->
-  <xacro:linear_elevator_link />
-  <xacro:linear_elevator_joint fixed="${fixed}" />
-  <!-- ================================================================== -->
-  <xacro:linear_head_base_link />
-  <xacro:linear_head_yaw_joint fixed="${fixed}" />
-  <!-- ================================================================== -->
-  <xacro:linear_head_main_link />
-  <xacro:linear_head_pitch_joint fixed="${fixed}" />
-  <!-- ================================================================== -->
-<!-- Load Sensors ######################################################### -->
-  <xacro:if value="${enable_sensors}" >
-    <xacro:if value="${enable_laser_sensor}" >
-      <xacro:laser_sensor fixed="${fixed}" />
-    </xacro:if>
-    <xacro:if value="${enable_kinect_sensor}" >
-      <xacro:kinect_sensor fixed="${fixed}" />
-    </xacro:if>
-    <xacro:if value="${enable_camera_sensors}" >
-      <!-- ================================================================ -->
-      <xacro:if value="${enable_left_camera_sensor}" >
-        <xacro:left_camera_sensor />
-      </xacro:if>
-      <!-- ================================================================ -->
-      <xacro:if value="${enable_right_camera_sensor}" >
-        <xacro:right_camera_sensor />
-      </xacro:if>
-      <!-- ================================================================ -->
-    </xacro:if>
-    <xacro:if value="${enable_sonar_sensors}" >
-      <!-- ================================================================ -->
-      <xacro:if value="${enable_linear_sonar_sensor}" >
-        <xacro:linear_sonar_sensor />
-      </xacro:if>
-      <!-- ================================================================ -->
-      <xacro:if value="${enable_left_sonar_sensor}" >
-        <xacro:left_sonar_sensor />
-      </xacro:if>
-      <!-- ================================================================ -->
-      <xacro:if value="${enable_right_sonar_sensor}" >
-        <xacro:right_sonar_sensor />
-      </xacro:if>
-      <!-- ================================================================ -->
-    </xacro:if>
-    <xacro:if value="${enable_thermal_sensors}" >
-      <!-- ================================================================ -->
-      <xacro:if value="${enable_middle_thermal_sensor}" >
-        <xacro:middle_thermal_sensor />
-      </xacro:if>
-      <!-- ================================================================ -->
-      <xacro:if value="${enable_left_thermal_sensor}" >
-        <xacro:left_thermal_sensor />
-      </xacro:if>
-      <!-- ================================================================ -->
-      <xacro:if value="${enable_right_thermal_sensor}" >
-        <xacro:right_thermal_sensor />
-      </xacro:if>
-      <!-- ================================================================ -->
-    </xacro:if>
-    <xacro:if value="${enable_co2_sensor}" >
-      <xacro:co2_sensor />
-    </xacro:if>
-    <xacro:if value="${enable_microphone_sensor}" >
-      <xacro:microphone_sensor />
-    </xacro:if>
-  </xacro:if>
-</xacro:macro>
-<!-- ###################################################################### -->
+<robot name="gears"
+       xmlns:xacro="http://ros.org/wiki/xacro" >
+  <!-- Import Files -->
+  <xacro:include filename="$(find pandora_urdf_properties)/xacro/*.xacro" />
+  <xacro:include filename="$(find pandora_robots_description)/gears/urdf/urdf_configurations.xacro" />
+  <xacro:include filename="$(find pandora_robots_description)/gears/urdf/parts/*.xacro" />
+  <xacro:include filename="$(find pandora_robots_description)/gears/urdf/sensors/*.xacro" />
+  <!-- Load Links & Joints -->
+  <xacro:base />
+  <xacro:side prefix_y="left" reflect_y="1" />
+  <xacro:side prefix_y="right" reflect_y="-1" />
+  <xacro:wheel prefix_y="left" prefix_x="front" reflect_y="1" reflect_x="1" />
+  <xacro:wheel prefix_y="left" prefix_x="rear" reflect_y="1" reflect_x="-1" />
+  <xacro:wheel prefix_y="right" prefix_x="front" reflect_y="-1" reflect_x="1" />
+  <xacro:wheel prefix_y="right" prefix_x="rear" reflect_y="-1" reflect_x="-1" />
+  <xacro:linear_elevator />
+  <xacro:linear_head />
+  <!-- Load Sensors -->
+  <xacro:laser_sensor />
+  <xacro:kinect_sensor />
+  <xacro:left_camera_sensor />
+  <xacro:right_camera_sensor />
+  <xacro:linear_sonar_sensor />
+  <xacro:left_sonar_sensor />
+  <xacro:right_sonar_sensor />
+  <xacro:co2_sensor />
+  <xacro:middle_thermal_sensor />
+  <xacro:left_thermal_sensor />
+  <xacro:right_thermal_sensor />
+  <xacro:microphone_sensor />
 </robot>

File: pandora_robots_description/gears/urdf/parts/base.urdf.xacro (robot description, xacro)
@@ -4,5 +4,5 @@
     <link name="base_link" >
       <inertial>
-        <origin xyz="-0.00968 -0.00122 0.19369" />
+        <origin xyz="-0.00968 -0.00122 0.17947" />
         <mass value="8.25079" />
         <inertia ixx="0.112701442"
@@ -15,5 +15,5 @@
       <visual>
         <geometry>
-          <mesh filename="package://pandora_robots_description/woody/meshes/base_link.dae" />
+          <mesh filename="package://pandora_robots_description/gears/meshes/base_link.dae" />
         </geometry>
         <material name="base" />
@@ -21,208 +21,8 @@
       <collision>
         <geometry>
-          <mesh filename="package://pandora_robots_description/woody/meshes/base_link.stl" />
+          <mesh filename="package://pandora_robots_description/gears/meshes/base_link.stl" />
         </geometry>
       </collision>
     </link>
-    <link name="miniitx" >
-      <inertial>
-        <origin xyz="0.0 0.0 0.0" />
-        <mass value="0.589" />
-        <inertia ixx="0.0014381417"
-                 ixy="0.0"
-                 ixz="0.0"
-                 iyy="0.0019829667"
-                 iyz="0.0"
-                 izz="0.0033818417" />
-      </inertial>
-    </link>
-    <joint name="miniitx_joint"
-           type="fixed" >
-      <parent link="base_link" />
-      <child link="miniitx" />
-      <origin xyz="0.03895 0.0 0.16181"
-              rpy="0.0 0.0 0.0" />
-    </joint>
-    <link name="ssd" >
-      <inertial>
-        <origin xyz="0.0 0.0 0.0" />
-        <mass value="0.078" />
-        <inertia ixx="0.0000325"
-                 ixy="0.0"
-                 ixz="0.0"
-                 iyy="0.00006565"
-                 iyz="0.0"
-                 izz="0.00009685" />
-      </inertial>
-    </link>
-    <joint name="ssd_joint"
-           type="fixed" >
-      <parent link="base_link" />
-      <child link="ssd" />
-      <origin xyz="0.059 -0.097 0.181"
-              rpy="${PI_2} 0.0 0.0" />
-    </joint>
-    <link name="raspberry" >
-      <xacro:solid_cuboid_inertial mass="0.062" x="0.095" y="0.070" z="0.025" >
-        <xacro:default_origin />
-      </xacro:solid_cuboid_inertial>
-    </link>
-    <joint name="raspberry_joint"
-           type="fixed" >
-      <parent link="base_link" />
-      <child link="raspberry" />
-      <origin xyz="0.071 0.076 0.24"
-              rpy="0.0 0.0 0.0" />
-    </joint>
-    <link name="arm" >
-      <xacro:solid_cuboid_inertial mass="0.050" x="0.064" y="0.104" z="0.030" >
-        <xacro:default_origin />
-      </xacro:solid_cuboid_inertial>
-    </link>
-    <joint name="arm_joint"
-           type="fixed" >
-      <parent link="base_link" />
-      <child link="arm" />
-      <origin xyz="-0.052 0.002 0.245"
-              rpy="0.0 0.0 ${PI_2}" />
-    </joint>
-    <link name="epos" >
-      <inertial>
-        <origin xyz="0.0 0.0 0.0" />
-        <mass value="0.136" />
-        <inertia ixx="0.0002266667"
-                 ixy="0.0"
-                 ixz="0.0"
-                 iyy="6.8283E-005"
-                 iyz="0.0"
-                 izz="0.0002858833" />
-      </inertial>
-    </link>
-    <joint name="epos_joint"
-           type="fixed" >
-      <parent link="base_link" />
-      <child link="epos" />
-      <origin xyz="-0.08263 0.0 0.03222"
-              rpy="0.0 0.0 0.0" />
-    </joint>
-    <link name="psu" >
-      <inertial>
-        <origin xyz="0.0 0.0 0.0" />
-        <mass value="0.178" />
-        <inertia ixx="0.0002241168"
-                 ixy="0.0"
-                 ixz="0.0"
-                 iyy="0.0001828208"
-                 iyz="0.0"
-                 izz="0.0004002627" />
-      </inertial>
-    </link>
-    <joint name="psu_joint"
-           type="fixed" >
-      <parent link="base_link" />
-      <child link="psu" />
-      <origin xyz="0.073 0.0 0.11023"
-              rpy="0.0 0.0 0.0" />
-    </joint>
-    <link name="motor_battery" >
-      <inertial>
-        <origin xyz="0.0 0.0 0.0" />
-        <mass value="0.8" />
-        <inertia ixx="0.0003576"
-                 ixy="0.0"
-                 ixz="0.0"
-                 iyy="0.0016806"
-                 iyz="0.0"
-                 izz="0.0015582" />
-      </inertial>
-    </link>
-    <joint name="motor_battery_joint"
-           type="fixed" >
-      <parent link="base_link" />
-      <child link="motor_battery" />
-      <origin xyz="0.10395 0.027 0.04822"
-              rpy="0.0 0.0 0.0" />
-    </joint>
-    <link name="pc_battery" >
-      <inertial>
-        <origin xyz="0.0 0.0 0.0" />
-        <mass value="0.8" />
-        <inertia ixx="0.0003576"
-                 ixy="0.0"
-                 ixz="0.0"
-                 iyy="0.0016806"
-                 iyz="0.0"
-                 izz="0.0015582" />
-      </inertial>
-    </link>
-    <joint name="pc_battery_joint"
-           type="fixed" >
-      <parent link="base_link" />
-      <child link="pc_battery" />
-      <origin xyz="0.10395 -0.027 0.04822"
-              rpy="0.0 0.0 0.0" />
-    </joint>
-    <link name="cables" >
-      <inertial>
-        <origin xyz="0.0 0.0 0.0" />
-        <mass value="0.6" />
-        <inertia ixx="0.00001"
-                 ixy="0.0"
-                 ixz="0.0"
-                 iyy="0.00001"
-                 iyz="0.0"
-                 izz="0.00001" />
-      </inertial>
-    </link>
-    <joint name="cables_joint"
-           type="fixed" >
-      <parent link="base_link" />
-      <child link="cables" />
-      <origin xyz="0.0 0.0 0.1"
-              rpy="0.0 0.0 0.0" />
-    </joint>
-    <link name="axis" >
-      <xacro:solid_cylinder_inertial mass="0.446" radius="0.03" height="0.267" >
-        <xacro:default_origin />
-      </xacro:solid_cylinder_inertial>
-    </link>
-    <joint name="axis_joint"
-           type="fixed" >
-      <parent link="base_link" />
-      <child link="axis" />
-      <origin xyz="0.0 0.0 0.0"
-              rpy="0.0 0.0 0.0" />
-    </joint>
-    <link name="imu" >
-      <xacro:solid_cuboid_inertial mass="0.05" x="0.057" y="0.045" z="0.024" >
-        <xacro:default_origin />
-      </xacro:solid_cuboid_inertial>
-    </link>/
-    <joint name="imu_joint"
-           type="fixed" >
-      <parent link="base_link" />
-      <child link="imu" />
-      <origin xyz="0.09013 -0.08006 0.24281"
-              rpy="0.0 0.0 0.0" />
-    </joint>
-<!--    <link name="differential" >-->
-<!--      <inertial>-->
-<!--        <origin xyz="0.0 0.0 0.0" />-->
-<!--        <mass value="0.31" />-->
-<!--        <inertia ixx="0.0001"-->
-<!--                 ixy="0.0"-->
-<!--                 ixz="0.0"-->
-<!--                 iyy="0.0001"-->
-<!--                 iyz="0.0"-->
-<!--                 izz="0.0001" />-->
-<!--      </inertial>-->
-<!--    </link>-->
-<!--    <joint name="differential_joint"-->
-<!--           type="fixed" >-->
-<!--      <parent link="base_link" />-->
-<!--      <child link="differential" />-->
-<!--      <origin xyz="-0.15 0.0 0.09031"-->
-<!--              rpy="0.0 0.0 0.0" />-->
-<!--    </joint>-->
   </xacro:macro>
 </robot>

File: pandora_robots_description/gears/urdf/parts/side.urdf.xacro (robot description, xacro)
@@ -18,5 +18,5 @@
                 rpy="0.0 0.0 ${ ( 1 - reflect_y ) * PI_2 }" />
         <geometry>
-          <mesh filename="package://pandora_robots_description/woody/meshes/side_link.dae" />
+          <mesh filename="package://pandora_robots_description/gears/meshes/side_link.dae" />
         </geometry>
         <material name="side" />
@@ -26,5 +26,5 @@
                 rpy="0.0 0.0 ${ ( 1 - reflect_y ) * PI_2 }" />
         <geometry>
-          <mesh filename="package://pandora_robots_description/woody/meshes/side_link.stl" />
+          <mesh filename="package://pandora_robots_description/gears/meshes/side_link.stl" />
         </geometry>
       </collision>
@@ -37,5 +37,5 @@
               rpy="${zero}" />
       <axis xyz="0 1 0" />
-      <dynamics damping="${side_joint_damping}" />
+      <dynamics damping="0.0" />
       <limit lower="${side_joint_min_limit}"
              upper="${side_joint_max_limit}"

File: pandora_robots_description/gears/urdf/parts/wheel.urdf.xacro (robot description, xacro)
@@ -18,5 +18,5 @@
                 rpy="0.0 0.0 ${ ( 1 - reflect_y ) * PI_2 }" />
         <geometry>
-          <mesh filename="package://pandora_robots_description/woody/meshes/wheel_link.dae" />
+          <mesh filename="package://pandora_robots_description/gears/meshes/wheel_link.dae" />
         </geometry>
         <material name="wheel" />
@@ -26,5 +26,5 @@
                 rpy="0.0 0.0 ${ ( 1 - reflect_y ) * PI_2 }" />
         <geometry>
-          <mesh filename="package://pandora_robots_description/woody/meshes/wheel_link.stl" />
+          <mesh filename="package://pandora_robots_description/gears/meshes/wheel_link.stl" />
         </geometry>
       </collision>
@@ -34,7 +34,8 @@
       <parent link="${prefix_y}_side_link" />
       <child link="${prefix_y}_${prefix_x}_wheel_link" />
-      <origin xyz="${ reflect_x * ( 0.17339 ) } ${ reflect_y * ( 0.06886 ) } -0.052795"
+      <origin xyz="${ reflect_x * ( 0.198785 ) } ${ reflect_y * ( 0.06886 ) } -0.052795"
               rpy="${zero}" />
       <axis xyz="0 1 0" />
+      <dynamics damping="0.0" />
       <limit effort="100.0"
              velocity="100.0" />
