Commit message: Merge gears' links and joints to parts

File: pandora_robots_description/gears/urdf/urdf_configurations.xacro (robot description, xacro)
@@ -1,108 +1,34 @@
 <?xml version="1.0"?>
 <robot xmlns:xacro="http://ros.org/wiki/xacro" >
-<!-- Elements' Status ##################################################### -->
-  <!-- Sensors ============================================================ -->
-  <xacro:property name="enable_sensors" value="true" />
-    <!-- ================================================================== -->
-    <xacro:property name="enable_laser_sensor" value="true" />
-    <!-- ================================================================== -->
-    <xacro:property name="enable_kinect_sensor" value="true" />
-    <!-- ================================================================== -->
-    <xacro:property name="enable_camera_sensors" value="true" />
-      <xacro:property name="enable_left_camera_sensor" value="true" />
-      <xacro:property name="enable_right_camera_sensor" value="true" />
-    <!-- ================================================================== -->
-    <xacro:property name="enable_sonar_sensors" value="true" />
-      <xacro:property name="enable_linear_sonar_sensor" value="true" />
-      <xacro:property name="enable_left_sonar_sensor" value="true" />
-      <xacro:property name="enable_right_sonar_sensor" value="true" />
-    <!-- ================================================================== -->
-    <xacro:property name="enable_thermal_sensors" value="true" />
-      <xacro:property name="enable_middle_thermal_sensor" value="true" />
-      <xacro:property name="enable_left_thermal_sensor" value="true" />
-      <xacro:property name="enable_right_thermal_sensor" value="true" />
-    <!-- ================================================================== -->
-    <xacro:property name="enable_co2_sensor" value="true" />
-    <!-- ================================================================== -->
-    <xacro:property name="enable_microphone_sensor" value="true" />
-  <!-- ==================================================================== -->
-<!-- Joint Physics ######################################################## -->
-  <!-- Joint Types ======================================================== -->
-  <xacro:property name="side_joint_type" value="revolute" />
-  <!-- ==================================================================== -->
-  <xacro:property name="wheel_joint_type" value="continuous" />
-  <!-- ==================================================================== -->
-  <xacro:property name="linear_elevator_joint_type" value="prismatic" />
-  <!-- ==================================================================== -->
-  <xacro:property name="linear_head_yaw_joint_type" value="revolute" />
-  <!-- ==================================================================== -->
-  <xacro:property name="linear_head_pitch_joint_type" value="revolute" />
-  <!-- ==================================================================== -->
-  <!-- Joint Damping ====================================================== -->
-  <xacro:property name="side_joint_damping" value="0.0" />
-  <!-- ==================================================================== -->
-  <xacro:property name="wheel_joint_damping" value="0.0" />
-  <!-- ==================================================================== -->
-  <xacro:property name="linear_elevator_joint_damping" value="5800.0" />
-  <!-- ==================================================================== -->
-  <xacro:property name="linear_head_pitch_joint_damping" value="0.0" />
-  <!-- ==================================================================== -->
-  <xacro:property name="linear_head_yaw_joint_damping" value="0.0" />
-  <!-- ==================================================================== -->
-  <!-- Joint Limits ======================================================= -->
-  <xacro:property name="side_joint_min_limit" value="-0.785" /> <!--FIXME-->
-  <xacro:property name="side_joint_max_limit" value="0.785" /> <!--FIXME-->
-  <!-- ==================================================================== -->
+  <!-- Joint limits -->
+  <xacro:property name="side_joint_min_limit" value="-0.785" />
+  <xacro:property name="side_joint_max_limit" value="0.785" />
   <xacro:property name="linear_elevator_joint_min_limit" value="0.0" />
-  <xacro:property name="linear_elevator_joint_max_limit" value="0.18" /> <!--FIXME-->
-  <!-- ==================================================================== -->
-  <xacro:property name="linear_head_yaw_joint_min_limit" value="-1.57" /> <!--FIXME-->
-  <xacro:property name="linear_head_yaw_joint_max_limit" value="1.57" /> <!--FIXME-->
-  <!-- ==================================================================== -->
-  <xacro:property name="linear_head_pitch_joint_min_limit" value="-1.57" /> <!--FIXME-->
-  <xacro:property name="linear_head_pitch_joint_max_limit" value="1.57" /> <!--FIXME-->
-  <!-- ==================================================================== -->
-  <xacro:property name="laser_roll_joint_min_limit" value="-1.57" /> <!--FIXME-->
-  <xacro:property name="laser_roll_joint_max_limit" value="1.57" /> <!--FIXME-->
-  <!-- ==================================================================== -->
-  <xacro:property name="laser_pitch_joint_min_limit" value="-1.57" /> <!--FIXME-->
-  <xacro:property name="laser_pitch_joint_max_limit" value="1.57" /> <!--FIXME-->
-  <!-- ==================================================================== -->
-  <xacro:property name="kinect_pitch_joint_min_limit" value="-1.57" /> <!--FIXME-->
-  <xacro:property name="kinect_pitch_joint_max_limit" value="1.57" /> <!--FIXME-->
-  <!-- ==================================================================== -->
-  <xacro:property name="kinect_yaw_joint_min_limit" value="-1.57" /> <!--FIXME-->
-  <xacro:property name="kinect_yaw_joint_max_limit" value="1.57" /> <!--FIXME-->
-  <!-- ==================================================================== -->
-<!-- Coefficients ######################################################### -->
-  <!-- Velocities ========================================================= -->
+  <xacro:property name="linear_elevator_joint_max_limit" value="0.18" />
+  <xacro:property name="linear_head_yaw_joint_min_limit" value="-1.57" />
+  <xacro:property name="linear_head_yaw_joint_max_limit" value="1.57" />
+  <xacro:property name="linear_head_pitch_joint_min_limit" value="-1.57" />
+  <xacro:property name="linear_head_pitch_joint_max_limit" value="1.57" />
+  <xacro:property name="laser_roll_joint_min_limit" value="-1.57" />
+  <xacro:property name="laser_roll_joint_max_limit" value="1.57" />
+  <xacro:property name="laser_pitch_joint_min_limit" value="-1.57" />
+  <xacro:property name="laser_pitch_joint_max_limit" value="1.57" />
+  <xacro:property name="kinect_pitch_joint_min_limit" value="-1.57" />
+  <xacro:property name="kinect_pitch_joint_max_limit" value="1.57" />
+  <xacro:property name="kinect_yaw_joint_min_limit" value="-1.57" />
+  <xacro:property name="kinect_yaw_joint_max_limit" value="1.57" />
+  <!-- Coefficients -->
   <xacro:property name="max_robot_linear_velocity" value="2.0" />
-  <!-- ==================================================================== -->
   <xacro:property name="max_robot_angular_velocity" value="2.0" />
-  <!-- ==================================================================== -->
   <xacro:property name="max_kinect_angular_velocity" value="2.5" />
-  <!-- ==================================================================== -->
   <xacro:property name="max_laser_angular_velocity" value="2.5" />
-  <!-- ==================================================================== -->
-  <!-- Accelerations ====================================================== -->
   <xacro:property name="max_robot_linear_acceleration" value="1.0" />
-  <!-- ==================================================================== -->
   <xacro:property name="max_robot_angular_acceleration" value="0.2" />
-  <!-- ==================================================================== -->
   <xacro:property name="max_kinect_angular_acceleration" value="0.0" />
-  <!-- ==================================================================== -->
   <xacro:property name="max_laser_angular_acceleration" value="0.0" />
-  <!-- ==================================================================== -->
-<!-- Dimensions ########################################################### -->
-  <!-- TODO -->
-  <!-- Wheels ============================================================= -->
+  <!-- Dimensions -->
   <xacro:property name="wheel_length" value="0.07985" />
-  <!-- ==================================================================== -->
   <xacro:property name="wheel_radius" value="0.09794" />
-  <!-- ==================================================================== -->
-  <xacro:property name="wheelbase" value="0.405" />
-  <xacro:property name="wheel_separation" value="0.344" />
   <xacro:property name="track" value="0.344" />
-  <!-- ==================================================================== -->
-<!-- ###################################################################### -->
+  <xacro:property name="wheelbase" value="0.34678" />
 </robot>

File: pandora_robots_description/woody/urdf/parts/side.urdf.xacro (robot description, xacro)
@@ -37,5 +37,5 @@
               rpy="${zero}" />
       <axis xyz="0 1 0" />
-      <dynamics damping="${side_joint_damping}" />
+      <dynamics damping="0.0" />
       <limit lower="${side_joint_min_limit}"
              upper="${side_joint_max_limit}"

File: pandora_robots_description/woody/urdf/parts/wheel.urdf.xacro (robot description, xacro)
@@ -37,4 +37,5 @@
               rpy="${zero}" />
       <axis xyz="0 1 0" />
+      <dynamics damping="0.0" />
       <limit effort="100.0"
              velocity="100.0" />

File: pandora_robots_description/woody/urdf/urdf_configurations.xacro (robot description, xacro)
@@ -1,7 +1,5 @@
 <?xml version="1.0"?>
 <robot xmlns:xacro="http://ros.org/wiki/xacro" >
-  <!-- Joints -->
-  <xacro:property name="side_joint_damping" value="0.0" />
-  <xacro:property name="wheel_joint_damping" value="0.0" />
+  <!-- Joint limits -->
   <xacro:property name="side_joint_min_limit" value="-0.785" />
   <xacro:property name="side_joint_max_limit" value="0.785" />
@@ -14,5 +12,5 @@
   <xacro:property name="kinect_yaw_joint_min_limit" value="-1.308" />
   <xacro:property name="kinect_yaw_joint_max_limit" value="1.308" />
-  <!-- TODO: Coefficients -->
+  <!-- Coefficients -->
   <xacro:property name="max_robot_linear_velocity" value="2.0" />
   <xacro:property name="max_robot_angular_velocity" value="2.0" />
