Commit message: Fix linear_elevator macro name

File: pandora_robots_description/gears/urdf/parts/linear_elevator.urdf.xacro (robot description, xacro)
@@ -1,5 +1,5 @@
 <?xml version="1.0" ?>
 <robot xmlns:xacro="http://ros.org/wiki/xacro" >
-  <xacro:macro name="linear_elevator_link" >
+  <xacro:macro name="linear_elevator" >
     <link name="linear_elevator_link" >
       <inertial>
