Commit message: Merge links and joints of each part

File: pandora_robots_description/woody/urdf/parts/base.urdf.xacro (robot description, xacro)
@@ -1,5 +1,5 @@
 <?xml version="1.0" ?>
 <robot xmlns:xacro="http://ros.org/wiki/xacro" >
-  <xacro:macro name="base_link" >
+  <xacro:macro name="base" >
     <link name="base_link" >
       <inertial>

File: pandora_robots_description/woody/urdf/parts/side.urdf.xacro (robot description, xacro)
@@ -1,5 +1,5 @@
 <?xml version="1.0" ?>
 <robot xmlns:xacro="http://ros.org/wiki/xacro" >
-  <xacro:macro name="side_link"
+  <xacro:macro name="side"
                params="prefix_y reflect_y" >
     <link name="${prefix_y}_side_link" >
@@ -30,4 +30,17 @@
       </collision>
     </link>
+    <joint name="${prefix_y}_side_joint"
+           type="revolute" >
+      <parent link="base_link" />
+      <child link="${prefix_y}_side_link" />
+      <origin xyz="0.0 ${ reflect_y * ( 0.10314 ) } 0.0"
+              rpy="${zero}" />
+      <axis xyz="0 1 0" />
+      <dynamics damping="${side_joint_damping}" />
+      <limit lower="${side_joint_min_limit}"
+             upper="${side_joint_max_limit}"
+             effort="150.0"
+             velocity="150.0" />
+    </joint>
   </xacro:macro>
 </robot>

File: pandora_robots_description/woody/urdf/parts/wheel.urdf.xacro (robot description, xacro)
@@ -1,5 +1,5 @@
 <?xml version="1.0" ?>
 <robot xmlns:xacro="http://ros.org/wiki/xacro" >
-  <xacro:macro name="wheel_link"
+  <xacro:macro name="wheel"
                params="prefix_y prefix_x reflect_y reflect_x" >
     <link name="${prefix_y}_${prefix_x}_wheel_link" >
@@ -30,4 +30,14 @@
       </collision>
     </link>
+    <joint name="${prefix_y}_${prefix_x}_wheel_joint"
+           type="continuous" >
+      <parent link="${prefix_y}_side_link" />
+      <child link="${prefix_y}_${prefix_x}_wheel_link" />
+      <origin xyz="${ reflect_x * ( 0.17339 ) } ${ reflect_y * ( 0.06886 ) } -0.052795"
+              rpy="${zero}" />
+      <axis xyz="0 1 0" />
+      <limit effort="100.0"
+             velocity="100.0" />
+    </joint>
   </xacro:macro>
 </robot>

File: pandora_robots_description/woody/urdf/woody.urdf.xacro (robot description, xacro)
@@ -3,43 +3,24 @@
        xmlns:xacro="http://ros.org/wiki/xacro" >
   <!-- Import Files ####################################################### -->
-  <xacro:include filename="$(find pandora_urdf_properties)/xacro/constants.xacro" />
-  <xacro:include filename="$(find pandora_urdf_properties)/xacro/defaults.xacro" />
-  <xacro:include filename="$(find pandora_urdf_properties)/xacro/materials.xacro" />
+  <xacro:include filename="$(find pandora_urdf_properties)/xacro/*.xacro" />
   <xacro:include filename="$(find pandora_robots_description)/woody/urdf/urdf_configurations.xacro" />
-  <xacro:include filename="$(find pandora_robots_description)/woody/urdf/links/base_link.urdf.xacro" />
-  <xacro:include filename="$(find pandora_robots_description)/woody/urdf/links/side_link.urdf.xacro" />
-  <xacro:include filename="$(find pandora_robots_description)/woody/urdf/links/wheel_link.urdf.xacro" />
-  <xacro:include filename="$(find pandora_robots_description)/woody/urdf/joints/side_joint.urdf.xacro" />
-  <xacro:include filename="$(find pandora_robots_description)/woody/urdf/joints/wheel_joint.urdf.xacro" />
-  <xacro:include filename="$(find pandora_robots_description)/woody/urdf/sensors/laser_sensor.xacro" />
-  <xacro:include filename="$(find pandora_robots_description)/woody/urdf/sensors/kinect_sensor.xacro" />
-  <xacro:include filename="$(find pandora_robots_description)/woody/urdf/sensors/flir_sensor.xacro" />
-  <xacro:include filename="$(find pandora_robots_description)/woody/urdf/sensors/camera_sensor.xacro" />
-  <xacro:include filename="$(find pandora_robots_description)/woody/urdf/sensors/sonar_sensor.xacro" />
-  <xacro:include filename="$(find pandora_robots_description)/woody/urdf/sensors/thermal_sensor.xacro" />
-  <xacro:include filename="$(find pandora_robots_description)/woody/urdf/sensors/co2_sensor.xacro" />
-  <xacro:include filename="$(find pandora_robots_description)/woody/urdf/sensors/microphone_sensor.xacro" />
+  <xacro:include filename="$(find pandora_robots_description)/woody/urdf/parts/*.xacro" />
+  <xacro:include filename="$(find pandora_robots_description)/woody/urdf/sensors/*.xacro" />
   <!-- Load Links & Joints ################################################ -->
-  <xacro:base_link />
-  <xacro:side_link prefix_y="left" reflect_y="1" />
-  <xacro:side_joint prefix_y="left" reflect_y="1" />
-  <xacro:side_link prefix_y="right" reflect_y="-1" />
-  <xacro:side_joint prefix_y="right" reflect_y="-1" />
-  <xacro:wheel_link prefix_y="left" prefix_x="front" reflect_y="1" reflect_x="1" />
-  <xacro:wheel_joint prefix_y="left" prefix_x="front" reflect_y="1" reflect_x="1" />
-  <xacro:wheel_link prefix_y="left" prefix_x="rear" reflect_y="1" reflect_x="-1" />
-  <xacro:wheel_joint prefix_y="left" prefix_x="rear" reflect_y="1" reflect_x="-1" />
-  <xacro:wheel_link prefix_y="right" prefix_x="front" reflect_y="-1" reflect_x="1" />
-  <xacro:wheel_joint prefix_y="right" prefix_x="front" reflect_y="-1" reflect_x="1" />
-  <xacro:wheel_link prefix_y="right" prefix_x="rear" reflect_y="-1" reflect_x="-1" />
-  <xacro:wheel_joint prefix_y="right" prefix_x="rear" reflect_y="-1" reflect_x="-1" />
+  <xacro:base />
+  <xacro:side prefix_y="left" reflect_y="1" />
+  <xacro:side prefix_y="right" reflect_y="-1" />
+  <xacro:wheel prefix_y="left" prefix_x="front" reflect_y="1" reflect_x="1" />
+  <xacro:wheel prefix_y="left" prefix_x="rear" reflect_y="1" reflect_x="-1" />
+  <xacro:wheel prefix_y="right" prefix_x="front" reflect_y="-1" reflect_x="1" />
+  <xacro:wheel prefix_y="right" prefix_x="rear" reflect_y="-1" reflect_x="-1" />
   <!-- Load Sensors ####################################################### -->
   <xacro:laser_sensor />
   <xacro:kinect_sensor />
-  <xacro:flir_sensor />
   <xacro:left_camera_sensor />
   <xacro:right_camera_sensor />
   <xacro:left_sonar_sensor />
   <xacro:right_sonar_sensor />
+  <xacro:flir_sensor />
   <xacro:thermal_sensor />
   <xacro:co2_sensor />

Commit message: Fix position of parts and sensors [ci skip]

File: pandora_robots_description/woody/urdf/parts/base.urdf.xacro (robot description, xacro)
@@ -13,6 +13,7 @@
       </visual>
       <collision>
+        <origin xyz="0.02514 0.0 0.14619" />
         <geometry>
-          <mesh filename="package://pandora_robots_description/woody/meshes/base_link.stl" />
+          <box size="0.336 0.225 0.315" />
         </geometry>
       </collision>
@@ -20,5 +21,4 @@
     <link name="miniitx" >
       <inertial>
-        <origin xyz="0.0 0.0 0.0" />
         <mass value="0.589" />
         <inertia ixx="0.0014381417"
@@ -34,10 +34,8 @@
       <parent link="base_link" />
       <child link="miniitx" />
-      <origin xyz="0.03895 0.0 0.16181"
-              rpy="0.0 0.0 0.0" />
+      <origin xyz="0.03895 0.0 0.16181" />
     </joint>
     <link name="ssd" >
       <inertial>
-        <origin xyz="0.0 0.0 0.0" />
         <mass value="0.078" />
         <inertia ixx="0.0000325"
@@ -65,5 +63,5 @@
       <parent link="base_link" />
       <child link="raspberry" />
-      <origin xyz="0.071 0.076 0.24"
+      <origin xyz="-0.07522 0.0 0.26906"
               rpy="0.0 0.0 0.0" />
     </joint>
@@ -77,10 +75,9 @@
       <parent link="base_link" />
       <child link="arm" />
-      <origin xyz="-0.052 0.002 0.245"
+      <origin xyz="-0.07371 0.0 0.24325"
               rpy="0.0 0.0 ${PI_2}" />
     </joint>
     <link name="epos" >
       <inertial>
-        <origin xyz="0.0 0.0 0.0" />
         <mass value="0.136" />
         <inertia ixx="0.0002266667"
@@ -96,10 +93,8 @@
       <parent link="base_link" />
       <child link="epos" />
-      <origin xyz="-0.08263 0.0 0.03222"
-              rpy="0.0 0.0 0.0" />
+      <origin xyz="-0.08263 0.0 0.03222" />
     </joint>
     <link name="psu" >
       <inertial>
-        <origin xyz="0.0 0.0 0.0" />
         <mass value="0.178" />
         <inertia ixx="0.0002241168"
@@ -115,10 +110,8 @@
       <parent link="base_link" />
       <child link="psu" />
-      <origin xyz="0.073 0.0 0.11023"
-              rpy="0.0 0.0 0.0" />
+      <origin xyz="0.073 0.0 0.11023" />
     </joint>
     <link name="motor_battery" >
       <inertial>
-        <origin xyz="0.0 0.0 0.0" />
         <mass value="0.8" />
         <inertia ixx="0.0003576"
@@ -134,10 +127,8 @@
       <parent link="base_link" />
       <child link="motor_battery" />
-      <origin xyz="0.10395 0.027 0.04822"
-              rpy="0.0 0.0 0.0" />
+      <origin xyz="0.10395 0.027 0.04822" />
     </joint>
     <link name="pc_battery" >
       <inertial>
-        <origin xyz="0.0 0.0 0.0" />
         <mass value="0.8" />
         <inertia ixx="0.0003576"
@@ -153,10 +144,8 @@
       <parent link="base_link" />
       <child link="pc_battery" />
-      <origin xyz="0.10395 -0.027 0.04822"
-              rpy="0.0 0.0 0.0" />
+      <origin xyz="0.10395 -0.027 0.04822" />
     </joint>
     <link name="cables" >
       <inertial>
-        <origin xyz="0.0 0.0 0.0" />
         <mass value="0.6" />
         <inertia ixx="0.00001"
@@ -172,9 +161,8 @@
       <parent link="base_link" />
       <child link="cables" />
-      <origin xyz="0.0 0.0 0.1"
-              rpy="0.0 0.0 0.0" />
+      <origin xyz="0.0 0.0 0.1" />
     </joint>
     <link name="axis" >
-      <xacro:solid_cylinder_inertial mass="0.446" radius="0.03" height="0.267" >
+      <xacro:solid_cylinder_inertial mass="0.446" radius="0.03" y="0.267" >
         <xacro:default_origin />
       </xacro:solid_cylinder_inertial>
@@ -184,6 +172,4 @@
       <parent link="base_link" />
       <child link="axis" />
-      <origin xyz="0.0 0.0 0.0"
-              rpy="0.0 0.0 0.0" />
     </joint>
     <link name="imu" >
@@ -196,6 +182,5 @@
       <parent link="base_link" />
       <child link="imu" />
-      <origin xyz="0.09013 -0.08006 0.24281"
-              rpy="0.0 0.0 0.0" />
+      <origin xyz="0.09013 -0.08006 0.24281" />
     </joint>
 <!--    <link name="differential" >-->

File: pandora_robots_description/woody/urdf/parts/side.urdf.xacro (robot description, xacro)
@@ -25,6 +25,7 @@
         <origin xyz="${zero}"
                 rpy="0.0 0.0 ${ ( 1 - reflect_y ) * PI_2 }" />
+        <origin xyz="0.0 0.0 -0.03018" />
         <geometry>
-          <mesh filename="package://pandora_robots_description/woody/meshes/side_link.stl" />
+          <box size="0.405 0.081 0.096" />
         </geometry>
       </collision>
@@ -34,6 +35,5 @@
       <parent link="base_link" />
       <child link="${prefix_y}_side_link" />
-      <origin xyz="0.0 ${ reflect_y * ( 0.10314 ) } 0.0"
-              rpy="${zero}" />
+      <origin xyz="0.0 ${ reflect_y * ( 0.10614 ) } 0.0" />
       <axis xyz="0 1 0" />
       <dynamics damping="0.0" />

File: pandora_robots_description/woody/urdf/parts/wheel.urdf.xacro (robot description, xacro)
@@ -4,14 +4,7 @@
                params="prefix_y prefix_x reflect_y reflect_x" >
     <link name="${prefix_y}_${prefix_x}_wheel_link" >
-      <inertial>
-        <origin xyz="${ reflect_y * ( -2.2235E-05 ) } ${ reflect_y * ( -0.00052624 ) } 2.4287E-05" />
-        <mass value="1.5" />
-        <inertia ixx="0.0040302"
-                 ixy="7.250E-08"
-                 ixz="${ reflect_y * ( 5.2121E-07 ) }"
-                 iyy="0.0067791"
-                 iyz="${ reflect_y * ( -7.9189E-08 ) }"
-                 izz="0.0040286" />
-      </inertial>
+      <xacro:solid_cylinder_inertial mass="0.970" radius="0.0922" y="0.0742" >
+        <origin xyz="0.0 ${ reflect_y * ( -0.00201 ) } 0.0" />
+      </xacro:solid_cylinder_inertial>
       <visual>
         <origin xyz="${zero}"
@@ -34,6 +27,5 @@
       <parent link="${prefix_y}_side_link" />
       <child link="${prefix_y}_${prefix_x}_wheel_link" />
-      <origin xyz="${ reflect_x * ( 0.17339 ) } ${ reflect_y * ( 0.06886 ) } -0.052795"
-              rpy="${zero}" />
+      <origin xyz="${ reflect_x * ( 0.17308 ) } ${ reflect_y * ( 0.07186 ) } -0.052795" />
       <axis xyz="0 1 0" />
       <dynamics damping="0.0" />

File: pandora_robots_description/woody/urdf/sensors/co2.xacro (robot description, xacro)
@@ -3,6 +3,6 @@
   <xacro:include filename="$(find pandora_sensors_description)/co2/urdf/*.urdf.xacro" />
   <xacro:macro name="co2" >
-    <xacro:dynament_gold parent="kinect_link" >
-      <origin xyz="0.0173 -0.0595 0.0"
+    <xacro:dynament_gold parent="kinect_platform_link" >
+      <origin xyz="0.04937 -0.07649 0.05345"
               rpy="${zero}" />
     </xacro:dynament_gold>

File: pandora_robots_description/woody/urdf/sensors/kinect.xacro (robot description, xacro)
@@ -8,5 +8,5 @@
                                yaw_min_limit="${kinect_yaw_joint_min_limit}"
                                yaw_max_limit="${kinect_yaw_joint_max_limit}" >
-      <origin xyz="0.11999 0.031 0.25781"
+      <origin xyz="0.11999 0.0 0.25921"
               rpy="0.0 0.0 0.0" />
     </xacro:asus_xtion_pro_live>

File: pandora_robots_description/woody/urdf/sensors/microphone.xacro (robot description, xacro)
@@ -3,6 +3,6 @@
   <xacro:include filename="$(find pandora_sensors_description)/microphone/urdf/*.urdf.xacro" />
   <xacro:macro name="microphone" >
-    <xacro:kinect_array parent="kinect_link" >
-      <origin xyz="-0.02175 -0.0374 0.09643"
+    <xacro:kinect_array parent="kinect_platform_link" >
+      <origin xyz="0.0015 0.0 0.07001"
               rpy="${zero}" />
     </xacro:kinect_array>

File: pandora_robots_description/woody/urdf/sensors/sonar.xacro (robot description, xacro)
@@ -5,5 +5,5 @@
     <xacro:devantech_srf05 name="left"
                            parent="base_link" >
-      <origin xyz="-0.146 0.1376 0.21406"
+      <origin xyz="-0.15974 0.11037 0.14973"
               rpy="0.0 0.0 ${- PI_6 }" />
     </xacro:devantech_srf05>
@@ -12,5 +12,5 @@
     <xacro:devantech_srf05 name="right"
                            parent="base_link" >
-      <origin xyz="-0.146 -0.1376 0.21406"
+      <origin xyz="-0.15974 -0.11037 0.14973"
               rpy="0.0 0.0 ${ PI_6 }" />
     </xacro:devantech_srf05>

File: pandora_robots_description/woody/urdf/sensors/thermal.xacro (robot description, xacro)
@@ -3,6 +3,6 @@
   <xacro:include filename="$(find pandora_sensors_description)/thermal/urdf/*.urdf.xacro" />
   <xacro:macro name="thermal" >
-    <xacro:flir_lepton parent="kinect_link" >
-      <origin xyz="0.0173 0.0747 0.0"
+    <xacro:flir_lepton parent="kinect_platform_link" >
+      <origin xyz="0.0575 0.07522 0.05166"
               rpy="0 0 0" />
     </xacro:flir_lepton>

File: pandora_robots_description/woody/urdf/urdf_configurations.xacro (robot description, xacro)
@@ -22,6 +22,6 @@
   <xacro:property name="max_laser_angular_acceleration" value="0.0" />
   <!-- Dimensions -->
-  <xacro:property name="wheel_length" value="0.07985" />
-  <xacro:property name="wheel_radius" value="0.09794" />
+  <xacro:property name="wheel_length" value="0.0742" />
+  <xacro:property name="wheel_radius" value="0.0922" />
   <xacro:property name="track" value="0.344" />
   <xacro:property name="wheelbase" value="0.34678" />

File: pandora_robots_description/woody/urdf/woody.urdf.xacro (robot description, xacro)
@@ -25,5 +25,5 @@
   <xacro:right_sonar />
   <xacro:co2 />
+  <xacro:microphone />
   <!--<xacro:temperature />-->
-  <!--<xacro:microphone />-->
 </robot>
