Commit message: Add new robot designs [ci skip]

File: pandora_sensors_description/kinect/urdf/asus_xtion_pro_live.urdf.xacro (robot description, xacro)
@@ -105,5 +105,5 @@
       <parent link="kinect_platform_link" />
       <child link="kinect_link" />
-      <origin xyz="0.03261 -0.00101 0.04261"
+      <origin xyz="0.01461 -0.00106 0.05011"
               rpy="0.0 0.0 0.0" />
     </joint>

Commit message: Fix collision box of kinect's platform [ci skip]

File: pandora_sensors_description/kinect/urdf/asus_xtion_pro_live.urdf.xacro (robot description, xacro)
@@ -48,8 +48,8 @@
       </visual>
       <collision>
-        <origin xyz="0.012 -0.00101 -0.019"
+        <origin xyz="0.0095 0.0 0.04851"
                 rpy="0 0 0" />
         <geometry>
-          <box size="0.100 0.120 0.041" />
+          <box size="0.096 0.180 0.043" />
         </geometry>
       </collision>
