Commit message: Fix pi_camera_link pitch offset [ci skip]

File: pandora_sensors_description/camera_effector/urdf/pi_camera.urdf.xacro (robot description, xacro)
@@ -123,6 +123,5 @@
       <parent link="pi_camera_platform_link" />
       <child link="pi_camera_link" />
-      <origin xyz="0.00034 -0.01925 0.04306"
-              rpy="0.0 -0.3490658504 0.0" />
+      <origin xyz="0.00034 -0.01925 0.04306" />
     </joint>
     <!-- Frames -->

Commit message: Add inertial elements in camera_effector's links [ci skip]

File: pandora_sensors_description/camera_effector/urdf/pi_camera.urdf.xacro (robot description, xacro)
@@ -6,8 +6,7 @@
                        pitch_min_limit pitch_max_limit" >
     <!-- Links -->
-    <!-- MASS = 0.076 -->
     <link name="camera_effector_pan_link" >
-      <xacro:solid_cuboid_inertial mass="0.01" x="0.01" y="0.01" z="0.01" >
-        <origin xyz="0.0 0.0 0.0" /> <!-- TODO -->
+      <xacro:solid_cuboid_inertial mass="0.020" x="0.012" y="0.032" z="0.029" >
+        <origin xyz="0.0 -0.00518 0.01887" />
       </xacro:solid_cuboid_inertial>
       <visual>
@@ -17,12 +16,13 @@
       </visual>
       <collision>
+        <origin xyz="0.0 -0.00518 0.01887" />
         <geometry>
-          <box size="0.01 0.01 0.01" /> <!-- TODO -->
+          <box size="0.012 0.032 0.029" />
         </geometry>
       </collision>
     </link>
     <link name="camera_effector_base_link" >
-      <xacro:solid_cuboid_inertial mass="0.01" x="0.01" y="0.01" z="0.01" >
-        <origin xyz="0.0 0.0 0.0" /> <!-- TODO -->
+      <xacro:solid_cuboid_inertial mass="0.010" x="0.051" y="0.053" z="0.005" >
+        <origin xyz="-0.0045 -0.00011 0.00069" />
       </xacro:solid_cuboid_inertial>
       <visual>
@@ -32,12 +32,13 @@
       </visual>
       <collision>
+        <origin xyz="-0.0045 -0.00011 0.00069" />
         <geometry>
-          <box size="0.01 0.01 0.01" /> <!-- TODO -->
+          <box size="0.051 0.053 0.005" />
         </geometry>
       </collision>
     </link>
     <link name="camera_effector_tilt_link" >
-      <xacro:solid_cuboid_inertial mass="0.01" x="0.01" y="0.01" z="0.01" >
-        <origin xyz="0.0 0.0 0.0" /> <!-- TODO -->
+      <xacro:solid_cuboid_inertial mass="0.020" x="0.012" y="0.029" z="0.032" >
+        <origin xyz="0.0 -0.01887 -0.00518" />
       </xacro:solid_cuboid_inertial>
       <visual>
@@ -47,12 +48,13 @@
       </visual>
       <collision>
+        <origin xyz="0.0 -0.01887 -0.00518" />
         <geometry>
-          <box size="0.01 0.01 0.01" /> <!-- TODO -->
+          <box size="0.012 0.029 0.032" />
         </geometry>
       </collision>
     </link>
     <link name="pi_camera_platform_link" >
-      <xacro:solid_cuboid_inertial mass="0.01" x="0.01" y="0.01" z="0.01" >
-        <origin xyz="0.0 0.0 0.0" /> <!-- TODO -->
+      <xacro:solid_cuboid_inertial mass="0.005" x="0.011" y="0.050" z="0.030" >
+        <origin xyz="0.0 -0.01085 0.01074" />
       </xacro:solid_cuboid_inertial>
       <visual>
@@ -62,12 +64,13 @@
       </visual>
       <collision>
+        <origin xyz="0.0 -0.01925 0.00324" />
         <geometry>
-          <box size="0.01 0.01 0.01" /> <!-- TODO -->
+          <box size="0.011 0.050 0.030" />
         </geometry>
       </collision>
     </link>
     <link name="pi_camera_link" >
-      <xacro:solid_cuboid_inertial mass="0.01" x="0.01" y="0.01" z="0.01" >
-        <origin xyz="0.0 0.0 0.0" /> <!-- TODO -->
+      <xacro:solid_cuboid_inertial mass="0.021" x="0.009" y="0.025" z="0.024" >
+        <origin xyz="-0.00058 0.0 0.00189" />
       </xacro:solid_cuboid_inertial>
       <visual>
@@ -77,6 +80,7 @@
       </visual>
       <collision>
+        <origin xyz="-0.00058 0.0 0.00189" />
         <geometry>
-          <box size="0.01 0.01 0.01" /> <!-- TODO -->
+          <box size="0.009 0.025 0.024" />
         </geometry>
       </collision>
@@ -111,5 +115,6 @@
       <parent link="camera_effector_tilt_link" />
       <child link="pi_camera_platform_link" />
-      <origin xyz="0.0 0.0 0.0" />
+      <origin xyz="0.0 0.0 0.0"
+              rpy="0.0 0.3490658504 0.0" />
       <axis xyz="0 1 0" />
       <dynamics damping="0.0" />
@@ -123,5 +128,6 @@
       <parent link="pi_camera_platform_link" />
       <child link="pi_camera_link" />
-      <origin xyz="0.00034 -0.01925 0.04306" />
+      <origin xyz="0.00034 -0.01925 0.04306"
+              rpy="0.0 -0.3490658504 0.0" />
     </joint>
     <!-- Frames -->
