Commit message: Fix linear_actuator_link's mesh and position [ci skip]

File: pandora_robots_description/gio/urdf/parts/linear.urdf.xacro (robot description, xacro)
@@ -44,5 +44,5 @@
       <parent link="linear_link" />
       <child link="linear_actuator_link" />
-      <origin xyz="0.0 0.0 0.2145" />
+      <origin xyz="0.0 0.0 0.06211" />
       <axis xyz="0 0 1" />
       <dynamics damping="5800.0" />

Commit message: Fix collisions of linear and camera_effector [ci skip]

File: pandora_robots_description/gio/urdf/parts/linear.urdf.xacro (robot description, xacro)
@@ -13,6 +13,7 @@
       </visual>
       <collision>
+        <origin xyz="-0.0015 0.0 0.10075" />
         <geometry>
-          <box size="0.02 0.018 0.207" />
+          <box size="0.020 0.018 0.213" />
         </geometry>
       </collision>
@@ -28,6 +29,7 @@
       </visual>
       <collision>
+        <origin xyz="0.0 0.0 0.0787" />
         <geometry>
-          <box size="0.009 0.009 0.100" />
+          <box size="0.009 0.009 0.157" />
         </geometry>
       </collision>

File: pandora_sensors_description/camera_effector/urdf/pi_camera.urdf.xacro (robot description, xacro)
@@ -16,5 +16,5 @@
       </visual>
       <collision>
-        <origin xyz="0.0 -0.00518 0.01887" />
+        <origin xyz="0.0 -0.00585 0.01588" />
         <geometry>
           <box size="0.012 0.032 0.029" />
@@ -32,5 +32,5 @@
       </visual>
       <collision>
-        <origin xyz="-0.0045 -0.00011 0.00069" />
+        <origin xyz="0.00027 -0.00042 0.00104" />
         <geometry>
           <box size="0.051 0.053 0.005" />
@@ -48,5 +48,5 @@
       </visual>
       <collision>
-        <origin xyz="0.0 -0.01887 -0.00518" />
+        <origin xyz="0.0 -0.01588 -0.00585" />
         <geometry>
           <box size="0.012 0.029 0.032" />
@@ -80,5 +80,5 @@
       </visual>
       <collision>
-        <origin xyz="-0.00058 0.0 0.00189" />
+        <origin xyz="0.00045 0.0 0.0025" />
         <geometry>
           <box size="0.009 0.025 0.024" />
