Commit message: Fix base_link collision [ci skip]

File: pandora_robots_description/gio/urdf/parts/base.urdf.xacro (robot description, xacro)
@@ -12,7 +12,6 @@
       </visual>
       <collision>
-        <origin xyz="0.02514 0.0 0.14619" />
         <geometry>
-          <box size="0.336 0.225 0.315" />
+          <mesh filename="package://pandora_robots_description/gio/meshes/base_link.stl" />
         </geometry>
       </collision>
@@ -166,4 +165,9 @@
         <xacro:default_origin />
       </xacro:solid_cylinder_inertial>
+      <collision>
+        <geometry>
+          <box size="0.057 0.267 0.025" />
+        </geometry>
+      </collision>
     </link>
     <joint name="axis_joint"

Commit message: Fix base_link inertial [ci skip]

File: pandora_robots_description/gio/urdf/parts/base.urdf.xacro (robot description, xacro)
@@ -18,13 +18,7 @@
     </link>
     <link name="miniitx" >
-      <inertial>
-        <mass value="0.589" />
-        <inertia ixx="0.0014381417"
-                 ixy="0.0"
-                 ixz="0.0"
-                 iyy="0.0019829667"
-                 iyz="0.0"
-                 izz="0.0033818417" />
-      </inertial>
+      <xacro:solid_cuboid_inertial mass="0.589" x="0.17" y="0.17" z="0.04" >
+        <origin xyz="0.0 0.0 0.0" />
+      </xacro:solid_cuboid_inertial>
     </link>
     <joint name="miniitx_joint"
@@ -35,13 +29,7 @@
     </joint>
     <link name="ssd" >
-      <inertial>
-        <mass value="0.078" />
-        <inertia ixx="0.0000325"
-                 ixy="0.0"
-                 ixz="0.0"
-                 iyy="0.00006565"
-                 iyz="0.0"
-                 izz="0.00009685" />
-      </inertial>
+      <xacro:solid_cuboid_inertial mass="0.078" x="0.1" y="0.01" z="0.07" >
+        <origin xyz="0.0 0.0 0.0" />
+      </xacro:solid_cuboid_inertial>
     </link>
     <joint name="ssd_joint"
@@ -77,13 +65,7 @@
     </joint>
     <link name="epos" >
-      <inertial>
-        <mass value="0.136" />
-        <inertia ixx="0.0002266667"
-                 ixy="0.0"
-                 ixz="0.0"
-                 iyy="6.8283E-005"
-                 iyz="0.0"
-                 izz="0.0002858833" />
-      </inertial>
+      <xacro:solid_cuboid_inertial mass="0.136" x="0.075" y="0.14" z="0.04" >
+        <origin xyz="0.0 0.0 0.0" />
+      </xacro:solid_cuboid_inertial>
     </link>
     <joint name="epos_joint"
@@ -94,13 +76,7 @@
     </joint>
     <link name="psu" >
-      <inertial>
-        <mass value="0.178" />
-        <inertia ixx="0.0002241168"
-                 ixy="0.0"
-                 ixz="0.0"
-                 iyy="0.0001828208"
-                 iyz="0.0"
-                 izz="0.0004002627" />
-      </inertial>
+      <xacro:solid_cuboid_inertial mass="0.178" x="0.094" y="0.122" z="0.02" >
+        <origin xyz="0.0 0.0 0.0" />
+      </xacro:solid_cuboid_inertial>
     </link>
     <joint name="psu_joint"
@@ -111,13 +87,7 @@
     </joint>
     <link name="motor_battery" >
-      <inertial>
-        <mass value="0.8" />
-        <inertia ixx="0.0003576"
-                 ixy="0.0"
-                 ixz="0.0"
-                 iyy="0.0016806"
-                 iyz="0.0"
-                 izz="0.0015582" />
-      </inertial>
+      <xacro:solid_cuboid_inertial mass="0.8" x="0.154" y="0.049" z="0.052" >
+        <origin xyz="0.0 0.0 0.0" />
+      </xacro:solid_cuboid_inertial>
     </link>
     <joint name="motor_battery_joint"
@@ -128,13 +98,7 @@
     </joint>
     <link name="pc_battery" >
-      <inertial>
-        <mass value="0.8" />
-        <inertia ixx="0.0003576"
-                 ixy="0.0"
-                 ixz="0.0"
-                 iyy="0.0016806"
-                 iyz="0.0"
-                 izz="0.0015582" />
-      </inertial>
+      <xacro:solid_cuboid_inertial mass="0.8" x="0.154" y="0.049" z="0.052" >
+        <origin xyz="0.0 0.0 0.0" />
+      </xacro:solid_cuboid_inertial>
     </link>
     <joint name="pc_battery_joint"
@@ -143,21 +107,4 @@
       <child link="pc_battery" />
       <origin xyz="0.10395 -0.027 0.04822" />
-    </joint>
-    <link name="cables" >
-      <inertial>
-        <mass value="0.6" />
-        <inertia ixx="0.00001"
-                 ixy="0.0"
-                 ixz="0.0"
-                 iyy="0.00001"
-                 iyz="0.0"
-                 izz="0.00001" />
-      </inertial>
-    </link>
-    <joint name="cables_joint"
-           type="fixed" >
-      <parent link="base_link" />
-      <child link="cables" />
-      <origin xyz="0.0 0.0 0.1" />
     </joint>
     <link name="axis" >
