Commit message: Fix sonar position

File: pandora_robots_description/gio/urdf/sensors/sonar.xacro (robot description, xacro)
@@ -5,6 +5,6 @@
     <xacro:devantech_srf05 name="left"
                            parent="base_link" >
-      <origin xyz="-0.15974 0.11037 0.14973"
-              rpy="0.0 0.0 ${- PI_6 }" />
+      <origin xyz="-0.15974 0.07913 0.14973"
+              rpy="0.0 0.0 0.0" />
     </xacro:devantech_srf05>
   </xacro:macro>
@@ -12,6 +12,6 @@
     <xacro:devantech_srf05 name="right"
                            parent="base_link" >
-      <origin xyz="-0.15974 -0.11037 0.14973"
-              rpy="0.0 0.0 ${ PI_6 }" />
+      <origin xyz="-0.15974 -0.07913 0.14973"
+              rpy="0.0 0.0 0.0" />
     </xacro:devantech_srf05>
   </xacro:macro>
