Commit message: Rename camera to webcam and fix orientation of webcams

File: pandora_robots_description/gio/urdf/sensors/webcam.xacro (robot description, xacro)
@@ -4,14 +4,14 @@
   <xacro:macro name="left_webcam" >
     <xacro:logitech_c310hd parent="base_link"
-                           prefix_y="left" >
-      <origin xyz="-0.08308 0.08308 0.23081"
-              rpy="0.0 0.0 ${ 3 * PI_4 }" />
+                           prefix="left" >
+      <origin xyz="-0.06887 0.08618 0.23081"
+              rpy="0.0 0.0 ${PI_2}" />
     </xacro:logitech_c310hd>
   </xacro:macro>
   <xacro:macro name="right_webcam" >
     <xacro:logitech_c310hd parent="base_link"
-                           prefix_y="right" >
-      <origin xyz="-0.08308 -0.08308 0.23081"
-              rpy="0.0 0.0 ${ 5 * PI_4 }" />
+                           prefix="right" >
+      <origin xyz="-0.06887 -0.08618 0.23081"
+              rpy="0.0 0.0 ${-PI_2}" />
     </xacro:logitech_c310hd>
   </xacro:macro>

File: pandora_sensors_description/webcam/urdf/logitech_c310hd.urdf.xacro (robot description, xacro)
@@ -2,7 +2,7 @@
 <robot xmlns:xacro="http://ros.org/wiki/xacro" >
   <xacro:macro name="logitech_c310hd"
-               params="parent prefix_y *origin" >
+               params="parent prefix *origin" >
     <!-- Links -->
-    <link name="${prefix_y}_camera_link" >
+    <link name="${prefix}_webcam_link" >
       <xacro:solid_cuboid_inertial mass="0.099" x="0.049" y="0.095" z="0.073" >
         <origin xyz="0.00972 0.0 0.04428" />
@@ -22,28 +22,28 @@
     </link>
     <!-- Joints -->
-    <joint name="${prefix_y}_camera_parent_joint"
+    <joint name="${prefix}_webcam_parent_joint"
            type="fixed" >
       <parent link="${parent}" />
-      <child link="${prefix_y}_camera_link" />
+      <child link="${prefix}_webcam_link" />
       <xacro:insert_block name="origin" />
     </joint>
     <!-- Frames -->
-    <link name="${prefix_y}_camera_frame" >
+    <link name="${prefix}_webcam_frame" >
       <xacro:point_mass_inertial />
     </link>
-    <link name="${prefix_y}_camera_optical_frame" >
+    <link name="${prefix}_webcam_optical_frame" >
       <xacro:point_mass_inertial />
     </link>
-    <joint name="${prefix_y}_camera_joint"
+    <joint name="${prefix}_webcam_joint"
            type="fixed" >
-      <parent link="${prefix_y}_camera_link" />
-      <child link="${prefix_y}_camera_frame" />
+      <parent link="${prefix}_webcam_link" />
+      <child link="${prefix}_webcam_frame" />
       <origin xyz="0.02499 0.0 0.05704"
               rpy="0.0 -0.2792 0.0" />
     </joint>
-    <joint name="${prefix_y}_camera_optical_joint"
+    <joint name="${prefix}_webcam_optical_joint"
            type="fixed" >
-      <parent link="${prefix_y}_camera_frame" />
-      <child link="${prefix_y}_camera_optical_frame" />
+      <parent link="${prefix}_webcam_frame" />
+      <child link="${prefix}_webcam_optical_frame" />
       <origin xyz="0.0 0.0 0.0"
               rpy="-1.5708 0.0 -1.5708" />
