Commit message: Fix laser's position [ci skip]

File: pandora_robots_description/gio/urdf/sensors/laser.xacro (robot description, xacro)
@@ -8,6 +8,5 @@
                            pitch_min_limit="${laser_pitch_joint_min_limit}"
                            pitch_max_limit="${laser_pitch_joint_max_limit}" >
-      <origin xyz="0.19015 -0.00248 0.12722"
-              rpy="0.0 0.0 0.035" /> <!-- yaw offset -->
+      <origin xyz="0.19015 -0.01352 0.11822" />
     </xacro:hokuyo_urg_04lx>
   </xacro:macro>
@@ -18,6 +17,5 @@
                            pitch_min_limit="${laser_pitch_joint_min_limit}"
                            pitch_max_limit="${laser_pitch_joint_max_limit}" >
-      <origin xyz="0.19015 -0.00248 0.12722"
-              rpy="0.0 0.0 0.0" />
+      <origin xyz="0.19015 -0.01352 0.11822" />
     </xacro:hokuyo_ust_20lx>
   </xacro:macro>

Commit message: Add laser roll, pitch offset params

File: pandora_robots_description/gio/urdf/sensors/laser.xacro (robot description, xacro)
@@ -6,6 +6,8 @@
                            roll_min_limit="${laser_roll_joint_min_limit}"
                            roll_max_limit="${laser_roll_joint_max_limit}"
+                           roll_offset="${laser_roll_joint_offset}"
                            pitch_min_limit="${laser_pitch_joint_min_limit}"
-                           pitch_max_limit="${laser_pitch_joint_max_limit}" >
+                           pitch_max_limit="${laser_pitch_joint_max_limit}"
+                           pitch_offset="${laser_pitch_joint_offset}" >
       <origin xyz="0.19015 -0.01352 0.11822" />
     </xacro:hokuyo_urg_04lx>
@@ -15,6 +17,8 @@
                            roll_min_limit="${laser_roll_joint_min_limit}"
                            roll_max_limit="${laser_roll_joint_max_limit}"
+                           roll_offset="${laser_roll_joint_offset}"
                            pitch_min_limit="${laser_pitch_joint_min_limit}"
-                           pitch_max_limit="${laser_pitch_joint_max_limit}" >
+                           pitch_max_limit="${laser_pitch_joint_max_limit}"
+                           pitch_offset="${laser_pitch_joint_offset}" >
       <origin xyz="0.19015 -0.01352 0.11822" />
     </xacro:hokuyo_ust_20lx>

File: pandora_robots_description/gio/urdf/urdf_configurations.xacro (robot description, xacro)
@@ -14,6 +14,8 @@
   <xacro:property name="laser_roll_joint_min_limit" value="-0.523" />
   <xacro:property name="laser_roll_joint_max_limit" value="0.523" />
+  <xacro:property name="laser_roll_joint_offset" value="-0.03" />
   <xacro:property name="laser_pitch_joint_min_limit" value="-0.523" />
   <xacro:property name="laser_pitch_joint_max_limit" value="0.523" />
+  <xacro:property name="laser_pitch_joint_offset" value="0.03" />
   <xacro:property name="kinect_pitch_joint_min_limit" value="-0.785" />
   <xacro:property name="kinect_pitch_joint_max_limit" value="0.785" />

File: pandora_robots_description/monstertruck/urdf/joint_limits.xacro (robot description, xacro)
@@ -5,6 +5,8 @@
   <xacro:property name="laser_roll_joint_min_limit" value="-0.523" />
   <xacro:property name="laser_roll_joint_max_limit" value="0.523" />
+  <xacro:property name="laser_roll_joint_offset" value="0.0" />
   <xacro:property name="laser_pitch_joint_min_limit" value="-0.523" />
   <xacro:property name="laser_pitch_joint_max_limit" value="0.523" />
+  <xacro:property name="laser_pitch_joint_offset" value="0.0" />
   <!-- wheel steer joint limits -->
   <xacro:property name="steer_joint_lower_limit" value="${-25*PI/180}" />

File: pandora_robots_description/monstertruck/urdf/sensors/laser04.urdf.xacro (robot description, xacro)
@@ -6,6 +6,8 @@
                            roll_min_limit="${laser_roll_joint_min_limit}"
                            roll_max_limit="${laser_roll_joint_max_limit}"
+                           roll_offset="${laser_roll_joint_offset}"
                            pitch_min_limit="${laser_pitch_joint_min_limit}"
-                           pitch_max_limit="${laser_pitch_joint_max_limit}" >
+                           pitch_max_limit="${laser_pitch_joint_max_limit}"
+                           pitch_offset="${laser_pitch_joint_offset}" >
       <origin xyz="0.137 0.0 0.06" />
     </xacro:hokuyo_urg_04lx>

File: pandora_sensors_description/laser/urdf/hokuyo_urg_04lx.urdf.xacro (robot description, xacro)
@@ -3,6 +3,6 @@
   <xacro:macro name="hokuyo_urg_04lx"
                params="parent *origin
-                       roll_min_limit roll_max_limit
-                       pitch_min_limit pitch_max_limit" >
+                       roll_min_limit roll_max_limit roll_offset
+                       pitch_min_limit pitch_max_limit pitch_offset">
     <!-- Links -->
     <link name="laser_roll_servo_link" >
@@ -69,5 +69,5 @@
       <child link="laser_pitch_servo_link" />
       <origin xyz="0.03999 0.0 0.0"
-              rpy="-0.03 0 0" />
+              rpy="${roll_offset} 0 0" />
       <axis xyz="1 0 0" />
       <limit lower="${roll_min_limit}"
@@ -81,5 +81,5 @@
       <child link="laser_main_link" />
       <origin xyz="0.0 0.0 0.02276"
-              rpy="0 0.03 0" />
+              rpy="0 ${pitch_offset} 0" />
       <axis xyz="0 1 0" />
       <limit lower="${pitch_min_limit}"

File: pandora_sensors_description/laser/urdf/hokuyo_ust_20lx.urdf.xacro (robot description, xacro)
@@ -3,6 +3,6 @@
   <xacro:macro name="hokuyo_ust_20lx"
                params="parent *origin
-                       roll_min_limit roll_max_limit
-                       pitch_min_limit pitch_max_limit" >
+                       roll_min_limit roll_max_limit roll_offset
+                       pitch_min_limit pitch_max_limit pitch_offset" >
     <!-- Links -->
     <link name="laser_roll_servo_link" >
@@ -69,5 +69,5 @@
       <child link="laser_pitch_servo_link" />
       <origin xyz="0.03999 0.0 0.0"
-              rpy="-0.03 0 0" />
+        rpy="${roll_offset} 0 0" />
       <axis xyz="1 0 0" />
       <limit lower="${roll_min_limit}"
@@ -81,5 +81,5 @@
       <child link="laser_main_link" />
       <origin xyz="0.0 0.0 0.02276"
-              rpy="0 0.03 0" />
+              rpy="0 ${pitch_offset} 0" />
       <axis xyz="0 1 0" />
       <limit lower="${pitch_min_limit}"
