Commit message: Rename robot

File: pandora_robots_description/gio/urdf/gio.urdf.xacro (robot description, xacro)
@@ -1,10 +1,10 @@
 <?xml version="1.0"?>
-<robot name="woody"
+<robot name="gio"
        xmlns:xacro="http://ros.org/wiki/xacro" >
   <!-- Import Files -->
   <xacro:include filename="$(find pandora_urdf_properties)/xacro/*.xacro" />
-  <xacro:include filename="$(find pandora_robots_description)/woody/urdf/urdf_configurations.xacro" />
-  <xacro:include filename="$(find pandora_robots_description)/woody/urdf/parts/*.xacro" />
-  <xacro:include filename="$(find pandora_robots_description)/woody/urdf/sensors/*.xacro" />
+  <xacro:include filename="$(find pandora_robots_description)/gio/urdf/urdf_configurations.xacro" />
+  <xacro:include filename="$(find pandora_robots_description)/gio/urdf/parts/*.xacro" />
+  <xacro:include filename="$(find pandora_robots_description)/gio/urdf/sensors/*.xacro" />
   <!-- Load Links & Joints -->
   <xacro:base />

File: pandora_robots_description/gio/urdf/parts/base.urdf.xacro (robot description, xacro)
@@ -8,5 +8,5 @@
       <visual>
         <geometry>
-          <mesh filename="package://pandora_robots_description/woody/meshes/base_link.dae" />
+          <mesh filename="package://pandora_robots_description/gio/meshes/base_link.dae" />
         </geometry>
         <material name="base" />

File: pandora_robots_description/gio/urdf/parts/side.urdf.xacro (robot description, xacro)
@@ -18,5 +18,5 @@
                 rpy="0.0 0.0 ${ ( 1 - reflect_y ) * PI_2 }" />
         <geometry>
-          <mesh filename="package://pandora_robots_description/woody/meshes/side_link.dae" />
+          <mesh filename="package://pandora_robots_description/gio/meshes/side_link.dae" />
         </geometry>
         <material name="side" />

File: pandora_robots_description/gio/urdf/parts/wheel.urdf.xacro (robot description, xacro)
@@ -11,5 +11,5 @@
                 rpy="0.0 0.0 ${ ( 1 - reflect_y ) * PI_2 }" />
         <geometry>
-          <mesh filename="package://pandora_robots_description/woody/meshes/wheel_link.dae" />
+          <mesh filename="package://pandora_robots_description/gio/meshes/wheel_link.dae" />
         </geometry>
         <material name="wheel" />
@@ -19,5 +19,5 @@
                 rpy="0.0 0.0 ${ ( 1 - reflect_y ) * PI_2 }" />
         <geometry>
-          <mesh filename="package://pandora_robots_description/woody/meshes/wheel_link.stl" />
+          <mesh filename="package://pandora_robots_description/gio/meshes/wheel_link.stl" />
         </geometry>
       </collision>

Commit message: Add differential link [ci skip]

File: pandora_robots_description/gio/urdf/gio.urdf.xacro (robot description, xacro)
@@ -9,4 +9,5 @@
   <!-- Load Links & Joints -->
   <xacro:base />
+  <xacro:differential />
   <xacro:side prefix_y="left" reflect_y="1" />
   <xacro:side prefix_y="right" reflect_y="-1" />
@@ -16,6 +17,5 @@
   <xacro:wheel prefix_y="right" prefix_x="rear" reflect_y="-1" reflect_x="-1" />
   <!-- Load Sensors -->
-  <xacro:laser_04 />
-  <!--<xacro:laser_20 />-->
+  <xacro:laser_04 /> <!--<xacro:laser_20 />-->
   <xacro:kinect />
   <xacro:thermal />

File: pandora_robots_description/gio/urdf/parts/base.urdf.xacro (robot description, xacro)
@@ -184,23 +184,4 @@
       <origin xyz="0.09013 -0.08006 0.24281" />
     </joint>
-<!--    <link name="differential" >-->
-<!--      <inertial>-->
-<!--        <origin xyz="0.0 0.0 0.0" />-->
-<!--        <mass value="0.31" />-->
-<!--        <inertia ixx="0.0001"-->
-<!--                 ixy="0.0"-->
-<!--                 ixz="0.0"-->
-<!--                 iyy="0.0001"-->
-<!--                 iyz="0.0"-->
-<!--                 izz="0.0001" />-->
-<!--      </inertial>-->
-<!--    </link>-->
-<!--    <joint name="differential_joint"-->
-<!--           type="fixed" >-->
-<!--      <parent link="base_link" />-->
-<!--      <child link="differential" />-->
-<!--      <origin xyz="-0.15 0.0 0.09031"-->
-<!--              rpy="0.0 0.0 0.0" />-->
-<!--    </joint>-->
   </xacro:macro>
 </robot>

File: pandora_robots_description/gio/urdf/parts/side.urdf.xacro (robot description, xacro)
@@ -23,7 +23,6 @@
       </visual>
       <collision>
-        <origin xyz="${zero}"
+        <origin xyz="0.0 0.0 -0.03018"
                 rpy="0.0 0.0 ${ ( 1 - reflect_y ) * PI_2 }" />
-        <origin xyz="0.0 0.0 -0.03018" />
         <geometry>
           <box size="0.405 0.081 0.096" />

File: pandora_robots_description/gio/urdf/urdf_configurations.xacro (robot description, xacro)
@@ -2,4 +2,6 @@
 <robot xmlns:xacro="http://ros.org/wiki/xacro" >
   <!-- Joint limits -->
+  <xacro:property name="differential_pin_joint_min_limit" value="-0.785" />
+  <xacro:property name="differential_pin_joint_max_limit" value="0.785" />
   <xacro:property name="side_joint_min_limit" value="-0.785" />
   <xacro:property name="side_joint_max_limit" value="0.785" />

Commit message: Add linear [ci skip]

File: pandora_robots_description/gio/urdf/gio.urdf.xacro (robot description, xacro)
@@ -9,4 +9,5 @@
   <!-- Load Links & Joints -->
   <xacro:base />
+  <xacro:linear />
   <xacro:differential />
   <xacro:side prefix_y="left" reflect_y="1" />
@@ -26,4 +27,3 @@
   <xacro:co2 />
   <xacro:microphone />
-  <!--<xacro:temperature />-->
 </robot>

File: pandora_robots_description/gio/urdf/urdf_configurations.xacro (robot description, xacro)
@@ -6,4 +6,6 @@
   <xacro:property name="side_joint_min_limit" value="-0.785" />
   <xacro:property name="side_joint_max_limit" value="0.785" />
+  <xacro:property name="linear_actuator_joint_min_limit" value="0.0" />
+  <xacro:property name="linear_actuator_joint_max_limit" value="0.14" />
   <xacro:property name="laser_roll_joint_min_limit" value="-0.523" />
   <xacro:property name="laser_roll_joint_max_limit" value="0.523" />

Commit message: Add camera_effector in urdf [ci skip]

File: pandora_robots_description/gio/urdf/gio.urdf.xacro (robot description, xacro)
@@ -20,4 +20,5 @@
   <xacro:laser_04 /> <!--<xacro:laser_20 />-->
   <xacro:kinect />
+  <xacro:camera_effector />
   <xacro:thermal />
   <xacro:left_webcam />

File: pandora_robots_description/gio/urdf/urdf_configurations.xacro (robot description, xacro)
@@ -8,4 +8,8 @@
   <xacro:property name="linear_actuator_joint_min_limit" value="0.0" />
   <xacro:property name="linear_actuator_joint_max_limit" value="0.14" />
+  <xacro:property name="camera_effector_pan_joint_min_limit" value="-1.3962" />
+  <xacro:property name="camera_effector_pan_joint_max_limit" value="1.3962" />
+  <xacro:property name="camera_effector_tilt_joint_min_limit" value="-0.6" />
+  <xacro:property name="camera_effector_tilt_joint_max_limit" value="0.6" />
   <xacro:property name="laser_roll_joint_min_limit" value="-0.523" />
   <xacro:property name="laser_roll_joint_max_limit" value="0.523" />

File: pandora_sensors_description/camera_effector/urdf/pi_camera.urdf.xacro (robot description, xacro)
@@ -84,5 +84,5 @@
     <!-- Joints -->
     <joint name="camera_effector_pan_joint"
-           type="fixed" >
+           type="revolute" >
       <parent link="${parent}" />
       <child link="camera_effector_pan_link" />
@@ -108,5 +108,5 @@
     </joint>
     <joint name="camera_effector_tilt_joint"
-           type="fixed" >
+           type="revolute" >
       <parent link="camera_effector_tilt_link" />
       <child link="pi_camera_platform_link" />

Commit message: Separate camera_effector and picam and add second picam

File: pandora_robots_description/gio/urdf/gio.urdf.xacro (robot description, xacro)
@@ -9,6 +9,7 @@
   <!-- Load Links & Joints -->
   <xacro:base />
+  <xacro:differential />
   <xacro:linear />
-  <xacro:differential />
+  <xacro:camera_effector />
   <xacro:side prefix_y="left" reflect_y="1" />
   <xacro:side prefix_y="right" reflect_y="-1" />
@@ -20,8 +21,9 @@
   <xacro:laser_20 /> <!--<xacro:laser_04 />-->
   <xacro:kinect />
-  <xacro:camera_effector />
-  <xacro:thermal />
+  <xacro:front_picam />
+  <xacro:rear_picam />
   <xacro:left_webcam />
   <xacro:right_webcam />
+  <xacro:thermal />
   <xacro:left_sonar />
   <xacro:right_sonar />

File: pandora_robots_description/gio/urdf/parts/camera_effector.xacro (robot description, xacro)
@@ -1,8 +1,5 @@
 <?xml version="1.0" ?>
 <robot xmlns:xacro="http://ros.org/wiki/xacro" >
-  <xacro:macro name="pi_camera"
-               params="parent *origin
-                       yaw_min_limit yaw_max_limit
-                       pitch_min_limit pitch_max_limit" >
+  <xacro:macro name="camera_effector" >
     <!-- Links -->
     <link name="camera_effector_pan_link" >
@@ -13,5 +10,5 @@
       <visual>
         <geometry>
-          <mesh filename="package://pandora_sensors_description/camera_effector/meshes/pan_servo_link.dae" />
+          <mesh filename="package://pandora_robots_description/gio/meshes/camera_effector_pan_servo_link.dae" />
         </geometry>
       </visual>
@@ -29,8 +26,8 @@
       <visual>
         <geometry>
-          <mesh filename="package://pandora_sensors_description/camera_effector/meshes/pan_base_link.dae" />
+          <mesh filename="package://pandora_robots_description/gio/meshes/camera_effector_pan_base_link.dae" />
         </geometry>
       </visual>
-      <collision>
+      <collision>picam/meshes/raspberry_pi_camera
         <origin xyz="0.00027 -0.00042 0.00104" />
         <geometry>
@@ -45,5 +42,5 @@
       <visual>
         <geometry>
-          <mesh filename="package://pandora_sensors_description/camera_effector/meshes/tilt_servo_link.dae" />
+          <mesh filename="package://pandora_robots_description/gio/meshes/camera_effector_tilt_servo_link.dae" />
         </geometry>
       </visual>
@@ -55,5 +52,5 @@
       </collision>
     </link>
-    <link name="pi_camera_platform_link" >
+    <link name="camera_effector_platform_link" >
       <!-- FIXME -->
       <inertial>
@@ -69,5 +66,5 @@
       <visual>
         <geometry>
-          <mesh filename="package://pandora_sensors_description/camera_effector/meshes/platform.dae" />
+          <mesh filename="package://pandora_robots_description/gio/meshes/camera_effector_platform.dae" />
         </geometry>
       </visual>
@@ -79,26 +76,10 @@
       </collision>
     </link>
-    <link name="pi_camera_link" >
-      <xacro:solid_cuboid_inertial mass="0.021" x="0.009" y="0.025" z="0.024" >
-        <origin xyz="-0.00058 0.0 0.00189" />
-      </xacro:solid_cuboid_inertial>
-      <visual>
-        <geometry>
-          <mesh filename="package://pandora_sensors_description/camera_effector/meshes/pi_camera.dae" />
-        </geometry>
-      </visual>
-      <collision>
-        <origin xyz="0.00045 0.0 0.0025" />
-        <geometry>
-          <box size="0.009 0.025 0.024" />
-        </geometry>
-      </collision>
-    </link>
     <!-- Joints -->
     <joint name="camera_effector_pan_joint"
            type="revolute" >
-      <parent link="${parent}" />
+      <parent link="linear_actuator_link" />
       <child link="camera_effector_pan_link" />
-      <xacro:insert_block name="origin" />
+      <origin xyz="0.0 0.0 0.15614" />
       <axis xyz="0 0 1" />
       <dynamics damping="0.0" />
@@ -123,5 +104,5 @@
            type="revolute" >
       <parent link="camera_effector_tilt_link" />
-      <child link="pi_camera_platform_link" />
+      <child link="camera_effector_platform_link" />
       <origin xyz="0.0 0.0 0.0"
               rpy="0.0 0.3490658504 0.0" />
@@ -133,31 +114,4 @@
              velocity="50.0" />
     </joint>
-    <joint name="pi_camera_platform_joint"
-           type="fixed" >
-      <parent link="pi_camera_platform_link" />
-      <child link="pi_camera_link" />
-      <origin xyz="0.00034 -0.01925 0.04306"
-              rpy="0.0 -0.3490658504 0.0" />
-    </joint>
-    <!-- Frames -->
-    <link name="pi_camera_frame" >
-      <xacro:point_mass_inertial />
-    </link>
-    <link name="pi_camera_optical_frame" >
-      <xacro:point_mass_inertial />
-    </link>
-    <joint name="pi_camera_joint"
-           type="fixed" >
-      <parent link="pi_camera_link" />
-      <child link="pi_camera_frame" />
-      <origin xyz="0.0045 0.0 0.0" />
-    </joint>
-    <joint name="pi_camera_optical_joint"
-           type="fixed" >
-      <parent link="pi_camera_frame" />
-      <child link="pi_camera_optical_frame" />
-      <origin xyz="0.0 0.0 0.0"
-              rpy="-1.5708 0.0 -1.5708" />
-    </joint>
   </xacro:macro>
 </robot>

Commit message: Replace rear picam with webcam

File: pandora_robots_description/gio/urdf/gio.urdf.xacro (robot description, xacro)
@@ -22,5 +22,5 @@
   <xacro:kinect />
   <xacro:front_picam />
-  <xacro:rear_picam />
+  <xacro:rear_webcam />
   <xacro:left_webcam />
   <xacro:right_webcam />

File: pandora_robots_description/gio/urdf/sensors/webcam.xacro (robot description, xacro)
@@ -16,3 +16,10 @@
     </xacro:logitech_c310hd>
   </xacro:macro>
+  <xacro:macro name="rear_webcam" >
+    <xacro:logitech_c310hd parent="base_link"
+                           prefix="rear" >
+      <origin xyz="-0.10937 0.0 0.26221"
+              rpy="0.0 0.0 ${- 2 * PI_2}" />
+    </xacro:logitech_c310hd>
+  </xacro:macro>
 </robot>

File: pandora_sensors_description/webcam/urdf/logitech_c310hd.urdf.xacro (robot description, xacro)
@@ -39,6 +39,6 @@
       <parent link="${prefix}_webcam_link" />
       <child link="${prefix}_webcam_frame" />
-      <origin xyz="0.02499 0.0 0.05704"
-              rpy="0.0 -0.2792 0.0" />
+      <origin xyz="0.02499 0.0 0.04"
+              rpy="0.0 0.0 0.0" />
     </joint>
     <joint name="${prefix}_webcam_optical_joint"
