Commit message: Add yellow material

File: pandora_urdf_properties/xacro/materials.xacro (robot description, xacro)
@@ -6,4 +6,7 @@
   <material name="black" >
     <color rgba="${0/255} ${0/255} ${0/255} 1.0" />
+  </material>
+  <material name="dark_grey" >
+    <color rgba="${10/255} ${10/255} ${10/255} 1.0" />
   </material>
   <material name="red" >
@@ -16,4 +19,7 @@
     <color rgba="${0/255} ${0/255} ${204/255} 1.0" />
   </material>
+  <material name="yellow" >
+    <color rgba="${255/255} ${255/255} ${0/255} 1.0" />
+  </material>
   <material name="solidworks_default" >
     <color rgba="${192/255} ${192/255} ${192/255} 1.0" />
