Commit message: Add null unertial macro

File: pandora_urdf_properties/xacro/defaults.xacro (robot description, xacro)
@@ -39,4 +39,16 @@
                iyz="0"
                izz="1.0E-6" />
+    </inertial>
+  </xacro:macro>
+  <xacro:macro name="null_inertial" >
+    <inertial>
+      <origin xyz="0.0 0.0 0.0" />
+      <mass value="0.001" />
+      <inertia ixx="0.001"
+               ixy="0"
+               ixz="0"
+               iyy="0.001"
+               iyz="0"
+               izz="0.001" />
     </inertial>
   </xacro:macro>
