Commit message: Add monstertruck model
- adds monstertruck urdf files
- adds meshes of parts

File: pandora_robots_description/monstertruck/urdf/dimensions.xacro (robot description, xacro)
@@ -1,5 +1,4 @@
 <?xml version="1.0"?>
 <robot xmlns:xacro="http://ros.org/wiki/xacro" >
-  <!-- PARAMETERS -->
   <!-- Dimensions -->
   <xacro:property name="wheel_width" value="0.08" />

File: pandora_robots_description/monstertruck/urdf/joint_limits.xacro (robot description, xacro)
@@ -1,15 +1,25 @@
 <?xml version="1.0"?>
 <robot xmlns:xacro="http://ros.org/wiki/xacro" >
-  <!-- TODO find/measure/compute actual joint limits -->
-  <!-- Joint limits -->
+  <!-- Joint Limits -->
+  <!-- laser joint limits -->
   <xacro:property name="laser_roll_joint_min_limit" value="-0.523" />
   <xacro:property name="laser_roll_joint_max_limit" value="0.523" />
   <xacro:property name="laser_pitch_joint_min_limit" value="-0.523" />
   <xacro:property name="laser_pitch_joint_max_limit" value="0.523" />
-  <xacro:property name="max_robot_linear_velocity" value="2.0" />
-  <xacro:property name="max_robot_angular_velocity" value="2.0" />
   <xacro:property name="max_laser_angular_velocity" value="2.5" />
-  <xacro:property name="max_robot_linear_acceleration" value="1.0" />
-  <xacro:property name="max_robot_angular_acceleration" value="0.2" />
   <xacro:property name="max_laser_angular_acceleration" value="0.0" />
+  <!-- robot steer and drive joint limits -->
+  <xacro:property name="steer_joint_min_limit" value="-PI/8" />
+  <xacro:property name="steer_joint_max_limit" value="PI/8" />
+  <xacro:property name="drive_joint_velocity_limit" value="0.22" />
+  <xacro:property name="drive_joint_effort_limit" value="100.0" />
+  <!-- axle suspension approximation joint limits -->
+  <xacro:property name="axle_z_joint_min_limit" value="0.0" />
+  <xacro:property name="axle_z_joint_max_limit" value="0.027" />
+  <xacro:property name="axle_z_joint_velocity_limit" value="5.0" />
+  <xacro:property name="axle_z_joint_effort_limit" value="100.0" />
+  <xacro:property name="axle_roll_joint_min_limit" value="${-PI/8}" />
+  <xacro:property name="axle_roll_joint_max_limit" value="${PI/8}" />
+  <xacro:property name="axle_velocity_limit" value="5.0" />
+  <xacro:property name="axle_effort_limit" value="100.0" />
 </robot>

File: pandora_robots_description/monstertruck/urdf/monstertruck.urdf.xacro (robot description, xacro)
@@ -4,18 +4,38 @@
   <xacro:include filename="$(find pandora_urdf_properties)/xacro/*.xacro" />
   <xacro:include filename="$(find pandora_robots_description)/monstertruck/urdf/joint_limits.xacro" />
-  <xacro:include filename="$(find pandora_robots_description)/monstertruck/urdf/urdf.xacro" />
+  <xacro:include filename="$(find pandora_robots_description)/monstertruck/urdf/dimensions.xacro" />
   <xacro:include filename="$(find pandora_robots_description)/monstertruck/urdf/parts/*.xacro" />
   <xacro:include filename="$(find pandora_robots_description)/monstertruck/urdf/sensors/*.xacro" />
   <!-- Load Links & Joints -->
+  <!-- Load base and boxes -->
   <xacro:base />
-  <xacro:side prefix_y="left" reflect_y="1" />
-  <xacro:side prefix_y="right" reflect_y="-1" />
-  <xacro:wheel prefix_y="left" prefix_x="front" reflect_y="1" reflect_x="1" />
-  <xacro:wheel prefix_y="left" prefix_x="rear" reflect_y="1" reflect_x="-1" />
-  <xacro:wheel prefix_y="right" prefix_x="front" reflect_y="-1" reflect_x="1" />
-  <xacro:wheel prefix_y="right" prefix_x="rear" reflect_y="-1" reflect_x="-1" />
+  <xacro:electronics_box />
+  <xacro:pc_box />
+  <!-- Load suspensions -->
+  <xacro:suspensions prefix_y="left" prefix_x="front" reflect_y="1" reflect_x="1" />
+  <xacro:suspensions prefix_y="right" prefix_x="front" reflect_y="-1" reflect_x="1" />
+  <xacro:suspensions prefix_y="left" prefix_x="rear" reflect_y="1" reflect_x="-1" />
+  <xacro:suspensions prefix_y="right" prefix_x="rear" reflect_y="-1" reflect_x="-1" />
+  <!-- Load front and rear axles -->
+  <xacro:axle prefix_x="front" reflect_x="1" />
+  <xacro:axle prefix_x="rear" reflect_x="-1" />
+  <!-- Load wheels -->
+  <xacro:offroad_wheel prefix_y="left" prefix_x="front" reflect_y="1" reflect_x="1" />
+  <xacro:offroad_wheel prefix_y="left" prefix_x="rear" reflect_y="1" reflect_x="-1" />
+  <xacro:offroad_wheel prefix_y="right" prefix_x="front" reflect_y="-1" reflect_x="1" />
+  <xacro:offroad_wheel prefix_y="right" prefix_x="rear" reflect_y="-1" reflect_x="-1" />
   <!-- Load Sensors -->
   <xacro:laser_04 />
-  <xacro:camera>
-  <xacro:compass>
+  <xacro:picam />
+  <xacro:compass_os4000 />
+  <!-- Load miscellaneous parts -->
+  <xacro:battery />
+  <xacro:pc_fan_40mm />
+  <xacro:pc_fan_60mm />
+  <xacro:m4_atx_psu />
+  <xacro:dc_dc_converter />
+  <xacro:electronics_power_distribution_board />
+  <xacro:motors_power_distribution_board />
+  <xacro:battery_power_distribution_board />
+  <xacro:epos_24_1 />
 </robot>
