Commit message: Add argument to enable/disable experimental suspension approximation

File: pandora_robots_description/monstertruck/urdf/monstertruck.urdf.xacro (robot description, xacro)
@@ -1,4 +1,5 @@
 <?xml version="1.0"?>
 <robot name="monstertruck" xmlns:xacro="http://ros.org/wiki/xacro" >
+  <xacro:arg name="suspension_approximation" default="false" />
   <!-- Import Files -->
   <xacro:include filename="$(find pandora_urdf_properties)/xacro/*.xacro" />
@@ -18,6 +19,6 @@
   <xacro:suspensions prefix_y="right" prefix_x="rear" reflect_y="-1" reflect_x="-1" />
   <!-- Load front and rear axles -->
-  <xacro:axle prefix_x="front" reflect_x="1" />
-  <xacro:axle prefix_x="rear" reflect_x="-1" />
+  <xacro:axle prefix_x="front" reflect_x="1" suspension_approximation="$(arg suspension_approximation)"/>
+  <xacro:axle prefix_x="rear" reflect_x="-1" suspension_approximation="$(arg suspension_approximation)"/>
   <!-- Load wheels -->
   <xacro:offroad_wheel prefix_y="left" prefix_x="front" reflect_y="1" reflect_x="1" />

File: pandora_robots_description/monstertruck/urdf/parts/axle.urdf.xacro (robot description, xacro)
@@ -1,52 +1,55 @@
 <?xml version="1.0" ?>
 <robot xmlns:xacro="http://ros.org/wiki/xacro" >
-  <xacro:macro name="axle" params="prefix_x reflect_x" >
-    <!-- <joint name="${prefix_x}_base_axle_joint" type="fixed"> -->
-      <!-- <parent link="base_link" /> -->
-      <!-- <child link="${prefix_x}_axle_link" /> -->
-      <!-- <origin xyz="${reflect_x*0.159+0.031} 0.0 -0.078" /> -->
-    <!-- </joint> -->
-<!-- ======================================================================= -->
-<!-- ========= Experimental Suspension Approximation for simulation =========-->
-<!-- ======================================================================= -->
-    <joint name="${prefix_x}_base_axle_sim_suspension_joint" type="prismatic" >
-      <parent link="base_link" />
-      <child link="${prefix_x}_axle_sim_suspension_link" />
-      <limit
-        effort="${axle_z_joint_effort_limit}"
-        velocity="${axle_z_joint_velocity_limit}"
-        lower="${axle_z_joint_min_limit}"
-        upper="${axle_z_joint_max_limit}" />
-      <origin xyz="${reflect_x*0.158+0.031} 0.0 0.035"  rpy="0.0 0.0 0.0" />
-      <axis xyz="0 0 1" />
-    </joint>
-    <link name="${prefix_x}_axle_sim_suspension_link" >
-      <xacro:solid_cylinder_intertial mass="0.00001" radius="0.001" y="0.1212" >
-        <origin xyz="0.0 0.0 0.0"/>
-      </xacro:solid_cylinder_intertial>
-      <visual>
-        <geometry>
-          <cylinder radius="0.001" length="0.1212" />
-        </geometry>
-        <origin xyz="0.0 0.0 ${-0.1212/2}" />
-      </visual>
-      <collision>
-        <geometry>
-          <cylinder radius="0.001" length="0.1212" />
-        </geometry>
-        <origin xyz="0.0 0.0 ${-0.1212/2}" />
-      </collision>
-    </link>
-    <joint name="${prefix_x}_axle_joint" type="revolute" >
-      <parent link="${prefix_x}_axle_sim_suspension_link" />
-      <child link="${prefix_x}_axle_link" />
-      <limit
-        effort="${axle_effort_limit}"
-        velocity="${axle_velocity_limit}"
-        lower="${axle_roll_joint_min_limit}"
-        upper="${axle_roll_joint_max_limit}" />
-      <origin xyz="0.0 0.0 -0.112"  rpy="0.0 0.0 0.0" />
-      <axis xyz="1 0 0" />
-    </joint>
+  <xacro:macro name="axle" params="prefix_x reflect_x suspension_approximation" >
+    <!-- No suspension  -->
+    <xacro:unless value="${suspension_approximation}">
+      <joint name="${prefix_x}_base_axle_joint" type="fixed">
+        <parent link="base_link" />
+        <child link="${prefix_x}_axle_link" />
+        <origin xyz="${reflect_x*0.159+0.031} 0.0 -0.078" />
+      </joint>
+    </xacro:unless>
+<!-- =============== Experimental Suspension Approximation ================= -->
+    <xacro:if value="${suspension_approximation}">
+      <joint name="${prefix_x}_base_axle_sim_suspension_joint" type="prismatic" >
+        <parent link="base_link" />
+        <child link="${prefix_x}_axle_sim_suspension_link" />
+        <limit
+          effort="${axle_z_joint_effort_limit}"
+          velocity="${axle_z_joint_velocity_limit}"
+          lower="${axle_z_joint_min_limit}"
+          upper="${axle_z_joint_max_limit}" />
+        <origin xyz="${reflect_x*0.158+0.031} 0.0 0.035"  rpy="0.0 0.0 0.0" />
+        <axis xyz="0 0 1" />
+      </joint>
+      <link name="${prefix_x}_axle_sim_suspension_link" >
+        <xacro:solid_cylinder_intertial mass="0.00001" radius="0.001" y="0.1212" >
+          <origin xyz="0.0 0.0 0.0"/>
+        </xacro:solid_cylinder_intertial>
+        <visual>
+          <geometry>
+            <cylinder radius="0.001" length="0.1212" />
+          </geometry>
+          <origin xyz="0.0 0.0 ${-0.1212/2}" />
+        </visual>
+        <collision>
+          <geometry>
+            <cylinder radius="0.001" length="0.1212" />
+          </geometry>
+          <origin xyz="0.0 0.0 ${-0.1212/2}" />
+        </collision>
+      </link>
+      <joint name="${prefix_x}_axle_joint" type="revolute" >
+        <parent link="${prefix_x}_axle_sim_suspension_link" />
+        <child link="${prefix_x}_axle_link" />
+        <limit
+          effort="${axle_effort_limit}"
+          velocity="${axle_velocity_limit}"
+          lower="${axle_roll_joint_min_limit}"
+          upper="${axle_roll_joint_max_limit}" />
+        <origin xyz="0.0 0.0 -0.112"  rpy="0.0 0.0 0.0" />
+        <axis xyz="1 0 0" />
+      </joint>
+    </xacro:if>
 <!-- ======================================================================= -->
     <link name="${prefix_x}_axle_link" >
