Commit message: Modify joint limits

File: pandora_robots_description/monstertruck/urdf/joint_limits.xacro (robot description, xacro)
@@ -12,14 +12,14 @@
   <xacro:property name="steer_joint_min_limit" value="-PI/8" />
   <xacro:property name="steer_joint_max_limit" value="PI/8" />
-  <xacro:property name="drive_joint_velocity_limit" value="0.22" />
-  <xacro:property name="drive_joint_effort_limit" value="100.0" />
+  <xacro:property name="drive_joint_velocity_limit" value="1.0" />
+  <xacro:property name="drive_joint_effort_limit" value="10.0" />
   <!-- axle suspension approximation joint limits -->
   <xacro:property name="axle_z_joint_min_limit" value="0.0" />
   <xacro:property name="axle_z_joint_max_limit" value="0.027" />
-  <xacro:property name="axle_z_joint_velocity_limit" value="5.0" />
-  <xacro:property name="axle_z_joint_effort_limit" value="100.0" />
+  <xacro:property name="axle_z_joint_velocity_limit" value="10.0" />
+  <xacro:property name="axle_z_joint_effort_limit" value="10.0" />
   <xacro:property name="axle_roll_joint_min_limit" value="${-PI/8}" />
   <xacro:property name="axle_roll_joint_max_limit" value="${PI/8}" />
-  <xacro:property name="axle_velocity_limit" value="5.0" />
-  <xacro:property name="axle_effort_limit" value="100.0" />
+  <xacro:property name="axle_velocity_limit" value="10.0" />
+  <xacro:property name="axle_effort_limit" value="10.0" />
 </robot>

Commit message: Fix offroad_wheel urdf

File: pandora_robots_description/monstertruck/urdf/joint_limits.xacro (robot description, xacro)
@@ -9,7 +9,10 @@
   <xacro:property name="max_laser_angular_velocity" value="2.5" />
   <xacro:property name="max_laser_angular_acceleration" value="0.0" />
-  <!-- robot steer and drive joint limits -->
-  <xacro:property name="steer_joint_min_limit" value="-PI/8" />
-  <xacro:property name="steer_joint_max_limit" value="PI/8" />
+  <!-- wheel steer joint limits -->
+  <xacro:property name="steer_joint_min_limit" value="${-PI/8}" />
+  <xacro:property name="steer_joint_max_limit" value="${PI/8}" />
+  <xacro:property name="steer_joint_velocity_limit" value="5.0" />
+  <xacro:property name="steer_joint_effort_limit" value="10.0" />
+  <!-- wheel drive joint limits -->
   <xacro:property name="drive_joint_velocity_limit" value="1.0" />
   <xacro:property name="drive_joint_effort_limit" value="10.0" />

File: pandora_robots_description/monstertruck/urdf/parts/offroad_wheel.urdf.xacro (robot description, xacro)
@@ -1,13 +1,35 @@
 <?xml version="1.0" ?>
 <robot xmlns:xacro="http://ros.org/wiki/xacro" >
-  <xacro:macro name="offroad_wheel" params="prefix_y prefix_x reflect_y reflect_x" >
-    <joint name="${prefix_y}_${prefix_x}_axle_to_wheel_steer_joint" type="fixed" >
+  <xacro:property name="wheelbase" value="0.32" />
+  <xacro:property name="track" value="0.26" />
+  <xacro:property name="steer_link_offset" value="0.115" />
+  <xacro:property name="steer_link_radius" value="0.008" />
+  <xacro:property name="steer_link_mass" value="0.001" />
+  <xacro:property name="drive_link_length" value="0.03" />
+  <xacro:property name="drive_link_radius" value="0.0025" />
+  <xacro:property name="drive_link_mass" value="0.001" />
+  <xacro:property name="wheel_link_radius" value="0.075" />
+  <xacro:property name="wheel_link_width" value="0.081" />
+  <xacro:property name="wheel_link_offset" value="-0.004" />
+  <xacro:property name="wheel_link_mass" value="0.281" />
+  <xacro:macro name="offroad_wheel"
+    params="prefix_y prefix_x reflect_y reflect_x" >
+    <joint name="${prefix_y}_${prefix_x}_wheel_steer_joint" type="revolute" >
       <parent link="${prefix_x}_axle_link" />
       <child link="${prefix_y}_${prefix_x}_wheel_steer_link" />
-      <origin xyz="0.0 ${reflect_y*0.112} 0.0" />
+      <origin xyz="0.0 ${reflect_y*steer_link_offset} 0.0" />
+      <axis xyz="0 0 1" />
+      <dynamics damping="0.0" />
+      <limit
+        lower="${steer_joint_min_limit}"
+        upper="${steer_joint_max_limit}"
+        effort="${steer_joint_effort_limit}"
+        velocity="${steer_joint_velocity_limit}"/>
     </joint>
     <!-- wheel steer link -->
     <link name="${prefix_y}_${prefix_x}_wheel_steer_link" >
-      <xacro:solid_sphere_inertial mass="0.05" radius="0.01" >
+      <xacro:solid_sphere_inertial
+        mass="${steer_link_mass}"
+        radius="${steer_link_radius}" >
         <origin xyz="0.0 0.0 0.0" />
       </xacro:solid_sphere_inertial>
@@ -15,5 +37,5 @@
         <origin xyz="0.0 0.0 0.0" rpy="0.0 0.0 0.0" />
         <geometry>
-          <sphere radius="0.01" />
+          <sphere radius="${steer_link_radius}" />
         </geometry>
         <material name="dark_grey" />
@@ -22,42 +44,41 @@
         <origin xyz="0.0 0.0 0.0" rpy="0.0 0.0 0.0" />
         <geometry>
-          <sphere radius="0.01" />
+          <sphere radius="${steer_link_radius}" />
         </geometry>
       </collision>
     </link>
     <!-- wheel steer link to drive link joint -->
-    <joint name="${prefix_y}_${prefix_x}_wheel_steer_joint"
-           type="revolute" >
+    <joint name="${prefix_y}_${prefix_x}_wheel_steer_link_to_drive_link_joint" type="fixed" >
       <parent link="${prefix_y}_${prefix_x}_wheel_steer_link" />
       <child link="${prefix_y}_${prefix_x}_wheel_drive_link" />
-      <axis xyz="0 0 1" />
-      <dynamics damping="0.0" />
-      <limit lower="${-PI/8}" upper="${PI/8}" effort="100" velocity="100"/>
+      <origin xyz="0.0 ${reflect_y*(steer_link_radius/2+drive_link_length/2)} 0.0" />
     </joint>
     <!-- wheel drive link -->
     <link name="${prefix_y}_${prefix_x}_wheel_drive_link" >
-      <xacro:solid_cylinder_inertial mass="0.01" radius="0.005" y="0.04">
-        <xacro:default_origin />
-      </xacro:solid_cylinder_inertial>
+      <!-- Using real inertia causes unexpected bahaviour -->
+      <!-- Works fine, only with null inertial -->
+      <xacro:null_inertial />
+      <!-- <xacro:solid_cylinder_inertial mass="0.01" radius="0.0025" y="0.03" > -->
+        <!-- <origin xyz="0.0 0.0 0.0" /> -->
+      <!-- </xacro:solid_cylinder_inertial> -->
       <visual>
-        <origin xyz="0.0 ${reflect_y*0.02} 0.0" rpy="${-PI/2} 0.0 0.0" />
+        <origin xyz="0.0 0.0 0.0" rpy="${PI/2} 0.0 0.0" />
         <geometry>
-          <cylinder radius="0.005" length="0.04" />
+          <cylinder radius="${drive_link_radius}" length="${drive_link_length}" />
         </geometry>
         <material name="dark_grey" />
       </visual>
       <collision>
-        <origin xyz="0.0 ${reflect_y*0.005} 0.0" rpy="${-PI/2} 0.0 0.0" />
+        <origin xyz="0.0 0.0 0.0" rpy="${PI/2} 0.0 0.0" />
         <geometry>
-          <cylinder radius="0.05" length="0.045" />
+          <cylinder radius="${drive_link_radius}" length="${drive_link_length}" />
         </geometry>
       </collision>
     </link>
     <!-- drive link to wheel joint -->
-    <joint name="${prefix_y}_${prefix_x}_wheel_drive_joint"
-           type="continuous" >
+    <joint name="${prefix_y}_${prefix_x}_wheel_drive_joint" type="continuous" >
       <parent link="${prefix_y}_${prefix_x}_wheel_drive_link" />
       <child link="${prefix_y}_${prefix_x}_wheel_link" />
-      <origin xyz="0.0 ${reflect_y*0.004} 0.0" />
+      <origin xyz="0.0 ${reflect_y*wheel_link_offset} 0.0" />
       <axis xyz="0 1 0" />
       <dynamics damping="0.0" />
@@ -68,14 +89,12 @@
     <!-- wheel_link -->
     <link name="${prefix_y}_${prefix_x}_wheel_link" >
-      <!-- <inertial> -->
-        <!-- <mass value="0.281"/> -->
-        <!-- <inertia ixx="0.000002" ixy="0.0" iyy="0.000003" iyz="0.0" izz="0.000002" ixz="0.0" /> -->
-        <!-- <origin xyz="-0.00001 ${reflect_y*0.0004} 0.000053" /> -->
-      <!-- </inertial> -->
-      <xacro:solid_cylinder_inertial mass="0.970" radius="0.075" y="0.08" >
-        <origin xyz="-0.00001 ${reflect_y*0.00004} 0.000053" />
+      <xacro:solid_cylinder_inertial
+        mass="${wheel_link_mass}"
+        radius="${wheel_link_radius}"
+        y="${wheel_link_width}" >
+        <origin xyz="0.0 0.0 0.0" />
       </xacro:solid_cylinder_inertial>
       <visual>
-        <origin xyz="0.0 ${reflect_y*0.019} 0.0" rpy="0.0 0.0 0.0" />
+        <origin xyz="0.0 0.0 0.0" rpy="0.0 0.0 0.0" />
         <geometry>
           <mesh filename="package://pandora_robots_description/monstertruck/meshes/${prefix_y}_offroad_wheel.dae" />
@@ -83,15 +102,10 @@
       </visual>
       <collision>
-        <origin xyz="0.0 ${reflect_y*0.019} 0.0" rpy="0.0 0.0 0.0" />
+        <origin xyz="0.0 0.0 0.0" rpy="${PI/2} 0.0 0.0" />
         <geometry>
-          <mesh filename="package://pandora_robots_description/monstertruck/meshes/${prefix_y}_offroad_wheel.stl" />
+          <!-- <mesh filename="package://pandora_robots_description/monstertruck/meshes/${prefix_y}_offroad_wheel.stl" /> -->
+          <cylinder radius="${wheel_link_radius}" length="${wheel_link_width}" />
         </geometry>
       </collision>
-      <collision_checking>
-        <origin xyz="0.0 ${reflect_y*0.019} 0.0" rpy="0.0 0.0 0.0" />
-        <geometry>
-          <cylinder length="0.084" radius="0.075"/>
-        </geometry>
-      </collision_checking>
     </link>
   </xacro:macro>

Commit message: Add an axle suspension using a prismatic and a revolute joint

File: pandora_robots_description/monstertruck/urdf/joint_limits.xacro (robot description, xacro)
@@ -10,18 +10,18 @@
   <xacro:property name="max_laser_angular_acceleration" value="0.0" />
   <!-- wheel steer joint limits -->
-  <xacro:property name="steer_joint_min_limit" value="${-PI/8}" />
-  <xacro:property name="steer_joint_max_limit" value="${PI/8}" />
-  <xacro:property name="steer_joint_velocity_limit" value="5.0" />
-  <xacro:property name="steer_joint_effort_limit" value="10.0" />
+  <xacro:property name="steer_joint_lower_limit" value="${-25*PI/180}" />
+  <xacro:property name="steer_joint_upper_limit" value="${25*PI/180}" />
+  <xacro:property name="steer_joint_velocity_limit" value="100.0" />
+  <xacro:property name="steer_joint_effort_limit" value="100.0" />
   <!-- wheel drive joint limits -->
-  <xacro:property name="drive_joint_velocity_limit" value="1.0" />
-  <xacro:property name="drive_joint_effort_limit" value="10.0" />
+  <xacro:property name="drive_joint_velocity_limit" value="100.0" />
+  <xacro:property name="drive_joint_effort_limit" value="100.0" />
   <!-- axle suspension approximation joint limits -->
-  <xacro:property name="axle_z_joint_min_limit" value="0.0" />
-  <xacro:property name="axle_z_joint_max_limit" value="0.027" />
-  <xacro:property name="axle_z_joint_velocity_limit" value="10.0" />
-  <xacro:property name="axle_z_joint_effort_limit" value="10.0" />
-  <xacro:property name="axle_roll_joint_min_limit" value="${-PI/8}" />
-  <xacro:property name="axle_roll_joint_max_limit" value="${PI/8}" />
+  <xacro:property name="virtual_suspension_joint_lower_limit" value="0.0" />
+  <xacro:property name="virtual_suspension_joint_upper_limit" value="0.027" />
+  <xacro:property name="virtual_suspension_joint_velocity_limit" value="10.0" />
+  <xacro:property name="virtual_suspension_joint_effort_limit" value="1.0" />
+  <xacro:property name="axle_roll_joint_lower_limit" value="${-PI*10/180}" />
+  <xacro:property name="axle_roll_joint_upper_limit" value="${PI*10/180}" />
   <xacro:property name="axle_velocity_limit" value="10.0" />
   <xacro:property name="axle_effort_limit" value="10.0" />

File: pandora_robots_description/monstertruck/urdf/monstertruck.urdf.xacro (robot description, xacro)
@@ -1,5 +1,4 @@
 <?xml version="1.0"?>
 <robot name="monstertruck" xmlns:xacro="http://ros.org/wiki/xacro" >
-  <xacro:arg name="suspension_approximation" default="false" />
   <!-- Import Files -->
   <xacro:include filename="$(find pandora_urdf_properties)/xacro/*.xacro" />
@@ -19,6 +18,6 @@
   <xacro:suspensions prefix_y="right" prefix_x="rear" reflect_y="-1" reflect_x="-1" />
   <!-- Load front and rear axles -->
-  <xacro:axle prefix_x="front" reflect_x="1" suspension_approximation="$(arg suspension_approximation)"/>
-  <xacro:axle prefix_x="rear" reflect_x="-1" suspension_approximation="$(arg suspension_approximation)"/>
+  <xacro:axle prefix_x="front" reflect_x="1" />
+  <xacro:axle prefix_x="rear" reflect_x="-1" />
   <!-- Load wheels -->
   <xacro:offroad_wheel prefix_y="left" prefix_x="front" reflect_y="1" reflect_x="1" />

File: pandora_robots_description/monstertruck/urdf/parts/axle.urdf.xacro (robot description, xacro)
@@ -1,56 +1,32 @@
 <?xml version="1.0" ?>
 <robot xmlns:xacro="http://ros.org/wiki/xacro" >
-  <xacro:macro name="axle" params="prefix_x reflect_x suspension_approximation" >
-    <!-- No suspension  -->
-    <xacro:unless value="${suspension_approximation}">
-      <joint name="${prefix_x}_base_axle_joint" type="fixed" >
-        <parent link="base_link" />
-        <child link="${prefix_x}_axle_link" />
-        <origin xyz="${reflect_x*0.159+0.031} 0.0 -0.078" />
-      </joint>
-    </xacro:unless>
-<!-- =============== Experimental Suspension Approximation ================= -->
-    <xacro:if value="${suspension_approximation}">
-      <joint name="${prefix_x}_virtual_suspension_joint" type="prismatic" >
-        <parent link="base_link" />
-        <child link="${prefix_x}_virtual_suspension_link" />
-        <limit
-          effort="${axle_z_joint_effort_limit}"
-          velocity="${axle_z_joint_velocity_limit}"
-          lower="${axle_z_joint_min_limit}"
-          upper="${axle_z_joint_max_limit}" />
-        <origin xyz="${reflect_x*0.158+0.031} 0.0 0.035"  rpy="0.0 0.0 0.0" />
-        <axis xyz="0 0 1" />
-      </joint>
-      <link name="${prefix_x}_virtual_suspension_link" >
-        <xacro:solid_cylinder_intertial mass="0.00001" radius="0.001" y="0.1212" >
-          <origin xyz="0.0 0.0 0.0"/>
-        </xacro:solid_cylinder_intertial>
-        <visual>
-          <geometry>
-            <cylinder radius="0.001" length="0.1212" />
-          </geometry>
-          <origin xyz="0.0 0.0 ${-0.1212/2}" />
-        </visual>
-        <collision>
-          <geometry>
-            <cylinder radius="0.001" length="0.1212" />
-          </geometry>
-          <origin xyz="0.0 0.0 ${-0.1212/2}" />
-        </collision>
-      </link>
-      <joint name="${prefix_x}_axle_joint" type="revolute" >
-        <parent link="${prefix_x}_virtual_suspension_link" />
-        <child link="${prefix_x}_axle_link" />
-        <limit
-          effort="${axle_effort_limit}"
-          velocity="${axle_velocity_limit}"
-          lower="${axle_roll_joint_min_limit}"
-          upper="${axle_roll_joint_max_limit}" />
-        <origin xyz="0.0 0.0 -0.112"  rpy="0.0 0.0 0.0" />
-        <axis xyz="1 0 0" />
-      </joint>
-    </xacro:if>
-<!-- ======================================================================= -->
+  <xacro:macro name="axle" params="prefix_x reflect_x" >
+    <joint name="${prefix_x}_virtual_suspension_joint" type="prismatic" >
+      <parent link="base_link" />
+      <child link="${prefix_x}_virtual_suspension_link" />
+      <limit
+        effort="${virtual_suspension_joint_effort_limit}"
+        velocity="${virtual_suspension_joint_velocity_limit}"
+        lower="${virtual_suspension_joint_lower_limit}"
+        upper="${virtual_suspension_joint_upper_limit}" />
+      <dynamics damping="100.0" />
+      <origin xyz="${reflect_x*0.158+0.031} 0.0 0.035"  rpy="0.0 0.0 0.0" />
+      <axis xyz="0 0 1" />
+    </joint>
+    <link name="${prefix_x}_virtual_suspension_link" >
+      <xacro:null_inertial />
+    </link>
+    <joint name="${prefix_x}_axle_joint" type="revolute" >
+      <parent link="${prefix_x}_virtual_suspension_link" />
+      <child link="${prefix_x}_axle_link" />
+      <origin xyz="0.0 0.0 -0.112"  rpy="0.0 0.0 0.0" />
+      <axis xyz="1 0 0" />
+      <dynamics damping="0.0" />
+      <limit
+        effort="${axle_effort_limit}"
+        velocity="${axle_velocity_limit}"
+        lower="${axle_roll_joint_lower_limit}"
+        upper="${axle_roll_joint_upper_limit}" />
+    </joint>
     <link name="${prefix_x}_axle_link" >
       <xacro:solid_cylinder_inertial mass="0.4" radius="0.03" y="0.12" >

File: pandora_robots_description/monstertruck/urdf/parts/offroad_wheel.urdf.xacro (robot description, xacro)
@@ -8,5 +8,5 @@
   <xacro:property name="drive_link_length" value="0.03" />
   <xacro:property name="drive_link_radius" value="0.0025" />
-  <xacro:property name="drive_link_mass" value="0.001" />
+  <xacro:property name="drive_link_mass" value="0.005" />
   <xacro:property name="wheel_link_radius" value="0.075" />
   <xacro:property name="wheel_link_width" value="0.081" />
@@ -22,6 +22,6 @@
       <dynamics damping="0.0" />
       <limit
-        lower="${steer_joint_min_limit}"
-        upper="${steer_joint_max_limit}"
+        lower="${steer_joint_lower_limit}"
+        upper="${steer_joint_upper_limit}"
         effort="${steer_joint_effort_limit}"
         velocity="${steer_joint_velocity_limit}"/>
@@ -29,9 +29,12 @@
     <!-- wheel steer link -->
     <link name="${prefix_y}_${prefix_x}_wheel_steer_link" >
-      <xacro:solid_sphere_inertial
-        mass="${steer_link_mass}"
-        radius="${steer_link_radius}" >
-        <origin xyz="0.0 0.0 0.0" />
-      </xacro:solid_sphere_inertial>
+      <!-- Using real inertia causes unexpected bahaviour -->
+      <!-- Works fine, only with null inertial -->
+      <!-- <xacro:solid_sphere_inertial -->
+        <!-- mass="${steer_link_mass}" -->
+        <!-- radius="${steer_link_radius}" > -->
+        <!-- <origin xyz="0.0 0.0 0.0" /> -->
+      <!-- </xacro:solid_sphere_inertial> -->
+      <xacro:null_inertial />
       <visual>
         <origin xyz="0.0 0.0 0.0" rpy="0.0 0.0 0.0" />
@@ -49,17 +52,23 @@
     </link>
     <!-- wheel steer link to drive link joint -->
-    <joint name="${prefix_y}_${prefix_x}_wheel_steer_link_to_drive_link_joint" type="fixed" >
+    <joint name="${prefix_y}_${prefix_x}_wheel_drive_joint" type="continuous" >
       <parent link="${prefix_y}_${prefix_x}_wheel_steer_link" />
       <child link="${prefix_y}_${prefix_x}_wheel_drive_link" />
       <origin xyz="0.0 ${reflect_y*(steer_link_radius/2+drive_link_length/2)} 0.0" />
+      <axis xyz="0 1 0" />
+      <dynamics damping="0.0" />
+      <limit
+        effort="${drive_joint_effort_limit}"
+        velocity="${drive_joint_velocity_limit}" />
     </joint>
     <!-- wheel drive link -->
     <link name="${prefix_y}_${prefix_x}_wheel_drive_link" >
-      <!-- Using real inertia causes unexpected bahaviour -->
-      <!-- Works fine, only with null inertial -->
-      <xacro:null_inertial />
-      <!-- <xacro:solid_cylinder_inertial mass="0.01" radius="0.0025" y="0.03" > -->
-        <!-- <origin xyz="0.0 0.0 0.0" /> -->
-      <!-- </xacro:solid_cylinder_inertial> -->
+      <!-- <xacro:null_inertial /> -->
+      <xacro:solid_cylinder_inertial
+        mass="${drive_link_mass}"
+        radius="${drive_link_radius}"
+        y="${drive_link_length}" >
+        <origin xyz="0.0 0.0 0.0" />
+      </xacro:solid_cylinder_inertial>
       <visual>
         <origin xyz="0.0 0.0 0.0" rpy="${PI/2} 0.0 0.0" />
@@ -77,13 +86,8 @@
     </link>
     <!-- drive link to wheel joint -->
-    <joint name="${prefix_y}_${prefix_x}_wheel_drive_joint" type="continuous" >
+    <joint name="${prefix_y}_${prefix_x}_wheel_joint" type="fixed" >
       <parent link="${prefix_y}_${prefix_x}_wheel_drive_link" />
       <child link="${prefix_y}_${prefix_x}_wheel_link" />
       <origin xyz="0.0 ${reflect_y*wheel_link_offset} 0.0" />
-      <axis xyz="0 1 0" />
-      <dynamics damping="0.0" />
-      <limit
-        effort="${drive_joint_effort_limit}"
-        velocity="${drive_joint_velocity_limit}" />
     </joint>
     <!-- wheel_link -->

Commit message: Modify suspension joint limits

File: pandora_robots_description/monstertruck/urdf/joint_limits.xacro (robot description, xacro)
@@ -19,10 +19,10 @@
   <!-- axle suspension approximation joint limits -->
   <xacro:property name="virtual_suspension_joint_lower_limit" value="0.0" />
-  <xacro:property name="virtual_suspension_joint_upper_limit" value="0.027" />
-  <xacro:property name="virtual_suspension_joint_velocity_limit" value="10.0" />
-  <xacro:property name="virtual_suspension_joint_effort_limit" value="1.0" />
+  <xacro:property name="virtual_suspension_joint_upper_limit" value="0.03" />
+  <xacro:property name="virtual_suspension_joint_velocity_limit" value="100.0" />
+  <xacro:property name="virtual_suspension_joint_effort_limit" value="50.0" />
   <xacro:property name="axle_roll_joint_lower_limit" value="${-PI*10/180}" />
   <xacro:property name="axle_roll_joint_upper_limit" value="${PI*10/180}" />
   <xacro:property name="axle_velocity_limit" value="10.0" />
-  <xacro:property name="axle_effort_limit" value="10.0" />
+  <xacro:property name="axle_effort_limit" value="1.0" />
 </robot>
