Commit message: Add a suspension in each wheel (replaces experimental axle suspension)

File: pandora_robots_description/monstertruck/urdf/joint_limits.xacro (robot description, xacro)
@@ -7,22 +7,25 @@
   <xacro:property name="laser_pitch_joint_min_limit" value="-0.523" />
   <xacro:property name="laser_pitch_joint_max_limit" value="0.523" />
-  <xacro:property name="max_laser_angular_velocity" value="2.5" />
-  <xacro:property name="max_laser_angular_acceleration" value="0.0" />
   <!-- wheel steer joint limits -->
   <xacro:property name="steer_joint_lower_limit" value="${-25*PI/180}" />
   <xacro:property name="steer_joint_upper_limit" value="${25*PI/180}" />
-  <xacro:property name="steer_joint_velocity_limit" value="100.0" />
-  <xacro:property name="steer_joint_effort_limit" value="100.0" />
+  <xacro:property name="steer_joint_velocity_limit" value="1.0" />
+  <xacro:property name="steer_joint_effort_limit" value="10.0" />
   <!-- wheel drive joint limits -->
   <xacro:property name="drive_joint_velocity_limit" value="100.0" />
   <xacro:property name="drive_joint_effort_limit" value="100.0" />
-  <!-- axle suspension approximation joint limits -->
-  <xacro:property name="virtual_suspension_joint_lower_limit" value="0.0" />
-  <xacro:property name="virtual_suspension_joint_upper_limit" value="0.03" />
-  <xacro:property name="virtual_suspension_joint_velocity_limit" value="100.0" />
-  <xacro:property name="virtual_suspension_joint_effort_limit" value="50.0" />
+  <!-- axle suspension joint limits -->
+  <xacro:property name="axle_suspension_joint_upper_limit" value="0.03" />
+  <xacro:property name="axle_suspension_joint_lower_limit" value="-0.015" />
+  <xacro:property name="axle_suspension_joint_velocity_limit" value="10.0" />
+  <xacro:property name="axle_suspension_joint_effort_limit" value="100.0" />
   <xacro:property name="axle_roll_joint_lower_limit" value="${-PI*10/180}" />
   <xacro:property name="axle_roll_joint_upper_limit" value="${PI*10/180}" />
   <xacro:property name="axle_velocity_limit" value="10.0" />
-  <xacro:property name="axle_effort_limit" value="1.0" />
+  <xacro:property name="axle_effort_limit" value="100.0" />
+  <!-- wheel suspension joint limits -->
+  <xacro:property name="wheel_suspension_joint_lower_limit" value="-0.01" />
+  <xacro:property name="wheel_suspension_joint_upper_limit" value="0.03" />
+  <xacro:property name="wheel_suspension_joint_velocity_limit" value="1.0" />
+  <xacro:property name="wheel_suspension_joint_effort_limit" value="30.0" />
 </robot>

File: pandora_robots_description/monstertruck/urdf/parts/axle.urdf.xacro (robot description, xacro)
@@ -2,25 +2,25 @@
 <robot xmlns:xacro="http://ros.org/wiki/xacro" >
   <xacro:macro name="axle" params="prefix_x reflect_x" >
-    <joint name="${prefix_x}_virtual_suspension_joint" type="prismatic" >
+    <joint name="${prefix_x}_axle_suspension_joint" type="prismatic" >
       <parent link="base_link" />
-      <child link="${prefix_x}_virtual_suspension_link" />
+      <child link="${prefix_x}_axle_suspension_link" />
       <limit
-        effort="${virtual_suspension_joint_effort_limit}"
-        velocity="${virtual_suspension_joint_velocity_limit}"
-        lower="${virtual_suspension_joint_lower_limit}"
-        upper="${virtual_suspension_joint_upper_limit}" />
+        effort="${axle_suspension_joint_effort_limit}"
+        velocity="${axle_suspension_joint_velocity_limit}"
+        lower="${axle_suspension_joint_lower_limit}"
+        upper="${axle_suspension_joint_upper_limit}" />
       <dynamics damping="100.0" />
       <origin xyz="${reflect_x*0.158+0.031} 0.0 0.035"  rpy="0.0 0.0 0.0" />
       <axis xyz="0 0 1" />
     </joint>
-    <link name="${prefix_x}_virtual_suspension_link" >
+    <link name="${prefix_x}_axle_suspension_link" >
       <xacro:null_inertial />
     </link>
     <joint name="${prefix_x}_axle_joint" type="revolute" >
-      <parent link="${prefix_x}_virtual_suspension_link" />
+      <parent link="${prefix_x}_axle_suspension_link" />
       <child link="${prefix_x}_axle_link" />
       <origin xyz="0.0 0.0 -0.112"  rpy="0.0 0.0 0.0" />
       <axis xyz="1 0 0" />
-      <dynamics damping="0.0" />
+      <dynamics damping="10.0" />
       <limit
         effort="${axle_effort_limit}"
@@ -39,10 +39,10 @@
         </geometry>
       </visual>
-      <collision>
-        <origin xyz="0.0 0.0 0.0" rpy="0.0 0.0 ${(1-reflect_x)*PI/2}" />
-        <geometry>
-          <mesh filename="package://pandora_robots_description/monstertruck/meshes/axle.stl" />
-        </geometry>
-      </collision>
+      <!-- <collision> -->
+        <!-- <origin xyz="0.0 0.0 0.0" rpy="0.0 0.0 ${(1-reflect_x)*PI/2}" /> -->
+        <!-- <geometry> -->
+          <!-- <mesh filename="package://pandora_robots_description/monstertruck/meshes/axle.stl" /> -->
+        <!-- </geometry> -->
+      <!-- </collision> -->
     </link>
   </xacro:macro>

File: pandora_robots_description/monstertruck/urdf/parts/base.urdf.xacro (robot description, xacro)
@@ -26,5 +26,5 @@
     <link name="motor_and_transmission_link" >
       <inertial>
-        <mass value="0.7" />
+        <mass value="2.0" />
         <inertia ixx= "0.00000016498" ixy="0.00000000129" ixz="-0.00000014688"
           iyy="0.00000043294" iyz="0.00000000125" izz="0.00000031516" />

File: pandora_robots_description/monstertruck/urdf/parts/offroad_wheel.urdf.xacro (robot description, xacro)
@@ -3,5 +3,7 @@
   <xacro:property name="wheelbase" value="0.32" />
   <xacro:property name="track" value="0.26" />
-  <xacro:property name="steer_link_offset" value="0.115" />
+  <xacro:property name="steer_link_x_offset" value="0.028" />
+  <xacro:property name="steer_link_y_offset" value="0.0525" />
+  <xacro:property name="steer_link_z_offset" value="-0.051" />
   <xacro:property name="steer_link_radius" value="0.008" />
   <xacro:property name="steer_link_mass" value="0.001" />
@@ -15,8 +17,23 @@
   <xacro:macro name="offroad_wheel"
     params="prefix_y prefix_x reflect_y reflect_x" >
+    <joint name="${prefix_y}_${prefix_x}_wheel_suspension_joint" type="prismatic" >
+      <parent link="base_link" />
+      <child link="${prefix_y}_${prefix_x}_wheel_suspension_link" />
+      <limit
+        effort="${wheel_suspension_joint_effort_limit}"
+        velocity="${wheel_suspension_joint_velocity_limit}"
+        lower="${wheel_suspension_joint_lower_limit}"
+        upper="${wheel_suspension_joint_upper_limit}" />
+      <dynamics damping="20.0" />
+      <origin xyz="${reflect_x*0.158+0.031} ${reflect_y*0.115} -0.077"  rpy="0.0 0.0 0.0" />
+      <axis xyz="0 0 1" />
+    </joint>
+    <link name="${prefix_y}_${prefix_x}_wheel_suspension_link">
+      <xacro:null_inertial />
+    </link>
     <joint name="${prefix_y}_${prefix_x}_wheel_steer_joint" type="revolute" >
-      <parent link="${prefix_x}_axle_link" />
+      <parent link="${prefix_y}_${prefix_x}_wheel_suspension_link" />
       <child link="${prefix_y}_${prefix_x}_wheel_steer_link" />
-      <origin xyz="0.0 ${reflect_y*steer_link_offset} 0.0" />
+      <origin xyz="0.0 0.0 0.0" />
       <axis xyz="0 0 1" />
       <dynamics damping="0.0" />
@@ -29,5 +46,5 @@
     <!-- wheel steer link -->
     <link name="${prefix_y}_${prefix_x}_wheel_steer_link" >
-      <!-- Using real inertia causes unexpected bahaviour -->
+      <!-- Using real inertia causes unstable bahaviour -->
       <!-- Works fine, only with null inertial -->
       <!-- <xacro:solid_sphere_inertial -->
@@ -64,5 +81,4 @@
     <!-- wheel drive link -->
     <link name="${prefix_y}_${prefix_x}_wheel_drive_link" >
-      <!-- <xacro:null_inertial /> -->
       <xacro:solid_cylinder_inertial
         mass="${drive_link_mass}"
