Commit message: Use more discreet colors

File: pandora_robots_description/monstertruck/urdf/parts/batteries_power_distribution_board.urdf.xacro (robot description, xacro)
@@ -15,5 +15,5 @@
           <box size="0.03 0.07 0.02" />
         </geometry>
-        <material name="yellow" />
+        <material name="dark_grey" />
       </visual>
     </link>

File: pandora_robots_description/monstertruck/urdf/parts/dc_dc_converter.urdf.xacro (robot description, xacro)
@@ -15,5 +15,5 @@
           <box size="0.05 0.03 0.05" />
         </geometry>
-        <material name="green" />
+        <material name="dark_grey" />
       </visual>
     </link>

File: pandora_robots_description/monstertruck/urdf/parts/electronics_power_distribution_board.urdf.xacro (robot description, xacro)
@@ -15,5 +15,5 @@
           <box size="0.035 0.02 0.06" />
         </geometry>
-        <material name="yellow" />
+        <material name="dark_grey" />
       </visual>
     </link>

File: pandora_robots_description/monstertruck/urdf/parts/epos_24_1.urdf.xacro (robot description, xacro)
@@ -16,5 +16,5 @@
           <box size="0.042 0.04 0.026" />
         </geometry>
-        <material name="green" />
+        <material name="dark_grey" />
       </visual>
       <!-- <collision> -->

File: pandora_robots_description/monstertruck/urdf/parts/m4_atx_psu.urdf.xacro (robot description, xacro)
@@ -15,5 +15,5 @@
           <box size="0.122 0.119 0.02" />
         </geometry>
-        <material name="green" />
+        <material name="dark_grey" />
       </visual>
     </link>

File: pandora_robots_description/monstertruck/urdf/parts/motors_power_distribution_board.urdf.xacro (robot description, xacro)
@@ -15,5 +15,5 @@
           <box size="0.04 0.02 0.05" />
         </geometry>
-        <material name="yellow" />
+        <material name="dark_grey" />
       </visual>
     </link>

File: pandora_robots_description/monstertruck/urdf/sensors/compass_os4000.urdf.xacro (robot description, xacro)
@@ -15,4 +15,5 @@
           <box size="0.05 0.04 0.04" />
         </geometry>
+        <material name="dark_grey" />
       </visual>
       <collision>
