Commit message: Modify motor mass

File: pandora_robots_description/monstertruck/urdf/parts/base.urdf.xacro (robot description, xacro)
@@ -26,5 +26,5 @@
     <link name="motor_and_transmission_link" >
       <inertial>
-        <mass value="2.0" />
+        <mass value="1.0" />
         <inertia ixx= "0.00000016498" ixy="0.00000000129" ixz="-0.00000014688"
           iyy="0.00000043294" iyz="0.00000000125" izz="0.00000031516" />
