Commit message: Minor changes in robot link masses and inertias

File: pandora_robots_description/monstertruck/urdf/parts/axle.urdf.xacro (robot description, xacro)
@@ -4,5 +4,5 @@
     <!-- No suspension  -->
     <xacro:unless value="${suspension_approximation}">
-      <joint name="${prefix_x}_base_axle_joint" type="fixed">
+      <joint name="${prefix_x}_base_axle_joint" type="fixed" >
         <parent link="base_link" />
         <child link="${prefix_x}_axle_link" />
@@ -54,11 +54,7 @@
 <!-- ======================================================================= -->
     <link name="${prefix_x}_axle_link" >
-      <inertial>
-        <origin xyz="0.000288 -0.010863 0.073460" />
-        <mass value="0.3" />
-        <inertia ixx="0.00000004383" ixy="0.0"
-          iyy="0.00000028948" iyz="0.0"
-          izz="0.00000026930" ixz="0.0" />
-      </inertial>
+      <xacro:solid_cylinder_inertial mass="0.4" radius="0.03" y="0.12" >
+        <origin xyz="0.0 0.0 0.0" />
+      </xacro:solid_cylinder_inertial>
       <visual>
         <origin xyz="0.0 0.0 0.0" rpy="0.0 0.0 ${(1-reflect_x)*PI/2}" />
@@ -73,10 +69,4 @@
         </geometry>
       </collision>
-      <collision_checking>
-        <origin xyz="0.0 0.0 0.0" rpy="0.0 0.0 ${(1-reflect_x)*PI/2}" />
-        <geometry>
-          <box size="0.0543 0.2153 0.0635" />
-        </geometry>
-      </collision_checking>
     </link>
   </xacro:macro>

File: pandora_robots_description/monstertruck/urdf/parts/base.urdf.xacro (robot description, xacro)
@@ -3,16 +3,7 @@
   <xacro:macro name="base" >
     <link name="base_link" >
-      <inertial>
-        <!-- TODO find actual mass -->
-        <mass value="1.2" />
-        <!-- TODO recalculate inertia -->
-        <inertia ixx="0.000001"
-          ixy="0.0"
-          ixz="0.0"
-          iyy="0.000001"
-          iyz="0.0"
-          izz="0.000001" />
-        <origin xyz="-0.030427 0.001012 0.005388" />
-      </inertial>
+      <xacro:solid_cuboid_inertial mass="0.8" x="0.385" y="0.09" z="0.14">
+        <origin xyz="0.0 0.0 0.04" />
+      </xacro:solid_cuboid_inertial>
       <visual>
         <geometry>
@@ -35,5 +26,5 @@
     <link name="motor_and_transmission_link" >
       <inertial>
-        <mass value="1.0" />
+        <mass value="0.7" />
         <inertia ixx= "0.00000016498" ixy="0.00000000129" ixz="-0.00000014688"
           iyy="0.00000043294" iyz="0.00000000125" izz="0.00000031516" />
@@ -58,5 +49,5 @@
     </joint>
     <link name="floor_board_link" >
-      <xacro:solid_cuboid_inertial mass="0.1" x="0.34" y="0.17" z="0.004" >
+      <xacro:solid_cuboid_inertial mass="0.3" x="0.34" y="0.17" z="0.004" >
         <origin xyz="0.0 0.0 0.0" />
       </xacro:solid_cuboid_inertial>

File: pandora_robots_description/monstertruck/urdf/parts/batteries_power_distribution_board.urdf.xacro (robot description, xacro)
@@ -8,5 +8,5 @@
     </joint>
     <link name="battery_power_distribution_board_link" >
-      <xacro:solid_cuboid_inertial mass="0.3" x="0.03" y="0.07" z="0.02" >
+      <xacro:solid_cuboid_inertial mass="0.03" x="0.03" y="0.07" z="0.02" >
         <origin xyz="0.0 0.0 0.0" />
       </xacro:solid_cuboid_inertial>
@@ -17,4 +17,9 @@
         <material name="dark_grey" />
       </visual>
+      <collision>
+        <geometry>
+          <box size="0.03 0.07 0.02" />
+        </geometry>
+      </collision>
     </link>
   </xacro:macro>

File: pandora_robots_description/monstertruck/urdf/parts/battery.urdf.xacro (robot description, xacro)
@@ -16,9 +16,9 @@
         </geometry>
       </visual>
-      <!-- <collision> -->
-        <!-- <geometry> -->
-          <!-- <mesh filename="package://pandora_robots_description/monstertruck/meshes/battery.stl"/> -->
-        <!-- </geometry> -->
-      <!-- </collision> -->
+      <collision>
+        <geometry>
+          <mesh filename="package://pandora_robots_description/monstertruck/meshes/battery.stl"/>
+        </geometry>
+      </collision>
     </link>
   </xacro:macro>

File: pandora_robots_description/monstertruck/urdf/parts/dc_dc_converter.urdf.xacro (robot description, xacro)
@@ -17,4 +17,9 @@
         <material name="dark_grey" />
       </visual>
+      <collision>
+        <geometry>
+          <box size="0.05 0.03 0.05" />
+        </geometry>
+      </collision>
     </link>
   </xacro:macro>

File: pandora_robots_description/monstertruck/urdf/parts/electronics_box.urdf.xacro (robot description, xacro)
@@ -9,5 +9,5 @@
     </joint>
     <link name="electronics_box_link" >
-      <xacro:solid_cuboid_inertial mass="0.3" x="0.31" y="0.17" z="0.07454" >
+      <xacro:solid_cuboid_inertial mass="1.0" x="0.31" y="0.17" z="0.07454" >
         <origin xyz="0.0 0.0 0.0" />
       </xacro:solid_cuboid_inertial>

File: pandora_robots_description/monstertruck/urdf/parts/electronics_power_distribution_board.urdf.xacro (robot description, xacro)
@@ -17,4 +17,9 @@
         <material name="dark_grey" />
       </visual>
+      <collision>
+        <geometry>
+          <box size="0.035 0.02 0.06" />
+        </geometry>
+      </collision>
     </link>
   </xacro:macro>

File: pandora_robots_description/monstertruck/urdf/parts/epos_24_1.urdf.xacro (robot description, xacro)
@@ -18,9 +18,9 @@
         <material name="dark_grey" />
       </visual>
-      <!-- <collision> -->
-        <!-- <geometry> -->
-          <!-- <box size="0.042 0.04 0.026" /> -->
-        <!-- </geometry> -->
-      <!-- </collision> -->
+      <collision>
+        <geometry>
+          <box size="0.042 0.04 0.026" />
+        </geometry>
+      </collision>
     </link>
   </xacro:macro>

File: pandora_robots_description/monstertruck/urdf/parts/m4_atx_psu.urdf.xacro (robot description, xacro)
@@ -17,4 +17,9 @@
         <material name="dark_grey" />
       </visual>
+      <collision>
+        <geometry>
+          <box size="0.122 0.119 0.02" />
+        </geometry>
+      </collision>
     </link>
   </xacro:macro>

File: pandora_robots_description/monstertruck/urdf/parts/motors_power_distribution_board.urdf.xacro (robot description, xacro)
@@ -17,4 +17,9 @@
         <material name="dark_grey" />
       </visual>
+      <collision>
+        <geometry>
+          <box size="0.04 0.02 0.05" />
+        </geometry>
+      </collision>
     </link>
   </xacro:macro>

File: pandora_robots_description/monstertruck/urdf/parts/offroad_wheel.urdf.xacro (robot description, xacro)
@@ -96,7 +96,8 @@
       </xacro:solid_cylinder_inertial>
       <visual>
-        <origin xyz="0.0 0.0 0.0" rpy="0.0 0.0 0.0" />
+        <origin xyz="0.0 0.0 0.0" rpy="${PI/2*0} 0.0 0.0" />
         <geometry>
           <mesh filename="package://pandora_robots_description/monstertruck/meshes/${prefix_y}_offroad_wheel.dae" />
+          <!-- <cylinder radius="${wheel_link_radius}" length="${wheel_link_width}" /> -->
         </geometry>
       </visual>

File: pandora_robots_description/monstertruck/urdf/parts/pc_box.urdf.xacro (robot description, xacro)
@@ -10,5 +10,5 @@
     <!-- TODO measure mass -->
     <link name="pc_box_link" >
-      <xacro:solid_cuboid_inertial mass="0.3" x="0.21" y="0.24" z="0.084" >
+      <xacro:solid_cuboid_inertial mass="0.8" x="0.21" y="0.24" z="0.084" >
         <origin xyz="0.0 0.0 0.0" />
       </xacro:solid_cuboid_inertial>

File: pandora_robots_description/monstertruck/urdf/parts/pc_fan_40mm.urdf.xacro (robot description, xacro)
@@ -19,5 +19,6 @@
       <collision>
         <geometry>
-          <mesh filename="package://pandora_robots_description/monstertruck/meshes/pc_fan_40mm.dae" />
+          <!-- <mesh filename="package://pandora_robots_description/monstertruck/meshes/pc_fan_40mm.dae" /> -->
+          <box size="0.04 0.01 0.04" />
         </geometry>
       </collision>

File: pandora_robots_description/monstertruck/urdf/parts/pc_fan_60mm.urdf.xacro (robot description, xacro)
@@ -19,5 +19,6 @@
       <collision>
         <geometry>
-          <mesh filename="package://pandora_robots_description/monstertruck/meshes/pc_fan_60mm.dae" />
+          <!-- <mesh filename="package://pandora_robots_description/monstertruck/meshes/pc_fan_60mm.dae" /> -->
+          <box size="0.06 0.015 0.06" />
         </geometry>
       </collision>

File: pandora_robots_description/monstertruck/urdf/parts/suspension.urdf.xacro (robot description, xacro)
@@ -2,15 +2,15 @@
 <robot xmlns:xacro="http://ros.org/wiki/xacro" >
   <xacro:macro name="suspensions" params="prefix_y prefix_x reflect_y reflect_x" >
-    <joint name="${prefix_y}_${prefix_x}_base_suspension_joint" type="fixed">
+    <joint name="${prefix_y}_${prefix_x}_base_suspension_joint" type="fixed" >
       <parent link="base_link" />
       <child link="${prefix_y}_${prefix_x}_suspension_link" />
-      <origin xyz="${reflect_x*0.116+0.0311} ${reflect_y*0.06} 0.026" />
+      <origin xyz="${reflect_x*0.13+0.0311} ${reflect_y*0.06} -0.0265" />
     </joint>
     <link name="${prefix_y}_${prefix_x}_suspension_link" >
-      <xacro:solid_cylinder_inertial mass="0.25" radius="0.02" y="0.1255" >
-        <origin xyz="0.0 0.0 0.0" rpy="0.0 0.0 0.0" />
+      <xacro:solid_cylinder_inertial mass="0.050" radius="0.02" y="0.1255" >
+        <origin xyz="0.0 0.0 0.0" rpy="${-PI/2} ${-reflect_x*PI/12} 0.0" />
       </xacro:solid_cylinder_inertial>
       <visual>
-        <origin xyz="${reflect_x*0.014} 0.0 -0.0525" rpy="${-PI/2} ${-reflect_x*PI/12} 0.0" />
+        <origin xyz="0.0 0.0 0.0" rpy="${-PI/2} ${-reflect_x*PI/12} 0.0" />
         <geometry>
           <mesh filename="package://pandora_robots_description/monstertruck/meshes/suspension.dae" />
@@ -18,5 +18,5 @@
       </visual>
       <!-- <collision> -->
-        <!-- <origin xyz="${reflect_x*0.014} 0.0 -0.0525" rpy="${-PI/2} ${-reflect_x*PI/12} 0.0" /> -->
+        <!-- <origin xyz="0.0 0.0 0.0" rpy="${-PI/2} ${-reflect_x*PI/12} 0.0" /> -->
         <!-- <geometry> -->
           <!-- <mesh filename="package://pandora_robots_description/monstertruck/meshes/suspension.stl" /> -->

Commit message: Rename experimental suspension joints and links

File: pandora_robots_description/monstertruck/urdf/parts/axle.urdf.xacro (robot description, xacro)
@@ -12,7 +12,7 @@
 <!-- =============== Experimental Suspension Approximation ================= -->
     <xacro:if value="${suspension_approximation}">
-      <joint name="${prefix_x}_base_axle_sim_suspension_joint" type="prismatic" >
+      <joint name="${prefix_x}_virtual_suspension_joint" type="prismatic" >
         <parent link="base_link" />
-        <child link="${prefix_x}_axle_sim_suspension_link" />
+        <child link="${prefix_x}_virtual_suspension_link" />
         <limit
           effort="${axle_z_joint_effort_limit}"
@@ -23,5 +23,5 @@
         <axis xyz="0 0 1" />
       </joint>
-      <link name="${prefix_x}_axle_sim_suspension_link" >
+      <link name="${prefix_x}_virtual_suspension_link" >
         <xacro:solid_cylinder_intertial mass="0.00001" radius="0.001" y="0.1212" >
           <origin xyz="0.0 0.0 0.0"/>
@@ -41,5 +41,5 @@
       </link>
       <joint name="${prefix_x}_axle_joint" type="revolute" >
-        <parent link="${prefix_x}_axle_sim_suspension_link" />
+        <parent link="${prefix_x}_virtual_suspension_link" />
         <child link="${prefix_x}_axle_link" />
         <limit

Commit message: Separate chassis from base_link and offset to center the model

File: pandora_robots_description/monstertruck/urdf/parts/axle.urdf.xacro (robot description, xacro)
@@ -3,5 +3,5 @@
   <xacro:macro name="axle" params="prefix_x reflect_x" >
     <joint name="${prefix_x}_axle_suspension_joint" type="prismatic" >
-      <parent link="base_link" />
+      <parent link="chassis_link" />
       <child link="${prefix_x}_axle_suspension_link" />
       <limit

File: pandora_robots_description/monstertruck/urdf/parts/base.urdf.xacro (robot description, xacro)
@@ -3,4 +3,12 @@
   <xacro:macro name="base" >
     <link name="base_link" >
+      <xacro:point_mass_inertial />
+    </link>
+    <joint name="base_to_chassis_link" type="fixed" >
+      <parent link="base_link" />
+      <child link="chassis_link" />
+      <origin xyz="-0.03 0.0 0.0" />
+    </joint>
+    <link name="chassis_link" >
       <xacro:solid_cuboid_inertial mass="0.8" x="0.385" y="0.09" z="0.14">
         <origin xyz="0.0 0.0 0.04" />
@@ -20,5 +28,5 @@
     <!-- Motor and Transmission -->
     <joint name="base_motor_and_transmission_joint" type="fixed" >
-      <parent link="base_link" />
+      <parent link="chassis_link" />
       <child link="motor_and_transmission_link" />
       <origin xyz="0.07 0.0 -0.0175" />
@@ -44,5 +52,5 @@
     <!-- chassis floor board -->
     <joint name="base_floor_board_joint" type="fixed" >
-      <parent link="base_link" />
+      <parent link="chassis_link" />
       <child link="floor_board_link" />
       <origin xyz="0.001042 0.0 0.066" />

File: pandora_robots_description/monstertruck/urdf/parts/epos_24_1.urdf.xacro (robot description, xacro)
@@ -4,5 +4,5 @@
     <!-- chassis floor board -->
     <joint name="base_epos_24_1_joint" type="fixed" >
-      <parent link="base_link" />
+      <parent link="chassis_link" />
       <child link="epos_24_1_link" />
       <origin xyz="0.05 0.0 0.043" />

File: pandora_robots_description/monstertruck/urdf/parts/suspension.urdf.xacro (robot description, xacro)
@@ -3,5 +3,5 @@
   <xacro:macro name="suspensions" params="prefix_y prefix_x reflect_y reflect_x" >
     <joint name="${prefix_y}_${prefix_x}_base_suspension_joint" type="fixed" >
-      <parent link="base_link" />
+      <parent link="chassis_link" />
       <child link="${prefix_y}_${prefix_x}_suspension_link" />
       <origin xyz="${reflect_x*0.13+0.0311} ${reflect_y*0.06} -0.0265" />
@@ -25,5 +25,5 @@
     </link>
     <joint name="${prefix_y}_${prefix_x}_wheel_suspension_joint" type="prismatic" >
-      <parent link="base_link" />
+      <parent link="chassis_link" />
       <child link="${prefix_y}_${prefix_x}_wheel_suspension_link" />
       <limit
